File: hardware/ntp-server-stm32/3v3-main-power.kicad_sch (KiCad schematic)
At the start: 52 parts, among them U28 MIC28516T-E/PHA, U29 AP3441SHE-7B, U30 INA228AQDGSRQ1, U31 INA228AQDGSRQ1, U32 INA228AQDGSRQ1, U33 RT9742VGJ5

Commit message: Standardize net/rail names: plain 3V3 style, _N active-low, voltage-format PG/alerts
22 net renames applied across all sheets and verified: removed/added net-name
sets match intent exactly and all node connectivity is preserved (kicad-cli
netlist re-parse).

Co-Authored-By: Claude Opus 4.8 (1M context) <noreply@anthropic.com>
Connections:
- net +3.3V renamed 3V3
- net +3.3V_STM renamed 3V3_STM
- net +5V renamed 5V
- net INA_ALERT_3.3V renamed INA_ALERT_3V3
- net INA_ALERT_3.3V_STM renamed INA_ALERT_3V3_STM
- net INA_ALERT_V_DISP_5V renamed INA_ALERT_5V_DISP
- net POE_PGO renamed POE_PG
- net V_DISP_5V renamed 5V_DISP
Changed lines of the file:
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@@
 		)
 	)
-	(global_label "INA_ALERT_3.3V_STM"
+	(global_label "INA_ALERT_3V3_STM"
 		(shape output)
 		(at 325.12 97.79 180)
@@
 		)
 	)
-	(global_label "INA_ALERT_3.3V"
+	(global_label "INA_ALERT_3V3"
 		(shape output)
 		(at 167.64 210.82 180)
@@
 		)
 	)
-	(global_label "POE_PGO"
+	(global_label "POE_PG"
 		(shape input)
 		(at 62.23 50.8 180)
@@
 		)
 	)
-	(global_label "INA_ALERT_V_DISP_5V"
+	(global_label "INA_ALERT_5V_DISP"
 		(shape output)
 		(at 326.39 194.31 180)
@@
 			)
 		)
-		(property "Value" "+3.3V"
+		(property "Value" "3V3"
 			(at 377.19 44.45 0)
 			(show_name no)
@@
 			)
 		)
-		(property "Value" "+3.3V"
+		(property "Value" "3V3"
 			(at 332.74 83.82 0)
 			(show_name no)
@@
 			)
 		)
-		(property "Value" "+3.3V_STM"
+		(property "Value" "3V3_STM"
 			(at 388.62 44.45 0)
 			(show_name no)
@@
 			)
 		)
-		(property "Value" "+5V"
+		(property "Value" "5V"
 			(at 109.22 29.21 0)
 			(show_name no)
@@
 			)
 		)
-		(property "Value" "+3.3V"
+		(property "Value" "3V3"
 			(at 384.81 96.52 0)
 			(show_name no)
@@
 			)
 		)
-		(property "Value" "+3.3V_STM"
+		(property "Value" "3V3_STM"
 			(at 347.98 127 0)
 			(show_name no)
@@
 			)
 		)
-		(property "Value" "+3.3V"
+		(property "Value" "3V3"
 			(at 386.08 193.04 0)
 			(show_name no)
@@
 			)
 		)
-		(property "Value" "+5V"
+		(property "Value" "5V"
 			(at 71.12 160.02 0)
 			(show_name no)
@@
 			)
 		)
-		(property "Value" "+3.3V"
+		(property "Value" "3V3"
 			(at 231.14 154.94 0)
 			(show_name no)
@@
 			)
 		)
-		(property "Value" "+5V"
+		(property "Value" "5V"
 			(at 327.66 129.54 0)
 			(show_name no)
@@
 			)
 		)
-		(property "Value" "V_DISP_5V"
+		(property "Value" "5V_DISP"
 			(at 389.89 134.62 0)
 			(show_name no)
@@
 			)
 		)
-		(property "Value" "+5V"
+		(property "Value" "5V"
 			(at 160.02 59.69 0)
 			(show_name no)
@@
 			)
 		)
-		(property "Value" "+3.3V"
+		(property "Value" "3V3"
 			(at 227.33 209.55 0)
 			(show_name no)

Commit message: Standardize + complete BOM; write fields back into KiCad symbols
- New sts1000_bom.csv: rebuilt from authoritative Value field (source MPN/footprint/
  description were corrupted by copy-paste). 338 standardized, 78 MPN-from-value,
  50 kept, ~64 flagged (SELECT/REVIEW-HV/SHUNT-REVIEW) each with full spec.
- Resistors -> deterministic Panasonic ERJ-2RKF 0402 1% 1/10W (consolidated 1 part/value).
- Caps -> verified Murata GRM parts where value matches; clean spec + footprint otherwise.
- 1633 symbol field updates (Value/Footprint/Description/MPN/Mfr/Digikey) written to
  .kicad_sch; netlist re-parse confirms connectivity byte-identical.
- Add docs/sts1000_net_naming.md naming reference.

Co-Authored-By: Claude Opus 4.8 (1M context) <noreply@anthropic.com>
Parts:
- C63, C67, C68, C69, C70: footprint 402 -> C_0402_1005Metric; MANUFACTURER (none) -> Murata
- C64, C65, C66, C73, C74, C76, C78, C81: footprint 805 -> C_0805_2012Metric; MANUFACTURER (none) -> Murata
- C71, C72: footprint 1210 -> C_1210_3225Metric; MANUFACTURER (none) -> Murata
- C75, C77, C80: value 2.2uF 100V -> 2.2uF; footprint 805 -> C_0805_2012Metric; MANUFACTURER (none) -> Murata
- C79: value 1uF 100V -> 1uF; footprint 603 -> C_0603_1608Metric; MANUFACTURER (none) -> Murata
- C82: footprint 603 -> C_0603_1608Metric; MANUFACTURER (none) -> Murata
- C83, C86, C87: footprint (none) -> C_0402_1005Metric; DIGIKEY_PART_NUMBER (none) -> 490-6328-2-ND; MANUFACTURER (none) -> Murata; MANUFACTURER_PART_NUMBER (none) -> GRM155R71C104KA88J
- C84, C85: footprint (none) -> C_0603_1608Metric
- L2: MANUFACTURER (none) -> Bourns Inc.
- L3: MANUFACTURER (none) -> Eaton - Electronics Division
- R100, R104, R90, R91, R92, R93, R94, R96, R97, R98, R99: footprint 402 -> R_0402_1005Metric; MANUFACTURER (none) -> Panasonic
- R101, R103: footprint 402 -> R_0402_1005Metric; MANUFACTURER (none) -> Panasonic; MANUFACTURER_PART_NUMBER ERJ-U02F2R20X -> ERJ-2RKF2R20X
- R105: footprint (none) -> R_0402_1005Metric; MANUFACTURER (none) -> Panasonic; MANUFACTURER_PART_NUMBER (none) -> ERJ-2RKF1002X
- R95: footprint 402 -> R_0402_1005Metric; MANUFACTURER (none) -> Panasonic; MANUFACTURER_PART_NUMBER ERJ-2RKF2051X -> ERJ-2RKF1002X
- U28: MANUFACTURER (none) -> Microchip Technology
- U29: MANUFACTURER (none) -> Diodes Incorporated
- U30, U31, U32: MANUFACTURER_PART_NUMBER (none) -> INA228AQDGSRQ1
- U33: MANUFACTURER (none) -> Richtek USA Inc.
