File: hardware/ntp-server-stm32/3v3-main-power.kicad_sch (KiCad schematic)
At the start: 52 parts, among them U28 MIC28516T-E/PHA, U29 AP3441SHE-7B, U30 INA228AQDGSRQ1, U31 INA228AQDGSRQ1, U32 INA228AQDGSRQ1, U33 RT9742VGJ5

Commit message: Updates
Parts:
- C63: footprint C_0402_1005Metric -> 0402 (1005 Metric); DIELECTRIC (none) -> X7R; DIGIKEY_PART_NUMBER 490-1313-2-ND -> 490-GRT155R71C103KE01JCT-ND; MANUFACTURER Murata -> Murata Electronics; MANUFACTURER_PART_NUMBER GRM155R71C103KA01D -> GRT155R71C103KE01J; TOLERANCE (none) -> 10%; VOLTAGE (none) -> 16V
- C64, C65, C66, C73, C74, C76, C78: footprint C_0805_2012Metric -> 1206 (3216 Metric); DIELECTRIC (none) -> X7R; DIGIKEY_PART_NUMBER 490-GRM21BZ71C106KE15LTR-ND -> 1276-6797-1-ND; MANUFACTURER Murata -> Samsung Electro-Mechanics; MANUFACTURER_PART_NUMBER GRM21BZ71C106KE15L -> CL31B106KOHVPNE; TOLERANCE (none) -> 10%; VOLTAGE (none) -> 16V
- C67, C68, C83, C86, C87: footprint C_0402_1005Metric -> 0402 (1005 Metric); DIELECTRIC (none) -> X7R; DIGIKEY_PART_NUMBER 490-6328-2-ND -> 490-4759-1-ND; MANUFACTURER_PART_NUMBER GRM155R71C104KA88J -> GCM155R71C104KA55D; TOLERANCE (none) -> 10%; VOLTAGE (none) -> 16V
- C69, C70: footprint C_0402_1005Metric -> 0402 (1005 Metric); DIELECTRIC (none) -> X7R; DIGIKEY_PART_NUMBER 490-6334-2-ND -> 399-17875-1-ND; MANUFACTURER Murata -> KEMET; MANUFACTURER_PART_NUMBER GRM155R71C472KA01D -> C0402C472K4RECAUTO; TOLERANCE (none) -> 10%; VOLTAGE (none) -> 16V
- C71, C72: footprint C_1210_3225Metric -> 1210 (3225 Metric); DIELECTRIC (none) -> X6S; DIGIKEY_PART_NUMBER 490-16309-2-ND -> 490-12494-1-ND; MANUFACTURER Murata -> Murata Electronics; MANUFACTURER_PART_NUMBER GRM32EC81C476KE15K -> GRT32EC81C476KE13L; TOLERANCE (none) -> 10%; VOLTAGE (none) -> 16V
- C75, C77, C80: footprint C_0805_2012Metric -> 2220 (5750 Metric); DIELECTRIC (none) -> X7T; DIGIKEY_PART_NUMBER 490-GRM21BD72A225ME01KTR-ND -> 445-7950-1-ND; MANUFACTURER Murata -> TDK; MANUFACTURER_PART_NUMBER GRM21BD72A225ME01K -> CGA9P3X7T2E225K250KA; TOLERANCE (none) -> 10%; VOLTAGE (none) -> 100V
- C79: footprint C_0603_1608Metric -> 0805 (2012 Metric); DIELECTRIC (none) -> X7T; DIGIKEY_PART_NUMBER 490-GRM188D72A105KE01WTR-ND -> 478-KAM21KR72A105KUCT-ND; MANUFACTURER Murata -> KYOCERA AVX; MANUFACTURER_PART_NUMBER GRM188D72A105KE01W -> 08051C105K4T2A; TOLERANCE (none) -> 10%; VOLTAGE (none) -> 100V
- C81: footprint C_0805_2012Metric -> 0805 (2012 Metric); DIELECTRIC (none) -> X7R; DIGIKEY_PART_NUMBER 490-GRM21BR71C475KE51KTR-ND -> 490-GRT21BR71C475KE13KCT-ND; MANUFACTURER Murata -> Murata Electronics; MANUFACTURER_PART_NUMBER GRM21BR71C475KE51K -> GRT21BR71C475KE13K; TOLERANCE (none) -> 10%; VOLTAGE (none) -> 16V
- C82: footprint C_0603_1608Metric -> 0805 (2012 Metric); DIELECTRIC (none) -> X7R; DIGIKEY_PART_NUMBER 490-GRM188Z71C225KE43DTR-ND -> 490-GRT21BR71C225KE01LCT-ND; MANUFACTURER Murata -> Murata Electronics; MANUFACTURER_PART_NUMBER GRM188Z71C225KE43D -> GRT21BR71C225KE01L; TOLERANCE (none) -> 10%; VOLTAGE (none) -> 16V
- C84, C85: footprint C_0603_1608Metric -> 0603 (1608 Metric); DIELECTRIC (none) -> X7R; DIGIKEY_PART_NUMBER (none) -> 399-17704-1-ND; MANUFACTURER (none) -> KEMET; MANUFACTURER_PART_NUMBER (none) -> C0603C105K4RACAUTO; TOLERANCE (none) -> 10%; VOLTAGE (none) -> 16V
- FB7: DIELECTRIC (none) -> Ferrite bead; MANUFACTURER Murata Electronics -> Murata; MANUFACTURER_PART_NUMBER BLM31KN601SN1L -> BLM31PG601SN1L; POWER (none) -> 3A
- L2: DIELECTRIC (none) -> Inductor; POWER (none) -> 11.5A
- L3: DIELECTRIC (none) -> Inductor; POWER (none) -> 4.15A
- R100: footprint R_0402_1005Metric -> 0402 (1005 Metric); DIELECTRIC (none) -> Thick-film; DIGIKEY_PART_NUMBER P2.20KLTR-ND -> P2.20KLCT-ND; MANUFACTURER Panasonic -> Panasonic Industry; POWER (none) -> 1/10W; TOLERANCE (none) -> 1%
- R101, R103: footprint R_0402_1005Metric -> 0402 (1005 Metric); DIELECTRIC (none) -> Thick-film; MANUFACTURER Panasonic -> Panasonic Industry; MANUFACTURER_PART_NUMBER ERJ-2RKF2R20X -> ERJ-U02F2R20X; POWER (none) -> 1/10W; TOLERANCE (none) -> 1%
- R102: footprint 0805 -> 0805 (2012 Metric); DIELECTRIC (none) -> Metal-strip shunt; DIGIKEY_PART_NUMBER 273-KDV08DR150ETCT-ND -> 10-ERJ-UP6D75R0VCT-ND; MANUFACTURER Ohmite -> Panasonic Industry; MANUFACTURER_PART_NUMBER KDV08DR150ET -> ERJ-UP6D75R0V; POWER (none) -> 1/4W; TOLERANCE (none) -> 0.5%
- R104, R92, R99: footprint R_0402_1005Metric -> 0402 (1005 Metric); DIELECTRIC (none) -> Thick-film; DIGIKEY_PART_NUMBER P10.0KLTR-ND -> P10.0KLCT-ND; MANUFACTURER Panasonic -> Panasonic Industry; POWER (none) -> 1/10W; TOLERANCE (none) -> 1%
- R105: footprint R_0402_1005Metric -> 0402 (1005 Metric); DIELECTRIC (none) -> Thick-film; DIGIKEY_PART_NUMBER (none) -> P10.0KLCT-ND; MANUFACTURER Panasonic -> Panasonic Industry; POWER (none) -> 1/10W; TOLERANCE (none) -> 1%
- R106: value 500m -> 15m; footprint 0805 -> 1206 (3216 Metric); DIELECTRIC (none) -> Metal-strip shunt; DIGIKEY_PART_NUMBER 273-KDV08DR150ETCT-ND -> 273-MCS1632R015DERCT-ND; MANUFACTURER_PART_NUMBER KDV08DR150ET -> MCS1632R015DER; POWER (none) -> 1/4W; TOLERANCE (none) -> 0.5%
- R107: footprint 0805 -> 1206 (3216 Metric); DIELECTRIC (none) -> Metal-strip shunt; DIGIKEY_PART_NUMBER 273-KDV08DR150ETCT-ND -> 273-KDV12DR100ETCT-ND; MANUFACTURER_PART_NUMBER KDV08DR150ET -> KDV12DR100ET; POWER (none) -> 1/4W; TOLERANCE (none) -> 0.5%
- R90: footprint R_0402_1005Metric -> 0402 (1005 Metric); DIELECTRIC (none) -> Thick-film; DIGIKEY_PART_NUMBER P200KLTR-ND -> P200KLCT-ND; MANUFACTURER Panasonic -> Panasonic Industry; POWER (none) -> 1/10W; TOLERANCE (none) -> 1%
- R91: footprint R_0402_1005Metric -> 0402 (1005 Metric); DIELECTRIC (none) -> Thick-film; DIGIKEY_PART_NUMBER P100KLTR-ND -> P100KLCT-ND; MANUFACTURER Panasonic -> Panasonic Industry; POWER (none) -> 1/10W; TOLERANCE (none) -> 1%
- R93: footprint R_0402_1005Metric -> 0402 (1005 Metric); DIELECTRIC (none) -> Thick-film; DIGIKEY_PART_NUMBER P2.21KLTR-ND -> P2.21KLCT-ND; MANUFACTURER Panasonic -> Panasonic Industry; POWER (none) -> 1/10W; TOLERANCE (none) -> 1%
- R94, R98: footprint R_0402_1005Metric -> 0402 (1005 Metric); DIELECTRIC (none) -> Thick-film; MANUFACTURER Panasonic -> Panasonic Industry; POWER (none) -> 1/10W; TOLERANCE (none) -> 1%
- R95: footprint R_0402_1005Metric -> 0402 (1005 Metric); DIELECTRIC (none) -> Thick-film; DIGIKEY_PART_NUMBER P2.05KLTR-ND -> P10.0KLCT-ND; MANUFACTURER Panasonic -> Panasonic Industry; POWER (none) -> 1/10W; TOLERANCE (none) -> 1%
- R96: footprint R_0402_1005Metric -> 0402 (1005 Metric); DIELECTRIC (none) -> Thick-film; DIGIKEY_PART_NUMBER P24.9KLTR-ND -> P24.9KLCT-ND; MANUFACTURER Panasonic -> Panasonic Industry; POWER (none) -> 1/10W; TOLERANCE (none) -> 1%
- R97: footprint R_0402_1005Metric -> 0402 (1005 Metric); DIELECTRIC (none) -> Thick-film; DIGIKEY_PART_NUMBER P15.0KLTR-ND -> 2019-RK73H1ETTP1502FCT-ND; MANUFACTURER Panasonic -> KOA Speer Electronics, Inc.; MANUFACTURER_PART_NUMBER ERJ-2RKF1502X -> RK73H1ETTP1502F; POWER (none) -> 1/10W; TOLERANCE (none) -> 1%
- U28: MANUFACTURER Microchip Technology -> Microchip
- U29: MANUFACTURER Diodes Incorporated -> Diodes Inc
- U30, U31, U32: MANUFACTURER (none) -> Texas Instruments
- U33: MANUFACTURER Richtek USA Inc. -> Richtek
Connections:
- net I2C_SCL: now also U30.2 (A0), U30.5 (SCL), U31.5 (SCL), U32.5 (SCL); no longer U30.4 (SDA), U31.4 (SDA), U32.2 (A0), U32.4 (SDA)
- net I2C_SDA: now also U30.4 (SDA), U31.4 (SDA), U32.2 (A0), U32.4 (SDA); no longer U30.2 (A0), U30.5 (SCL), U31.5 (SCL), U32.5 (SCL)
- net VOUT_P renamed V_POE
Other:
- note added: "PG pulled to VIN When power good"

Commit message: Bom updates
Parts:
- FB7: footprint 1206 -> 1206 (3216 Metric)
- R102: value 75m -> 50m; footprint 0805 (2012 Metric) -> 1206 (3216 Metric); DIGIKEY_PART_NUMBER 10-ERJ-UP6D75R0VCT-ND -> WSLC-.05CT-ND; MANUFACTURER Panasonic Industry -> Vishay Dale; MANUFACTURER_PART_NUMBER ERJ-UP6D75R0V -> WSL1206R0500FEA
- R106: value 15m -> 100m; DIGIKEY_PART_NUMBER 273-MCS1632R015DERCT-ND -> WSLC-.10CT-ND; MANUFACTURER Ohmite -> Vishay Dale; MANUFACTURER_PART_NUMBER MCS1632R015DER -> WSL1206R1000FEA
- R107: DIGIKEY_PART_NUMBER 273-KDV12DR100ETCT-ND -> WSLC-.10CT-ND; MANUFACTURER Ohmite -> Vishay Dale; MANUFACTURER_PART_NUMBER KDV12DR100ET -> WSL1206R1000FEA
- U30, U31, U32: DIGIKEY_PART_NUMBER (none) -> 296-INA228AQDGSRQ1CT-ND
Changed lines of the file:
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@@
 			)
 		)
-		(property "Value" "75m"
+		(property "Value" "50m"
 			(at 228.346 168.91 90)
 			(show_name no)
@@
 			)
 		)
-		(property "Footprint" "0805 (2012 Metric)"
+		(property "Footprint" "1206 (3216 Metric)"
 			(at 226.06 164.592 90)
 			(hide yes)
@@
 			)
 		)
-		(property "Datasheet" "https://industrial.panasonic.com/cdbs/www-data/pdf/RDM0000/DMM0000COL9.pdf"
+		(property "Datasheet" "https://www.vishay.com/docs/30100/wsl.pdf"
 			(at 226.06 166.37 0)
 			(hide yes)
@@
 			)
 		)
-		(property "Description" "RES 75 OHM 0.5% 1/2W 0805"
+		(property "Description" "RES 0.05 OHM 1% 1/4W 1206"
 			(at 226.06 166.37 90)
 			(hide yes)
@@
 			)
 		)
-		(property "DIGIKEY_PART_NUMBER" "10-ERJ-UP6D75R0VCT-ND"
+		(property "DIGIKEY_PART_NUMBER" "WSLC-.05CT-ND"
 			(at 226.06 166.37 90)
 			(hide yes)
@@
 			)
 		)
-		(property "MANUFACTURER_PART_NUMBER" "ERJ-UP6D75R0V"
+		(property "MANUFACTURER_PART_NUMBER" "WSL1206R0500FEA"
 			(at 226.06 166.37 90)
 			(hide yes)
@@
 			)
 		)
-		(property "MANUFACTURER" "Panasonic Industry"
+		(property "MANUFACTURER" "Vishay Dale"
 			(at 226.06 166.37 90)
 			(hide yes)
@@
 			)
 		)
-		(property "Footprint" "1206"
+		(property "Footprint" "1206 (3216 Metric)"
 			(at 391.668 146.05 90)
 			(hide yes)
@@
 			)
 		)
-		(property "Datasheet" "https://www.ohmite.com/assets/images/res-kdv.pdf"
+		(property "Datasheet" "https://www.vishay.com/docs/30100/wsl.pdf"
 			(at 383.54 152.4 0)
 			(hide yes)
@@
 			)
 		)
-		(property "Description" "RES 0.1 OHM 0.5% 1/2W 1206"
+		(property "Description" "RES 0.1 OHM 1% 1/4W 1206"
 			(at 383.54 152.4 90)
 			(hide yes)
@@
 			)
 		)
-		(property "DIGIKEY_PART_NUMBER" "273-KDV12DR100ETCT-ND"
+		(property "DIGIKEY_PART_NUMBER" "WSLC-.10CT-ND"
 			(at 383.54 152.4 90)
 			(hide yes)
@@
 			)
 		)
-		(property "MANUFACTURER_PART_NUMBER" "KDV12DR100ET"
+		(property "MANUFACTURER_PART_NUMBER" "WSL1206R1000FEA"
 			(at 383.54 152.4 90)
 			(hide yes)
@@
 			)
 		)
-		(property "MANUFACTURER" "Ohmite"
+		(property "MANUFACTURER" "Vishay Dale"
 			(at 383.54 152.4 90)
 			(hide yes)
@@
 			)
 		)
-		(property "Datasheet" "https://www.ti.com/lit/gpn/ina228-q1"
+		(property "Datasheet" "https://www.ti.com/lit/ds/symlink/ina228-q1.pdf"
 			(at 176.53 205.74 0)
 			(hide yes)
@@
 			)
 		)
-		(property "Description" "Current/power monitor 20-bit I2C"
+		(property "Description" "IC PWR MONITOR 10VSSOP"
 			(at 176.53 205.74 0)
 			(hide yes)
@@
 			)
 		)
+		(property "DIGIKEY_PART_NUMBER" "296-INA228AQDGSRQ1CT-ND"
+			(at 176.53 205.74 0)
+			(hide yes)
+			(show_name no)
+			(do_not_autoplace no)
+			(effects
+				(font
+					(size 1.27 1.27)
+				)
+			)
+		)
 		(pin "2"
 		)
@@
 			)
 		)
-		(property "Value" "15m"
+		(property "Value" "100m"
 			(at 384.556 58.42 90)
 			(show_name no)
@@
 			)
 		)
-		(property "Datasheet" "https://www.ohmite.com/assets/images/res-mcs.pdf"
+		(property "Datasheet" "https://www.vishay.com/docs/30100/wsl.pdf"
 			(at 382.27 55.88 0)
 			(hide yes)
@@
 			)
 		)
-		(property "Description" "1W 0.015 OHM METAL ALLOY CS 1% C"
+		(property "Description" "RES 0.1 OHM 1% 1/4W 1206"
 			(at 382.27 55.88 90)
 			(hide yes)
@@
 			)
 		)
-		(property "DIGIKEY_PART_NUMBER" "273-MCS1632R015DERCT-ND"
+		(property "DIGIKEY_PART_NUMBER" "WSLC-.10CT-ND"
 			(at 382.27 55.88 90)
 			(hide yes)
@@
 			)
 		)
-		(property "MANUFACTURER_PART_NUMBER" "MCS1632R015DER"
+		(property "MANUFACTURER_PART_NUMBER" "WSL1206R1000FEA"
 			(at 382.27 55.88 90)
 			(hide yes)
@@
 			)
 		)
-		(property "MANUFACTURER" "Ohmite"
+		(property "MANUFACTURER" "Vishay Dale"
 			(at 382.27 55.88 90)
 			(hide yes)
@@
 			)
 		)
-		(property "Datasheet" "https://www.ti.com/lit/gpn/ina228-q1"
+		(property "Datasheet" "https://www.ti.com/lit/ds/symlink/ina228-q1.pdf"
 			(at 335.28 189.23 0)
 			(hide yes)
@@
 			)
 		)
-		(property "Description" "Current/power monitor 20-bit I2C"
+		(property "Description" "IC PWR MONITOR 10VSSOP"
 			(at 335.28 189.23 0)
 			(hide yes)
@@
 			)
 		)
+		(property "DIGIKEY_PART_NUMBER" "296-INA228AQDGSRQ1CT-ND"
+			(at 335.28 189.23 0)
+			(hide yes)
+			(show_name no)
+			(do_not_autoplace no)
+			(effects
+				(font
+					(size 1.27 1.27)
+				)
+			)
+		)
 		(pin "2"
 		)
@@
 			)
 		)
-		(property "Datasheet" "https://www.ti.com/lit/gpn/ina228-q1"
+		(property "Datasheet" "https://www.ti.com/lit/ds/symlink/ina228-q1.pdf"
 			(at 334.01 92.71 0)
 			(hide yes)
@@
 			)
 		)
-		(property "Description" "Current/power monitor 20-bit I2C"
+		(property "Description" "IC PWR MONITOR 10VSSOP"
 			(at 334.01 92.71 0)
 			(hide yes)
@@
 			(hide yes)
 			(show_name no)
+			(do_not_autoplace no)
+			(effects
+				(font
+					(size 1.27 1.27)
+				)
+			)
+		)
+		(property "DIGIKEY_PART_NUMBER" "296-INA228AQDGSRQ1CT-ND"
+			(at 334.01 92.71 0)
+			(hide yes)
+			(show_name no)

Commit message: Bom updates
Parts:
- U30, U31, U32: footprint VSSOP10_DGS_TEX -> sts1000:VSSOP10_DGS_TEX
Changed lines of the file:
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@@
 			)
 		)
-		(property "Footprint" "VSSOP10_DGS_TEX"
+		(property "Footprint" "sts1000:VSSOP10_DGS_TEX"
 			(at 176.53 205.74 0)
 			(hide yes)
@@
 			)
 		)
-		(property "Footprint" "VSSOP10_DGS_TEX"
+		(property "Footprint" "sts1000:VSSOP10_DGS_TEX"
 			(at 335.28 189.23 0)
 			(hide yes)
@@
 			)
 		)
-		(property "Footprint" "VSSOP10_DGS_TEX"
+		(property "Footprint" "sts1000:VSSOP10_DGS_TEX"
 			(at 334.01 92.71 0)
 			(hide yes)

Commit message: Add files via upload
Updated, completed placement
Parts:
- C63, C67, C68, C69, C70, C83, C86, C87: footprint 0402 (1005 Metric) -> copy_ref:C_0402_1005Metric
- C64, C65, C66, C73, C74, C76, C78: footprint 1206 (3216 Metric) -> copy_ref:C_1206_3216Metric
- C71, C72: footprint 1210 (3225 Metric) -> copy_ref:C_1210_3225Metric
- C75, C77, C80: footprint 2220 (5750 Metric) -> Capacitor_SMD:C_2220_5750Metric
- C79, C81, C82: footprint 0805 (2012 Metric) -> copy_ref:C_0805_2012Metric
- C84, C85: footprint 0603 (1608 Metric) -> copy_ref:C_0603_1608Metric
- FB7: footprint 1206 (3216 Metric) -> copy_ref:1206
- L2: footprint (none) -> dowload:SRP1265A-6R8M
- L3: footprint (none) -> dowload:DR73-2R2-R
- R100, R101, R103, R104, R105, R90, R91, R92, R93, R94, R95, R96, R97, R98, R99: footprint 0402 (1005 Metric) -> copy_ref:R_0402_1005Metric
- R102, R106, R107: footprint 1206 (3216 Metric) -> copy_ref:R_1206_3216Metric
- U28: footprint 32-PowerVQFN -> copy_ref:MIC28516T-EPHA
- U29: footprint 8-UFDFN (Exposed Pad) -> dowload:AP3441SHE-7B_DIO-M
- U33: footprint TSOT-23-5 -> Package_TO_SOT_SMD:TSOT-23-5
Changed lines of the file:
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@@
 			)
 		)
-		(property "Footprint" "32-PowerVQFN"
+		(property "Footprint" "copy_ref:MIC28516T-EPHA"
 			(at 237.49 45.72 0)
 			(hide yes)
@@
 			)
 		)
-		(property "Footprint" "1206 (3216 Metric)"
+		(property "Footprint" "copy_ref:C_1206_3216Metric"
 			(at 93.0148 175.26 0)
 			(hide yes)
@@
 			)
 		)
-		(property "Footprint" "TSOT-23-5"
+		(property "Footprint" "Package_TO_SOT_SMD:TSOT-23-5"
 			(at 336.55 162.56 0)
 			(hide yes)
@@
 			)
 		)
-		(property "Footprint" "1206 (3216 Metric)"
+		(property "Footprint" "copy_ref:C_1206_3216Metric"
 			(at 167.3352 175.26 0)
 			(hide yes)
@@
 			)
 		)
-		(property "Footprint" "0805 (2012 Metric)"
+		(property "Footprint" "copy_ref:C_0805_2012Metric"
 			(at 221.9452 55.88 0)
 			(hide yes)
@@
 			)
 		)
-		(property "Footprint" "0402 (1005 Metric)"
+		(property "Footprint" "copy_ref:R_0402_1005Metric"
 			(at 121.412 72.39 90)
 			(hide yes)
@@
 			)
 		)
-		(property "Footprint" "1206 (3216 Metric)"
+		(property "Footprint" "copy_ref:R_1206_3216Metric"
 			(at 226.06 164.592 90)
 			(hide yes)
@@
 			)
 		)
-		(property "Footprint" "2220 (5750 Metric)"
+		(property "Footprint" "Capacitor_SMD:C_2220_5750Metric"
 			(at 209.8548 74.93 0)
 			(hide yes)
@@
 			)
 		)
-		(property "Footprint" "0402 (1005 Metric)"
+		(property "Footprint" "copy_ref:C_0402_1005Metric"
 			(at 113.9952 85.09 0)
 			(hide yes)
@@
 			)
 		)
-		(property "Footprint" "0402 (1005 Metric)"
+		(property "Footprint" "copy_ref:R_0402_1005Metric"
 			(at 196.85 88.392 90)
 			(hide yes)
@@
 			)
 		)
-		(property "Footprint" "8-UFDFN (Exposed Pad)"
+		(property "Footprint" "dowload:AP3441SHE-7B_DIO-M"
 			(at 114.3 173.99 0)
 			(hide yes)
@@
 			)
 		)
-		(property "Footprint" "0402 (1005 Metric)"
+		(property "Footprint" "copy_ref:R_0402_1005Metric"
 			(at 346.202 137.16 90)
 			(hide yes)
@@
 			)
 		)
-		(property "Footprint" ""
+		(property "Footprint" "dowload:DR73-2R2-R"
 			(at 133.35 166.37 0)
 			(hide yes)
@@
 			)
 		)
-		(property "Footprint" "0805 (2012 Metric)"
+		(property "Footprint" "copy_ref:C_0805_2012Metric"
 			(at 226.3648 85.09 0)
 			(hide yes)
@@
 			)
 		)
-		(property "Footprint" "0402 (1005 Metric)"
+		(property "Footprint" "copy_ref:C_0402_1005Metric"
 			(at 385.7752 110.49 0)
 			(hide yes)
@@
 			)
 		)
-		(property "Footprint" "0402 (1005 Metric)"
+		(property "Footprint" "copy_ref:R_0402_1005Metric"
 			(at 41.402 60.96 90)
 			(hide yes)
@@
 			)
 		)
-		(property "Footprint" "0805 (2012 Metric)"
+		(property "Footprint" "copy_ref:C_0805_2012Metric"
 			(at 205.4352 99.06 0)
 			(hide yes)
@@
 			)
 		)
-		(property "Footprint" "0402 (1005 Metric)"
+		(property "Footprint" "copy_ref:R_0402_1005Metric"
 			(at 88.9 149.098 90)
 			(hide yes)
@@
 			)
 		)
-		(property "Footprint" "1206 (3216 Metric)"
+		(property "Footprint" "copy_ref:1206"
 			(at 391.668 146.05 90)
 			(hide yes)
@@
 			)
 		)
-		(property "Footprint" "2220 (5750 Metric)"
+		(property "Footprint" "Capacitor_SMD:C_2220_5750Metric"
 			(at 197.1548 74.93 0)
 			(hide yes)
@@
 			)
 		)
-		(property "Footprint" "1206 (3216 Metric)"
+		(property "Footprint" "copy_ref:C_1206_3216Metric"
 			(at 81.5848 175.26 0)
 			(hide yes)
@@
 			)
 		)
-		(property "Footprint" "0402 (1005 Metric)"
+		(property "Footprint" "copy_ref:R_0402_1005Metric"
 			(at 84.328 151.13 90)
 			(hide yes)
@@
 			)
 		)
-		(property "Footprint" "0402 (1005 Metric)"
+		(property "Footprint" "copy_ref:R_0402_1005Metric"
 			(at 225.552 60.96 90)
 			(hide yes)
@@
 			)
 		)
-		(property "Footprint" "0402 (1005 Metric)"
+		(property "Footprint" "copy_ref:R_0402_1005Metric"
 			(at 107.442 40.64 90)
 			(hide yes)
@@
 			)
 		)
-		(property "Footprint" "0402 (1005 Metric)"
+		(property "Footprint" "copy_ref:C_0402_1005Metric"
 			(at 61.9252 69.85 0)
 			(hide yes)
@@
 			)
 		)
-		(property "Footprint" "0402 (1005 Metric)"
+		(property "Footprint" "copy_ref:C_0402_1005Metric"
 			(at 134.3152 76.2 0)
 			(hide yes)
@@
 			)
 		)
-		(property "Footprint" "1206 (3216 Metric)"
+		(property "Footprint" "copy_ref:C_1206_3216Metric"
 			(at 70.1548 175.26 0)
 			(hide yes)
@@
 			)
 		)
-		(property "Footprint" "1210 (3225 Metric)"
+		(property "Footprint" "copy_ref:C_1210_3225Metric"
 			(at 147.0152 76.2 0)
 			(hide yes)
@@
 			)
 		)
-		(property "Footprint" "0402 (1005 Metric)"
+		(property "Footprint" "copy_ref:R_0402_1005Metric"
 			(at 150.622 181.61 90)
 			(hide yes)
@@
 			)
 		)
-		(property "Footprint" "0402 (1005 Metric)"
+		(property "Footprint" "copy_ref:C_0402_1005Metric"
 			(at 141.9352 175.26 0)
 			(hide yes)
@@
 			)
 		)
-		(property "Footprint" "1206 (3216 Metric)"
+		(property "Footprint" "copy_ref:R_1206_3216Metric"
 			(at 383.54 150.622 90)
 			(hide yes)
@@
 			)
 		)
-		(property "Footprint" "0402 (1005 Metric)"
+		(property "Footprint" "copy_ref:R_0402_1005Metric"
 			(at 121.412 93.98 90)
 			(hide yes)
@@
 			)
 		)
-		(property "Footprint" "0402 (1005 Metric)"
+		(property "Footprint" "copy_ref:R_0402_1005Metric"
 			(at 111.252 72.39 90)
 			(hide yes)
@@
 			)
 		)
-		(property "Footprint" "1206 (3216 Metric)"
+		(property "Footprint" "copy_ref:C_1206_3216Metric"
 			(at 191.4652 175.26 0)
 			(hide yes)
@@
 			)
 		)
-		(property "Footprint" "0402 (1005 Metric)"
+		(property "Footprint" "copy_ref:C_0402_1005Metric"
 			(at 387.0452 207.01 0)
 			(hide yes)
@@
 			)
 		)
-		(property "Footprint" "2220 (5750 Metric)"
+		(property "Footprint" "Capacitor_SMD:C_2220_5750Metric"
 			(at 184.4548 74.93 0)
 			(hide yes)
@@
 			)
 		)
-		(property "Footprint" "0402 (1005 Metric)"
+		(property "Footprint" "copy_ref:R_0402_1005Metric"
 			(at 36.83 57.658 90)
 			(hide yes)
@@
 			)
 		)
-		(property "Footprint" "0402 (1005 Metric)"
+		(property "Footprint" "copy_ref:C_0402_1005Metric"
 			(at 117.8052 58.42 0)
 			(hide yes)
@@
 			)
 		)
-		(property "Footprint" "1206 (3216 Metric)"
+		(property "Footprint" "copy_ref:R_1206_3216Metric"
 			(at 382.27 54.102 90)
 			(hide yes)
@@
 			)
 		)
-		(property "Footprint" "0402 (1005 Metric)"
+		(property "Footprint" "copy_ref:R_0402_1005Metric"
 			(at 150.622 171.45 90)
 			(hide yes)
@@
 			)
 		)
-		(property "Footprint" "1206 (3216 Metric)"
+		(property "Footprint" "copy_ref:C_1206_3216Metric"
 			(at 178.7652 175.26 0)
 			(hide yes)
@@
 			)
 		)
-		(property "Footprint" "0402 (1005 Metric)"
+		(property "Footprint" "copy_ref:C_0402_1005Metric"
 			(at 228.2952 223.52 0)
 			(hide yes)
@@
 			)
 		)
-		(property "Footprint" "0603 (1608 Metric)"
+		(property "Footprint" "copy_ref:C_0603_1608Metric"
 			(at 317.8048 147.32 0)
 			(hide yes)
@@
 			)
 		)
-		(property "Footprint" "32-PowerVQFN"
+		(property "Footprint" "copy_ref:MIC28516T-EPHA"
 			(at 64.77 50.8 0)
 			(hide yes)
@@
 			)
 		)
-		(property "Footprint" "1206 (3216 Metric)"
+		(property "Footprint" "copy_ref:C_1206_3216Metric"
 			(at 202.8952 175.26 0)
 			(hide yes)
@@
 			)
 		)
-		(property "Footprint" ""
+		(property "Footprint" "dowload:SRP1265A-6R8M"
 			(at 118.11 67.31 0)
 			(hide yes)
@@
 			)
 		)
-		(property "Footprint" "0402 (1005 Metric)"
+		(property "Footprint" "copy_ref:R_0402_1005Metric"
 			(at 85.09 86.868 90)
 			(hide yes)
@@
 			)
 		)
-		(property "Footprint" "0402 (1005 Metric)"
+		(property "Footprint" "copy_ref:R_0402_1005Metric"
 			(at 328.168 162.56 90)
 			(hide yes)
@@
 			)
 		)
-		(property "Footprint" "1210 (3225 Metric)"
+		(property "Footprint" "copy_ref:C_1210_3225Metric"
 			(at 160.9852 76.2 0)
 			(hide yes)
@@
 			)
 		)
-		(property "Footprint" "0603 (1608 Metric)"
+		(property "Footprint" "copy_ref:C_0603_1608Metric"
 			(at 366.0648 161.29 0)
 			(hide yes)

Commit message: PCB / 3D updates
Parts:
- U32: value INA228AQDGSRQ1 -> RT9742VGJ5
Changed lines of the file:
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@@
 			)
 		)
-		(property "Value" "INA228AQDGSRQ1"
+		(property "Value" "RT9742VGJ5"
 			(at 355.6 181.61 0)
 			(show_name no)
