File: hardware/ntp-server-stm32/batt-supplies.kicad_sch (KiCad schematic)
At the start: 24 parts, among them U34 TPS61094DSSR, U35 TPS61094DSSR

Commit message: Standardize net/rail names: plain 3V3 style, _N active-low, voltage-format PG/alerts
22 net renames applied across all sheets and verified: removed/added net-name
sets match intent exactly and all node connectivity is preserved (kicad-cli
netlist re-parse).

Co-Authored-By: Claude Opus 4.8 (1M context) <noreply@anthropic.com>
Connections:
- net +3.3V renamed 3V3
Changed lines of the file:
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@@
 			)
 		)
-		(property "Value" "+3.3V"
+		(property "Value" "3V3"
 			(at 99.06 154.94 0)
 			(show_name no)
@@
 			)
 		)
-		(property "Value" "+3.3V"
+		(property "Value" "3V3"
 			(at 99.06 63.5 0)
 			(show_name no)

Commit message: Standardize + complete BOM; write fields back into KiCad symbols
- New sts1000_bom.csv: rebuilt from authoritative Value field (source MPN/footprint/
  description were corrupted by copy-paste). 338 standardized, 78 MPN-from-value,
  50 kept, ~64 flagged (SELECT/REVIEW-HV/SHUNT-REVIEW) each with full spec.
- Resistors -> deterministic Panasonic ERJ-2RKF 0402 1% 1/10W (consolidated 1 part/value).
- Caps -> verified Murata GRM parts where value matches; clean spec + footprint otherwise.
- 1633 symbol field updates (Value/Footprint/Description/MPN/Mfr/Digikey) written to
  .kicad_sch; netlist re-parse confirms connectivity byte-identical.
- Add docs/sts1000_net_naming.md naming reference.

Co-Authored-By: Claude Opus 4.8 (1M context) <noreply@anthropic.com>
Parts:
- C88, C89: footprint (none) -> C_0805_2012Metric; DIGIKEY_PART_NUMBER (none) -> 490-GRM21BZ71C106KE15LTR-ND; MANUFACTURER (none) -> Murata; MANUFACTURER_PART_NUMBER (none) -> GRM21BZ71C106KE15L
- C92, C93, C94, C95, C96, C97: footprint (none) -> C_0805_2012Metric
- R108, R109, R110, R111: footprint (none) -> R_0402_1005Metric; MANUFACTURER (none) -> Panasonic; MANUFACTURER_PART_NUMBER (none) -> ERJ-2RKF1003X
- R112, R113: footprint (none) -> R_0402_1005Metric; MANUFACTURER (none) -> Panasonic; MANUFACTURER_PART_NUMBER (none) -> ERJ-2RKF6651X
- R114, R115: footprint (none) -> R_0402_1005Metric; MANUFACTURER (none) -> Panasonic; MANUFACTURER_PART_NUMBER (none) -> ERJ-2RKF9531X
- R116, R117: footprint (none) -> R_0402_1005Metric; MANUFACTURER (none) -> Panasonic; MANUFACTURER_PART_NUMBER (none) -> ERJ-2RKF3091X
- U34, U35: MANUFACTURER_PART_NUMBER (none) -> TPS61094DSSR
