File: hardware/ntp-server-stm32/ethernet-input.kicad_sch (KiCad schematic)
At the start: 5 parts, among them J1 0826-1X1T-HS-F, U1 TPD4EUSB30

Commit message: Updates
Parts:
- C1: footprint C_0402_1005Metric -> 1812 (4532 Metric); DIELECTRIC (none) -> X7R; DIGIKEY_PART_NUMBER 490-6334-2-ND -> 399-16791-1-ND; MANUFACTURER Murata -> KEMET; MANUFACTURER_PART_NUMBER GRM155R71C472KA01D -> C1812C472KGRACAUTO; TOLERANCE (none) -> 10%; VOLTAGE (none) -> 2kV
- C2: footprint C_0402_1005Metric -> 0402 (1005 Metric); DIELECTRIC (none) -> X7R; DIGIKEY_PART_NUMBER 490-3542-2-ND -> 399-C0402C223J5RACAUTOCT-ND; MANUFACTURER (none) -> KEMET; MANUFACTURER_PART_NUMBER GRM31CR72E104KW03L -> C0402C223J5RACAUTO; TOLERANCE (none) -> 10%; VOLTAGE (none) -> 50V
- J1: MANUFACTURER Bel Fuse -> Bel/Stewart
- R1: footprint R_0402_1005Metric -> 0402 (1005 Metric); DIELECTRIC (none) -> Thick-film; DIGIKEY_PART_NUMBER (none) -> P1.00MLCT-ND; MANUFACTURER Panasonic -> Panasonic Industry; POWER (none) -> 1/10W; TOLERANCE (none) -> 1%
Changed lines of the file:
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@@
 			)
 		)
-		(property "Description" "CONN JACK 1PORT 1000 BASE-T PCB"
+		(property "Description" "RJ45 magjack 1000BASE-T"
 			(at 138.43 116.84 0)
 			(hide yes)
@@
 			)
 		)
-		(property "MANUFACTURER" "Bel Fuse"
+		(property "MANUFACTURER" "Bel/Stewart"
 			(at 138.43 116.84 0)
 			(hide yes)
@@
 			)
 		)
-		(property "Footprint" "R_0402_1005Metric"
+		(property "Footprint" "0402 (1005 Metric)"
 			(at 97.028 160.02 90)
 			(hide yes)
@@
 			)
 		)
-		(property "Datasheet" ""
+		(property "Datasheet" "https://industrial.panasonic.com/cdbs/www-data/pdf/RDA0000/AOA0000C304.pdf"
 			(at 95.25 160.02 0)
 			(hide yes)
@@
 			)
 		)
-		(property "MANUFACTURER" "Panasonic"
+		(property "POWER" "1/10W"
+			(at 0 0 0)
+			(hide yes)
+			(show_name no)
+			(do_not_autoplace no)
+			(effects
+				(font
+					(size 1.27 1.27)
+				)
+			)
+		)
+		(property "DIELECTRIC" "Thick-film"
+			(at 0 0 0)
+			(hide yes)
+			(show_name no)
+			(do_not_autoplace no)
+			(effects
+				(font
+					(size 1.27 1.27)
+				)
+			)
+		)
+		(property "TOLERANCE" "1%"
+			(at 0 0 0)
+			(hide yes)
+			(show_name no)
+			(do_not_autoplace no)
+			(effects
+				(font
+					(size 1.27 1.27)
+				)
+			)
+		)
+		(property "MANUFACTURER" "Panasonic Industry"
 			(at 0 0 0)
 			(hide yes)
@@
 		(property "MANUFACTURER_PART_NUMBER" "ERJ-2RKF1004X"
 			(at 0 0 0)
+			(hide yes)
+			(show_name no)
+			(do_not_autoplace no)
+			(effects
+				(font
+					(size 1.27 1.27)
+				)
+			)
+		)
+		(property "DIGIKEY_PART_NUMBER" "P1.00MLCT-ND"
+			(at 95.25 160.02 0)
 			(hide yes)
 			(show_name no)
@@
 		)
 		(property "Value" "4.7nF"
-			(at 107.95 161.2899 0)
+			(at 104.648 162.56 0)
 			(show_name no)
 			(do_not_autoplace no)
@@
 			)
 		)
-		(property "Footprint" "C_0402_1005Metric"
+		(property "Footprint" "1812 (4532 Metric)"
 			(at 103.8352 163.83 0)
 			(hide yes)
@@
 			)
 		)
-		(property "Datasheet" "https://product.tdk.com/system/files/dam/doc/product/capacitor/ceramic/mlcc/catalog/mlcc_commercial_general_en.pdf"
+		(property "Datasheet" "https://yageogroup.com/content/datasheet/asset/file/KEM_C1076_X7R_HV_AUTO_SMD"
 			(at 102.87 160.02 0)
 			(hide yes)
@@
 			)
 		)
-		(property "Description" "CAP CER 4.7nF 16V X7R 0402"
+		(property "Description" "CAP CER 1812 4.7NF 2000V X7R 10%"
 			(at 102.87 160.02 0)
 			(hide yes)
@@
 			)
 		)
-		(property "DIGIKEY_PART_NUMBER" "490-6334-2-ND"
+		(property "DIELECTRIC" "X7R"
+			(at 0 0 0)
+			(hide yes)
+			(show_name no)
+			(do_not_autoplace no)
+			(effects
+				(font
+					(size 1.27 1.27)
+				)
+			)
+		)
+		(property "TOLERANCE" "10%"
+			(at 0 0 0)
+			(hide yes)
+			(show_name no)
+			(do_not_autoplace no)
+			(effects
+				(font
+					(size 1.27 1.27)
+				)
+			)
+		)
+		(property "VOLTAGE" "2kV"
+			(at 0 0 0)
+			(hide yes)
+			(show_name no)
+			(do_not_autoplace no)
+			(effects
+				(font
+					(size 1.27 1.27)
+				)
+			)
+		)
+		(property "DIGIKEY_PART_NUMBER" "399-16791-1-ND"
 			(at 102.87 160.02 0)
 			(hide yes)
@@
 			)
 		)
-		(property "MANUFACTURER" "Murata"
+		(property "MANUFACTURER" "KEMET"
 			(at 102.87 160.02 0)
 			(hide yes)
@@
 			)
 		)
-		(property "MANUFACTURER_PART_NUMBER" "GRM155R71C472KA01D"
+		(property "MANUFACTURER_PART_NUMBER" "C1812C472KGRACAUTO"
 			(at 102.87 160.02 0)
 			(hide yes)
@@
 			)
 		)
-		(property "Footprint" "C_0402_1005Metric"
+		(property "Footprint" "0402 (1005 Metric)"
 			(at 120.3452 163.83 0)
 			(hide yes)
@@
 			)
 		)
-		(property "Datasheet" "https://search.murata.co.jp/Ceramy/image/img/A01X/G101/ENG/GRM31CR72E104KW03-01.pdf"
+		(property "Datasheet" "https://yageogroup.com/content/datasheet/asset/file/KEM_C1023_X7R_AUTO_SMD"
 			(at 119.38 160.02 0)
 			(hide yes)
@@
 			)
 		)
-		(property "Description" "CAP CER 0.022uF 50V X7R 0402"
+		(property "Description" "CAP CER 0.022UF 50V X7R 0402"
 			(at 119.38 160.02 0)
 			(hide yes)
@@
 			)
 		)
-		(property "DIGIKEY_PART_NUMBER" "490-3542-2-ND"
+		(property "DIELECTRIC" "X7R"
+			(at 0 0 0)
+			(hide yes)
+			(show_name no)
+			(do_not_autoplace no)
+			(effects
+				(font
+					(size 1.27 1.27)
+				)
+			)
+		)
+		(property "TOLERANCE" "10%"
+			(at 0 0 0)
+			(hide yes)
+			(show_name no)
+			(do_not_autoplace no)
+			(effects
+				(font
+					(size 1.27 1.27)
+				)
+			)
+		)
+		(property "VOLTAGE" "50V"
+			(at 0 0 0)
+			(hide yes)
+			(show_name no)
+			(do_not_autoplace no)
+			(effects
+				(font
+					(size 1.27 1.27)
+				)
+			)
+		)
+		(property "MANUFACTURER" "KEMET"
+			(at 0 0 0)
+			(hide yes)
+			(show_name no)
+			(do_not_autoplace no)
+			(effects
+				(font
+					(size 1.27 1.27)
+				)
+			)
+		)
+		(property "DIGIKEY_PART_NUMBER" "399-C0402C223J5RACAUTOCT-ND"
 			(at 119.38 160.02 0)
 			(hide yes)
@@
 			)
 		)
-		(property "MANUFACTURER_PART_NUMBER" "GRM31CR72E104KW03L"
+		(property "MANUFACTURER_PART_NUMBER" "C0402C223J5RACAUTO"
 			(at 119.38 160.02 0)
 			(hide yes)
@@
 			)
 		)
-		(property "Description" "TVS DIODE 5.5VWM 8VC 10USON"
+		(property "Description" "USB ESD array"
 			(at 78.74 43.18 0)
 			(hide yes)

Commit message: Bom updates
Parts:
- U1: DIGIKEY_PART_NUMBER 296-28063-2-ND -> 296-28063-1-ND
Changed lines of the file:
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@@
 			)
 		)
-		(property "DIGIKEY_PART_NUMBER" "296-28063-2-ND"
+		(property "DIGIKEY_PART_NUMBER" "296-28063-1-ND"
 			(at 78.74 43.18 0)
 			(hide yes)

Commit message: Add files via upload
Updated, completed placement
Parts:
- C1: footprint 1812 (4532 Metric) -> Capacitor_SMD:C_1812_4532Metric
- C2: footprint 0402 (1005 Metric) -> copy_ref:C_0402_1005Metric
- J1: footprint (none) -> copy_ref:BEL_0826-1X1T-GH-F
- R1: footprint 0402 (1005 Metric) -> copy_ref:R_0402_1005Metric
- U1: footprint 10-USON -> dowload:TPD4E02B04DQAR
Changed lines of the file:
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@@
 			)
 		)
-		(property "Footprint" ""
+		(property "Footprint" "copy_ref:BEL_0826-1X1T-GH-F"
 			(at 138.43 116.84 0)
 			(hide yes)
@@
 			)
 		)
-		(property "Footprint" "0402 (1005 Metric)"
+		(property "Footprint" "copy_ref:R_0402_1005Metric"
 			(at 97.028 160.02 90)
 			(hide yes)
@@
 			)
 		)
-		(property "Footprint" "1812 (4532 Metric)"
+		(property "Footprint" "Capacitor_SMD:C_1812_4532Metric"
 			(at 103.8352 163.83 0)
 			(hide yes)
@@
 			)
 		)
-		(property "Footprint" "0402 (1005 Metric)"
+		(property "Footprint" "copy_ref:C_0402_1005Metric"
 			(at 120.3452 163.83 0)
 			(hide yes)
@@
 			)
 		)
-		(property "Footprint" "10-USON"
+		(property "Footprint" "dowload:TPD4E02B04DQAR"
 			(at 54.61 53.34 0)
 			(hide yes)
