File: hardware/ntp-server-stm32/ethernet-phy.kicad_sch (KiCad schematic)
At the start: 26 parts, among them U11 LAN8742AI-CZ-TR, Y1 25MHz

Commit message: Standardize net/rail names: plain 3V3 style, _N active-low, voltage-format PG/alerts
22 net renames applied across all sheets and verified: removed/added net-name
sets match intent exactly and all node connectivity is preserved (kicad-cli
netlist re-parse).

Co-Authored-By: Claude Opus 4.8 (1M context) <noreply@anthropic.com>
Connections:
- net +3.3V renamed 3V3
- net +3.3V_LAN renamed 3V3_LAN
- net LAN_nRST renamed LAN_RST_N
Changed lines of the file:
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@@
 		)
 	)
-	(global_label "LAN_nRST"
+	(global_label "LAN_RST_N"
 		(shape input)
 		(at 46.99 80.01 180)
@@
 			)
 		)
-		(property "Value" "+3.3V"
+		(property "Value" "3V3"
 			(at 133.35 40.64 0)
 			(show_name no)
@@
 			)
 		)
-		(property "Value" "+3.3V_LAN"
+		(property "Value" "3V3_LAN"
 			(at 36.83 19.05 0)
 			(show_name no)
@@
 			)
 		)
-		(property "Value" "+3.3V_LAN"
+		(property "Value" "3V3_LAN"
 			(at 200.66 57.15 0)
 			(show_name no)
@@
 			)
 		)
-		(property "Value" "+3.3V_LAN"
+		(property "Value" "3V3_LAN"
 			(at 63.5 55.88 0)
 			(show_name no)
@@
 			)
 		)
-		(property "Value" "+3.3V"
+		(property "Value" "3V3"
 			(at 24.13 20.32 0)
 			(show_name no)
@@
 			)
 		)
-		(property "Value" "+3.3V_LAN"
+		(property "Value" "3V3_LAN"
 			(at 223.52 121.92 0)
 			(show_name no)
@@
 			)
 		)
-		(property "Value" "+3.3V_LAN"
+		(property "Value" "3V3_LAN"
 			(at 214.63 58.42 0)
 			(show_name no)

Commit message: Standardize + complete BOM; write fields back into KiCad symbols
- New sts1000_bom.csv: rebuilt from authoritative Value field (source MPN/footprint/
  description were corrupted by copy-paste). 338 standardized, 78 MPN-from-value,
  50 kept, ~64 flagged (SELECT/REVIEW-HV/SHUNT-REVIEW) each with full spec.
- Resistors -> deterministic Panasonic ERJ-2RKF 0402 1% 1/10W (consolidated 1 part/value).
- Caps -> verified Murata GRM parts where value matches; clean spec + footprint otherwise.
- 1633 symbol field updates (Value/Footprint/Description/MPN/Mfr/Digikey) written to
  .kicad_sch; netlist re-parse confirms connectivity byte-identical.
- Add docs/sts1000_net_naming.md naming reference.

Co-Authored-By: Claude Opus 4.8 (1M context) <noreply@anthropic.com>
Parts:
- C13: footprint (none) -> C_0805_2012Metric; DIGIKEY_PART_NUMBER (none) -> 490-GRM21BR71C475KE51KTR-ND; MANUFACTURER (none) -> Murata; MANUFACTURER_PART_NUMBER (none) -> GRM21BR71C475KE51K
- C14, C16, C17: footprint (none) -> C_0402_1005Metric
- C15, C19, C20: footprint (none) -> C_0402_1005Metric; DIGIKEY_PART_NUMBER (none) -> 490-6328-2-ND; MANUFACTURER (none) -> Murata; MANUFACTURER_PART_NUMBER (none) -> GRM155R71C104KA88J
- C18: footprint (none) -> C_0603_1608Metric
- R31, R32, R33, R34: footprint (none) -> R_0402_1005Metric; MANUFACTURER (none) -> Panasonic; MANUFACTURER_PART_NUMBER (none) -> ERJ-2RKF1000X
- R35: footprint (none) -> R_0402_1005Metric; MANUFACTURER (none) -> Panasonic; MANUFACTURER_PART_NUMBER (none) -> ERJ-2RKF1002X
- R36: footprint (none) -> R_0402_1005Metric; MANUFACTURER (none) -> Panasonic; MANUFACTURER_PART_NUMBER (none) -> ERJ-2RKF1501X
- R37: footprint (none) -> R_0402_1005Metric; MANUFACTURER (none) -> Panasonic; MANUFACTURER_PART_NUMBER (none) -> ERJ-2RKF1212X
- R38, R39: footprint (none) -> R_0402_1005Metric; MANUFACTURER (none) -> Panasonic; MANUFACTURER_PART_NUMBER (none) -> ERJ-2RKF3300X
- R40, R41: footprint (none) -> R_0402_1005Metric; MANUFACTURER (none) -> Panasonic; MANUFACTURER_PART_NUMBER (none) -> ERJ-2RKF4751X
- R42, R43, R44, R45: footprint (none) -> R_0402_1005Metric; MANUFACTURER (none) -> Panasonic; MANUFACTURER_PART_NUMBER (none) -> ERJ-2RKF49R9X
- U11: MANUFACTURER_PART_NUMBER (none) -> LAN8742AI-CZ-TR
