File: hardware/ntp-server-stm32/gps-antenna.kicad_sch (KiCad schematic)
At the start: 40 parts, among them Q11 NSS40300MZ4T1G, Q12 BC857W, Q13 BC857W, Q14 BC847W, U24 INA181A1IDBVR, U25 LMV393, U26 INA228AQDGSRQ1, U27 RT9742VGJ5

Commit message: Standardize net/rail names: plain 3V3 style, _N active-low, voltage-format PG/alerts
22 net renames applied across all sheets and verified: removed/added net-name
sets match intent exactly and all node connectivity is preserved (kicad-cli
netlist re-parse).

Co-Authored-By: Claude Opus 4.8 (1M context) <noreply@anthropic.com>
Connections:
- net +3.3V renamed 3V3
- net +3.3V_GPS renamed 3V3_GPS
- net +5V renamed 5V
Changed lines of the file:
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@@
 			)
 		)
-		(property "Value" "+3.3V_GPS"
+		(property "Value" "3V3_GPS"
 			(at 179.07 125.73 0)
 			(show_name no)
@@
 			)
 		)
-		(property "Value" "+5V"
+		(property "Value" "5V"
 			(at 292.1 146.05 0)
 			(show_name no)
@@
 			)
 		)
-		(property "Value" "+3.3V"
+		(property "Value" "3V3"
 			(at 346.71 194.31 0)
 			(show_name no)
@@
 			)
 		)
-		(property "Value" "+3.3V_GPS"
+		(property "Value" "3V3_GPS"
 			(at 104.14 113.03 0)
 			(show_name no)
@@
 			)
 		)
-		(property "Value" "+3.3V_GPS"
+		(property "Value" "3V3_GPS"
 			(at 116.84 60.96 0)
 			(show_name no)
@@
 			)
 		)
-		(property "Value" "+3.3V_GPS"
+		(property "Value" "3V3_GPS"
 			(at 143.51 116.84 0)
 			(show_name no)
@@
 			)
 		)
-		(property "Value" "+3.3V"
+		(property "Value" "3V3"
 			(at 294.64 181.61 0)
 			(show_name no)
@@
 			)
 		)
-		(property "Value" "+5V"
+		(property "Value" "5V"
 			(at 219.71 73.66 0)
 			(show_name no)
@@
 			)
 		)
-		(property "Value" "+3.3V_GPS"
+		(property "Value" "3V3_GPS"
 			(at 146.05 71.12 0)
 			(show_name no)

Commit message: Standardize + complete BOM; write fields back into KiCad symbols
- New sts1000_bom.csv: rebuilt from authoritative Value field (source MPN/footprint/
  description were corrupted by copy-paste). 338 standardized, 78 MPN-from-value,
  50 kept, ~64 flagged (SELECT/REVIEW-HV/SHUNT-REVIEW) each with full spec.
- Resistors -> deterministic Panasonic ERJ-2RKF 0402 1% 1/10W (consolidated 1 part/value).
- Caps -> verified Murata GRM parts where value matches; clean spec + footprint otherwise.
- 1633 symbol field updates (Value/Footprint/Description/MPN/Mfr/Digikey) written to
  .kicad_sch; netlist re-parse confirms connectivity byte-identical.
- Add docs/sts1000_net_naming.md naming reference.

Co-Authored-By: Claude Opus 4.8 (1M context) <noreply@anthropic.com>
Parts:
- C52, C57: footprint (none) -> C_0603_1608Metric
- C53, C54, C55, C56, C58, C60, C61: footprint (none) -> C_0402_1005Metric; DIGIKEY_PART_NUMBER (none) -> 490-6328-2-ND; MANUFACTURER (none) -> Murata; MANUFACTURER_PART_NUMBER (none) -> GRM155R71C104KA88J
- C59: footprint (none) -> C_0805_2012Metric; DIGIKEY_PART_NUMBER (none) -> 490-GRM21BZ71C106KE15LTR-ND; MANUFACTURER (none) -> Murata; MANUFACTURER_PART_NUMBER (none) -> GRM21BZ71C106KE15L
- C62: footprint (none) -> C_0402_1005Metric; DIGIKEY_PART_NUMBER (none) -> 490-GRM1555C1H102FA01JTR-ND; MANUFACTURER (none) -> Murata; MANUFACTURER_PART_NUMBER (none) -> GRM1555C1H102FA01J
- Q12, Q13: MANUFACTURER_PART_NUMBER (none) -> BC857W
- Q14: MANUFACTURER_PART_NUMBER (none) -> BC847W
- R73: footprint (none) -> R_0402_1005Metric; MANUFACTURER (none) -> Panasonic; MANUFACTURER_PART_NUMBER (none) -> ERJ-2RKF2201X
- R74, R79, R84, R87: footprint (none) -> R_0402_1005Metric; MANUFACTURER (none) -> Panasonic; MANUFACTURER_PART_NUMBER (none) -> ERJ-2RKF1002X
- R75: footprint (none) -> R_0402_1005Metric; MANUFACTURER (none) -> Panasonic; MANUFACTURER_PART_NUMBER (none) -> ERJ-2RKF4701X
- R76: footprint (none) -> R_0402_1005Metric; MANUFACTURER (none) -> Panasonic; MANUFACTURER_PART_NUMBER (none) -> ERJ-2RKF2200X
- R78, R80, R81, R82, R85: footprint (none) -> R_0402_1005Metric; MANUFACTURER (none) -> Panasonic; MANUFACTURER_PART_NUMBER (none) -> ERJ-2RKF1003X
- R83: footprint (none) -> R_0402_1005Metric; MANUFACTURER (none) -> Panasonic; MANUFACTURER_PART_NUMBER (none) -> ERJ-2RKF3002X
- R86: footprint (none) -> R_0402_1005Metric; MANUFACTURER (none) -> Panasonic; MANUFACTURER_PART_NUMBER (none) -> ERJ-2RKF1102X
- R88: footprint 402 -> R_0402_1005Metric; MANUFACTURER (none) -> Panasonic
- U24: MANUFACTURER_PART_NUMBER (none) -> INA181A1IDBVR
- U25: MANUFACTURER_PART_NUMBER (none) -> LMV393
- U26: MANUFACTURER_PART_NUMBER (none) -> INA228AQDGSRQ1
- U27: MANUFACTURER (none) -> Richtek USA Inc.
