File: hardware/ntp-server-stm32/gps-antenna.kicad_sch (KiCad schematic)
At the start: 40 parts, among them Q11 NSS40300MZ4T1G, Q12 BC857W, Q13 BC857W, Q14 BC847W, U24 INA181A1IDBVR, U25 LMV393, U26 INA228AQDGSRQ1, U27 RT9742VGJ5

Commit message: Updates
Parts:
- added C204: 47pF, 0402 (1005 Metric), symbol Device:C
- added R200: 10k, 0402 (1005 Metric), symbol Device:R
- C52, C57: footprint C_0603_1608Metric -> 0603 (1608 Metric); DIELECTRIC (none) -> X7R; DIGIKEY_PART_NUMBER (none) -> 399-17704-1-ND; MANUFACTURER (none) -> KEMET; MANUFACTURER_PART_NUMBER (none) -> C0603C105K4RACAUTO; TOLERANCE (none) -> 10%; VOLTAGE (none) -> 16V
- C53, C54, C55, C56, C58, C60, C61: footprint C_0402_1005Metric -> 0402 (1005 Metric); DIELECTRIC (none) -> X7R; DIGIKEY_PART_NUMBER 490-6328-2-ND -> 490-4759-1-ND; MANUFACTURER_PART_NUMBER GRM155R71C104KA88J -> GCM155R71C104KA55D; TOLERANCE (none) -> 10%; VOLTAGE (none) -> 16V
- C59: footprint C_0805_2012Metric -> 1206 (3216 Metric); DIELECTRIC (none) -> X7R; DIGIKEY_PART_NUMBER 490-GRM21BZ71C106KE15LTR-ND -> 1276-6797-1-ND; MANUFACTURER Murata -> Samsung Electro-Mechanics; MANUFACTURER_PART_NUMBER GRM21BZ71C106KE15L -> CL31B106KOHVPNE; TOLERANCE (none) -> 10%; VOLTAGE (none) -> 16V
- C62: footprint C_0402_1005Metric -> 0402 (1005 Metric); DIELECTRIC (none) -> C0G; DIGIKEY_PART_NUMBER 490-GRM1555C1H102FA01JTR-ND -> 399-C0402C102J5GECAUTOCT-ND; MANUFACTURER Murata -> KEMET; MANUFACTURER_PART_NUMBER GRM1555C1H102FA01J -> C0402C102J5GECAUTO; TOLERANCE (none) -> 5%; VOLTAGE (none) -> 50V
- FB4: DIELECTRIC (none) -> Ferrite bead; MANUFACTURER Murata Electronics -> Murata; MANUFACTURER_PART_NUMBER BLM15HB121SH1D -> BLM15HD121SN1D; POWER (none) -> 500mA
- FB5, FB6: DIELECTRIC (none) -> Ferrite bead; MANUFACTURER Murata Electronics -> Murata; MANUFACTURER_PART_NUMBER BLM31KN601SN1L -> BLM31PG601SN1L; POWER (none) -> 3A
- L1: footprint 0402 -> 0402 (1005 Metric); DIELECTRIC (none) -> Inductor; MANUFACTURER Murata Electronics -> Murata; POWER (none) -> 300mA
- Q11: footprint Package_TO_SOT_SMD:SOT-223-3_TabPin2 -> SOT-223 (TO-261); DIELECTRIC (none) -> Transistor
- Q12, Q13: footprint Package_TO_SOT_SMD:SOT-323_SC-70 -> SOT-323; DIELECTRIC (none) -> Transistor; DIGIKEY_PART_NUMBER (none) -> 1727-BC857W,135CT-ND; MANUFACTURER (none) -> Nexperia USA Inc.; MANUFACTURER_PART_NUMBER BC857W -> BC857W,135
- Q14: footprint Package_TO_SOT_SMD:SOT-323_SC-70 -> SOT-323; DIELECTRIC (none) -> Transistor; DIGIKEY_PART_NUMBER (none) -> 1727-BC847W,135CT-ND; MANUFACTURER (none) -> Nexperia USA Inc.; MANUFACTURER_PART_NUMBER BC847W -> BC847W,135
- R73: footprint R_0402_1005Metric -> 0402 (1005 Metric); DIELECTRIC (none) -> Thick-film; DIGIKEY_PART_NUMBER (none) -> P2.20KLCT-ND; MANUFACTURER Panasonic -> Panasonic Industry; POWER (none) -> 1/10W; TOLERANCE (none) -> 1%
- R74, R79, R84, R87: footprint R_0402_1005Metric -> 0402 (1005 Metric); DIELECTRIC (none) -> Thick-film; DIGIKEY_PART_NUMBER (none) -> P10.0KLCT-ND; MANUFACTURER Panasonic -> Panasonic Industry; POWER (none) -> 1/10W; TOLERANCE (none) -> 1%
- R75: footprint R_0402_1005Metric -> 0402 (1005 Metric); DIELECTRIC (none) -> Thick-film; DIGIKEY_PART_NUMBER (none) -> P4.70KLCT-ND; MANUFACTURER Panasonic -> Panasonic Industry; POWER (none) -> 1/10W; TOLERANCE (none) -> 1%
- R76: footprint R_0402_1005Metric -> 0402 (1005 Metric); DIELECTRIC (none) -> Thick-film; DIGIKEY_PART_NUMBER (none) -> P220LCT-ND; MANUFACTURER Panasonic -> Panasonic Industry; POWER (none) -> 1/10W; TOLERANCE (none) -> 1%
- R77: value 3.3 1% 0.25W -> 3.3; footprint (none) -> 0402 (1005 Metric); DIELECTRIC (none) -> Thick-film; DIGIKEY_PART_NUMBER (none) -> 2019-RK73H1ETTP3R30FCT-ND; MANUFACTURER (none) -> KOA Speer Electronics, Inc.; MANUFACTURER_PART_NUMBER (none) -> RK73H1ETTP3R30F; POWER (none) -> 1/4W; TOLERANCE (none) -> 1%
- R78, R80, R81, R82, R85: footprint R_0402_1005Metric -> 0402 (1005 Metric); DIELECTRIC (none) -> Thick-film; DIGIKEY_PART_NUMBER (none) -> P100KLCT-ND; MANUFACTURER Panasonic -> Panasonic Industry; POWER (none) -> 1/10W; TOLERANCE (none) -> 1%
- R83: footprint R_0402_1005Metric -> 0402 (1005 Metric); DIELECTRIC (none) -> Thick-film; DIGIKEY_PART_NUMBER (none) -> 2019-RK73H1ETTP3002FCT-ND; MANUFACTURER Panasonic -> KOA Speer Electronics, Inc.; MANUFACTURER_PART_NUMBER ERJ-2RKF3002X -> RK73H1ETTP3002F; POWER (none) -> 1/10W; TOLERANCE (none) -> 1%
- R86: footprint R_0402_1005Metric -> 0402 (1005 Metric); DIELECTRIC (none) -> Thick-film; DIGIKEY_PART_NUMBER (none) -> P11.0KLCT-ND; MANUFACTURER Panasonic -> Panasonic Industry; POWER (none) -> 1/10W; TOLERANCE (none) -> 1%
- R88: footprint R_0402_1005Metric -> 0402 (1005 Metric); DIELECTRIC (none) -> Thick-film; DIGIKEY_PART_NUMBER P10.0KLTR-ND -> P10.0KLCT-ND; MANUFACTURER Panasonic -> Panasonic Industry; POWER (none) -> 1/10W; TOLERANCE (none) -> 1%
- R89: footprint 0805 -> 1206 (3216 Metric); DIELECTRIC (none) -> Metal-strip shunt; DIGIKEY_PART_NUMBER 273-KDV08DR150ETCT-ND -> 273-KDV12DR100ETCT-ND; MANUFACTURER_PART_NUMBER KDV08DR150ET -> KDV12DR100ET; POWER (none) -> 1/4W; TOLERANCE (none) -> 0.5%
- U24, U26: MANUFACTURER (none) -> Texas Instruments
- U25: MANUFACTURER (none) -> Texas Instruments; MANUFACTURER_PART_NUMBER LMV393 -> LMV393IDGKR
- U27: MANUFACTURER Richtek USA Inc. -> Richtek
Connections:
- net GPS_RF_IN: now also C204.2; no longer L1.1
- net I2C_SCL: now also U26.5 (SCL); no longer U26.4 (SDA)
- net I2C_SDA: now also U26.4 (SDA); no longer U26.5 (SCL)
- net V_ANT: now also Q13.2 (E); no longer Q13.3 (C)
- net V_ANT_EN_FAULT: now also R200.2
- net at Q11.1 (B), Q12.3 (C), R73.1: now also Q13.3 (C); no longer Q13.2 (E)
- new net: C204.1, L1.1
- new net 3V3_STM: R200.1
Other:
- moved on the sheet: Q13

Commit message: Bom updates
Parts:
- FB4: footprint 0402 -> 0402 (1005 Metric)
- FB5, FB6: footprint 1206 -> 1206 (3216 Metric)
- R89: value 100m -> 150m; DIGIKEY_PART_NUMBER 273-KDV12DR100ETCT-ND -> WSLC-.15CT-ND; MANUFACTURER Ohmite -> Vishay Dale; MANUFACTURER_PART_NUMBER KDV12DR100ET -> WSL1206R1500FEA
- U24: footprint DBV0006A_N -> SOT-23-6; DIGIKEY_PART_NUMBER (none) -> 296-47656-1-ND
- U25: footprint (none) -> 8-VSSOP; DIGIKEY_PART_NUMBER (none) -> 296-13993-1-ND
- U26: DIGIKEY_PART_NUMBER (none) -> 296-INA228AQDGSRQ1CT-ND
Changed lines of the file:
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@@
 			)
 		)
-		(property "Datasheet" "https://www.ti.com/lit/gpn/ina228-q1"
+		(property "Datasheet" "https://www.ti.com/lit/ds/symlink/ina228-q1.pdf"
 			(at 295.91 190.5 0)
 			(hide yes)
@@
 			)
 		)
-		(property "Description" "Current/power monitor 20-bit I2C"
+		(property "Description" "IC PWR MONITOR 10VSSOP"
 			(at 295.91 190.5 0)
 			(hide yes)
@@
 			)
 		)
+		(property "DIGIKEY_PART_NUMBER" "296-INA228AQDGSRQ1CT-ND"
+			(at 295.91 190.5 0)
+			(hide yes)
+			(show_name no)
+			(do_not_autoplace no)
+			(effects
+				(font
+					(size 1.27 1.27)
+				)
+			)
+		)
 		(pin "2"
 		)
@@
 			)
 		)
-		(property "Footprint" ""
+		(property "Footprint" "8-VSSOP"
 			(at 137.16 88.9 0)
 			(hide yes)
@@
 			)
 		)
-		(property "Datasheet" "http://www.ti.com/lit/ds/symlink/lmv331.pdf"
+		(property "Datasheet" "https://www.ti.com/general/docs/suppproductinfo.tsp?distId=10&gotoUrl=https%3A%2F%2Fwww.ti.com%2Flit%2Fgpn%2Flmv393"
 			(at 137.16 88.9 0)
 			(hide yes)
@@
 			)
 		)
-		(property "Description" "Dual comparator low-voltage"
+		(property "Description" "IC COMPARATOR 2CH 8-VSSOP"
 			(at 137.16 88.9 0)
 			(hide yes)
@@
 			)
 		)
+		(property "DIGIKEY_PART_NUMBER" "296-13993-1-ND"
+			(at 137.16 88.9 0)
+			(hide yes)
+			(show_name no)
+			(do_not_autoplace no)
+			(effects
+				(font
+					(size 1.27 1.27)
+				)
+			)
+		)
 		(pin "6"
 		)
@@
 			)
 		)
-		(property "Value" "100m"
+		(property "Value" "150m"
 			(at 347.726 156.21 90)
 			(show_name no)
@@
 			)
 		)
-		(property "Datasheet" "https://www.ohmite.com/assets/images/res-kdv.pdf"
+		(property "Datasheet" "https://www.vishay.com/docs/30100/wsl.pdf"
 			(at 345.44 153.67 0)
 			(hide yes)
@@
 			)
 		)
-		(property "Description" "RES 0.1 OHM 0.5% 1/2W 1206"
+		(property "Description" "RES 0.15 OHM 1% 1/4W 1206"
 			(at 345.44 153.67 90)
 			(hide yes)
@@
 			)
 		)
-		(property "DIGIKEY_PART_NUMBER" "273-KDV12DR100ETCT-ND"
+		(property "DIGIKEY_PART_NUMBER" "WSLC-.15CT-ND"
 			(at 345.44 153.67 90)
 			(hide yes)
@@
 			)
 		)
-		(property "MANUFACTURER_PART_NUMBER" "KDV12DR100ET"
+		(property "MANUFACTURER_PART_NUMBER" "WSL1206R1500FEA"
 			(at 345.44 153.67 90)
 			(hide yes)
@@
 			)
 		)
-		(property "MANUFACTURER" "Ohmite"
+		(property "MANUFACTURER" "Vishay Dale"
 			(at 345.44 153.67 90)
 			(hide yes)
@@
 			)
 		)
-		(property "Footprint" "DBV0006A_N"
+		(property "Footprint" "SOT-23-6"
 			(at 120.65 148.59 0)
 			(hide yes)
@@
 			)
 		)
-		(property "Description" "Current-sense amp gain-20 SOT-23-6"
+		(property "Description" "Current Sense Amplifier 1 Circuit Rail-to-Rail SOT-23-6"
 			(at 120.65 148.59 0)
 			(hide yes)
@@
 			)
 		)
+		(property "DIGIKEY_PART_NUMBER" "296-47656-1-ND"
+			(at 120.65 148.59 0)
+			(hide yes)
+			(show_name no)
+			(do_not_autoplace no)
+			(effects
+				(font
+					(size 1.27 1.27)
+				)
+			)
+		)
 		(pin "6"
 		)
@@
 			)
 		)
-		(property "Footprint" "1206"
+		(property "Footprint" "1206 (3216 Metric)"
 			(at 221.488 85.09 90)
 			(hide yes)
@@
 			)
 		)
-		(property "Footprint" "1206"
+		(property "Footprint" "1206 (3216 Metric)"
 			(at 356.87 151.892 90)
 			(hide yes)
@@
 			)
 		)
-		(property "Footprint" "0402"
+		(property "Footprint" "0402 (1005 Metric)"
 			(at 84.328 109.22 90)
 			(hide yes)
@@
 			)
 		)
-		(property "Footprint" ""
+		(property "Footprint" "8-VSSOP"
 			(at 228.6 100.33 0)
 			(hide yes)
@@
 			)
 		)
-		(property "Datasheet" "http://www.ti.com/lit/ds/symlink/lmv331.pdf"
+		(property "Datasheet" "https://www.ti.com/general/docs/suppproductinfo.tsp?distId=10&gotoUrl=https%3A%2F%2Fwww.ti.com%2Flit%2Fgpn%2Flmv393"
 			(at 228.6 100.33 0)
 			(hide yes)
@@
 			)
 		)
-		(property "Description" "Dual comparator low-voltage"
+		(property "Description" "IC COMPARATOR 2CH 8-VSSOP"
 			(at 228.6 100.33 0)
 			(hide yes)
@@
 			)
 		)
+		(property "DIGIKEY_PART_NUMBER" "296-13993-1-ND"
+			(at 228.6 100.33 0)
+			(hide yes)
+			(show_name no)
+			(do_not_autoplace no)
+			(effects
+				(font
+					(size 1.27 1.27)
+				)
+			)
+		)
 		(pin "6"
 		)
@@
 			)
 		)
-		(property "Footprint" ""
+		(property "Footprint" "8-VSSOP"
 			(at 170.18 143.51 0)
 			(hide yes)
@@
 			)
 		)
-		(property "Datasheet" "http://www.ti.com/lit/ds/symlink/lmv331.pdf"
+		(property "Datasheet" "https://www.ti.com/general/docs/suppproductinfo.tsp?distId=10&gotoUrl=https%3A%2F%2Fwww.ti.com%2Flit%2Fgpn%2Flmv393"
 			(at 170.18 143.51 0)
 			(hide yes)
@@
 			)
 		)
-		(property "Description" "Dual comparator low-voltage"
+		(property "Description" "IC COMPARATOR 2CH 8-VSSOP"
 			(at 170.18 143.51 0)
 			(hide yes)
@@
 			(hide yes)
 			(show_name no)
+			(do_not_autoplace no)
+			(effects
+				(font
+					(size 1.27 1.27)
+				)
+			)
+		)
+		(property "DIGIKEY_PART_NUMBER" "296-13993-1-ND"
+			(at 170.18 143.51 0)
+			(hide yes)
+			(show_name no)

Commit message: Bom updates
Parts:
- removed C204: 47pF, 0402 (1005 Metric), symbol Device:C
- R77: footprint 0402 (1005 Metric) -> 1206 (3216 Metric); DIGIKEY_PART_NUMBER 2019-RK73H1ETTP3R30FCT-ND -> 738-RMCF1206FT3R30CT-ND; MANUFACTURER KOA Speer Electronics, Inc. -> Stackpole Electronics Inc; MANUFACTURER_PART_NUMBER RK73H1ETTP3R30F -> RMCF1206FT3R30
- U26: footprint VSSOP10_DGS_TEX -> sts1000:VSSOP10_DGS_TEX
Connections:
- net GPS_RF_IN: now also L1.1
Changed lines of the file:
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@@
 	(wire
 		(pts
-			(xy 87.63 76.2) (xy 91.44 76.2)
-		)
-		(stroke
-			(width 0)
-			(type default)
-		)
-	)
-	(wire
-		(pts
 			(xy 82.55 113.03) (xy 82.55 116.84)
 		)
@@
 	(wire
 		(pts
-			(xy 73.66 76.2) (xy 80.01 76.2)
+			(xy 73.66 76.2) (xy 91.44 76.2)
 		)
 		(stroke
@@
 			)
 		)
-		(property "Footprint" "VSSOP10_DGS_TEX"
+		(property "Footprint" "sts1000:VSSOP10_DGS_TEX"
 			(at 295.91 190.5 0)
 			(hide yes)
@@
 	)
 	(symbol
-		(lib_id "Device:C")
-		(at 83.82 76.2 90)
-		(mirror x)
-		(unit 1)
-		(body_style 1)
-		(exclude_from_sim no)
-		(in_bom yes)
-		(on_board yes)
-		(in_pos_files yes)
-		(dnp no)
-		(property "Reference" "C204"
-			(at 83.82 83.82 90)
-			(show_name no)
-			(do_not_autoplace no)
-			(effects
-				(font
-					(size 1.27 1.27)
-				)
-			)
-		)
-		(property "Value" "47pF"
-			(at 83.82 81.28 90)
-			(show_name no)
-			(do_not_autoplace no)
-			(effects
-				(font
-					(size 1.27 1.27)
-				)
-			)
-		)
-		(property "Footprint" "0402 (1005 Metric)"
-			(at 87.63 77.1652 0)
-			(hide yes)
-			(show_name no)
-			(do_not_autoplace no)
-			(effects
-				(font
-					(size 1.27 1.27)
-				)
-			)
-		)
-		(property "Datasheet" "https://pim.murata.com/asset/pim4/ceramicCapacitorSMD/GCM1555C1HR50BA16-01A-EN_PDF_CERAMICCAPACITORSMD"
-			(at 83.82 76.2 0)
-			(hide yes)
-			(show_name no)
-			(do_not_autoplace no)
-			(effects
-				(font
-					(size 1.27 1.27)
-				)
-			)
-		)
-		(property "Description" "CAP CER 47PF 50V C0G/NP0 0402"
-			(at 83.82 76.2 0)
-			(hide yes)
-			(show_name no)
-			(do_not_autoplace no)
-			(effects
-				(font
-					(size 1.27 1.27)
-				)
-			)
-		)
-		(property "DIELECTRIC" "X7R"
-			(at -39.37 -27.94 0)
-			(hide yes)
-			(show_name no)
-			(do_not_autoplace no)
-			(effects
-				(font
-					(size 1.27 1.27)
-				)
-			)
-		)
-		(property "TOLERANCE" "10%"
-			(at -39.37 -27.94 0)
-			(hide yes)
-			(show_name no)
-			(do_not_autoplace no)
-			(effects
-				(font
-					(size 1.27 1.27)
-				)
-			)
-		)
-		(property "VOLTAGE" "16V"
-			(at -39.37 -27.94 0)
-			(hide yes)
-			(show_name no)
-			(do_not_autoplace no)
-			(effects
-				(font
-					(size 1.27 1.27)
-				)
-			)
-		)
-		(property "MANUFACTURER" "Murata Electronics"
-			(at -39.37 -27.94 0)
-			(hide yes)
-			(show_name no)
-			(do_not_autoplace no)
-			(effects
-				(font
-					(size 1.27 1.27)
-				)
-			)
-		)
-		(property "MANUFACTURER_PART_NUMBER" "GCM1555C1H470FA16D"
-			(at -39.37 -27.94 0)
-			(hide yes)
-			(show_name no)
-			(do_not_autoplace no)
-			(effects
-				(font
-					(size 1.27 1.27)
-				)
-			)
-		)
-		(property "DIGIKEY_PART_NUMBER" "490-16445-1-ND"
-			(at -39.37 -27.94 0)
-			(hide yes)
-			(show_name no)
-			(do_not_autoplace no)
-			(effects
-				(font
-					(size 1.27 1.27)
-				)
-			)
-		)
-		(pin "2"
-		)
-		(pin "1"
-		)
-		(instances
-			(project "ntp-server-stm32"
-				(path "/4c8fa883-5b85-4079-9006-ac22e5786016/c4e88dde-49ac-40b9-90f6-1d5d3c2b8d55"
-					(reference "C204")
-					(unit 1)
-				)
-			)
-		)
-	)
-	(symbol
 		(lib_id "power:GND")
 		(at 97.79 97.79 0)
@@
 			)
 		)
-		(property "Footprint" "0402 (1005 Metric)"
+		(property "Footprint" "1206 (3216 Metric)"
 			(at 72.39 117.602 90)
 			(hide yes)
@@
 			)
 		)
-		(property "Datasheet" "https://www.koaspeer.com/pdfs/RK73H.pdf"
+		(property "Datasheet" "https://www.seielect.com/catalog/SEI-RMCF_RMCP.pdf"
 			(at 72.39 119.38 0)
 			(hide yes)
@@
 			)
 		)
-		(property "Description" "RES 3.3 OHM 1% 1/10W 0402"
+		(property "Description" "RES 3.3 OHM 1% 1/4W 1206"
 			(at 72.39 119.38 0)
 			(hide yes)
@@
 			)
 		)
-		(property "MANUFACTURER_PART_NUMBER" "RK73H1ETTP3R30F"
+		(property "MANUFACTURER_PART_NUMBER" "RMCF1206FT3R30"
 			(at 0 0 0)
 			(hide yes)
@@
 			)
 		)
-		(property "MANUFACTURER" "KOA Speer Electronics, Inc."
+		(property "MANUFACTURER" "Stackpole Electronics Inc"
 			(at 0 0 0)
 			(hide yes)
@@
 			)
 		)
-		(property "DIGIKEY_PART_NUMBER" "2019-RK73H1ETTP3R30FCT-ND"
+		(property "DIGIKEY_PART_NUMBER" "738-RMCF1206FT3R30CT-ND"
 			(at 72.39 119.38 90)
 			(hide yes)

Commit message: Add files via upload
Updated, completed placement
Parts:
- C52, C57: footprint 0603 (1608 Metric) -> copy_ref:C_0603_1608Metric
- C53, C54, C55, C56, C58, C60, C61, C62: footprint 0402 (1005 Metric) -> copy_ref:C_0402_1005Metric
- C59: footprint 1206 (3216 Metric) -> copy_ref:C_1206_3216Metric
- FB4: footprint 0402 (1005 Metric) -> copy_ref:402
- FB5, FB6: footprint 1206 (3216 Metric) -> copy_ref:1206
- L1: footprint 0402 (1005 Metric) -> Inductor_SMD:L_0402_1005Metric
- Q11: footprint SOT-223 (TO-261) -> Package_TO_SOT_SMD:SOT-223
- Q12, Q13, Q14: footprint SOT-323 -> Package_TO_SOT_SMD:SOT-323_SC-70
- R200, R73, R74, R75, R76, R78, R79, R80, R81, R82, R83, R84, R85, R86, R87, R88: footprint 0402 (1005 Metric) -> copy_ref:R_0402_1005Metric
- R77, R89: footprint 1206 (3216 Metric) -> copy_ref:R_1206_3216Metric
- U24: footprint SOT-23-6 -> Package_TO_SOT_SMD:SOT-23-6
- U25: footprint 8-VSSOP -> dowload:LMV393
- U27: footprint TSOT-23-5 -> Package_TO_SOT_SMD:TSOT-23-5
Changed lines of the file:
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@@
 			)
 		)
-		(property "Footprint" "8-VSSOP"
+		(property "Footprint" "dowload:LMV393"
 			(at 137.16 88.9 0)
 			(hide yes)
@@
 			)
 		)
-		(property "Footprint" "0402 (1005 Metric)"
+		(property "Footprint" "copy_ref:R_0402_1005Metric"
 			(at 71.628 38.1 90)
 			(hide yes)
@@
 			)
 		)
-		(property "Footprint" "0402 (1005 Metric)"
+		(property "Footprint" "copy_ref:R_0402_1005Metric"
 			(at 149.352 152.4 90)
 			(hide yes)
@@
 			)
 		)
-		(property "Footprint" "0402 (1005 Metric)"
+		(property "Footprint" "copy_ref:C_0402_1005Metric"
 			(at 218.7448 104.14 0)
 			(hide yes)
@@
 			)
 		)
-		(property "Footprint" "0402 (1005 Metric)"
+		(property "Footprint" "Inductor_SMD:L_0402_1005Metric"
 			(at 73.66 81.28 0)
 			(hide yes)
@@
 			)
 		)
-		(property "Footprint" "SOT-323"
+		(property "Footprint" "Package_TO_SOT_SMD:SOT-323_SC-70"
 			(at 67.31 61.595 0)
 			(hide yes)
@@
 			)
 		)
-		(property "Footprint" "1206 (3216 Metric)"
+		(property "Footprint" "copy_ref:R_1206_3216Metric"
 			(at 345.44 151.892 90)
 			(hide yes)
@@
 			)
 		)
-		(property "Footprint" "0402 (1005 Metric)"
+		(property "Footprint" "copy_ref:C_0402_1005Metric"
 			(at 117.8052 74.93 0)
 			(hide yes)
@@
 			)
 		)
-		(property "Footprint" "0402 (1005 Metric)"
+		(property "Footprint" "copy_ref:C_0402_1005Metric"
 			(at 83.5152 125.73 0)
 			(hide yes)
@@
 			)
 		)
-		(property "Footprint" "0402 (1005 Metric)"
+		(property "Footprint" "copy_ref:C_0402_1005Metric"
 			(at 374.9548 162.56 0)
 			(hide yes)
@@
 			)
 		)
-		(property "Footprint" "1206 (3216 Metric)"
+		(property "Footprint" "copy_ref:C_1206_3216Metric"
 			(at 330.5048 162.56 0)
 			(hide yes)
@@
 			)
 		)
-		(property "Footprint" "TSOT-23-5"
+		(property "Footprint" "Package_TO_SOT_SMD:TSOT-23-5"
 			(at 300.99 163.83 0)
 			(hide yes)
@@
 			)
 		)
-		(property "Footprint" "SOT-223 (TO-261)"
+		(property "Footprint" "Package_TO_SOT_SMD:SOT-223"
 			(at 43.18 97.155 0)
 			(hide yes)
@@
 			)
 		)
-		(property "Footprint" "1206 (3216 Metric)"
+		(property "Footprint" "copy_ref:R_1206_3216Metric"
 			(at 72.39 117.602 90)
 			(hide yes)
@@
 			)
 		)
-		(property "Footprint" "SOT-23-6"
+		(property "Footprint" "Package_TO_SOT_SMD:SOT-23-6"
 			(at 120.65 148.59 0)
 			(hide yes)
@@
 			)
 		)
-		(property "Footprint" "0402 (1005 Metric)"
+		(property "Footprint" "copy_ref:R_0402_1005Metric"
 			(at 96.012 92.71 90)
 			(hide yes)
@@
 			)
 		)
-		(property "Footprint" "0402 (1005 Metric)"
+		(property "Footprint" "copy_ref:C_0402_1005Metric"
 			(at 144.4752 130.81 0)
 			(hide yes)
@@
 			)
 		)
-		(property "Footprint" "0402 (1005 Metric)"
+		(property "Footprint" "copy_ref:R_0402_1005Metric"
 			(at 292.608 163.83 90)
 			(hide yes)
@@
 			)
 		)
-		(property "Footprint" "1206 (3216 Metric)"
+		(property "Footprint" "copy_ref:1206"
 			(at 221.488 85.09 90)
 			(hide yes)
@@
 			)
 		)
-		(property "Footprint" "0402 (1005 Metric)"
+		(property "Footprint" "copy_ref:R_0402_1005Metric"
 			(at 113.03 89.662 90)
 			(hide yes)
@@
 			)
 		)
-		(property "Footprint" "0603 (1608 Metric)"
+		(property "Footprint" "copy_ref:C_0603_1608Metric"
 			(at 74.6252 95.25 0)
 			(hide yes)
@@
 			)
 		)
-		(property "Footprint" "1206 (3216 Metric)"
+		(property "Footprint" "copy_ref:1206"
 			(at 356.87 151.892 90)
 			(hide yes)
@@
 			)
 		)
-		(property "Footprint" "0402 (1005 Metric)"
+		(property "Footprint" "copy_ref:R_0402_1005Metric"
 			(at 72.39 116.078 90)
 			(hide yes)
@@
 			)
 		)
-		(property "Footprint" "0402 (1005 Metric)"
+		(property "Footprint" "copy_ref:402"
 			(at 84.328 109.22 90)
 			(hide yes)
@@
 			)
 		)
-		(property "Footprint" "0402 (1005 Metric)"
+		(property "Footprint" "copy_ref:R_0402_1005Metric"
 			(at 71.628 48.26 90)
 			(hide yes)
@@
 			)
 		)
-		(property "Footprint" "8-VSSOP"
+		(property "Footprint" "dowload:LMV393"
 			(at 228.6 100.33 0)
 			(hide yes)
@@
 			)
 		)
-		(property "Footprint" "0603 (1608 Metric)"
+		(property "Footprint" "copy_ref:C_0603_1608Metric"
 			(at 206.0448 104.14 0)
 			(hide yes)
@@
 			)
 		)
-		(property "Footprint" "0402 (1005 Metric)"
+		(property "Footprint" "copy_ref:R_0402_1005Metric"
 			(at 64.77 97.028 90)
 			(hide yes)
@@
 			)
 		)
-		(property "Footprint" "SOT-323"
+		(property "Footprint" "Package_TO_SOT_SMD:SOT-323_SC-70"
 			(at 59.69 111.125 0)
 			(hide yes)
@@
 			)
 		)
-		(property "Footprint" "0402 (1005 Metric)"
+		(property "Footprint" "copy_ref:R_0402_1005Metric"
 			(at 146.05 144.272 90)
 			(hide yes)
@@
 			)
 		)
-		(property "Footprint" "0402 (1005 Metric)"
+		(property "Footprint" "copy_ref:C_0402_1005Metric"
 			(at 347.6752 208.28 0)
 			(hide yes)
@@
 			)
 		)
-		(property "Footprint" "0402 (1005 Metric)"
+		(property "Footprint" "copy_ref:R_0402_1005Metric"
 			(at 75.692 64.77 90)
 			(hide yes)
@@
 			)
 		)
-		(property "Footprint" "0402 (1005 Metric)"
+		(property "Footprint" "copy_ref:R_0402_1005Metric"
 			(at 92.71 84.582 90)
 			(hide yes)
@@
 			)
 		)
-		(property "Footprint" "0402 (1005 Metric)"
+		(property "Footprint" "copy_ref:R_0402_1005Metric"
 			(at 83.82 61.468 90)
 			(hide yes)
@@
 			)
 		)
-		(property "Footprint" "SOT-323"
+		(property "Footprint" "Package_TO_SOT_SMD:SOT-323_SC-70"
 			(at 54.61 41.275 0)
 			(hide yes)
@@
 			)
 		)
-		(property "Footprint" "0402 (1005 Metric)"
+		(property "Footprint" "copy_ref:R_0402_1005Metric"
 			(at 314.198 139.7 90)
 			(hide yes)
@@
 			)
 		)
-		(property "Footprint" "0402 (1005 Metric)"
+		(property "Footprint" "copy_ref:R_0402_1005Metric"
 			(at 116.332 97.79 90)
 			(hide yes)
@@
 			)
 		)
-		(property "Footprint" "0402 (1005 Metric)"
+		(property "Footprint" "copy_ref:C_0402_1005Metric"
 			(at 363.5248 162.56 0)
 			(hide yes)
@@
 			)
 		)
-		(property "Footprint" "8-VSSOP"
+		(property "Footprint" "dowload:LMV393"
 			(at 170.18 143.51 0)
 			(hide yes)
@@
 			)
 		)
-		(property "Footprint" "0402 (1005 Metric)"
+		(property "Footprint" "copy_ref:R_0402_1005Metric"
 			(at 144.272 81.28 90)
 			(hide yes)
@@
 			)
 		)
-		(property "Footprint" "0402 (1005 Metric)"
+		(property "Footprint" "copy_ref:R_0402_1005Metric"
 			(at 177.292 135.89 90)
 			(hide yes)
@@
 			)
 		)
-		(property "Footprint" "0402 (1005 Metric)"
+		(property "Footprint" "copy_ref:C_0402_1005Metric"
 			(at 105.1052 127 0)
 			(hide yes)
