File: hardware/ntp-server-stm32/gps.kicad_sch (KiCad schematic)
At the start: 15 parts, among them U21 ZED-F9T-00B, U22 LT3045xDD, U23 INA228AQDGSRQ1

Commit message: Standardize net/rail names: plain 3V3 style, _N active-low, voltage-format PG/alerts
22 net renames applied across all sheets and verified: removed/added net-name
sets match intent exactly and all node connectivity is preserved (kicad-cli
netlist re-parse).

Co-Authored-By: Claude Opus 4.8 (1M context) <noreply@anthropic.com>
Connections:
- net +3.3V renamed 3V3
- net +3.3V_GPS renamed 3V3_GPS
- net +5V renamed 5V
- net 3V3_LDO_GPS_PG renamed 3V3_GPS_LDO_PG
- net GPS_nRST renamed GPS_RST_N
- net GPS_nSAFEBOOT renamed GPS_SAFEBOOT_N
- net INA_ALERT_3.3V_GPS renamed INA_ALERT_3V3_GPS
Changed lines of the file:
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@@
 		)
 	)
-	(global_label "INA_ALERT_3.3V_GPS"
+	(global_label "INA_ALERT_3V3_GPS"
 		(shape output)
 		(at 283.21 111.76 180)
@@
 		)
 	)
-	(global_label "3V3_LDO_GPS_PG"
+	(global_label "3V3_GPS_LDO_PG"
 		(shape output)
 		(at 308.61 59.69 0)
@@
 		)
 	)
-	(global_label "GPS_nSAFEBOOT"
+	(global_label "GPS_SAFEBOOT_N"
 		(shape input)
 		(at 148.59 194.31 0)
@@
 		)
 	)
-	(global_label "GPS_nRST"
+	(global_label "GPS_RST_N"
 		(shape input)
 		(at 148.59 227.33 0)
@@
 			)
 		)
-		(property "Value" "+3.3V_GPS"
+		(property "Value" "3V3_GPS"
 			(at 346.71 58.42 0)
 			(show_name no)
@@
 			)
 		)
-		(property "Value" "+3.3V_GPS"
+		(property "Value" "3V3_GPS"
 			(at 48.26 224.79 0)
 			(show_name no)
@@
 			)
 		)
-		(property "Value" "+3.3V_GPS"
+		(property "Value" "3V3_GPS"
 			(at 219.71 173.99 0)
 			(show_name no)
@@
 			)
 		)
-		(property "Value" "+3.3V"
+		(property "Value" "3V3"
 			(at 289.306 97.79 0)
 			(show_name no)
@@
 			)
 		)
-		(property "Value" "+5V"
+		(property "Value" "5V"
 			(at 220.98 50.8 0)
 			(show_name no)
@@
 			)
 		)
-		(property "Value" "+3.3V"
+		(property "Value" "3V3"
 			(at 342.646 111.76 0)
 			(show_name no)

Commit message: Standardize + complete BOM; write fields back into KiCad symbols
- New sts1000_bom.csv: rebuilt from authoritative Value field (source MPN/footprint/
  description were corrupted by copy-paste). 338 standardized, 78 MPN-from-value,
  50 kept, ~64 flagged (SELECT/REVIEW-HV/SHUNT-REVIEW) each with full spec.
- Resistors -> deterministic Panasonic ERJ-2RKF 0402 1% 1/10W (consolidated 1 part/value).
- Caps -> verified Murata GRM parts where value matches; clean spec + footprint otherwise.
- 1633 symbol field updates (Value/Footprint/Description/MPN/Mfr/Digikey) written to
  .kicad_sch; netlist re-parse confirms connectivity byte-identical.
- Add docs/sts1000_net_naming.md naming reference.

Co-Authored-By: Claude Opus 4.8 (1M context) <noreply@anthropic.com>
Parts:
- C45, C47, C49: footprint (none) -> C_0603_1608Metric
- C46: footprint 0805 -> C_0805_2012Metric; DIGIKEY_PART_NUMBER 445-5972-1-ND -> 490-GRM21BR71C475KE51KTR-ND; MANUFACTURER TDK -> Murata; MANUFACTURER_PART_NUMBER C2012X7R1E475K125AB -> GRM21BR71C475KE51K
- C48, C51: footprint (none) -> C_0402_1005Metric; DIGIKEY_PART_NUMBER (none) -> 490-6328-2-ND; MANUFACTURER (none) -> Murata; MANUFACTURER_PART_NUMBER (none) -> GRM155R71C104KA88J
- C50: footprint 1206 -> C_0805_2012Metric; DIGIKEY_PART_NUMBER 445-7705-1-ND -> 490-GRM21BZ71C106KE15LTR-ND; MANUFACTURER TDK -> Murata; MANUFACTURER_PART_NUMBER C3216X7R1E106K160AB -> GRM21BZ71C106KE15L
- R69: footprint (none) -> R_0402_1005Metric; MANUFACTURER (none) -> Panasonic; MANUFACTURER_PART_NUMBER (none) -> ERJ-2RKF1003X
- R70: footprint (none) -> R_0402_1005Metric; MANUFACTURER (none) -> Panasonic; MANUFACTURER_PART_NUMBER (none) -> ERJ-2RKF3740X
- R71: footprint (none) -> R_0402_1005Metric; MANUFACTURER (none) -> Panasonic; MANUFACTURER_PART_NUMBER (none) -> ERJ-2RKF3322X
- U21: MANUFACTURER_PART_NUMBER (none) -> ZED-F9T-00B
- U22: MANUFACTURER_PART_NUMBER (none) -> LT3045xDD
- U23: MANUFACTURER_PART_NUMBER (none) -> INA228AQDGSRQ1
Changed lines of the file:
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@@
 			)
 		)
+		(property "MANUFACTURER_PART_NUMBER" "LT3045xDD"
+			(at 0 0 0)
+			(hide yes)
+			(show_name no)
+			(do_not_autoplace no)
+			(effects
+				(font
+					(size 1.27 1.27)
+				)
+			)
+		)
 		(pin "7"
 		)
@@
 			)
 		)
-		(property "Description" "RES 0.15 OHM 0.5% 1/4W 0805"
+		(property "Description" "RES 500m OHM 0.5% SENSE 0805 (value TBD per rail)"
 			(at 341.63 68.58 90)
 			(hide yes)
@@
 			)
 		)
-		(property "Footprint" ""
+		(property "Footprint" "C_0603_1608Metric"
 			(at 232.1052 190.5 0)
 			(hide yes)
@@
 			)
 		)
-		(property "Description" "Unpolarized capacitor"
+		(property "Description" "CAP CER 1uF 16V X7R 0603"
 			(at 231.14 186.69 0)
 			(hide yes)
@@
 			)
 		)
-		(property "Description" ""
+		(property "Description" "INA228AQDGSRQ1"
 			(at 292.1 106.68 0)
 			(hide yes)
@@
 			)
 		)
+		(property "MANUFACTURER_PART_NUMBER" "INA228AQDGSRQ1"
+			(at 0 0 0)
+			(hide yes)
+			(show_name no)
+			(do_not_autoplace no)
+			(effects
+				(font
+					(size 1.27 1.27)
+				)
+			)
+		)
 		(pin "2"
 		)
@@
 			)
 		)
-		(property "Footprint" ""
+		(property "Footprint" "C_0402_1005Metric"
 			(at 343.8652 124.46 0)
 			(hide yes)
@@
 			)
 		)
-		(property "Description" "Unpolarized capacitor"
+		(property "Description" "CAP CER 0.1uF 16V X7R 0402"
 			(at 342.9 120.65 0)
 			(hide yes)
@@
 			)
 		)
+		(property "MANUFACTURER" "Murata"
+			(at 0 0 0)
+			(hide yes)
+			(show_name no)
+			(do_not_autoplace no)
+			(effects
+				(font
+					(size 1.27 1.27)
+				)
+			)
+		)
+		(property "MANUFACTURER_PART_NUMBER" "GRM155R71C104KA88J"
+			(at 0 0 0)
+			(hide yes)
+			(show_name no)
+			(do_not_autoplace no)
+			(effects
+				(font
+					(size 1.27 1.27)
+				)
+			)
+		)
+		(property "DIGIKEY_PART_NUMBER" "490-6328-2-ND"
+			(at 0 0 0)
+			(hide yes)
+			(show_name no)
+			(do_not_autoplace no)
+			(effects
+				(font
+					(size 1.27 1.27)
+				)
+			)
+		)
 		(pin "2"
 		)
@@
 			)
 		)
-		(property "Footprint" ""
+		(property "Footprint" "C_0402_1005Metric"
 			(at 251.1552 190.5 0)
 			(hide yes)
@@
 			)
 		)
-		(property "Description" "Unpolarized capacitor"
+		(property "Description" "CAP CER 0.1uF 16V X7R 0402"
 			(at 250.19 186.69 0)
 			(hide yes)
@@
 			)
 		)
+		(property "MANUFACTURER" "Murata"
+			(at 0 0 0)
+			(hide yes)
+			(show_name no)
+			(do_not_autoplace no)
+			(effects
+				(font
+					(size 1.27 1.27)
+				)
+			)
+		)
+		(property "MANUFACTURER_PART_NUMBER" "GRM155R71C104KA88J"
+			(at 0 0 0)
+			(hide yes)
+			(show_name no)
+			(do_not_autoplace no)
+			(effects
+				(font
+					(size 1.27 1.27)
+				)
+			)
+		)
+		(property "DIGIKEY_PART_NUMBER" "490-6328-2-ND"
+			(at 0 0 0)
+			(hide yes)
+			(show_name no)
+			(do_not_autoplace no)
+			(effects
+				(font
+					(size 1.27 1.27)
+				)
+			)
+		)
 		(pin "2"
 		)
@@
 			)
 		)
-		(property "Description" ""
+		(property "Description" "ZED-F9T-00B"
 			(at 116.84 207.01 0)
 			(hide yes)
@@
 			)
 		)
+		(property "MANUFACTURER_PART_NUMBER" "ZED-F9T-00B"
+			(at 0 0 0)
+			(hide yes)
+			(show_name no)
+			(do_not_autoplace no)
+			(effects
+				(font
+					(size 1.27 1.27)
+				)
+			)
+		)
 		(property "MAXIMUM_PACKAGE_HEIGHT" "2.6mm"
 			(at 116.84 207.01 0)
@@
 			)
 		)
-		(property "Footprint" ""
+		(property "Footprint" "C_0603_1608Metric"
 			(at 272.7452 87.63 0)
 			(hide yes)
@@
 			)
 		)
-		(property "Description" "Unpolarized capacitor"
+		(property "Description" "CAP CER 0.47uF 16V X7R 0603"
 			(at 271.78 83.82 0)
 			(hide yes)
@@
 			)
 		)
-		(property "Footprint" ""
+		(property "Footprint" "R_0402_1005Metric"
 			(at 246.888 83.82 90)
 			(hide yes)
@@
 			)
 		)
-		(property "Description" "Resistor"
+		(property "Description" "RES SMD 100k OHM 1% 1/10W 0402"
 			(at 245.11 83.82 0)
 			(hide yes)
@@
 			)
 		)
+		(property "MANUFACTURER" "Panasonic"
+			(at 0 0 0)
+			(hide yes)
+			(show_name no)
+			(do_not_autoplace no)
+			(effects
+				(font
+					(size 1.27 1.27)
+				)
+			)
+		)
+		(property "MANUFACTURER_PART_NUMBER" "ERJ-2RKF1003X"
+			(at 0 0 0)
+			(hide yes)
+			(show_name no)
+			(do_not_autoplace no)
+			(effects
+				(font
+					(size 1.27 1.27)
+				)
+			)
+		)
 		(pin "1"
 		)
@@
 			)
 		)
-		(property "Footprint" "1206"
+		(property "Footprint" "C_0805_2012Metric"
 			(at 313.3852 77.47 0)
 			(hide yes)
@@
 			)
 		)
-		(property "Description" "CAP CER 10UF 25V X7R 1206"
+		(property "Description" "CAP CER 10uF 16V X7R 0805"
 			(at 312.42 73.66 0)
 			(hide yes)
@@
 			)
 		)
-		(property "DIGIKEY_PART_NUMBER" "445-7705-1-ND"
+		(property "DIGIKEY_PART_NUMBER" "490-GRM21BZ71C106KE15LTR-ND"
 			(at 312.42 73.66 0)
 			(hide yes)
@@
 			)
 		)
-		(property "MANUFACTURER" "TDK"
+		(property "MANUFACTURER" "Murata"
 			(at 312.42 73.66 0)
 			(hide yes)
@@
 			)
 		)
-		(property "MANUFACTURER_PART_NUMBER" "C3216X7R1E106K160AB"
+		(property "MANUFACTURER_PART_NUMBER" "GRM21BZ71C106KE15L"
 			(at 312.42 73.66 0)
 			(hide yes)
@@
 			)
 		)
-		(property "Footprint" ""
+		(property "Footprint" "C_0603_1608Metric"
 			(at 220.6752 190.5 0)
 			(hide yes)
@@
 			)
 		)
-		(property "Description" "Unpolarized capacitor"
+		(property "Description" "CAP CER 1uF 16V X7R 0603"
 			(at 219.71 186.69 0)
 			(hide yes)
@@
 			)
 		)
-		(property "Footprint" "0805"
+		(property "Footprint" "C_0805_2012Metric"
 			(at 220.0148 86.36 0)
 			(hide yes)
@@
 			)
 		)
-		(property "Description" "CAP CER 4.7UF 25V X7R 0805"
+		(property "Description" "CAP CER 4.7uF 16V X7R 0805"
 			(at 220.98 82.55 0)
 			(hide yes)
@@
 			)
 		)
-		(property "DIGIKEY_PART_NUMBER" "445-5972-1-ND"
+		(property "DIGIKEY_PART_NUMBER" "490-GRM21BR71C475KE51KTR-ND"
 			(at 220.98 82.55 0)
 			(hide yes)
@@
 			)
 		)
-		(property "MANUFACTURER" "TDK"
+		(property "MANUFACTURER" "Murata"
 			(at 220.98 82.55 0)
 			(hide yes)
@@
 			)
 		)
-		(property "MANUFACTURER_PART_NUMBER" "C2012X7R1E475K125AB"
+		(property "MANUFACTURER_PART_NUMBER" "GRM21BR71C475KE51K"
 			(at 220.98 82.55 0)
 			(hide yes)
@@
 			)
 		)
-		(property "Footprint" ""
+		(property "Footprint" "R_0402_1005Metric"
 			(at 267.208 83.82 90)
 			(hide yes)
@@
 			)
 		)
-		(property "Description" "Resistor"
+		(property "Description" "RES SMD 33.2k OHM 1% 1/10W 0402"
 			(at 265.43 83.82 0)
 			(hide yes)
@@
 			)
 		)
+		(property "MANUFACTURER" "Panasonic"
+			(at 0 0 0)
+			(hide yes)
+			(show_name no)
+			(do_not_autoplace no)
+			(effects
+				(font
+					(size 1.27 1.27)
+				)
+			)
+		)
+		(property "MANUFACTURER_PART_NUMBER" "ERJ-2RKF3322X"
+			(at 0 0 0)
+			(hide yes)
+			(show_name no)
+			(do_not_autoplace no)
+			(effects
+				(font
+					(size 1.27 1.27)
+				)
+			)
+		)
 		(pin "1"
 		)
@@
 			)
 		)
-		(property "Footprint" ""
+		(property "Footprint" "R_0402_1005Metric"
 			(at 257.048 83.82 90)
 			(hide yes)
@@
 			)
 		)
-		(property "Description" "Resistor"
+		(property "Description" "RES SMD 374 OHM 1% 1/10W 0402"
 			(at 255.27 83.82 0)
 			(hide yes)
 			(show_name no)
+			(do_not_autoplace no)
+			(effects
+				(font
+					(size 1.27 1.27)
+				)
+			)
+		)
+		(property "MANUFACTURER" "Panasonic"
+			(at 0 0 0)
+			(hide yes)
+			(show_name no)
+			(do_not_autoplace no)
+			(effects
+				(font
+					(size 1.27 1.27)
+				)
+			)
+		)
+		(property "MANUFACTURER_PART_NUMBER" "ERJ-2RKF3740X"
+			(at 0 0 0)
+			(hide yes)
+			(show_name no)
