File: hardware/ntp-server-stm32/gps.kicad_sch (KiCad schematic)
At the start: 15 parts, among them U21 ZED-F9T-00B, U22 LT3045xDD, U23 INA228AQDGSRQ1

Commit message: Updates
Parts:
- added R197: 453k, R_0402_1005Metric, symbol Device:R
- added R214: 49.9k, R_0402_1005Metric, symbol Device:R
- added R215: 10k, 0402 (1005 Metric), symbol Device:R
- C45, C47: footprint C_0603_1608Metric -> 0603 (1608 Metric); DIELECTRIC (none) -> X7R; DIGIKEY_PART_NUMBER (none) -> 399-17704-1-ND; MANUFACTURER (none) -> KEMET; MANUFACTURER_PART_NUMBER (none) -> C0603C105K4RACAUTO; TOLERANCE (none) -> 10%; VOLTAGE (none) -> 16V
- C46: footprint C_0805_2012Metric -> 0805 (2012 Metric); DIELECTRIC (none) -> X7R; DIGIKEY_PART_NUMBER 490-GRM21BR71C475KE51KTR-ND -> 490-GRT21BR71C475KE13KCT-ND; MANUFACTURER Murata -> Murata Electronics; MANUFACTURER_PART_NUMBER GRM21BR71C475KE51K -> GRT21BR71C475KE13K; TOLERANCE (none) -> 10%; VOLTAGE (none) -> 16V
- C48, C51: footprint C_0402_1005Metric -> 0402 (1005 Metric); DIELECTRIC (none) -> X7R; DIGIKEY_PART_NUMBER 490-6328-2-ND -> 490-4759-1-ND; MANUFACTURER_PART_NUMBER GRM155R71C104KA88J -> GCM155R71C104KA55D; TOLERANCE (none) -> 10%; VOLTAGE (none) -> 16V
- C49: footprint C_0603_1608Metric -> 0603 (1608 Metric); DIELECTRIC (none) -> X7R; DIGIKEY_PART_NUMBER (none) -> 490-GRT188R71C474KE01DCT-ND; MANUFACTURER (none) -> Murata Electronics; MANUFACTURER_PART_NUMBER (none) -> GRT188R71C474KE01D; TOLERANCE (none) -> 10%; VOLTAGE (none) -> 16V
- C50: footprint C_0805_2012Metric -> 1206 (3216 Metric); DIELECTRIC (none) -> X7R; DIGIKEY_PART_NUMBER 490-GRM21BZ71C106KE15LTR-ND -> 1276-6797-1-ND; MANUFACTURER Murata -> Samsung Electro-Mechanics; MANUFACTURER_PART_NUMBER GRM21BZ71C106KE15L -> CL31B106KOHVPNE; TOLERANCE (none) -> 10%; VOLTAGE (none) -> 16V
- FB3: DIELECTRIC (none) -> Ferrite bead; MANUFACTURER Murata Electronics -> Murata; MANUFACTURER_PART_NUMBER BLM31KN601SN1L -> BLM31PG601SN1L; POWER (none) -> 3A
- R69: footprint R_0402_1005Metric -> 0402 (1005 Metric); DIELECTRIC (none) -> Thick-film; DIGIKEY_PART_NUMBER (none) -> P100KLCT-ND; MANUFACTURER Panasonic -> Panasonic Industry; POWER (none) -> 1/10W; TOLERANCE (none) -> 1%
- R70: footprint R_0402_1005Metric -> 0402 (1005 Metric); DIELECTRIC (none) -> Thick-film; DIGIKEY_PART_NUMBER (none) -> P374LCT-ND; MANUFACTURER Panasonic -> Panasonic Industry; POWER (none) -> 1/10W; TOLERANCE (none) -> 1%
- R71: footprint R_0402_1005Metric -> 0402 (1005 Metric); DIELECTRIC (none) -> Thick-film; DIGIKEY_PART_NUMBER (none) -> P33.2KLCT-ND; MANUFACTURER Panasonic -> Panasonic Industry; POWER (none) -> 1/10W; TOLERANCE (none) -> 1%
- R72: value 500m -> 100m; footprint 0805 -> 1206 (3216 Metric); DIELECTRIC (none) -> Metal-strip shunt; DIGIKEY_PART_NUMBER 273-KDV08DR150ETCT-ND -> 273-KDV12DR100ETCT-ND; MANUFACTURER_PART_NUMBER KDV08DR150ET -> KDV12DR100ET; POWER (none) -> 1/4W; TOLERANCE (none) -> 0.5%
- U21: MANUFACTURER U-Blox -> u-blox
- U22: MANUFACTURER (none) -> Analog Devices; MANUFACTURER_PART_NUMBER LT3045xDD -> LT3045EDD#TRPBF
- U23: MANUFACTURER (none) -> Texas Instruments
Connections:
- net 3V3: no longer U23.1 (A1)
- net 3V3_GPS_LDO_PG: now also R215.2
- net GND: now also R214.2; no longer U23.2 (A0)
- net I2C_SCL: now also U23.5 (SCL); no longer U23.4 (SDA)
- net I2C_SDA: now also U23.1 (A1), U23.2 (A0), U23.4 (SDA); no longer U23.5 (SCL)
- net at C46.1, FB3.1, U22.1 (IN)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: no longer U22.6 (PGFB)
- net at C50.1, R72.1, U22.10 (OUT)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: now also R197.1
- new net: R197.2, R214.1, U22.6 (PGFB)
- new net 3V3_STM: R215.1
Other:
- note added: "I2C Address: 0x4A"
- note removed: "I2C Address: 0x44"
- moved on the sheet: C46, C49, C50, FB3, R69, R70, R71, R72, U22

Commit message: Bom updates
Parts:
- FB3: footprint 1206 -> 1206 (3216 Metric)
- R197: footprint R_0402_1005Metric -> 0402 (1005 Metric); DIGIKEY_PART_NUMBER (none) -> P453KLCT-ND; MANUFACTURER Panasonic -> Panasonic Industry
- R214: footprint R_0402_1005Metric -> 0402 (1005 Metric); DIGIKEY_PART_NUMBER (none) -> P49.9KLCT-ND; MANUFACTURER Panasonic -> Panasonic Industry
- R72: value 100m -> 75m; DIGIKEY_PART_NUMBER 273-KDV12DR100ETCT-ND -> 541-10064-1-ND; MANUFACTURER Ohmite -> Vishay Dale; MANUFACTURER_PART_NUMBER KDV12DR100ET -> WSL1206R0750FEA
- U21: DIGIKEY_PART_NUMBER (none) -> 672-1197-1-ND
- U22: DIGIKEY_PART_NUMBER (none) -> 505-LT3045EDD#TRPBFCT-ND
- U23: DIGIKEY_PART_NUMBER (none) -> 296-INA228AQDGSRQ1CT-ND
Changed lines of the file:
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@@
 			)
 		)
-		(property "Description" "LDO 500mA ultralow-noise DFN-10"
+		(property "Description" "IC REG LIN POS ADJ 500MA 10DFN"
 			(at 287.02 67.31 0)
 			(hide yes)
@@
 			)
 		)
+		(property "DIGIKEY_PART_NUMBER" "505-LT3045EDD#TRPBFCT-ND"
+			(at 287.02 67.31 0)
+			(hide yes)
+			(show_name no)
+			(do_not_autoplace no)
+			(effects
+				(font
+					(size 1.27 1.27)
+				)
+			)
+		)
 		(pin "7"
 		)
@@
 			)
 		)
-		(property "Footprint" "1206"
+		(property "Footprint" "1206 (3216 Metric)"
 			(at 222.758 58.42 90)
 			(hide yes)
@@
 			)
 		)
-		(property "Value" "100m"
+		(property "Value" "75m"
 			(at 343.916 67.31 90)
 			(show_name no)
@@
 			)
 		)
-		(property "Datasheet" "https://www.ohmite.com/assets/images/res-kdv.pdf"
+		(property "Datasheet" "https://www.vishay.com/docs/30100/wsl.pdf"
 			(at 341.63 64.77 0)
 			(hide yes)
@@
 			)
 		)
-		(property "Description" "RES 0.1 OHM 0.5% 1/2W 1206"
+		(property "Description" "RES 0.075 OHM 1% 1/4W 1206"
 			(at 341.63 64.77 90)
 			(hide yes)
@@
 			)
 		)
-		(property "DIGIKEY_PART_NUMBER" "273-KDV12DR100ETCT-ND"
+		(property "DIGIKEY_PART_NUMBER" "541-10064-1-ND"
 			(at 341.63 64.77 90)
 			(hide yes)
@@
 			)
 		)
-		(property "MANUFACTURER_PART_NUMBER" "KDV12DR100ET"
+		(property "MANUFACTURER_PART_NUMBER" "WSL1206R0750FEA"
 			(at 341.63 64.77 90)
 			(hide yes)
@@
 			)
 		)
-		(property "MANUFACTURER" "Ohmite"
+		(property "MANUFACTURER" "Vishay Dale"
 			(at 341.63 64.77 90)
 			(hide yes)
@@
 			)
 		)
-		(property "Footprint" "R_0402_1005Metric"
+		(property "Footprint" "0402 (1005 Metric)"
 			(at 318.008 69.85 90)
 			(hide yes)
@@
 			)
 		)
-		(property "Datasheet" ""
+		(property "Datasheet" "https://industrial.panasonic.com/cdbs/www-data/pdf/RDA0000/AOA0000C304.pdf"
 			(at 316.23 69.85 0)
 			(hide yes)
@@
 			)
 		)
-		(property "Description" "RES 453k 1% 1/10W 0402"
+		(property "Description" "RES SMD 453K OHM 1% 1/10W 0402"
 			(at 316.23 69.85 0)
 			(hide yes)
@@
 			)
 		)
-		(property "MANUFACTURER" "Panasonic"
+		(property "MANUFACTURER" "Panasonic Industry"
 			(at 50.8 -13.97 0)
 			(hide yes)
@@
 			)
 		)
+		(property "DIGIKEY_PART_NUMBER" "P453KLCT-ND"
+			(at 316.23 69.85 0)
+			(hide yes)
+			(show_name no)
+			(do_not_autoplace no)
+			(effects
+				(font
+					(size 1.27 1.27)
+				)
+			)
+		)
 		(pin "1"
 		)
@@
 			)
 		)
-		(property "Datasheet" "https://www.ti.com/lit/gpn/ina228-q1"
+		(property "Datasheet" "https://www.ti.com/lit/ds/symlink/ina228-q1.pdf"
 			(at 292.1 106.68 0)
 			(hide yes)
@@
 			)
 		)
-		(property "Description" "Current/power monitor 20-bit I2C"
+		(property "Description" "IC PWR MONITOR 10VSSOP"
 			(at 292.1 106.68 0)
 			(hide yes)
@@
 			)
 		)
+		(property "DIGIKEY_PART_NUMBER" "296-INA228AQDGSRQ1CT-ND"
+			(at 292.1 106.68 0)
+			(hide yes)
+			(show_name no)
+			(do_not_autoplace no)
+			(effects
+				(font
+					(size 1.27 1.27)
+				)
+			)
+		)
 		(pin "2"
 		)
@@
 			)
 		)
-		(property "Datasheet" ""
+		(property "Datasheet" "https://www.u-blox.com/en/docs/UBX-18053713"
 			(at 116.84 207.01 0)
 			(hide yes)
@@
 			)
 		)
-		(property "Description" "GNSS timing receiver module"
+		(property "Description" "RF RECEIVER GNSS/GPS 54LGA"
 			(at 116.84 207.01 0)
 			(hide yes)
@@
 			)
 		)
+		(property "DIGIKEY_PART_NUMBER" "672-1197-1-ND"
+			(at 116.84 207.01 0)
+			(hide yes)
+			(show_name no)
+			(do_not_autoplace no)
+			(effects
+				(font
+					(size 1.27 1.27)
+				)
+			)
+		)
 		(pin "19"
 		)
@@
 			)
 		)
-		(property "Footprint" "R_0402_1005Metric"
+		(property "Footprint" "0402 (1005 Metric)"
 			(at 318.008 80.01 90)
 			(hide yes)
@@
 			)
 		)
-		(property "Datasheet" ""
+		(property "Datasheet" "https://industrial.panasonic.com/cdbs/www-data/pdf/RDA0000/AOA0000C304.pdf"
 			(at 316.23 80.01 0)
 			(hide yes)
@@
 			)
 		)
-		(property "Description" "RES 49.9k 1% 1/10W 0402"
+		(property "Description" "RES SMD 49.9K OHM 1% 1/10W 0402"
 			(at 316.23 80.01 0)
 			(hide yes)
@@
 			)
 		)
-		(property "MANUFACTURER" "Panasonic"
+		(property "MANUFACTURER" "Panasonic Industry"
 			(at 50.8 -3.81 0)
 			(hide yes)
@@
 			(hide yes)
 			(show_name no)
+			(do_not_autoplace no)
+			(effects
+				(font
+					(size 1.27 1.27)
+				)
+			)
+		)
+		(property "DIGIKEY_PART_NUMBER" "P49.9KLCT-ND"
+			(at 316.23 80.01 0)
+			(hide yes)
+			(show_name no)

Commit message: Bom updates
Parts:
- U23: footprint VSSOP10_DGS_TEX -> sts1000:VSSOP10_DGS_TEX
Changed lines of the file:
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@@
 			)
 		)
-		(property "Footprint" "VSSOP10_DGS_TEX"
+		(property "Footprint" "sts1000:VSSOP10_DGS_TEX"
 			(at 292.1 106.68 0)
 			(hide yes)

Commit message: Add files via upload
Updated, completed placement
Parts:
- C45, C47, C49: footprint 0603 (1608 Metric) -> copy_ref:C_0603_1608Metric
- C46: footprint 0805 (2012 Metric) -> copy_ref:C_0805_2012Metric
- C48, C51: footprint 0402 (1005 Metric) -> copy_ref:C_0402_1005Metric
- C50: footprint 1206 (3216 Metric) -> copy_ref:C_1206_3216Metric
- FB3: footprint 1206 (3216 Metric) -> copy_ref:1206
- R197, R214, R215, R69, R70, R71: footprint 0402 (1005 Metric) -> copy_ref:R_0402_1005Metric
- R72: footprint 1206 (3216 Metric) -> copy_ref:R_1206_3216Metric
Changed lines of the file:
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@@
 			)
 		)
-		(property "Footprint" "1206 (3216 Metric)"
+		(property "Footprint" "copy_ref:1206"
 			(at 222.758 58.42 90)
 			(hide yes)
@@
 			)
 		)
-		(property "Footprint" "0402 (1005 Metric)"
+		(property "Footprint" "copy_ref:R_0402_1005Metric"
 			(at 306.578 50.8 90)
 			(hide yes)
@@
 			)
 		)
-		(property "Footprint" "1206 (3216 Metric)"
+		(property "Footprint" "copy_ref:R_1206_3216Metric"
 			(at 341.63 62.992 90)
 			(hide yes)
@@
 			)
 		)
-		(property "Footprint" "0603 (1608 Metric)"
+		(property "Footprint" "copy_ref:C_0603_1608Metric"
 			(at 232.1052 190.5 0)
 			(hide yes)
@@
 			)
 		)
-		(property "Footprint" "0402 (1005 Metric)"
+		(property "Footprint" "copy_ref:R_0402_1005Metric"
 			(at 318.008 69.85 90)
 			(hide yes)
@@
 			)
 		)
-		(property "Footprint" "0402 (1005 Metric)"
+		(property "Footprint" "copy_ref:C_0402_1005Metric"
 			(at 343.8652 124.46 0)
 			(hide yes)
@@
 			)
 		)
-		(property "Footprint" "0402 (1005 Metric)"
+		(property "Footprint" "copy_ref:C_0402_1005Metric"
 			(at 251.1552 190.5 0)
 			(hide yes)
@@
 			)
 		)
-		(property "Footprint" "0603 (1608 Metric)"
+		(property "Footprint" "copy_ref:C_0603_1608Metric"
 			(at 272.7452 83.82 0)
 			(hide yes)
@@
 			)
 		)
-		(property "Footprint" "0402 (1005 Metric)"
+		(property "Footprint" "copy_ref:R_0402_1005Metric"
 			(at 246.888 80.01 90)
 			(hide yes)
@@
 			)
 		)
-		(property "Footprint" "1206 (3216 Metric)"
+		(property "Footprint" "copy_ref:C_1206_3216Metric"
 			(at 324.8152 73.66 0)
 			(hide yes)
@@
 			)
 		)
-		(property "Footprint" "0603 (1608 Metric)"
+		(property "Footprint" "copy_ref:C_0603_1608Metric"
 			(at 220.6752 190.5 0)
 			(hide yes)
@@
 			)
 		)
-		(property "Footprint" "0805 (2012 Metric)"
+		(property "Footprint" "copy_ref:C_0805_2012Metric"
 			(at 220.0148 82.55 0)
 			(hide yes)
@@
 			)
 		)
-		(property "Footprint" "0402 (1005 Metric)"
+		(property "Footprint" "copy_ref:R_0402_1005Metric"
 			(at 318.008 80.01 90)
 			(hide yes)
@@
 			)
 		)
-		(property "Footprint" "0402 (1005 Metric)"
+		(property "Footprint" "copy_ref:R_0402_1005Metric"
 			(at 267.208 80.01 90)
 			(hide yes)
@@
 			)
 		)
-		(property "Footprint" "0402 (1005 Metric)"
+		(property "Footprint" "copy_ref:R_0402_1005Metric"
 			(at 257.048 80.01 90)
 			(hide yes)
