File: hardware/ntp-server-stm32/i2c-gpio.kicad_sch (KiCad schematic)
At the start: 23 parts, among them U54 MCP23017T-E/ML, U55 MCP23017T-E/ML

Commit message: Standardize net/rail names: plain 3V3 style, _N active-low, voltage-format PG/alerts
22 net renames applied across all sheets and verified: removed/added net-name
sets match intent exactly and all node connectivity is preserved (kicad-cli
netlist re-parse).

Co-Authored-By: Claude Opus 4.8 (1M context) <noreply@anthropic.com>
Connections:
- net +3.3V_STM renamed 3V3_STM
- net 3.0V_RF_LDO_PG renamed 3V0_RF_LDO_PG
- net 3V3_LDO_GPS_PG renamed 3V3_GPS_LDO_PG
- net EXP_RESET renamed EXP_RST_N
- net INA_ALERT_3.3V renamed INA_ALERT_3V3
- net INA_ALERT_3.3V_GPS renamed INA_ALERT_3V3_GPS
- net INA_ALERT_3.3V_STM renamed INA_ALERT_3V3_STM
- net INA_ALERT_V_DISP_5V renamed INA_ALERT_5V_DISP
- net POE_PGO renamed POE_PG
Changed lines of the file:
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@@
 		)
 	)
-	(global_label "INA_ALERT_V_DISP_5V"
+	(global_label "INA_ALERT_5V_DISP"
 		(shape input)
 		(at 182.88 186.69 180)
@@
 		)
 	)
-	(global_label "3V3_LDO_GPS_PG"
+	(global_label "3V3_GPS_LDO_PG"
 		(shape input)
 		(at 187.96 68.58 180)
@@
 		)
 	)
-	(global_label "EXP_RESET"
+	(global_label "EXP_RST_N"
 		(shape input)
 		(at 215.9 179.07 0)
@@
 		)
 	)
-	(global_label "INA_ALERT_3.3V_STM"
+	(global_label "INA_ALERT_3V3_STM"
 		(shape input)
 		(at 182.88 184.15 180)
@@
 		)
 	)
-	(global_label "POE_PGO"
+	(global_label "POE_PG"
 		(shape input)
 		(at 187.96 86.36 180)
@@
 		)
 	)
-	(global_label "EXP_RESET"
+	(global_label "EXP_RST_N"
 		(shape input)
 		(at 233.68 91.44 0)
@@
 		)
 	)
-	(global_label "3.0V_RF_LDO_PG"
+	(global_label "3V0_RF_LDO_PG"
 		(shape input)
 		(at 187.96 73.66 180)
@@
 		)
 	)
-	(global_label "INA_ALERT_3.3V_GPS"
+	(global_label "INA_ALERT_3V3_GPS"
 		(shape input)
 		(at 182.88 189.23 180)
@@
 		)
 	)
-	(global_label "INA_ALERT_3.3V"
+	(global_label "INA_ALERT_3V3"
 		(shape input)
 		(at 182.88 181.61 180)
@@
 			)
 		)
-		(property "Value" "+3.3V_STM"
+		(property "Value" "3V3_STM"
 			(at 208.28 133.3499 0)
 			(show_name no)
@@
 			)
 		)
-		(property "Value" "+3.3V_STM"
+		(property "Value" "3V3_STM"
 			(at 214.63 45.7199 0)
 			(show_name no)
@@
 			)
 		)
-		(property "Value" "+3.3V_STM"
+		(property "Value" "3V3_STM"
 			(at 166.37 138.4299 0)
 			(show_name no)
@@
 			)
 		)
-		(property "Value" "+3.3V_STM"
+		(property "Value" "3V3_STM"
 			(at 82.55 138.4299 0)
 			(show_name no)
@@
 			)
 		)
-		(property "Value" "+3.3V_STM"
+		(property "Value" "3V3_STM"
 			(at 257.81 158.7499 0)
 			(show_name no)
@@
 			)
 		)
-		(property "Value" "+3.3V_STM"
+		(property "Value" "3V3_STM"
 			(at 49.53 138.4299 0)
 			(show_name no)
@@
 			)
 		)
-		(property "Value" "+3.3V_STM"
+		(property "Value" "3V3_STM"
 			(at 246.38 72.3899 0)
 			(show_name no)
@@
 			)
 		)
-		(property "Value" "+3.3V_STM"
+		(property "Value" "3V3_STM"
 			(at 219.71 187.9599 0)
 			(show_name no)
@@
 			)
 		)
-		(property "Value" "+3.3V_STM"
+		(property "Value" "3V3_STM"
 			(at 116.84 138.4299 0)
 			(show_name no)
@@
 			)
 		)
-		(property "Value" "+3.3V_STM"
+		(property "Value" "3V3_STM"
 			(at 133.35 138.4299 0)
 			(show_name no)
@@
 			)
 		)
-		(property "Value" "+3.3V_STM"
+		(property "Value" "3V3_STM"
 			(at 241.3 158.7499 0)
 			(show_name no)
@@
 			)
 		)
-		(property "Value" "+3.3V_STM"
+		(property "Value" "3V3_STM"
 			(at 66.04 138.4299 0)
 			(show_name no)
@@
 			)
 		)
-		(property "Value" "+3.3V_STM"
+		(property "Value" "3V3_STM"
 			(at 149.86 138.4299 0)
 			(show_name no)
@@
 			)
 		)
-		(property "Value" "+3.3V_STM"
+		(property "Value" "3V3_STM"
 			(at 99.06 138.4299 0)
 			(show_name no)

Commit message: Standardize + complete BOM; write fields back into KiCad symbols
- New sts1000_bom.csv: rebuilt from authoritative Value field (source MPN/footprint/
  description were corrupted by copy-paste). 338 standardized, 78 MPN-from-value,
  50 kept, ~64 flagged (SELECT/REVIEW-HV/SHUNT-REVIEW) each with full spec.
- Resistors -> deterministic Panasonic ERJ-2RKF 0402 1% 1/10W (consolidated 1 part/value).
- Caps -> verified Murata GRM parts where value matches; clean spec + footprint otherwise.
- 1633 symbol field updates (Value/Footprint/Description/MPN/Mfr/Digikey) written to
  .kicad_sch; netlist re-parse confirms connectivity byte-identical.
- Add docs/sts1000_net_naming.md naming reference.

Co-Authored-By: Claude Opus 4.8 (1M context) <noreply@anthropic.com>
Parts:
- C161, C162, C163, C164, C165, C166, C167, C168, C169: footprint 0805 -> C_0402_1005Metric; DIGIKEY_PART_NUMBER 445-5972-1-ND -> 490-6328-2-ND; MANUFACTURER TDK -> Murata; MANUFACTURER_PART_NUMBER C2012X7R1E475K125AB -> GRM155R71C104KA88J
- R190, R191, R192, R193, R194, R195, R196, R197, R198, R199, R200, R201: footprint (none) -> R_0402_1005Metric; MANUFACTURER (none) -> Panasonic; MANUFACTURER_PART_NUMBER (none) -> ERJ-2RKF1002X
- U54, U55: MANUFACTURER_PART_NUMBER (none) -> MCP23017T-E/ML
