File: hardware/ntp-server-stm32/i2c-gpio.kicad_sch (KiCad schematic)
At the start: 23 parts, among them U54 MCP23017T-E/ML, U55 MCP23017T-E/ML

Commit message: Updates
Parts:
- removed C168, C169: 0.1uF, C_0402_1005Metric, symbol Device:C
- removed R197, R198, R199, R200, R201: 10k, R_0402_1005Metric, symbol Device:R
- removed U54, U55: MCP23017T-E/ML, Package_DFN_QFN:QFN-28-1EP_6x6mm_P0.65mm_EP4.25x4.25mm, symbol Interface_Expansion:MCP23017x-x-ML
- added C187, C202: 0.1uF, 0402 (1005 Metric), symbol Device:C
- added C201: 1nF, 0402 (1005 Metric), symbol Device:C
- added R220, R221, R222, R223, R224, R225, R226, R227, R236, R254, R265: 10k, 0402 (1005 Metric), symbol Device:R
- C161, C162, C163, C164, C165, C166, C167: footprint C_0402_1005Metric -> 0402 (1005 Metric); DIELECTRIC (none) -> X7R; DIGIKEY_PART_NUMBER 490-6328-2-ND -> 490-4759-1-ND; MANUFACTURER_PART_NUMBER GRM155R71C104KA88J -> GCM155R71C104KA55D; TOLERANCE (none) -> 10%; VOLTAGE (none) -> 16V
- R190, R191, R192, R193, R194, R195, R196: footprint R_0402_1005Metric -> 0402 (1005 Metric); DIELECTRIC (none) -> Thick-film; DIGIKEY_PART_NUMBER (none) -> P10.0KLCT-ND; MANUFACTURER Panasonic -> Panasonic Industry; POWER (none) -> 1/10W; TOLERANCE (none) -> 1%
Connections:
- net 3V3_STM: now also R220.1, R221.1, R222.1, R223.1, R224.1, R225.1, R226.1, R227.1, R236.1, R254.1, R265.1
- net GND: now also C187.2, C201.2, C202.2
- net INA_ALERT_3V3: now also R221.2
- net INA_ALERT_3V3_GPS: now also R224.2
- net INA_ALERT_3V3_STM: now also R222.2
- net INA_ALERT_5V_DISP: now also R223.2
- net INA_ALERT_OCXO: now also R226.2
- net INA_ALERT_VCC_RB: now also R265.2
- net INA_ALERT_V_ANT: now also R225.2
- net INA_ALERT_V_POE: now also R220.2
- new net ENC_BUTTON: C187.1, R236.2
- new net INA_ALERT_5V_PANEL: R227.2
- new net PROX_WAKE: C202.1, R254.2
- new net RTC_TAMPER: C201.1
- no-connect marks 5 -> 0
Other:
- note removed: "I2C Address: 0x20"
- note removed: "I2C Address: 0x21"
- moved on the sheet: C161, C162, C163, C164, C165, C166, C167, R190, R191, R192, R193, R194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

Commit message: Add files via upload
Updated, completed placement
Parts:
- C161, C162, C163, C164, C165, C166, C167, C187, C201, C202: footprint 0402 (1005 Metric) -> copy_ref:C_0402_1005Metric
- R190, R191, R192, R193, R194, R195, R196, R220, R221, R222, R223, R224, R225, R226, R227, R236, R254, R265: footprint 0402 (1005 Metric) -> copy_ref:R_0402_1005Metric
Changed lines of the file:
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@@
 			)
 		)
-		(property "Footprint" "0402 (1005 Metric)"
+		(property "Footprint" "copy_ref:R_0402_1005Metric"
 			(at 151.892 157.48 90)
 			(hide yes)
@@
 			)
 		)
-		(property "Footprint" "0402 (1005 Metric)"
+		(property "Footprint" "copy_ref:R_0402_1005Metric"
 			(at 117.602 157.48 90)
 			(hide yes)
@@
 			)
 		)
-		(property "Footprint" "0402 (1005 Metric)"
+		(property "Footprint" "copy_ref:C_0402_1005Metric"
 			(at 120.3452 203.2 0)
 			(hide yes)
@@
 			)
 		)
-		(property "Footprint" "0402 (1005 Metric)"
+		(property "Footprint" "copy_ref:C_0402_1005Metric"
 			(at 154.6352 203.2 0)
 			(hide yes)
@@
 			)
 		)
-		(property "Footprint" "0402 (1005 Metric)"
+		(property "Footprint" "copy_ref:R_0402_1005Metric"
 			(at 267.462 168.91 90)
 			(hide yes)
@@
 			)
 		)
-		(property "Footprint" "0402 (1005 Metric)"
+		(property "Footprint" "copy_ref:R_0402_1005Metric"
 			(at 311.912 168.91 90)
 			(hide yes)
@@
 			)
 		)
-		(property "Footprint" "0402 (1005 Metric)"
+		(property "Footprint" "copy_ref:C_0402_1005Metric"
 			(at 87.3252 203.2 0)
 			(hide yes)
@@
 			)
 		)
-		(property "Footprint" "0402 (1005 Metric)"
+		(property "Footprint" "copy_ref:R_0402_1005Metric"
 			(at 168.402 157.48 90)
 			(hide yes)
@@
 			)
 		)
-		(property "Footprint" "0402 (1005 Metric)"
+		(property "Footprint" "copy_ref:R_0402_1005Metric"
 			(at 357.632 168.91 90)
 			(hide yes)
@@
 			)
 		)
-		(property "Footprint" "0402 (1005 Metric)"
+		(property "Footprint" "copy_ref:C_0402_1005Metric"
 			(at 136.8552 203.2 0)
 			(hide yes)
@@
 			)
 		)
-		(property "Footprint" "0402 (1005 Metric)"
+		(property "Footprint" "copy_ref:R_0402_1005Metric"
 			(at 84.582 157.48 90)
 			(hide yes)
@@
 			)
 		)
-		(property "Footprint" "0402 (1005 Metric)"
+		(property "Footprint" "copy_ref:R_0402_1005Metric"
 			(at 126.492 90.17 90)
 			(hide yes)
@@
 			)
 		)
-		(property "Footprint" "0402 (1005 Metric)"
+		(property "Footprint" "copy_ref:R_0402_1005Metric"
 			(at 383.032 168.91 90)
 			(hide yes)
@@
 			)
 		)
-		(property "Footprint" "0402 (1005 Metric)"
+		(property "Footprint" "copy_ref:R_0402_1005Metric"
 			(at 134.112 157.48 90)
 			(hide yes)
@@
 			)
 		)
-		(property "Footprint" "0402 (1005 Metric)"
+		(property "Footprint" "copy_ref:R_0402_1005Metric"
 			(at 296.672 168.91 90)
 			(hide yes)
@@
 			)
 		)
-		(property "Footprint" "0402 (1005 Metric)"
+		(property "Footprint" "copy_ref:R_0402_1005Metric"
 			(at 184.912 157.48 90)
 			(hide yes)
@@
 			)
 		)
-		(property "Footprint" "0402 (1005 Metric)"
+		(property "Footprint" "copy_ref:R_0402_1005Metric"
 			(at 83.312 90.17 90)
 			(hide yes)
@@
 			)
 		)
-		(property "Footprint" "0402 (1005 Metric)"
+		(property "Footprint" "copy_ref:C_0402_1005Metric"
 			(at 103.8352 203.2 0)
 			(hide yes)
@@
 			)
 		)
-		(property "Footprint" "0402 (1005 Metric)"
+		(property "Footprint" "copy_ref:C_0402_1005Metric"
 			(at 86.0552 104.14 0)
 			(hide yes)
@@
 			)
 		)
-		(property "Footprint" "0402 (1005 Metric)"
+		(property "Footprint" "copy_ref:R_0402_1005Metric"
 			(at 342.392 168.91 90)
 			(hide yes)
@@
 			)
 		)
-		(property "Footprint" "0402 (1005 Metric)"
+		(property "Footprint" "copy_ref:C_0402_1005Metric"
 			(at 171.1452 203.2 0)
 			(hide yes)
@@
 			)
 		)
-		(property "Footprint" "0402 (1005 Metric)"
+		(property "Footprint" "copy_ref:R_0402_1005Metric"
 			(at 327.152 168.91 90)
 			(hide yes)
@@
 			)
 		)
-		(property "Footprint" "0402 (1005 Metric)"
+		(property "Footprint" "copy_ref:C_0402_1005Metric"
 			(at 129.2352 104.14 0)
 			(hide yes)
@@
 			)
 		)
-		(property "Footprint" "0402 (1005 Metric)"
+		(property "Footprint" "copy_ref:R_0402_1005Metric"
 			(at 282.702 168.91 90)
 			(hide yes)
@@
 			)
 		)
-		(property "Footprint" "0402 (1005 Metric)"
+		(property "Footprint" "copy_ref:R_0402_1005Metric"
 			(at 101.092 157.48 90)
 			(hide yes)
@@
 			)
 		)
-		(property "Footprint" "0402 (1005 Metric)"
+		(property "Footprint" "copy_ref:C_0402_1005Metric"
 			(at 187.6552 203.2 0)
 			(hide yes)
@@
 			)
 		)
-		(property "Footprint" "0402 (1005 Metric)"
+		(property "Footprint" "copy_ref:C_0402_1005Metric"
 			(at 166.6748 105.41 0)
 			(hide yes)
@@
 			)
 		)
-		(property "Footprint" "0402 (1005 Metric)"
+		(property "Footprint" "copy_ref:R_0402_1005Metric"
 			(at 370.332 168.91 90)
 			(hide yes)
