File: hardware/ntp-server-stm32/i2c-peripherals.kicad_sch (KiCad schematic)
At the start: 13 parts, among them U57 TMP117xxDRV, U58 TMP117xxDRV, U59 LIS2DH12TR, U60 ATECC608B-SSHDA, U61 IIS2MDCTR

Commit message: Standardize net/rail names: plain 3V3 style, _N active-low, voltage-format PG/alerts
22 net renames applied across all sheets and verified: removed/added net-name
sets match intent exactly and all node connectivity is preserved (kicad-cli
netlist re-parse).

Co-Authored-By: Claude Opus 4.8 (1M context) <noreply@anthropic.com>
Connections:
- net +3.3V_STM renamed 3V3_STM
Changed lines of the file:
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@@
 			)
 		)
-		(property "Value" "+3.3V_STM"
+		(property "Value" "3V3_STM"
 			(at 85.09 119.38 0)
 			(show_name no)
@@
 			)
 		)
-		(property "Value" "+3.3V_STM"
+		(property "Value" "3V3_STM"
 			(at 283.21 88.9 0)
 			(show_name no)
@@
 			)
 		)
-		(property "Value" "+3.3V_STM"
+		(property "Value" "3V3_STM"
 			(at 250.19 182.88 0)
 			(show_name no)
@@
 			)
 		)
-		(property "Value" "+3.3V_STM"
+		(property "Value" "3V3_STM"
 			(at 48.26 54.61 0)
 			(show_name no)
@@
 			)
 		)
-		(property "Value" "+3.3V_STM"
+		(property "Value" "3V3_STM"
 			(at 83.82 29.21 0)
 			(show_name no)
@@
 			)
 		)
-		(property "Value" "+3.3V_STM"
+		(property "Value" "3V3_STM"
 			(at 148.59 92.71 0)
 			(show_name no)
@@
 			)
 		)
-		(property "Value" "+3.3V_STM"
+		(property "Value" "3V3_STM"
 			(at 361.95 76.2 0)
 			(show_name no)
@@
 			)
 		)
-		(property "Value" "+3.3V_STM"
+		(property "Value" "3V3_STM"
 			(at 226.06 81.28 0)
 			(show_name no)

Commit message: Standardize + complete BOM; write fields back into KiCad symbols
- New sts1000_bom.csv: rebuilt from authoritative Value field (source MPN/footprint/
  description were corrupted by copy-paste). 338 standardized, 78 MPN-from-value,
  50 kept, ~64 flagged (SELECT/REVIEW-HV/SHUNT-REVIEW) each with full spec.
- Resistors -> deterministic Panasonic ERJ-2RKF 0402 1% 1/10W (consolidated 1 part/value).
- Caps -> verified Murata GRM parts where value matches; clean spec + footprint otherwise.
- 1633 symbol field updates (Value/Footprint/Description/MPN/Mfr/Digikey) written to
  .kicad_sch; netlist re-parse confirms connectivity byte-identical.
- Add docs/sts1000_net_naming.md naming reference.

Co-Authored-By: Claude Opus 4.8 (1M context) <noreply@anthropic.com>
Parts:
- C171, C172, C173, C174, C175, C177, C178: footprint 0805 -> C_0402_1005Metric; DIGIKEY_PART_NUMBER 445-5972-1-ND -> 490-6328-2-ND; MANUFACTURER TDK -> Murata; MANUFACTURER_PART_NUMBER C2012X7R1E475K125AB -> GRM155R71C104KA88J
- C176: footprint 0805 -> C_0402_1005Metric
- U57, U58: MANUFACTURER_PART_NUMBER (none) -> TMP117xxDRV
- U59: MANUFACTURER_PART_NUMBER (none) -> LIS2DH12TR
- U60: MANUFACTURER_PART_NUMBER (none) -> ATECC608B-SSHDA
- U61: MANUFACTURER_PART_NUMBER (none) -> IIS2MDCTR
Changed lines of the file:
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@@
 			)
 		)
-		(property "Footprint" "0805"
+		(property "Footprint" "C_0402_1005Metric"
 			(at 227.0252 95.25 0)
 			(hide yes)
@@
 			)
 		)
-		(property "Description" "CAP CER 4.7UF 25V X7R 0805"
+		(property "Description" "CAP CER 0.1uF 16V X7R 0402"
 			(at 226.06 91.44 0)
 			(hide yes)
@@
 			)
 		)
-		(property "DIGIKEY_PART_NUMBER" "445-5972-1-ND"
+		(property "DIGIKEY_PART_NUMBER" "490-6328-2-ND"
 			(at 226.06 91.44 0)
 			(hide yes)
@@
 			)
 		)
-		(property "MANUFACTURER" "TDK"
+		(property "MANUFACTURER" "Murata"
 			(at 226.06 91.44 0)
 			(hide yes)
@@
 			)
 		)
-		(property "MANUFACTURER_PART_NUMBER" "C2012X7R1E475K125AB"
+		(property "MANUFACTURER_PART_NUMBER" "GRM155R71C104KA88J"
 			(at 226.06 91.44 0)
 			(hide yes)
@@
 			)
 		)
-		(property "Footprint" "0805"
+		(property "Footprint" "C_0402_1005Metric"
 			(at 86.0552 133.35 0)
 			(hide yes)
@@
 			)
 		)
-		(property "Description" "CAP CER 4.7UF 25V X7R 0805"
+		(property "Description" "CAP CER 0.1uF 16V X7R 0402"
 			(at 85.09 129.54 0)
 			(hide yes)
@@
 			)
 		)
-		(property "DIGIKEY_PART_NUMBER" "445-5972-1-ND"
+		(property "DIGIKEY_PART_NUMBER" "490-6328-2-ND"
 			(at 85.09 129.54 0)
 			(hide yes)
@@
 			)
 		)
-		(property "MANUFACTURER" "TDK"
+		(property "MANUFACTURER" "Murata"
 			(at 85.09 129.54 0)
 			(hide yes)
@@
 			)
 		)
-		(property "MANUFACTURER_PART_NUMBER" "C2012X7R1E475K125AB"
+		(property "MANUFACTURER_PART_NUMBER" "GRM155R71C104KA88J"
 			(at 85.09 129.54 0)
 			(hide yes)
@@
 			)
 		)
-		(property "Footprint" "0805"
+		(property "Footprint" "C_0402_1005Metric"
 			(at 275.8948 123.19 0)
 			(hide yes)
@@
 			)
 		)
-		(property "Description" "CAP CER 4.7UF 25V X7R 0805"
+		(property "Description" "CAP CER 220nF 16V X7R 0402"
 			(at 276.86 119.38 0)
 			(hide yes)
@@
 			)
 		)
-		(property "Footprint" "0805"
+		(property "Footprint" "C_0402_1005Metric"
 			(at 362.9152 90.17 0)
 			(hide yes)
@@
 			)
 		)
-		(property "Description" "CAP CER 4.7UF 25V X7R 0805"
+		(property "Description" "CAP CER 0.1uF 16V X7R 0402"
 			(at 361.95 86.36 0)
 			(hide yes)
@@
 			)
 		)
-		(property "DIGIKEY_PART_NUMBER" "445-5972-1-ND"
+		(property "DIGIKEY_PART_NUMBER" "490-6328-2-ND"
 			(at 361.95 86.36 0)
 			(hide yes)
@@
 			)
 		)
-		(property "MANUFACTURER" "TDK"
+		(property "MANUFACTURER" "Murata"
 			(at 361.95 86.36 0)
 			(hide yes)
@@
 			)
 		)
-		(property "MANUFACTURER_PART_NUMBER" "C2012X7R1E475K125AB"
+		(property "MANUFACTURER_PART_NUMBER" "GRM155R71C104KA88J"
 			(at 361.95 86.36 0)
 			(hide yes)
@@
 			)
 		)
-		(property "Description" "Digital Temperature Sensor with I2C/SMBus Interface, 16 bits, ±0.3°C, one-shot conversion, alert, nist traceable, EEPROM, WSON"
+		(property "Description" "Digital Temperature Sensor with I2C/SMBus Interface, 16 bits, Â±0.3Â°C, one-shot conversion, alert, nist traceable, EEPROM, WSON"
 			(at 78.74 59.69 0)
+			(hide yes)
+			(show_name no)
+			(do_not_autoplace no)
+			(effects
+				(font
+					(size 1.27 1.27)
+				)
+			)
+		)
+		(property "MANUFACTURER_PART_NUMBER" "TMP117xxDRV"
+			(at 0 0 0)
 			(hide yes)
 			(show_name no)
@@
 			)
 		)
-		(property "Footprint" "0805"
+		(property "Footprint" "C_0402_1005Metric"
 			(at 376.8852 90.17 0)
 			(hide yes)
@@
 			)
 		)
-		(property "Description" "CAP CER 4.7UF 25V X7R 0805"
+		(property "Description" "CAP CER 0.1uF 16V X7R 0402"
 			(at 375.92 86.36 0)
 			(hide yes)
@@
 			)
 		)
-		(property "DIGIKEY_PART_NUMBER" "445-5972-1-ND"
+		(property "DIGIKEY_PART_NUMBER" "490-6328-2-ND"
 			(at 375.92 86.36 0)
 			(hide yes)
@@
 			)
 		)
-		(property "MANUFACTURER" "TDK"
+		(property "MANUFACTURER" "Murata"
 			(at 375.92 86.36 0)
 			(hide yes)
@@
 			)
 		)
-		(property "MANUFACTURER_PART_NUMBER" "C2012X7R1E475K125AB"
+		(property "MANUFACTURER_PART_NUMBER" "GRM155R71C104KA88J"
 			(at 375.92 86.36 0)
 			(hide yes)
@@
 			)
 		)
-		(property "Description" ""
+		(property "Description" "LIS2DH12TR"
 			(at 152.4 101.6 0)
+			(hide yes)
+			(show_name no)
+			(do_not_autoplace no)
+			(effects
+				(font
+					(size 1.27 1.27)
+				)
+			)
+		)
+		(property "MANUFACTURER_PART_NUMBER" "LIS2DH12TR"
+			(at 0 0 0)
 			(hide yes)
 			(show_name no)
@@
 			)
 		)
-		(property "Description" ""
+		(property "Description" "IIS2MDCTR"
 			(at 285.75 99.06 0)
+			(hide yes)
+			(show_name no)
+			(do_not_autoplace no)
+			(effects
+				(font
+					(size 1.27 1.27)
+				)
+			)
+		)
+		(property "MANUFACTURER_PART_NUMBER" "IIS2MDCTR"
+			(at 0 0 0)
 			(hide yes)
 			(show_name no)
@@
 			)
 		)
+		(property "MANUFACTURER_PART_NUMBER" "ATECC608B-SSHDA"
+			(at 0 0 0)
+			(hide yes)
+			(show_name no)
+			(do_not_autoplace no)
+			(effects
+				(font
+					(size 1.27 1.27)
+				)
+			)
+		)
 		(pin "5"
 		)
@@
 			)
 		)
-		(property "Footprint" "0805"
+		(property "Footprint" "C_0402_1005Metric"
 			(at 240.9952 95.25 0)
 			(hide yes)
@@
 			)
 		)
-		(property "Description" "CAP CER 4.7UF 25V X7R 0805"
+		(property "Description" "CAP CER 0.1uF 16V X7R 0402"
 			(at 240.03 91.44 0)
 			(hide yes)
@@
 			)
 		)
-		(property "DIGIKEY_PART_NUMBER" "445-5972-1-ND"
+		(property "DIGIKEY_PART_NUMBER" "490-6328-2-ND"
 			(at 240.03 91.44 0)
 			(hide yes)
@@
 			)
 		)
-		(property "MANUFACTURER" "TDK"
+		(property "MANUFACTURER" "Murata"
 			(at 240.03 91.44 0)
 			(hide yes)
@@
 			)
 		)
-		(property "MANUFACTURER_PART_NUMBER" "C2012X7R1E475K125AB"
+		(property "MANUFACTURER_PART_NUMBER" "GRM155R71C104KA88J"
 			(at 240.03 91.44 0)
 			(hide yes)
@@
 			)
 		)
-		(property "Description" "Digital Temperature Sensor with I2C/SMBus Interface, 16 bits, ±0.3°C, one-shot conversion, alert, nist traceable, EEPROM, WSON"
+		(property "Description" "Digital Temperature Sensor with I2C/SMBus Interface, 16 bits, Â±0.3Â°C, one-shot conversion, alert, nist traceable, EEPROM, WSON"
 			(at 80.01 149.86 0)
+			(hide yes)
+			(show_name no)
+			(do_not_autoplace no)
+			(effects
+				(font
+					(size 1.27 1.27)
+				)
+			)
+		)
+		(property "MANUFACTURER_PART_NUMBER" "TMP117xxDRV"
+			(at 0 0 0)
 			(hide yes)
 			(show_name no)
@@
 			)
 		)
-		(property "Footprint" "0805"
+		(property "Footprint" "C_0402_1005Metric"
 			(at 251.1552 196.85 0)
 			(hide yes)
@@
 			)
 		)
-		(property "Description" "CAP CER 4.7UF 25V X7R 0805"
+		(property "Description" "CAP CER 0.1uF 16V X7R 0402"
 			(at 250.19 193.04 0)
 			(hide yes)
@@
 			)
 		)
-		(property "DIGIKEY_PART_NUMBER" "445-5972-1-ND"
+		(property "DIGIKEY_PART_NUMBER" "490-6328-2-ND"
 			(at 250.19 193.04 0)
 			(hide yes)
@@
 			)
 		)
-		(property "MANUFACTURER" "TDK"
+		(property "MANUFACTURER" "Murata"
 			(at 250.19 193.04 0)
 			(hide yes)
@@
 			)
 		)
-		(property "MANUFACTURER_PART_NUMBER" "C2012X7R1E475K125AB"
+		(property "MANUFACTURER_PART_NUMBER" "GRM155R71C104KA88J"
 			(at 250.19 193.04 0)
 			(hide yes)
@@
 			)
 		)
-		(property "Footprint" "0805"
+		(property "Footprint" "C_0402_1005Metric"
 			(at 84.7852 43.18 0)
 			(hide yes)
@@
 			)
 		)
-		(property "Description" "CAP CER 4.7UF 25V X7R 0805"
+		(property "Description" "CAP CER 0.1uF 16V X7R 0402"
 			(at 83.82 39.37 0)
 			(hide yes)
@@
 			)
 		)
-		(property "DIGIKEY_PART_NUMBER" "445-5972-1-ND"
+		(property "DIGIKEY_PART_NUMBER" "490-6328-2-ND"
 			(at 83.82 39.37 0)
 			(hide yes)
@@
 			)
 		)
-		(property "MANUFACTURER" "TDK"
+		(property "MANUFACTURER" "Murata"
 			(at 83.82 39.37 0)
 			(hide yes)
@@
 			)
 		)
-		(property "MANUFACTURER_PART_NUMBER" "C2012X7R1E475K125AB"
+		(property "MANUFACTURER_PART_NUMBER" "GRM155R71C104KA88J"
 			(at 83.82 39.37 0)
 			(hide yes)
