File: hardware/ntp-server-stm32/led.kicad_sch (KiCad schematic)
At the start: 13 parts, among them Q10 BC847W, Q8 BC847W, Q9 BC847W

Commit message: Standardize net/rail names: plain 3V3 style, _N active-low, voltage-format PG/alerts
22 net renames applied across all sheets and verified: removed/added net-name
sets match intent exactly and all node connectivity is preserved (kicad-cli
netlist re-parse).

Co-Authored-By: Claude Opus 4.8 (1M context) <noreply@anthropic.com>
Connections:
- net +5V renamed 5V
Changed lines of the file:
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@@
 			)
 		)
-		(property "Value" "+5V"
+		(property "Value" "5V"
 			(at 200.66 67.31 0)
 			(show_name no)
@@
 			)
 		)
-		(property "Value" "+5V"
+		(property "Value" "5V"
 			(at 191.77 67.31 0)
 			(show_name no)
@@
 			)
 		)
-		(property "Value" "+5V"
+		(property "Value" "5V"
 			(at 209.55 67.31 0)
 			(show_name no)

Commit message: Standardize + complete BOM; write fields back into KiCad symbols
- New sts1000_bom.csv: rebuilt from authoritative Value field (source MPN/footprint/
  description were corrupted by copy-paste). 338 standardized, 78 MPN-from-value,
  50 kept, ~64 flagged (SELECT/REVIEW-HV/SHUNT-REVIEW) each with full spec.
- Resistors -> deterministic Panasonic ERJ-2RKF 0402 1% 1/10W (consolidated 1 part/value).
- Caps -> verified Murata GRM parts where value matches; clean spec + footprint otherwise.
- 1633 symbol field updates (Value/Footprint/Description/MPN/Mfr/Digikey) written to
  .kicad_sch; netlist re-parse confirms connectivity byte-identical.
- Add docs/sts1000_net_naming.md naming reference.

Co-Authored-By: Claude Opus 4.8 (1M context) <noreply@anthropic.com>
Parts:
- D5: MANUFACTURER (none) -> Inolux
- Q10, Q8, Q9: MANUFACTURER_PART_NUMBER (none) -> BC847W
- R55: footprint (none) -> R_0402_1005Metric; MANUFACTURER (none) -> Panasonic; MANUFACTURER_PART_NUMBER (none) -> ERJ-2RKF1001X
- R56, R58, R63: footprint (none) -> R_0402_1005Metric; MANUFACTURER (none) -> Panasonic; MANUFACTURER_PART_NUMBER (none) -> ERJ-2RKF1002X
- R57: footprint (none) -> R_0402_1005Metric; MANUFACTURER (none) -> Panasonic; MANUFACTURER_PART_NUMBER (none) -> ERJ-2RKF1501X
- R59: footprint (none) -> R_0402_1005Metric; MANUFACTURER (none) -> Panasonic; MANUFACTURER_PART_NUMBER (none) -> ERJ-2RKF60R4X
- R60: footprint (none) -> R_0402_1005Metric; MANUFACTURER (none) -> Panasonic; MANUFACTURER_PART_NUMBER (none) -> ERJ-2RKF1740X
- R61: footprint (none) -> R_0402_1005Metric; MANUFACTURER (none) -> Panasonic; MANUFACTURER_PART_NUMBER (none) -> ERJ-2RKF2210X
- R62: footprint (none) -> R_0402_1005Metric; MANUFACTURER (none) -> Panasonic; MANUFACTURER_PART_NUMBER (none) -> ERJ-2RKF3011X
