File: hardware/ntp-server-stm32/led.kicad_sch (KiCad schematic)
At the start: 13 parts, among them Q10 BC847W, Q8 BC847W, Q9 BC847W

Commit message: Updates
Parts:
- added C168: 10uF, 1206 (3216 Metric), symbol Device:C
- added C169, C185: 0.1uF, 0402 (1005 Metric), symbol Device:C
- added C200: 1nF, 0402 (1005 Metric), symbol Device:C
- added FB12: 600, 1206, symbol Device:FerriteBead
- added Q22: NSS40300MZ4T1G, SOT-223 (TO-261), symbol Transistor_BJT:BCP51
- added Q23: BC847W, SOT-323, symbol Transistor_BJT:BC847W
- added R198, R201, R235: 10k, 0402 (1005 Metric), symbol Device:R
- added R199: 220m, 0805, symbol Device:R
- added R216: 4.7k, 0805, symbol Device:R
- added R217: 820, 0805, symbol Device:R
- added R234: 4.7k, 0402 (1005 Metric), symbol Device:R
- added R247, R248, R249, R250, R251, R252: 91, 0805, symbol Device:R
- added R253: 150, 0805, symbol Device:R
- added U54: INA228AQDGSRQ1, VSSOP10_DGS_TEX, symbol INA228AQDGSRQ1:INA228AQDGSRQ1
- added U55: RT9742VGJ5, TSOT-23-5, symbol CM5IO:RT9742GGJ5
- D5: DIELECTRIC (none) -> Diode
- Q10, Q8, Q9: footprint Package_TO_SOT_SMD:SOT-323_SC-70 -> SOT-323; DIELECTRIC (none) -> Transistor; DIGIKEY_PART_NUMBER (none) -> 1727-BC847W,135CT-ND; MANUFACTURER (none) -> Nexperia USA Inc.; MANUFACTURER_PART_NUMBER BC847W -> BC847W,135
- R55: footprint R_0402_1005Metric -> 0402 (1005 Metric); DIELECTRIC (none) -> Thick-film; DIGIKEY_PART_NUMBER (none) -> P1.00KLCT-ND; MANUFACTURER Panasonic -> Panasonic Industry; POWER (none) -> 1/10W; TOLERANCE (none) -> 1%
- R56, R58, R63: footprint R_0402_1005Metric -> 0402 (1005 Metric); DIELECTRIC (none) -> Thick-film; DIGIKEY_PART_NUMBER (none) -> P10.0KLCT-ND; MANUFACTURER Panasonic -> Panasonic Industry; POWER (none) -> 1/10W; TOLERANCE (none) -> 1%
- R57: footprint R_0402_1005Metric -> 0402 (1005 Metric); DIELECTRIC (none) -> Thick-film; DIGIKEY_PART_NUMBER (none) -> P1.50KLCT-ND; MANUFACTURER Panasonic -> Panasonic Industry; POWER (none) -> 1/10W; TOLERANCE (none) -> 1%
- R59: footprint R_0402_1005Metric -> 0402 (1005 Metric); DIELECTRIC (none) -> Thick-film; DIGIKEY_PART_NUMBER (none) -> 2019-RK73H1ETTP60R4FCT-ND; MANUFACTURER Panasonic -> KOA Speer Electronics, Inc.; MANUFACTURER_PART_NUMBER ERJ-2RKF60R4X -> RK73H1ETTP60R4F; POWER (none) -> 1/10W; TOLERANCE (none) -> 1%
- R60: footprint R_0402_1005Metric -> 0402 (1005 Metric); DIELECTRIC (none) -> Thick-film; DIGIKEY_PART_NUMBER (none) -> P174LCT-ND; MANUFACTURER Panasonic -> Panasonic Industry; POWER (none) -> 1/10W; TOLERANCE (none) -> 1%
- R61: footprint R_0402_1005Metric -> 0402 (1005 Metric); DIELECTRIC (none) -> Thick-film; DIGIKEY_PART_NUMBER (none) -> 2019-RK73H1ETTP2210FCT-ND; MANUFACTURER Panasonic -> KOA Speer Electronics, Inc.; MANUFACTURER_PART_NUMBER ERJ-2RKF2210X -> RK73H1ETTP2210F; POWER (none) -> 1/10W; TOLERANCE (none) -> 1%
- R62: footprint R_0402_1005Metric -> 0402 (1005 Metric); DIELECTRIC (none) -> Thick-film; DIGIKEY_PART_NUMBER (none) -> 2019-RK73H1ETTP3011FCT-ND; MANUFACTURER Panasonic -> KOA Speer Electronics, Inc.; MANUFACTURER_PART_NUMBER ERJ-2RKF3011X -> RK73H1ETTP3011F; POWER (none) -> 1/10W; TOLERANCE (none) -> 1%
Connections:
- net 5V: now also U55.5 (IN)
- net GND: now also C168.2, C169.2, C185.2, C200.2, Q23.2 (E), R198.2, R235.2, R247.2, R248.2, R249.2, R250.2, R251.2, R252.2, R253.2, U54.2 (A0), U54.7 (GND), U55.2 (GND)
- new net: Q23.1 (B), R216.2, R235.1
- new net: C168.1, R199.1, U54.10 (IN+), U55.1 (OUT)
- new net: Q22.1 (B), R217.2, R234.2
- new net: FB12.2, R199.2, U54.8 (VBUS), U54.9 (IN-)
- new net: Q23.3 (C), R217.1
- new net 3V3: C169.1, U54.6 (VS)
- new net 3V3_STM: R201.1
- new net I2C_SCL: U54.1 (A1), U54.5 (SCL)
- new net I2C_SDA: U54.4 (SDA)
- new net INA_ALERT_5V_PANEL: U54.3 (ALERT)
- new net PANEL_LEDS_P: Q22.2 (C)
- new net PANEL_LED_EN: R198.1, U55.4 (EN)
- new net PANEL_LED_FAULT: R201.2, U55.3 (nFLG)
- new net PANEL_LED_PWM: R216.1
- new net PANEL_LED_RED_N_1: R253.1
- new net PANEL_LED_WHITE_N_1: R247.1
- new net PANEL_LED_WHITE_N_2: R248.1
- new net PANEL_LED_WHITE_N_3: R249.1
- new net PANEL_LED_WHITE_N_4: R250.1
- new net PANEL_LED_WHITE_N_5: R251.1
- new net PANEL_LED_WHITE_N_6: R252.1
- new net V_PANEL_LED: C185.1, C200.1, FB12.1, Q22.3 (E), R234.1
Other:
- note added: "I2C Address: 0x4C"
- moved on the sheet: D5, Q10, Q8, Q9, R55, R56, R57, R58, R59, R60, R61, R62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

Commit message: Bom updates
Parts:
- FB12: footprint 1206 -> 1206 (3216 Metric)
- R199: value 220m -> 150m; footprint 0805 -> 1206 (3216 Metric); DIGIKEY_PART_NUMBER 273-KDV08DR150ETCT-ND -> WSLC-.15CT-ND; MANUFACTURER Ohmite -> Vishay Dale; MANUFACTURER_PART_NUMBER KDV08DR150ET -> WSL1206R1500FEA
- R216: footprint 0805 -> 0805 (2012 Metric); DIGIKEY_PART_NUMBER 273-KDV08DR150ETCT-ND -> P4.70KCCT-ND; MANUFACTURER Panasonic -> Panasonic Industry
- R217: footprint 0805 -> 0805 (2012 Metric); DIGIKEY_PART_NUMBER 273-KDV08DR150ETCT-ND -> P820CCT-ND; MANUFACTURER Panasonic -> Panasonic Industry
- R247, R248, R249, R250, R251, R252: footprint 0805 -> 0805 (2012 Metric); DIGIKEY_PART_NUMBER 273-KDV08DR150ETCT-ND -> P91.0CCT-ND; MANUFACTURER Panasonic -> Panasonic Industry
- R253: footprint 0805 -> 0805 (2012 Metric); DIGIKEY_PART_NUMBER 273-KDV08DR150ETCT-ND -> P150CCT-ND; MANUFACTURER Panasonic -> Panasonic Industry
- U54: DIGIKEY_PART_NUMBER (none) -> 296-INA228AQDGSRQ1CT-ND
Changed lines of the file:
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@@
 			)
 		)
-		(property "Footprint" "0805"
+		(property "Footprint" "0805 (2012 Metric)"
 			(at 132.08 238.252 90)
 			(hide yes)
@@
 			)
 		)
-		(property "Datasheet" "https://www.ohmite.com/assets/images/res-kdv.pdf"
+		(property "Datasheet" "https://industrial.panasonic.com/cdbs/www-data/pdf/RDA0000/AOA0000C304.pdf"
 			(at 132.08 240.03 0)
 			(hide yes)
@@
 			)
 		)
-		(property "Description" "RES 91 1% 1/8W 0805"
+		(property "Description" "RES SMD 91 OHM 1% 1/8W 0805"
 			(at 132.08 240.03 90)
 			(hide yes)
@@
 			)
 		)
-		(property "DIGIKEY_PART_NUMBER" "273-KDV08DR150ETCT-ND"
+		(property "DIGIKEY_PART_NUMBER" "P91.0CCT-ND"
 			(at 132.08 240.03 90)
 			(hide yes)
@@
 			)
 		)
-		(property "MANUFACTURER" "Panasonic"
+		(property "MANUFACTURER" "Panasonic Industry"
 			(at 132.08 240.03 90)
 			(hide yes)
@@
 			)
 		)
-		(property "Footprint" "0805"
+		(property "Footprint" "0805 (2012 Metric)"
 			(at 132.08 233.172 90)
 			(hide yes)
@@
 			)
 		)
-		(property "Datasheet" "https://www.ohmite.com/assets/images/res-kdv.pdf"
+		(property "Datasheet" "https://industrial.panasonic.com/cdbs/www-data/pdf/RDA0000/AOA0000C304.pdf"
 			(at 132.08 234.95 0)
 			(hide yes)
@@
 			)
 		)
-		(property "Description" "RES 91 1% 1/8W 0805"
+		(property "Description" "RES SMD 91 OHM 1% 1/8W 0805"
 			(at 132.08 234.95 90)
 			(hide yes)
@@
 			)
 		)
-		(property "DIGIKEY_PART_NUMBER" "273-KDV08DR150ETCT-ND"
+		(property "DIGIKEY_PART_NUMBER" "P91.0CCT-ND"
 			(at 132.08 234.95 90)
 			(hide yes)
@@
 			)
 		)
-		(property "MANUFACTURER" "Panasonic"
+		(property "MANUFACTURER" "Panasonic Industry"
 			(at 132.08 234.95 90)
 			(hide yes)
@@
 			)
 		)
-		(property "Footprint" "0805"
+		(property "Footprint" "0805 (2012 Metric)"
 			(at 99.06 169.672 90)
 			(hide yes)
@@
 			)
 		)
-		(property "Datasheet" "https://www.ohmite.com/assets/images/res-kdv.pdf"
+		(property "Datasheet" "https://industrial.panasonic.com/cdbs/www-data/pdf/RDA0000/AOA0000C304.pdf"
 			(at 99.06 171.45 0)
 			(hide yes)
@@
 			)
 		)
-		(property "Description" "RES 4.7k 1% 1/8W 0805"
+		(property "Description" "RES SMD 4.7K OHM 1% 1/8W 0805"
 			(at 99.06 171.45 90)
 			(hide yes)
@@
 			)
 		)
-		(property "DIGIKEY_PART_NUMBER" "273-KDV08DR150ETCT-ND"
+		(property "DIGIKEY_PART_NUMBER" "P4.70KCCT-ND"
 			(at 99.06 171.45 90)
 			(hide yes)
@@
 			)
 		)
-		(property "MANUFACTURER" "Panasonic"
+		(property "MANUFACTURER" "Panasonic Industry"
 			(at 99.06 171.45 90)
 			(hide yes)
@@
 			)
 		)
-		(property "Footprint" "0805"
+		(property "Footprint" "0805 (2012 Metric)"
 			(at 132.08 243.332 90)
 			(hide yes)
@@
 			)
 		)
-		(property "Datasheet" "https://www.ohmite.com/assets/images/res-kdv.pdf"
+		(property "Datasheet" "https://industrial.panasonic.com/cdbs/www-data/pdf/RDA0000/AOA0000C304.pdf"
 			(at 132.08 245.11 0)
 			(hide yes)
@@
 			)
 		)
-		(property "Description" "RES 150 1% 1/8W 0805"
+		(property "Description" "RES SMD 150 OHM 1% 1/8W 0805"
 			(at 132.08 245.11 90)
 			(hide yes)
@@
 			)
 		)
-		(property "DIGIKEY_PART_NUMBER" "273-KDV08DR150ETCT-ND"
+		(property "DIGIKEY_PART_NUMBER" "P150CCT-ND"
 			(at 132.08 245.11 90)
 			(hide yes)
@@
 			)
 		)
-		(property "MANUFACTURER" "Panasonic"
+		(property "MANUFACTURER" "Panasonic Industry"
 			(at 132.08 245.11 90)
 			(hide yes)
@@
 			)
 		)
-		(property "Footprint" "0805"
+		(property "Footprint" "0805 (2012 Metric)"
 			(at 132.08 223.012 90)
 			(hide yes)
@@
 			)
 		)
-		(property "Datasheet" "https://www.ohmite.com/assets/images/res-kdv.pdf"
+		(property "Datasheet" "https://industrial.panasonic.com/cdbs/www-data/pdf/RDA0000/AOA0000C304.pdf"
 			(at 132.08 224.79 0)
 			(hide yes)
@@
 			)
 		)
-		(property "Description" "RES 91 1% 1/8W 0805"
+		(property "Description" "RES SMD 91 OHM 1% 1/8W 0805"
 			(at 132.08 224.79 90)
 			(hide yes)
@@
 			)
 		)
-		(property "DIGIKEY_PART_NUMBER" "273-KDV08DR150ETCT-ND"
+		(property "DIGIKEY_PART_NUMBER" "P91.0CCT-ND"
 			(at 132.08 224.79 90)
 			(hide yes)
@@
 			)
 		)
-		(property "MANUFACTURER" "Panasonic"
+		(property "MANUFACTURER" "Panasonic Industry"
 			(at 132.08 224.79 90)
 			(hide yes)
@@
 			)
 		)
-		(property "Datasheet" "https://www.ti.com/lit/gpn/ina228-q1"
+		(property "Datasheet" "https://www.ti.com/lit/ds/symlink/ina228-q1.pdf"
 			(at 60.96 93.98 0)
 			(hide yes)
@@
 			)
 		)
-		(property "Description" "Current/power monitor 20-bit I2C"
+		(property "Description" "IC PWR MONITOR 10VSSOP"
 			(at 60.96 93.98 0)
 			(hide yes)
@@
 			)
 		)
+		(property "DIGIKEY_PART_NUMBER" "296-INA228AQDGSRQ1CT-ND"
+			(at 60.96 93.98 0)
+			(hide yes)
+			(show_name no)
+			(do_not_autoplace no)
+			(effects
+				(font
+					(size 1.27 1.27)
+				)
+			)
+		)
 		(pin "2"
 		)
@@
 			)
 		)
-		(property "Footprint" "0805"
+		(property "Footprint" "0805 (2012 Metric)"
 			(at 133.35 160.782 90)
 			(hide yes)
@@
 			)
 		)
-		(property "Datasheet" "https://www.ohmite.com/assets/images/res-kdv.pdf"
+		(property "Datasheet" "https://industrial.panasonic.com/cdbs/www-data/pdf/RDA0000/AOA0000C304.pdf"
 			(at 133.35 162.56 0)
 			(hide yes)
@@
 			)
 		)
-		(property "Description" "RES 820 1% 1/8W 0805"
+		(property "Description" "RES SMD 820 OHM 1% 1/8W 0805"
 			(at 133.35 162.56 90)
 			(hide yes)
@@
 			)
 		)
-		(property "DIGIKEY_PART_NUMBER" "273-KDV08DR150ETCT-ND"
+		(property "DIGIKEY_PART_NUMBER" "P820CCT-ND"
 			(at 133.35 162.56 90)
 			(hide yes)
@@
 			)
 		)
-		(property "MANUFACTURER" "Panasonic"
+		(property "MANUFACTURER" "Panasonic Industry"
 			(at 133.35 162.56 90)
 			(hide yes)
@@
 			)
 		)
-		(property "Footprint" "0805"
+		(property "Footprint" "0805 (2012 Metric)"
 			(at 132.08 212.852 90)
 			(hide yes)
@@
 			)
 		)
-		(property "Datasheet" "https://www.ohmite.com/assets/images/res-kdv.pdf"
+		(property "Datasheet" "https://industrial.panasonic.com/cdbs/www-data/pdf/RDA0000/AOA0000C304.pdf"
 			(at 132.08 214.63 0)
 			(hide yes)
@@
 			)
 		)
-		(property "Description" "RES 91 1% 1/8W 0805"
+		(property "Description" "RES SMD 91 OHM 1% 1/8W 0805"
 			(at 132.08 214.63 90)
 			(hide yes)
@@
 			)
 		)
-		(property "DIGIKEY_PART_NUMBER" "273-KDV08DR150ETCT-ND"
+		(property "DIGIKEY_PART_NUMBER" "P91.0CCT-ND"
 			(at 132.08 214.63 90)
 			(hide yes)
@@
 			)
 		)
-		(property "MANUFACTURER" "Panasonic"
+		(property "MANUFACTURER" "Panasonic Industry"
 			(at 132.08 214.63 90)
 			(hide yes)
@@
 			)
 		)
-		(property "Footprint" "0805"
+		(property "Footprint" "0805 (2012 Metric)"
 			(at 132.08 228.092 90)
 			(hide yes)
@@
 			)
 		)
-		(property "Datasheet" "https://www.ohmite.com/assets/images/res-kdv.pdf"
+		(property "Datasheet" "https://industrial.panasonic.com/cdbs/www-data/pdf/RDA0000/AOA0000C304.pdf"
 			(at 132.08 229.87 0)
 			(hide yes)
@@
 			)
 		)
-		(property "Description" "RES 91 1% 1/8W 0805"
+		(property "Description" "RES SMD 91 OHM 1% 1/8W 0805"
 			(at 132.08 229.87 90)
 			(hide yes)
@@
 			)
 		)
-		(property "DIGIKEY_PART_NUMBER" "273-KDV08DR150ETCT-ND"
+		(property "DIGIKEY_PART_NUMBER" "P91.0CCT-ND"
 			(at 132.08 229.87 90)
 			(hide yes)
@@
 			)
 		)
-		(property "MANUFACTURER" "Panasonic"
+		(property "MANUFACTURER" "Panasonic Industry"
 			(at 132.08 229.87 90)
 			(hide yes)
@@
 			)
 		)
-		(property "Footprint" "0805"
+		(property "Footprint" "0805 (2012 Metric)"
 			(at 132.08 217.932 90)
 			(hide yes)
@@
 			)
 		)
-		(property "Datasheet" "https://www.ohmite.com/assets/images/res-kdv.pdf"
+		(property "Datasheet" "https://industrial.panasonic.com/cdbs/www-data/pdf/RDA0000/AOA0000C304.pdf"
 			(at 132.08 219.71 0)
 			(hide yes)
@@
 			)
 		)
-		(property "Description" "RES 91 1% 1/8W 0805"
+		(property "Description" "RES SMD 91 OHM 1% 1/8W 0805"
 			(at 132.08 219.71 90)
 			(hide yes)
@@
 			)
 		)
-		(property "DIGIKEY_PART_NUMBER" "273-KDV08DR150ETCT-ND"
+		(property "DIGIKEY_PART_NUMBER" "P91.0CCT-ND"
 			(at 132.08 219.71 90)
 			(hide yes)
@@
 			)
 		)
-		(property "MANUFACTURER" "Panasonic"
+		(property "MANUFACTURER" "Panasonic Industry"
 			(at 132.08 219.71 90)
 			(hide yes)
@@
 			)
 		)
-		(property "Value" "220m"
+		(property "Value" "150m"
 			(at 112.776 59.69 90)
 			(show_name no)
@@
 			)
 		)
-		(property "Footprint" "0805"
+		(property "Footprint" "1206 (3216 Metric)"
 			(at 110.49 55.372 90)
 			(hide yes)
@@
 			)
 		)
-		(property "Datasheet" "https://www.ohmite.com/assets/images/res-kdv.pdf"
+		(property "Datasheet" "https://www.vishay.com/docs/30100/wsl.pdf"
 			(at 110.49 57.15 0)
 			(hide yes)
@@
 			)
 		)
-		(property "Description" "RES 220m SENSE 0.5% 0805"
+		(property "Description" "RES 0.15 OHM 1% 1/4W 1206"
 			(at 110.49 57.15 90)
 			(hide yes)
@@
 			)
 		)
-		(property "DIGIKEY_PART_NUMBER" "273-KDV08DR150ETCT-ND"
+		(property "DIGIKEY_PART_NUMBER" "WSLC-.15CT-ND"
 			(at 110.49 57.15 90)
 			(hide yes)
@@
 			)
 		)
-		(property "MANUFACTURER_PART_NUMBER" "KDV08DR150ET"
+		(property "MANUFACTURER_PART_NUMBER" "WSL1206R1500FEA"
 			(at 110.49 57.15 90)
 			(hide yes)
@@
 			)
 		)
-		(property "MANUFACTURER" "Ohmite"
+		(property "MANUFACTURER" "Vishay Dale"
 			(at 110.49 57.15 90)
 			(hide yes)
@@
 			)
 		)
-		(property "Footprint" "1206"
+		(property "Footprint" "1206 (3216 Metric)"
 			(at 121.92 55.372 90)
 			(hide yes)

Commit message: Bom updates
Parts:
- U54: footprint VSSOP10_DGS_TEX -> sts1000:VSSOP10_DGS_TEX
Changed lines of the file:
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@@
 			)
 		)
-		(property "Footprint" "VSSOP10_DGS_TEX"
+		(property "Footprint" "sts1000:VSSOP10_DGS_TEX"
 			(at 60.96 93.98 0)
 			(hide yes)

Commit message: Add files via upload
Updated, completed placement
Parts:
- C168: footprint 1206 (3216 Metric) -> copy_ref:C_1206_3216Metric
- C169, C185, C200: footprint 0402 (1005 Metric) -> copy_ref:C_0402_1005Metric
- D5: footprint Library:LED_IN-P55TATRGB -> copy_ref:LED_IN-P55TATRGB
- FB12: footprint 1206 (3216 Metric) -> copy_ref:1206
- Q10, Q23, Q8, Q9: footprint SOT-323 -> Package_TO_SOT_SMD:SOT-323_SC-70
- Q22: footprint SOT-223 (TO-261) -> Package_TO_SOT_SMD:SOT-223
- R198, R201, R234, R235, R55, R56, R57, R58, R59, R60, R61, R62, R63: footprint 0402 (1005 Metric) -> copy_ref:R_0402_1005Metric
- R199: footprint 1206 (3216 Metric) -> copy_ref:R_1206_3216Metric
- R216, R217, R247, R248, R249, R250, R251, R252, R253: footprint 0805 (2012 Metric) -> copy_ref:R_0805_2012Metric
- U55: footprint TSOT-23-5 -> Package_TO_SOT_SMD:TSOT-23-5
Changed lines of the file:
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@@
 			)
 		)
-		(property "Footprint" "0402 (1005 Metric)"
+		(property "Footprint" "copy_ref:R_0402_1005Metric"
 			(at 352.298 62.23 90)
 			(hide yes)
@@
 			)
 		)
-		(property "Footprint" "0402 (1005 Metric)"
+		(property "Footprint" "copy_ref:R_0402_1005Metric"
 			(at 79.248 43.18 90)
 			(hide yes)
@@
 			)
 		)
-		(property "Footprint" "0402 (1005 Metric)"
+		(property "Footprint" "copy_ref:R_0402_1005Metric"
 			(at 376.428 118.11 90)
 			(hide yes)
@@
 			)
 		)
-		(property "Footprint" "0402 (1005 Metric)"
+		(property "Footprint" "copy_ref:R_0402_1005Metric"
 			(at 109.982 177.8 90)
 			(hide yes)
@@
 			)
 		)
-		(property "Footprint" "0402 (1005 Metric)"
+		(property "Footprint" "copy_ref:R_0402_1005Metric"
 			(at 318.77 140.208 90)
 			(hide yes)
@@
 			)
 		)
-		(property "Footprint" "TSOT-23-5"
+		(property "Footprint" "Package_TO_SOT_SMD:TSOT-23-5"
 			(at 66.04 67.31 0)
 			(hide yes)
@@
 			)
 		)
-		(property "Footprint" "0402 (1005 Metric)"
+		(property "Footprint" "copy_ref:R_0402_1005Metric"
 			(at 143.002 156.21 90)
 			(hide yes)
@@
 			)
 		)
-		(property "Footprint" "0805 (2012 Metric)"
+		(property "Footprint" "copy_ref:R_0805_2012Metric"
 			(at 132.08 238.252 90)
 			(hide yes)
@@
 			)
 		)
-		(property "Footprint" "0805 (2012 Metric)"
+		(property "Footprint" "copy_ref:R_0805_2012Metric"
 			(at 132.08 233.172 90)
 			(hide yes)
@@
 			)
 		)
-		(property "Footprint" "0402 (1005 Metric)"
+		(property "Footprint" "copy_ref:C_0402_1005Metric"
 			(at 128.5748 66.04 0)
 			(hide yes)
@@
 			)
 		)
-		(property "Footprint" "0402 (1005 Metric)"
+		(property "Footprint" "copy_ref:R_0402_1005Metric"
 			(at 331.978 146.05 90)
 			(hide yes)
@@
 			)
 		)
-		(property "Footprint" "SOT-323"
+		(property "Footprint" "Package_TO_SOT_SMD:SOT-323_SC-70"
 			(at 344.17 140.335 0)
 			(hide yes)
@@
 			)
 		)
-		(property "Footprint" "0805 (2012 Metric)"
+		(property "Footprint" "copy_ref:R_0805_2012Metric"
 			(at 99.06 169.672 90)
 			(hide yes)
@@
 			)
 		)
-		(property "Footprint" "0805 (2012 Metric)"
+		(property "Footprint" "copy_ref:R_0805_2012Metric"
 			(at 132.08 243.332 90)
 			(hide yes)
@@
 			)
 		)
-		(property "Footprint" "0402 (1005 Metric)"
+		(property "Footprint" "copy_ref:R_0402_1005Metric"
 			(at 316.738 118.11 90)
 			(hide yes)
@@
 			)
 		)
-		(property "Footprint" "0805 (2012 Metric)"
+		(property "Footprint" "copy_ref:R_0805_2012Metric"
 			(at 132.08 223.012 90)
 			(hide yes)
@@
 			)
 		)
-		(property "Footprint" "0402 (1005 Metric)"
+		(property "Footprint" "copy_ref:R_0402_1005Metric"
 			(at 57.658 67.31 90)
 			(hide yes)
@@
 			)
 		)
-		(property "Footprint" "SOT-323"
+		(property "Footprint" "Package_TO_SOT_SMD:SOT-323_SC-70"
 			(at 388.62 112.395 0)
 			(hide yes)
@@
 			)
 		)
-		(property "Footprint" "SOT-323"
+		(property "Footprint" "Package_TO_SOT_SMD:SOT-323_SC-70"
 			(at 328.93 112.395 0)
 			(hide yes)
@@
 			)
 		)
-		(property "Footprint" "Library:LED_IN-P55TATRGB"
+		(property "Footprint" "copy_ref:LED_IN-P55TATRGB"
 			(at 333.502 76.2 0)
 			(hide yes)
@@
 			)
 		)
-		(property "Footprint" "0402 (1005 Metric)"
+		(property "Footprint" "copy_ref:R_0402_1005Metric"
 			(at 334.518 62.23 90)
 			(hide yes)
@@
 			)
 		)
-		(property "Footprint" "SOT-223 (TO-261)"
+		(property "Footprint" "Package_TO_SOT_SMD:SOT-223"
 			(at 160.02 160.655 0)
 			(hide yes)
@@
 			)
 		)
-		(property "Footprint" "0805 (2012 Metric)"
+		(property "Footprint" "copy_ref:R_0805_2012Metric"
 			(at 133.35 160.782 90)
 			(hide yes)
@@
 			)
 		)
-		(property "Footprint" "0402 (1005 Metric)"
+		(property "Footprint" "copy_ref:C_0402_1005Metric"
 			(at 140.0048 66.04 0)
 			(hide yes)
@@
 			)
 		)
-		(property "Footprint" "0402 (1005 Metric)"
+		(property "Footprint" "copy_ref:C_0402_1005Metric"
 			(at 112.7252 111.76 0)
 			(hide yes)
@@
 			)
 		)
-		(property "Footprint" "SOT-323"
+		(property "Footprint" "Package_TO_SOT_SMD:SOT-323_SC-70"
 			(at 125.73 173.355 0)
 			(hide yes)
@@
 			)
 		)
-		(property "Footprint" "0805 (2012 Metric)"
+		(property "Footprint" "copy_ref:R_0805_2012Metric"
 			(at 132.08 212.852 90)
 			(hide yes)
@@
 			)
 		)
-		(property "Footprint" "0402 (1005 Metric)"
+		(property "Footprint" "copy_ref:R_0402_1005Metric"
 			(at 303.53 112.268 90)
 			(hide yes)
@@
 			)
 		)
-		(property "Footprint" "0805 (2012 Metric)"
+		(property "Footprint" "copy_ref:R_0805_2012Metric"
 			(at 132.08 228.092 90)
 			(hide yes)
@@
 			)
 		)
-		(property "Footprint" "0402 (1005 Metric)"
+		(property "Footprint" "copy_ref:R_0402_1005Metric"
 			(at 343.408 62.23 90)
 			(hide yes)
@@
 			)
 		)
-		(property "Footprint" "0805 (2012 Metric)"
+		(property "Footprint" "copy_ref:R_0805_2012Metric"
 			(at 132.08 217.932 90)
 			(hide yes)
@@
 			)
 		)
-		(property "Footprint" "0402 (1005 Metric)"
+		(property "Footprint" "copy_ref:R_0402_1005Metric"
 			(at 363.22 112.268 90)
 			(hide yes)
@@
 			)
 		)
-		(property "Footprint" "1206 (3216 Metric)"
+		(property "Footprint" "copy_ref:R_1206_3216Metric"
 			(at 110.49 55.372 90)
 			(hide yes)
@@
 			)
 		)
-		(property "Footprint" "1206 (3216 Metric)"
+		(property "Footprint" "copy_ref:1206"
 			(at 121.92 55.372 90)
 			(hide yes)
@@
 			)
 		)
-		(property "Footprint" "1206 (3216 Metric)"
+		(property "Footprint" "copy_ref:C_1206_3216Metric"
 			(at 95.5548 66.04 0)
 			(hide yes)
