File: hardware/ntp-server-stm32/ocxo.kicad_sch (KiCad schematic)
At the start: 42 parts, among them U36 OPA320AIDBVT, U37 INA228AQDGSRQ1, U38 AP3441SHE-7B, U39 TPS7A5201QRGRRQ1, Y3 OH300

Commit message: Standardize net/rail names: plain 3V3 style, _N active-low, voltage-format PG/alerts
22 net renames applied across all sheets and verified: removed/added net-name
sets match intent exactly and all node connectivity is preserved (kicad-cli
netlist re-parse).

Co-Authored-By: Claude Opus 4.8 (1M context) <noreply@anthropic.com>
Connections:
- net +3.3V renamed 3V3
- net +5V renamed 5V
Changed lines of the file:
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@@
 			)
 		)
-		(property "Value" "+3.3V"
+		(property "Value" "3V3"
 			(at 195.326 151.13 0)
 			(show_name no)
@@
 			)
 		)
-		(property "Value" "+3.3V"
+		(property "Value" "3V3"
 			(at 248.666 165.1 0)
 			(show_name no)
@@
 			)
 		)
-		(property "Value" "+5V"
+		(property "Value" "5V"
 			(at 180.34 64.77 0)
 			(show_name no)
@@
 			)
 		)
-		(property "Value" "+3.3V"
+		(property "Value" "3V3"
 			(at 292.1 102.87 0)
 			(show_name no)

Commit message: Standardize + complete BOM; write fields back into KiCad symbols
- New sts1000_bom.csv: rebuilt from authoritative Value field (source MPN/footprint/
  description were corrupted by copy-paste). 338 standardized, 78 MPN-from-value,
  50 kept, ~64 flagged (SELECT/REVIEW-HV/SHUNT-REVIEW) each with full spec.
- Resistors -> deterministic Panasonic ERJ-2RKF 0402 1% 1/10W (consolidated 1 part/value).
- Caps -> verified Murata GRM parts where value matches; clean spec + footprint otherwise.
- 1633 symbol field updates (Value/Footprint/Description/MPN/Mfr/Digikey) written to
  .kicad_sch; netlist re-parse confirms connectivity byte-identical.
- Add docs/sts1000_net_naming.md naming reference.

Co-Authored-By: Claude Opus 4.8 (1M context) <noreply@anthropic.com>
Parts:
- C100, C101, C118, C98, C99: footprint 805 -> C_0402_1005Metric; DIGIKEY_PART_NUMBER 490-GRM21BZ71C106KE15LTR-ND -> 490-6328-2-ND; MANUFACTURER (none) -> Murata; MANUFACTURER_PART_NUMBER GRM21BZ71C106KE15L -> GRM155R71C104KA88J
- C102, C103, C104, C105, C111, C112, C113, C114, C115: footprint 805 -> C_0805_2012Metric; MANUFACTURER (none) -> Murata
- C106: value 0.01uF -> 10nF; footprint 805 -> C_0402_1005Metric; DIGIKEY_PART_NUMBER 490-GRM21BZ71C106KE15LTR-ND -> 490-1313-2-ND; MANUFACTURER (none) -> Murata; MANUFACTURER_PART_NUMBER GRM21BZ71C106KE15L -> GRM155R71C103KA01D
- C107: footprint (none) -> C_0402_1005Metric; DIGIKEY_PART_NUMBER (none) -> 490-6328-2-ND; MANUFACTURER (none) -> Murata; MANUFACTURER_PART_NUMBER (none) -> GRM155R71C104KA88J
- C108: footprint 402 -> C_0402_1005Metric; MANUFACTURER (none) -> Murata
- C109, C117: footprint 805 -> C_0805_2012Metric
- C110, C116: footprint 805 -> C_0402_1005Metric; DIGIKEY_PART_NUMBER 490-GRM21BZ71C106KE15LTR-ND -> 490-1313-2-ND; MANUFACTURER (none) -> Murata; MANUFACTURER_PART_NUMBER GRM21BZ71C106KE15L -> GRM155R71C103KA01D
- D10: MANUFACTURER_PART_NUMBER (none) -> BAT54J
- L6: MANUFACTURER (none) -> Eaton - Electronics Division
- R118, R119, R120: footprint 402 -> R_0402_1005Metric; MANUFACTURER (none) -> Panasonic; MANUFACTURER_PART_NUMBER ERJ-2RKF2201X -> ERJ-2RKF1003X
- R121: footprint 402 -> R_0402_1005Metric; MANUFACTURER (none) -> Panasonic; MANUFACTURER_PART_NUMBER ERJ-2RKF2201X -> ERJ-2RKF1005X
- R122: footprint 402 -> R_0402_1005Metric; MANUFACTURER (none) -> Panasonic; MANUFACTURER_PART_NUMBER ERJ-2RKF2201X -> ERJ-2RKF1001X
- R123: footprint 402 -> R_0402_1005Metric; MANUFACTURER (none) -> Panasonic; MANUFACTURER_PART_NUMBER ERJ-2RKF2201X -> ERJ-2RKF22R0X
- R124, R125: footprint 402 -> R_0402_1005Metric; MANUFACTURER (none) -> Panasonic
- R127: footprint 402 -> R_0402_1005Metric; MANUFACTURER (none) -> Panasonic; MANUFACTURER_PART_NUMBER ERJ-2RKF1002X -> ERJ-2RKF1242X
- R128: footprint 402 -> R_0402_1005Metric; MANUFACTURER (none) -> Panasonic; MANUFACTURER_PART_NUMBER ERJ-2RKF2201X -> ERJ-2RKF2401X
- R131: footprint 402 -> R_0402_1005Metric; MANUFACTURER (none) -> Panasonic; MANUFACTURER_PART_NUMBER ERJ-2RKF2201X -> ERJ-2RKF1002X
- U36: MANUFACTURER_PART_NUMBER (none) -> OPA320AIDBVT
- U37: MANUFACTURER_PART_NUMBER (none) -> INA228AQDGSRQ1
- U38: MANUFACTURER (none) -> Diodes Incorporated
- U39: MANUFACTURER_PART_NUMBER (none) -> TPS7A5201QRGRRQ1
