File: hardware/ntp-server-stm32/ocxo.kicad_sch (KiCad schematic)
At the start: 42 parts, among them U36 OPA320AIDBVT, U37 INA228AQDGSRQ1, U38 AP3441SHE-7B, U39 TPS7A5201QRGRRQ1, Y3 OH300

Commit message: Updates
Parts:
- C100, C107, C118: footprint C_0402_1005Metric -> 0402 (1005 Metric); DIELECTRIC (none) -> X7R; DIGIKEY_PART_NUMBER 490-6328-2-ND -> 490-4759-1-ND; MANUFACTURER_PART_NUMBER GRM155R71C104KA88J -> GCM155R71C104KA55D; TOLERANCE (none) -> 10%; VOLTAGE (none) -> 16V
- C101, C98, C99: footprint C_0402_1005Metric -> 1210 (3225 Metric); DIELECTRIC (none) -> C0G/film; DIGIKEY_PART_NUMBER 490-6328-2-ND -> 399-15804-1-ND; MANUFACTURER Murata -> KEMET; MANUFACTURER_PART_NUMBER GRM155R71C104KA88J -> C1210C104J5GACAUTO; TOLERANCE (none) -> 5%; VOLTAGE (none) -> 16V
- C102, C103, C104, C105, C111, C112, C113, C114, C115: footprint C_0805_2012Metric -> 1206 (3216 Metric); DIELECTRIC (none) -> X7R; DIGIKEY_PART_NUMBER 490-GRM21BZ71C106KE15LTR-ND -> 1276-6797-1-ND; MANUFACTURER Murata -> Samsung Electro-Mechanics; MANUFACTURER_PART_NUMBER GRM21BZ71C106KE15L -> CL31B106KOHVPNE; TOLERANCE (none) -> 10%; VOLTAGE (none) -> 16V
- C106, C110, C116: footprint C_0402_1005Metric -> 0402 (1005 Metric); DIELECTRIC (none) -> X7R; DIGIKEY_PART_NUMBER 490-1313-2-ND -> 490-GRT155R71C103KE01JCT-ND; MANUFACTURER Murata -> Murata Electronics; MANUFACTURER_PART_NUMBER GRM155R71C103KA01D -> GRT155R71C103KE01J; TOLERANCE (none) -> 10%; VOLTAGE (none) -> 16V
- C108: footprint C_0402_1005Metric -> 0402 (1005 Metric); DIELECTRIC (none) -> X7R; DIGIKEY_PART_NUMBER 490-6334-2-ND -> 399-17875-1-ND; MANUFACTURER Murata -> KEMET; MANUFACTURER_PART_NUMBER GRM155R71C472KA01D -> C0402C472K4RECAUTO; TOLERANCE (none) -> 10%; VOLTAGE (none) -> 16V
- C109, C117: footprint C_0805_2012Metric -> 0805 (2012 Metric); DIELECTRIC (none) -> X5R; DIGIKEY_PART_NUMBER 490-GRM21BZ71C106KE15LTR-ND -> 490-GRT21BR61C226ME13KCT-ND; MANUFACTURER (none) -> Murata Electronics; MANUFACTURER_PART_NUMBER GRM21BZ71C106KE15L -> GRT21BR61C226ME13K; TOLERANCE (none) -> 10%; VOLTAGE (none) -> 16V
- D10: footprint Diode_SMD:D_SOD-323F -> SOD-323F; DIELECTRIC (none) -> Diode; DIGIKEY_PART_NUMBER (none) -> 1727-BAT54J-QXCT-ND; MANUFACTURER (none) -> Nexperia USA Inc.; MANUFACTURER_PART_NUMBER BAT54J -> BAT54J-QX
- L6: DIELECTRIC (none) -> Inductor; POWER (none) -> 4.15A
- R118, R119, R120: footprint R_0402_1005Metric -> 0402 (1005 Metric); DIELECTRIC (none) -> Thick-film; DIGIKEY_PART_NUMBER P2.20KLTR-ND -> P100KLCT-ND; MANUFACTURER Panasonic -> Panasonic Industry; POWER (none) -> 1/10W; TOLERANCE (none) -> 1%
- R121: footprint R_0402_1005Metric -> 0402 (1005 Metric); DIELECTRIC (none) -> Thick-film; DIGIKEY_PART_NUMBER P2.20KLTR-ND -> 2019-RK73H1ETTP1005FCT-ND; MANUFACTURER Panasonic -> KOA Speer Electronics, Inc.; MANUFACTURER_PART_NUMBER ERJ-2RKF1005X -> RK73H1ETTP1005F; POWER (none) -> 1/10W; TOLERANCE (none) -> 1%
- R122: footprint R_0402_1005Metric -> 0402 (1005 Metric); DIELECTRIC (none) -> Thick-film; DIGIKEY_PART_NUMBER P2.20KLTR-ND -> P1.00KLCT-ND; MANUFACTURER Panasonic -> Panasonic Industry; POWER (none) -> 1/10W; TOLERANCE (none) -> 1%
- R123: footprint R_0402_1005Metric -> 0402 (1005 Metric); DIELECTRIC (none) -> Thick-film; DIGIKEY_PART_NUMBER P2.20KLTR-ND -> P22.0LCT-ND; MANUFACTURER Panasonic -> Panasonic Industry; POWER (none) -> 1/10W; TOLERANCE (none) -> 1%
- R124: footprint R_0402_1005Metric -> 0402 (1005 Metric); DIELECTRIC (none) -> Thick-film; DIGIKEY_PART_NUMBER P10.0KLTR-ND -> P10.0KLCT-ND; MANUFACTURER Panasonic -> Panasonic Industry; POWER (none) -> 1/10W; TOLERANCE (none) -> 1%
- R125: value 6.81k -> 3.57k; footprint R_0402_1005Metric -> 0402 (1005 Metric); DIELECTRIC (none) -> Thick-film; DIGIKEY_PART_NUMBER P6.81KLTR-ND -> P3.57KLCT-ND; MANUFACTURER Panasonic -> Panasonic Industry; MANUFACTURER_PART_NUMBER ERJ-2RKF6811X -> ERJ-2RKF3571X; POWER (none) -> 1/10W; TOLERANCE (none) -> 1%
- R126: footprint 0805 -> 0805Wide 3015 (7638 Metric), 1530; DIELECTRIC (none) -> Metal-strip shunt; DIGIKEY_PART_NUMBER 273-KDV08DR150ETCT-ND -> 273-FCSL76R025DERCT-ND; MANUFACTURER_PART_NUMBER KDV08DR150ET -> FCSL76R025DER; POWER (none) -> 1/4W; TOLERANCE (none) -> 0.5%
- R127: footprint R_0402_1005Metric -> 0402 (1005 Metric); DIELECTRIC (none) -> Thick-film; DIGIKEY_PART_NUMBER P10.0KLTR-ND -> P12.4KLCT-ND; MANUFACTURER Panasonic -> Panasonic Industry; POWER (none) -> 1/10W; TOLERANCE (none) -> 1%
- R128: footprint R_0402_1005Metric -> 0402 (1005 Metric); DIELECTRIC (none) -> Thick-film; DIGIKEY_PART_NUMBER P2.20KLTR-ND -> P12.4KLCT-ND; MANUFACTURER Panasonic -> Panasonic Industry; POWER (none) -> 1/10W; TOLERANCE (none) -> 1%
- R129, R130: footprint 0603 -> 0603 (1608 Metric); DIELECTRIC (none) -> Thin-film; MANUFACTURER TE Connectivity Passive Product -> TE Connectivity; POWER (none) -> 1/10W; TOLERANCE (none) -> 0.1%
- R131: footprint R_0402_1005Metric -> 0402 (1005 Metric); DIELECTRIC (none) -> Thick-film; DIGIKEY_PART_NUMBER P2.20KLTR-ND -> P10.0KLCT-ND; MANUFACTURER Panasonic -> Panasonic Industry; POWER (none) -> 1/10W; TOLERANCE (none) -> 1%
- U36, U37, U39: MANUFACTURER (none) -> Texas Instruments
- U38: MANUFACTURER Diodes Incorporated -> Diodes Inc
- Y3: MANUFACTURER Connor Winfield -> Connor-Winfield
Connections:
- net I2C_SCL: now also U37.5 (SCL); no longer U37.2 (A0), U37.4 (SDA)
- net I2C_SDA: now also U37.2 (A0), U37.4 (SDA); no longer U37.5 (SCL)
Other:
- note added: "3.7V ->"
- note added: "<- 3.7V"
- note added: "PG pulled to VIN When power good"

Commit message: bom updates
Parts:
- Y3: MANUFACTURER Connor-Winfield -> Panasonic Industry
Changed lines of the file:
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@@
 			)
 		)
-		(property "MANUFACTURER" "Connor-Winfield"
+		(property "MANUFACTURER" "Panasonic Industry"
 			(at 162.56 133.35 0)
 			(hide yes)

Commit message: Bom updates
Parts:
- R126: footprint 0805Wide 3015 (7638 Metric), 1530 -> 1206 (3216 Metric); DIGIKEY_PART_NUMBER 273-FCSL76R025DERCT-ND -> WSLC-.025CT-ND; MANUFACTURER Ohmite -> Vishay Dale; MANUFACTURER_PART_NUMBER FCSL76R025DER -> WSL1206R0250FEA
- U36: DIGIKEY_PART_NUMBER (none) -> 296-29510-1-ND
- U37: DIGIKEY_PART_NUMBER (none) -> 296-INA228AQDGSRQ1CT-ND
- U39: DIGIKEY_PART_NUMBER (none) -> 296-50505-1-ND
Changed lines of the file:
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@@
 			)
 		)
-		(property "Datasheet" ""
+		(property "Datasheet" "https://www.ti.com/general/docs/suppproductinfo.tsp?distId=10&gotoUrl=https%3A%2F%2Fwww.ti.com%2Flit%2Fgpn%2Fopa320"
 			(at 101.6 135.89 0)
 			(hide yes)
@@
 			)
 		)
+		(property "DIGIKEY_PART_NUMBER" "296-29510-1-ND"
+			(at 101.6 135.89 0)
+			(hide yes)
+			(show_name no)
+			(do_not_autoplace no)
+			(effects
+				(font
+					(size 1.27 1.27)
+				)
+			)
+		)
 		(pin "5"
 		)
@@
 			)
 		)
-		(property "Datasheet" "https://www.ti.com/lit/gpn/tps7a52-q1"
+		(property "Datasheet" "https://www.ti.com/general/docs/suppproductinfo.tsp?distId=10&gotoUrl=https%3A%2F%2Fwww.ti.com%2Flit%2Fgpn%2Ftps7a52-q1"
 			(at 299.72 125.73 0)
 			(hide yes)
@@
 			)
 		)
+		(property "DIGIKEY_PART_NUMBER" "296-50505-1-ND"
+			(at 299.72 125.73 0)
+			(hide yes)
+			(show_name no)
+			(do_not_autoplace no)
+			(effects
+				(font
+					(size 1.27 1.27)
+				)
+			)
+		)
 		(pin "18"
 		)
@@
 			)
 		)
-		(property "Datasheet" "https://www.ti.com/lit/gpn/ina228-q1"
+		(property "Datasheet" "https://www.ti.com/lit/ds/symlink/ina228-q1.pdf"
 			(at 198.12 160.02 0)
 			(hide yes)
@@
 			)
 		)
-		(property "Description" "Current/power monitor 20-bit I2C"
+		(property "Description" "IC PWR MONITOR 10VSSOP"
 			(at 198.12 160.02 0)
 			(hide yes)
@@
 			)
 		)
+		(property "DIGIKEY_PART_NUMBER" "296-INA228AQDGSRQ1CT-ND"
+			(at 198.12 160.02 0)
+			(hide yes)
+			(show_name no)
+			(do_not_autoplace no)
+			(effects
+				(font
+					(size 1.27 1.27)
+				)
+			)
+		)
 		(pin "2"
 		)
@@
 			)
 		)
-		(property "Footprint" "0805Wide 3015 (7638 Metric), 1530"
+		(property "Footprint" "1206 (3216 Metric)"
 			(at 247.65 120.142 90)
 			(hide yes)
@@
 			)
 		)
-		(property "Datasheet" "https://www.ohmite.com/assets/images/res-fcsl.pdf"
+		(property "Datasheet" "https://www.vishay.com/docs/30100/wsl.pdf"
 			(at 247.65 121.92 0)
 			(hide yes)
@@
 			)
 		)
-		(property "Description" "RES 0.025 OHM 0.5% 3W 3015"
+		(property "Description" "RES 0.025 OHM 1% 1/4W 1206"
 			(at 247.65 121.92 90)
 			(hide yes)
@@
 			)
 		)
-		(property "DIGIKEY_PART_NUMBER" "273-FCSL76R025DERCT-ND"
+		(property "DIGIKEY_PART_NUMBER" "WSLC-.025CT-ND"
 			(at 247.65 121.92 90)
 			(hide yes)
@@
 			)
 		)
-		(property "MANUFACTURER_PART_NUMBER" "FCSL76R025DER"
+		(property "MANUFACTURER_PART_NUMBER" "WSL1206R0250FEA"
 			(at 247.65 121.92 90)
 			(hide yes)
@@
 			)
 		)
-		(property "MANUFACTURER" "Ohmite"
+		(property "MANUFACTURER" "Vishay Dale"
 			(at 247.65 121.92 90)
 			(hide yes)

Commit message: Bom updates
Parts:
- U37: footprint VSSOP10_DGS_TEX -> sts1000:VSSOP10_DGS_TEX
- U39: footprint RGR20_2P05X2P05_TEX -> sts1000:RGR20_2P05X2P05_TEX
Changed lines of the file:
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@@
 			)
 		)
-		(property "Footprint" "RGR20_2P05X2P05_TEX"
+		(property "Footprint" "sts1000:RGR20_2P05X2P05_TEX"
 			(at 299.72 125.73 0)
 			(hide yes)
@@
 			)
 		)
-		(property "Footprint" "VSSOP10_DGS_TEX"
+		(property "Footprint" "sts1000:VSSOP10_DGS_TEX"
 			(at 198.12 160.02 0)
 			(hide yes)

Commit message: Add files via upload
Updated, completed placement
Parts:
- C100, C106, C107, C108, C110, C116, C118: footprint 0402 (1005 Metric) -> copy_ref:C_0402_1005Metric
- C101, C98, C99: footprint 1210 (3225 Metric) -> copy_ref:C_1210_3225Metric
- C102, C103, C104, C105, C111, C112, C113, C114, C115: footprint 1206 (3216 Metric) -> copy_ref:C_1206_3216Metric
- C109, C117: footprint 0805 (2012 Metric) -> copy_ref:C_0805_2012Metric
- D10: footprint SOD-323F -> Diode_SMD:D_SOD-323F
- L6: footprint (none) -> dowload:DR73-2R2-R
- R118, R119, R120, R121, R122, R123, R124, R125, R127, R128, R131: footprint 0402 (1005 Metric) -> copy_ref:R_0402_1005Metric
- R126: footprint 1206 (3216 Metric) -> copy_ref:R_1206_3216Metric
- R129, R130: footprint 0603 (1608 Metric) -> Resistor_SMD:R_0603_1608Metric
- U38: footprint 8-UFDFN (Exposed Pad) -> dowload:AP3441SHE-7B_DIO-M
- Y3: footprint Oscillator:Oscillator_SMD_OCXO_ConnorWinfield_OH300 -> copy_ref:Oscillator_SMD_OCXO_ConnorWinfield_OH300
Changed lines of the file:
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@@
 			)
 		)
-		(property "Footprint" "0402 (1005 Metric)"
+		(property "Footprint" "copy_ref:C_0402_1005Metric"
 			(at 251.1552 80.01 0)
 			(hide yes)
@@
 			)
 		)
-		(property "Footprint" "1206 (3216 Metric)"
+		(property "Footprint" "copy_ref:C_1206_3216Metric"
 			(at 300.6852 80.01 0)
 			(hide yes)
@@
 			)
 		)
-		(property "Footprint" "0402 (1005 Metric)"
+		(property "Footprint" "copy_ref:R_0402_1005Metric"
 			(at 128.27 131.572 90)
 			(hide yes)
@@
 			)
 		)
-		(property "Footprint" "0402 (1005 Metric)"
+		(property "Footprint" "copy_ref:C_0402_1005Metric"
 			(at 249.8852 177.8 0)
 			(hide yes)
@@
 			)
 		)
-		(property "Footprint" "1210 (3225 Metric)"
+		(property "Footprint" "copy_ref:C_1210_3225Metric"
 			(at 133.6548 140.97 0)
 			(hide yes)
@@
 			)
 		)
-		(property "Footprint" "1206 (3216 Metric)"
+		(property "Footprint" "copy_ref:C_1206_3216Metric"
 			(at 190.8048 80.01 0)
 			(hide yes)
@@
 			)
 		)
-		(property "Footprint" "1206 (3216 Metric)"
+		(property "Footprint" "copy_ref:C_1206_3216Metric"
 			(at 347.0148 157.48 0)
 			(hide yes)
@@
 			)
 		)
-		(property "Footprint" "0805 (2012 Metric)"
+		(property "Footprint" "copy_ref:C_0805_2012Metric"
 			(at 259.3848 129.54 0)
 			(hide yes)
@@
 			)
 		)
-		(property "Footprint" "0402 (1005 Metric)"
+		(property "Footprint" "copy_ref:R_0402_1005Metric"
 			(at 193.548 55.88 90)
 			(hide yes)
@@
 			)
 		)
-		(property "Footprint" "0402 (1005 Metric)"
+		(property "Footprint" "copy_ref:R_0402_1005Metric"
 			(at 198.12 53.848 90)
 			(hide yes)
@@
 			)
 		)
-		(property "Footprint" "0402 (1005 Metric)"
+		(property "Footprint" "copy_ref:C_0402_1005Metric"
 			(at 124.7648 107.95 0)
 			(hide yes)
@@
 			)
 		)
-		(property "Footprint" "0805 (2012 Metric)"
+		(property "Footprint" "copy_ref:C_0805_2012Metric"
 			(at 368.6048 152.4 0)
 			(hide yes)
@@
 			)
 		)
-		(property "Footprint" "0402 (1005 Metric)"
+		(property "Footprint" "copy_ref:R_0402_1005Metric"
 			(at 45.212 107.95 90)
 			(hide yes)
@@
 			)
 		)
-		(property "Footprint" "1206 (3216 Metric)"
+		(property "Footprint" "copy_ref:C_1206_3216Metric"
 			(at 202.2348 80.01 0)
 			(hide yes)
@@
 			)
 		)
-		(property "Footprint" "1210 (3225 Metric)"
+		(property "Footprint" "copy_ref:C_1210_3225Metric"
 			(at 54.9148 110.49 0)
 			(hide yes)
@@
 			)
 		)
-		(property "Footprint" "8-UFDFN (Exposed Pad)"
+		(property "Footprint" "dowload:AP3441SHE-7B_DIO-M"
 			(at 223.52 78.74 0)
 			(hide yes)
@@
 			)
 		)
-		(property "Footprint" "0402 (1005 Metric)"
+		(property "Footprint" "copy_ref:R_0402_1005Metric"
 			(at 184.15 131.572 90)
 			(hide yes)
@@
 			)
 		)
-		(property "Footprint" "0402 (1005 Metric)"
+		(property "Footprint" "copy_ref:R_0402_1005Metric"
 			(at 48.26 131.572 90)
 			(hide yes)
@@
 			)
 		)
-		(property "Footprint" "0402 (1005 Metric)"
+		(property "Footprint" "copy_ref:C_0402_1005Metric"
 			(at 270.8148 129.54 0)
 			(hide yes)
@@
 			)
 		)
-		(property "Footprint" "1206 (3216 Metric)"
+		(property "Footprint" "copy_ref:C_1206_3216Metric"
 			(at 179.3748 80.01 0)
 			(hide yes)
@@
 			)
 		)
-		(property "Footprint" "0402 (1005 Metric)"
+		(property "Footprint" "copy_ref:R_0402_1005Metric"
 			(at 293.878 113.03 90)
 			(hide yes)
@@
 			)
 		)
-		(property "Footprint" "0402 (1005 Metric)"
+		(property "Footprint" "copy_ref:R_0402_1005Metric"
 			(at 259.842 76.2 90)
 			(hide yes)
@@
 			)
 		)
-		(property "Footprint" "SOD-323F"
+		(property "Footprint" "Diode_SMD:D_SOD-323F"
 			(at 358.775 133.35 0)
 			(hide yes)
@@
 			)
 		)
-		(property "Footprint" "1206 (3216 Metric)"
+		(property "Footprint" "copy_ref:C_1206_3216Metric"
 			(at 276.5552 80.01 0)
 			(hide yes)
@@
 			)
 		)
-		(property "Footprint" "1206 (3216 Metric)"
+		(property "Footprint" "copy_ref:C_1206_3216Metric"
 			(at 213.6648 133.35 0)
 			(hide yes)
@@
 			)
 		)
-		(property "Footprint" "1206 (3216 Metric)"
+		(property "Footprint" "copy_ref:R_1206_3216Metric"
 			(at 247.65 120.142 90)
 			(hide yes)
@@
 			)
 		)
-		(property "Footprint" ""
+		(property "Footprint" "dowload:DR73-2R2-R"
 			(at 242.57 71.12 0)
 			(hide yes)
@@
 			)
 		)
-		(property "Footprint" "0402 (1005 Metric)"
+		(property "Footprint" "copy_ref:C_0402_1005Metric"
 			(at 228.9048 133.35 0)
 			(hide yes)
@@
 			)
 		)
-		(property "Footprint" "1210 (3225 Metric)"
+		(property "Footprint" "copy_ref:C_1210_3225Metric"
 			(at 53.6448 142.24 0)
 			(hide yes)
@@
 			)
 		)
-		(property "Footprint" "0402 (1005 Metric)"
+		(property "Footprint" "copy_ref:R_0402_1005Metric"
 			(at 39.37 99.822 90)
 			(hide yes)
@@
 			)
 		)
-		(property "Footprint" "0402 (1005 Metric)"
+		(property "Footprint" "copy_ref:C_0402_1005Metric"
 			(at 358.4448 157.48 0)
 			(hide yes)
@@
 			)
 		)
-		(property "Footprint" "0402 (1005 Metric)"
+		(property "Footprint" "copy_ref:R_0402_1005Metric"
 			(at 259.842 86.36 90)
 			(hide yes)
@@
 			)
 		)
-		(property "Footprint" "1206 (3216 Metric)"
+		(property "Footprint" "copy_ref:C_1206_3216Metric"
 			(at 312.1152 80.01 0)
 			(hide yes)
@@
 			)
 		)
-		(property "Footprint" "0402 (1005 Metric)"
+		(property "Footprint" "copy_ref:C_0402_1005Metric"
 			(at 380.0348 152.4 0)
 			(hide yes)
@@
 			)
 		)
-		(property "Footprint" "0603 (1608 Metric)"
+		(property "Footprint" "Resistor_SMD:R_0603_1608Metric"
 			(at 284.988 125.73 90)
 			(hide yes)
@@
 			)
 		)
-		(property "Footprint" "0402 (1005 Metric)"
+		(property "Footprint" "copy_ref:R_0402_1005Metric"
 			(at 63.5 99.822 90)
 			(hide yes)
@@
 			)
 		)
-		(property "Footprint" "1206 (3216 Metric)"
+		(property "Footprint" "copy_ref:C_1206_3216Metric"
 			(at 287.9852 80.01 0)
 			(hide yes)
@@
 			)
 		)
-		(property "Footprint" "0603 (1608 Metric)"
+		(property "Footprint" "Resistor_SMD:R_0603_1608Metric"
 			(at 284.988 135.89 90)
 			(hide yes)
@@
 			)
 		)
-		(property "Footprint" "Oscillator:Oscillator_SMD_OCXO_ConnorWinfield_OH300"
+		(property "Footprint" "copy_ref:Oscillator_SMD_OCXO_ConnorWinfield_OH300"
 			(at 162.56 142.24 0)
 			(hide yes)
