File: hardware/ntp-server-stm32/rb-io.kicad_sch (KiCad schematic)
At the start: 33 parts, among them K1 G6K-2F-Y DC3, Q21 BC847W, U46 SN65C3221EPWR, U47 PESD15VL2BT, U48 APC-817C1

Commit message: Standardize net/rail names: plain 3V3 style, _N active-low, voltage-format PG/alerts
22 net renames applied across all sheets and verified: removed/added net-name
sets match intent exactly and all node connectivity is preserved (kicad-cli
netlist re-parse).

Co-Authored-By: Claude Opus 4.8 (1M context) <noreply@anthropic.com>
Connections:
- net +3.3V renamed 3V3
Changed lines of the file:
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@@
 			)
 		)
-		(property "Value" "+3.3V"
+		(property "Value" "3V3"
 			(at 184.15 77.47 0)
 			(show_name no)
@@
 			)
 		)
-		(property "Value" "+3.3V"
+		(property "Value" "3V3"
 			(at 41.91 48.26 0)
 			(show_name no)
@@
 			)
 		)
-		(property "Value" "+3.3V"
+		(property "Value" "3V3"
 			(at 66.04 93.98 0)
 			(show_name no)
@@
 			)
 		)
-		(property "Value" "+3.3V"
+		(property "Value" "3V3"
 			(at 116.84 72.39 0)
 			(show_name no)
@@
 			)
 		)
-		(property "Value" "+3.3V"
+		(property "Value" "3V3"
 			(at 361.95 26.67 0)
 			(show_name no)

Commit message: Standardize + complete BOM; write fields back into KiCad symbols
- New sts1000_bom.csv: rebuilt from authoritative Value field (source MPN/footprint/
  description were corrupted by copy-paste). 338 standardized, 78 MPN-from-value,
  50 kept, ~64 flagged (SELECT/REVIEW-HV/SHUNT-REVIEW) each with full spec.
- Resistors -> deterministic Panasonic ERJ-2RKF 0402 1% 1/10W (consolidated 1 part/value).
- Caps -> verified Murata GRM parts where value matches; clean spec + footprint otherwise.
- 1633 symbol field updates (Value/Footprint/Description/MPN/Mfr/Digikey) written to
  .kicad_sch; netlist re-parse confirms connectivity byte-identical.
- Add docs/sts1000_net_naming.md naming reference.

Co-Authored-By: Claude Opus 4.8 (1M context) <noreply@anthropic.com>
Parts:
- C139, C140, C144, C145: footprint 402 -> C_0402_1005Metric; DIGIKEY_PART_NUMBER 490-3229-2-ND -> 490-6328-2-ND; MANUFACTURER (none) -> Murata; MANUFACTURER_PART_NUMBER GRM1555C1H151JA01D -> GRM155R71C104KA88J
- C141, C142, C146, C147: footprint 402 -> C_0402_1005Metric
- C143: footprint 402 -> C_0603_1608Metric
- C148: footprint 402 -> C_0402_1005Metric; DIGIKEY_PART_NUMBER 490-3229-2-ND -> 490-1313-2-ND; MANUFACTURER (none) -> Murata; MANUFACTURER_PART_NUMBER GRM1555C1H151JA01D -> GRM155R71C103KA01D
- D12: MANUFACTURER_PART_NUMBER (none) -> BAT54S
- D13, D14: MANUFACTURER (none) -> WÃ¼rth Elektronik
- D15, D17: MANUFACTURER_PART_NUMBER (none) -> BAT54J
- K1: MANUFACTURER_PART_NUMBER (none) -> G6K-2F-Y DC3
- L8, L9: MANUFACTURER (none) -> Fair-Rite Products Corp.
- Q21: MANUFACTURER_PART_NUMBER (none) -> BC847W
- R164: footprint (none) -> R_0402_1005Metric; MANUFACTURER (none) -> Panasonic; MANUFACTURER_PART_NUMBER (none) -> ERJ-2RKF1003X
- R165, R166: footprint 402 -> R_0402_1005Metric; MANUFACTURER (none) -> Panasonic
- R167: footprint (none) -> R_0402_1005Metric; MANUFACTURER (none) -> Panasonic; MANUFACTURER_PART_NUMBER (none) -> ERJ-2RKF2200X
- R168, R169: footprint (none) -> R_0402_1005Metric; MANUFACTURER (none) -> Panasonic; MANUFACTURER_PART_NUMBER (none) -> ERJ-2RKF1002X
- R170, R172: footprint (none) -> R_0402_1005Metric; MANUFACTURER (none) -> Panasonic; MANUFACTURER_PART_NUMBER (none) -> ERJ-2RKF4700X
- R171: footprint (none) -> R_0402_1005Metric; MANUFACTURER (none) -> Panasonic; MANUFACTURER_PART_NUMBER (none) -> ERJ-2RKF4701X
- R173: footprint (none) -> R_0402_1005Metric; MANUFACTURER (none) -> Panasonic; MANUFACTURER_PART_NUMBER (none) -> ERJ-2RKF2202X
- U46: MANUFACTURER_PART_NUMBER (none) -> SN65C3221EPWR
- U47: MANUFACTURER (none) -> Nexperia USA Inc.
