File: hardware/ntp-server-stm32/rb-io.kicad_sch (KiCad schematic)
At the start: 33 parts, among them K1 G6K-2F-Y DC3, Q21 BC847W, U46 SN65C3221EPWR, U47 PESD15VL2BT, U48 APC-817C1

Commit message: Updates
Parts:
- C139, C140, C144, C145: footprint C_0402_1005Metric -> 0402 (1005 Metric); DIELECTRIC (none) -> X7R; DIGIKEY_PART_NUMBER 490-6328-2-ND -> 490-4759-1-ND; MANUFACTURER_PART_NUMBER GRM155R71C104KA88J -> GCM155R71C104KA55D; TOLERANCE (none) -> 10%; VOLTAGE (none) -> 16V
- C141, C142, C146, C147: footprint C_0402_1005Metric -> 0402 (1005 Metric); DIELECTRIC (none) -> C0G; DIGIKEY_PART_NUMBER 490-3229-2-ND -> 490-16445-1-ND; MANUFACTURER (none) -> Murata Electronics; MANUFACTURER_PART_NUMBER GRM1555C1H151JA01D -> GCM1555C1H470FA16D; TOLERANCE (none) -> 5%; VOLTAGE (none) -> 50V
- C143: footprint C_0603_1608Metric -> 0603 (1608 Metric); DIELECTRIC (none) -> X7R; DIGIKEY_PART_NUMBER 490-3229-2-ND -> 399-17704-1-ND; MANUFACTURER (none) -> KEMET; MANUFACTURER_PART_NUMBER GRM1555C1H151JA01D -> C0603C105K4RACAUTO; TOLERANCE (none) -> 10%; VOLTAGE (none) -> 16V
- C148: footprint C_0402_1005Metric -> 0402 (1005 Metric); DIELECTRIC (none) -> X7R; DIGIKEY_PART_NUMBER 490-1313-2-ND -> 490-GRT155R71C103KE01JCT-ND; MANUFACTURER Murata -> Murata Electronics; MANUFACTURER_PART_NUMBER GRM155R71C103KA01D -> GRT155R71C103KE01J; TOLERANCE (none) -> 10%; VOLTAGE (none) -> 16V
- D12: footprint Package_TO_SOT_SMD:SOT-23 -> SOT-23-3 (TO-236); DIELECTRIC (none) -> Diode; DIGIKEY_PART_NUMBER (none) -> 4878-BAT54SCT-ND; MANUFACTURER (none) -> Diotec Semiconductor
- D13, D14: DIELECTRIC (none) -> Diode; MANUFACTURER WÃ¼rth Elektronik -> Würth Elektronik
- D15, D17: footprint Diode_SMD:D_SOD-323F -> SOD-323F; DIELECTRIC (none) -> Diode; DIGIKEY_PART_NUMBER (none) -> 1727-BAT54J-QXCT-ND; MANUFACTURER (none) -> Nexperia USA Inc.; MANUFACTURER_PART_NUMBER BAT54J -> BAT54J-QX
- D16: footprint (none) -> SOT-23-3 (TO-236); DIELECTRIC (none) -> Diode; DIGIKEY_PART_NUMBER (none) -> BZX84C3V3LT1GOSCT-ND; MANUFACTURER (none) -> onsemi; MANUFACTURER_PART_NUMBER (none) -> BZX84C3V3LT1G
- K1: DIGIKEY_PART_NUMBER (none) -> 39-G6K-2F-YDC3-ND; MANUFACTURER (none) -> Aratas America LLC
- L8, L9: footprint (none) -> 0805 (2012 Metric); DIELECTRIC (none) -> Ferrite bead; POWER (none) -> 3A
- Q21: footprint Package_TO_SOT_SMD:SOT-323_SC-70 -> SOT-323; DIELECTRIC (none) -> Transistor; DIGIKEY_PART_NUMBER (none) -> 1727-BC847W,135CT-ND; MANUFACTURER (none) -> Nexperia USA Inc.; MANUFACTURER_PART_NUMBER BC847W -> BC847W,135
- R164: footprint R_0402_1005Metric -> 0402 (1005 Metric); DIELECTRIC (none) -> Thick-film; DIGIKEY_PART_NUMBER (none) -> P100KLCT-ND; MANUFACTURER Panasonic -> Panasonic Industry; POWER (none) -> 1/10W; TOLERANCE (none) -> 1%
- R165, R166, R170, R172, R173: DIELECTRIC (none) -> Thick-film; POWER (none) -> 1/10W; TOLERANCE (none) -> 1%
- R167: footprint R_0402_1005Metric -> 0402 (1005 Metric); DIELECTRIC (none) -> Thick-film; DIGIKEY_PART_NUMBER (none) -> P220LCT-ND; MANUFACTURER Panasonic -> Panasonic Industry; POWER (none) -> 1/10W; TOLERANCE (none) -> 1%
- R168, R169: footprint R_0402_1005Metric -> 0402 (1005 Metric); DIELECTRIC (none) -> Thick-film; DIGIKEY_PART_NUMBER (none) -> P10.0KLCT-ND; MANUFACTURER Panasonic -> Panasonic Industry; POWER (none) -> 1/10W; TOLERANCE (none) -> 1%
- R171: footprint R_0402_1005Metric -> 0402 (1005 Metric); DIELECTRIC (none) -> Thick-film; DIGIKEY_PART_NUMBER (none) -> P4.70KLCT-ND; MANUFACTURER Panasonic -> Panasonic Industry; POWER (none) -> 1/10W; TOLERANCE (none) -> 1%
- U46: MANUFACTURER (none) -> Texas Instruments
- U47: MANUFACTURER Nexperia USA Inc. -> Nexperia
- U48: MANUFACTURER American Bright Optoelectronics Corporation -> American Bright
Other:
- moved on the sheet: C139, C140, C143, C144, C145, D12, D15, K1, Q21, R164, R167, R168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

Commit message: Bom updates
Parts:
- R165, R166: footprint R_0402_1005Metric -> 0402 (1005 Metric); DIGIKEY_PART_NUMBER P51.0LTR-ND -> P51.0LCT-ND; MANUFACTURER Panasonic -> Panasonic Industry
- R170, R172: footprint R_0402_1005Metric -> 0402 (1005 Metric); DIGIKEY_PART_NUMBER (none) -> P470LCT-ND; MANUFACTURER Panasonic -> Panasonic Industry
- R173: footprint R_0402_1005Metric -> 0402 (1005 Metric); DIGIKEY_PART_NUMBER (none) -> P22.0KLCT-ND; MANUFACTURER Panasonic -> Panasonic Industry
- U46: DIGIKEY_PART_NUMBER (none) -> 296-20992-1-ND
- U47: DIGIKEY_PART_NUMBER 1727-3813-2-ND -> 1727-3813-1-ND
Changed lines of the file:
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@@
 			)
 		)
-		(property "Datasheet" ""
+		(property "Datasheet" "https://www.ti.com/lit/ds/symlink/sn65c3221e.pdf"
 			(at 127 144.78 0)
 			(hide yes)
@@
 			)
 		)
+		(property "DIGIKEY_PART_NUMBER" "296-20992-1-ND"
+			(at 127 144.78 0)
+			(hide yes)
+			(show_name no)
+			(do_not_autoplace no)
+			(effects
+				(font
+					(size 1.27 1.27)
+				)
+			)
+		)
 		(pin "1"
 		)
@@
 			)
 		)
-		(property "DIGIKEY_PART_NUMBER" "1727-3813-2-ND"
+		(property "DIGIKEY_PART_NUMBER" "1727-3813-1-ND"
 			(at 124.46 40.64 90)
 			(hide yes)
@@
 			)
 		)
-		(property "Footprint" "R_0402_1005Metric"
+		(property "Footprint" "0402 (1005 Metric)"
 			(at 363.728 38.1 90)
 			(hide yes)
@@
 			)
 		)
-		(property "Datasheet" ""
+		(property "Datasheet" "https://industrial.panasonic.com/cdbs/www-data/pdf/RDA0000/AOA0000C304.pdf"
 			(at 361.95 38.1 0)
 			(hide yes)
@@
 			)
 		)
-		(property "Description" "RES 22k 1% 1/10W 0402"
+		(property "Description" "RES SMD 22K OHM 1% 1/10W 0402"
 			(at 361.95 38.1 0)
 			(hide yes)
@@
 			)
 		)
-		(property "MANUFACTURER" "Panasonic"
+		(property "MANUFACTURER" "Panasonic Industry"
 			(at 0 0 0)
 			(hide yes)
@@
 			)
 		)
+		(property "DIGIKEY_PART_NUMBER" "P22.0KLCT-ND"
+			(at 361.95 38.1 0)
+			(hide yes)
+			(show_name no)
+			(do_not_autoplace no)
+			(effects
+				(font
+					(size 1.27 1.27)
+				)
+			)
+		)
 		(pin "1"
 		)
@@
 			)
 		)
-		(property "Footprint" "R_0402_1005Metric"
+		(property "Footprint" "0402 (1005 Metric)"
 			(at 321.31 47.498 90)
 			(hide yes)
@@
 			)
 		)
-		(property "Datasheet" ""
+		(property "Datasheet" "https://industrial.panasonic.com/cdbs/www-data/pdf/RDA0000/AOA0000C304.pdf"
 			(at 321.31 45.72 0)
 			(hide yes)
@@
 			)
 		)
-		(property "Description" "RES 470 1% 1/10W 0402"
+		(property "Description" "RES SMD 470 OHM 1% 1/10W 0402"
 			(at 321.31 45.72 0)
 			(hide yes)
@@
 			)
 		)
-		(property "MANUFACTURER" "Panasonic"
+		(property "MANUFACTURER" "Panasonic Industry"
 			(at 0 0 0)
 			(hide yes)
@@
 			)
 		)
+		(property "DIGIKEY_PART_NUMBER" "P470LCT-ND"
+			(at 321.31 45.72 90)
+			(hide yes)
+			(show_name no)
+			(do_not_autoplace no)
+			(effects
+				(font
+					(size 1.27 1.27)
+				)
+			)
+		)
 		(pin "1"
 		)
@@
 			)
 		)
-		(property "Footprint" "R_0402_1005Metric"
+		(property "Footprint" "0402 (1005 Metric)"
 			(at 331.978 140.97 90)
 			(hide yes)
@@
 			)
 		)
-		(property "Datasheet" ""
+		(property "Datasheet" "https://industrial.panasonic.com/cdbs/www-data/pdf/RDA0000/AOA0000C304.pdf"
 			(at 330.2 140.97 0)
 			(hide yes)
@@
 			)
 		)
-		(property "Description" "RES 470 1% 1/10W 0402"
+		(property "Description" "RES SMD 470 OHM 1% 1/10W 0402"
 			(at 330.2 140.97 0)
 			(hide yes)
@@
 			)
 		)
-		(property "MANUFACTURER" "Panasonic"
+		(property "MANUFACTURER" "Panasonic Industry"
 			(at 95.25 41.91 0)
 			(hide yes)
@@
 			)
 		)
+		(property "DIGIKEY_PART_NUMBER" "P470LCT-ND"
+			(at 330.2 140.97 0)
+			(hide yes)
+			(show_name no)
+			(do_not_autoplace no)
+			(effects
+				(font
+					(size 1.27 1.27)
+				)
+			)
+		)
 		(pin "1"
 		)
@@
 			)
 		)
-		(property "Footprint" "R_0402_1005Metric"
+		(property "Footprint" "0402 (1005 Metric)"
 			(at 142.24 28.702 90)
 			(hide yes)
@@
 			)
 		)
-		(property "Description" "RES 51 1% 1/10W 0402"
+		(property "Description" "RES SMD 51 OHM 1% 1/10W 0402"
 			(at 142.24 30.48 90)
 			(hide yes)
@@
 			)
 		)
-		(property "MANUFACTURER" "Panasonic"
+		(property "MANUFACTURER" "Panasonic Industry"
 			(at 0 0 0)
 			(hide yes)
@@
 			)
 		)
-		(property "DIGIKEY_PART_NUMBER" "P51.0LTR-ND"
+		(property "DIGIKEY_PART_NUMBER" "P51.0LCT-ND"
 			(at 142.24 30.48 90)
 			(hide yes)
@@
 			)
 		)
-		(property "Footprint" "R_0402_1005Metric"
+		(property "Footprint" "0402 (1005 Metric)"
 			(at 142.24 27.178 90)
 			(hide yes)
@@
 			)
 		)
-		(property "Description" "RES 51 1% 1/10W 0402"
+		(property "Description" "RES SMD 51 OHM 1% 1/10W 0402"
 			(at 142.24 25.4 90)
 			(hide yes)
@@
 			)
 		)
-		(property "MANUFACTURER" "Panasonic"
+		(property "MANUFACTURER" "Panasonic Industry"
 			(at 0 0 0)
 			(hide yes)
@@
 			)
 		)
-		(property "DIGIKEY_PART_NUMBER" "P51.0LTR-ND"
+		(property "DIGIKEY_PART_NUMBER" "P51.0LCT-ND"
 			(at 142.24 25.4 90)
 			(hide yes)

Commit message: Add files via upload
Updated, completed placement
Parts:
- C139, C140, C141, C142, C144, C145, C146, C147, C148: footprint 0402 (1005 Metric) -> copy_ref:C_0402_1005Metric
- C143: footprint 0603 (1608 Metric) -> copy_ref:C_0603_1608Metric
- D12, D16: footprint SOT-23-3 (TO-236) -> copy_ref:SOT-23-3
- D13, D14: footprint DO-214AC -> dowload:DO-214AC
- D15, D17: footprint SOD-323F -> Diode_SMD:D_SOD-323F
- K1: footprint (none) -> dowload:G6K-2F-Y DC3
- L8, L9: footprint 0805 (2012 Metric) -> copy_ref:L_0805_2012Metric
- Q21: footprint SOT-323 -> Package_TO_SOT_SMD:SOT-323_SC-70
- R164, R165, R166, R167, R168, R169, R170, R171, R172, R173: footprint 0402 (1005 Metric) -> copy_ref:R_0402_1005Metric
- U47: footprint TO-236AB -> Package_TO_SOT_SMD:TSOT-23
- U48: footprint 4-SMD -> dowload:APC817C1SL
Changed lines of the file:
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@@
 			)
 		)
-		(property "Footprint" "SOT-23-3 (TO-236)"
+		(property "Footprint" "copy_ref:SOT-23-3"
 			(at 291.465 191.135 0)
 			(hide yes)
@@
 			)
 		)
-		(property "Footprint" ""
+		(property "Footprint" "dowload:G6K-2F-Y DC3"
 			(at 289.56 154.94 0)
 			(hide yes)
@@
 			)
 		)
-		(property "Footprint" "SOD-323F"
+		(property "Footprint" "Diode_SMD:D_SOD-323F"
 			(at 289.56 135.255 0)
 			(hide yes)
@@
 			)
 		)
-		(property "Footprint" "0402 (1005 Metric)"
+		(property "Footprint" "copy_ref:C_0402_1005Metric"
 			(at 110.1852 40.64 0)
 			(hide yes)
@@
 			)
 		)
-		(property "Footprint" "0402 (1005 Metric)"
+		(property "Footprint" "copy_ref:C_0402_1005Metric"
 			(at 369.2652 53.34 0)
 			(hide yes)
@@
 			)
 		)
-		(property "Footprint" "TO-236AB"
+		(property "Footprint" "Package_TO_SOT_SMD:TSOT-23"
 			(at 124.46 40.64 0)
 			(hide yes)
@@
 			)
 		)
-		(property "Footprint" "0402 (1005 Metric)"
+		(property "Footprint" "copy_ref:R_0402_1005Metric"
 			(at 275.59 171.958 90)
 			(hide yes)
@@
 			)
 		)
-		(property "Footprint" "0402 (1005 Metric)"
+		(property "Footprint" "copy_ref:R_0402_1005Metric"
 			(at 323.342 142.24 90)
 			(hide yes)
@@
 			)
 		)
-		(property "Footprint" "0402 (1005 Metric)"
+		(property "Footprint" "copy_ref:R_0402_1005Metric"
 			(at 274.32 159.258 90)
 			(hide yes)
@@
 			)
 		)
-		(property "Footprint" "0603 (1608 Metric)"
+		(property "Footprint" "copy_ref:C_0603_1608Metric"
 			(at 154.6352 118.11 0)
 			(hide yes)
@@
 			)
 		)
-		(property "Footprint" "SOD-323F"
+		(property "Footprint" "Diode_SMD:D_SOD-323F"
 			(at 324.485 49.53 0)
 			(hide yes)
@@
 			)
 		)
-		(property "Footprint" "SOT-323"
+		(property "Footprint" "Package_TO_SOT_SMD:SOT-323_SC-70"
 			(at 311.15 139.065 0)
 			(hide yes)
@@
 			)
 		)
-		(property "Footprint" "4-SMD"
+		(property "Footprint" "dowload:APC817C1SL"
 			(at 345.44 50.8 0)
 			(hide yes)
@@
 			)
 		)
-		(property "Footprint" "0402 (1005 Metric)"
+		(property "Footprint" "copy_ref:C_0402_1005Metric"
 			(at 167.3352 118.11 0)
 			(hide yes)
@@
 			)
 		)
-		(property "Footprint" "0402 (1005 Metric)"
+		(property "Footprint" "copy_ref:R_0402_1005Metric"
 			(at 363.728 38.1 90)
 			(hide yes)
@@
 			)
 		)
-		(property "Footprint" "0402 (1005 Metric)"
+		(property "Footprint" "copy_ref:C_0402_1005Metric"
 			(at 164.7952 50.8 0)
 			(hide yes)
@@
 			)
 		)
-		(property "Footprint" "0805 (2012 Metric)"
+		(property "Footprint" "copy_ref:L_0805_2012Metric"
 			(at 154.94 25.4 0)
 			(hide yes)
@@
 			)
 		)
-		(property "Footprint" "0402 (1005 Metric)"
+		(property "Footprint" "copy_ref:R_0402_1005Metric"
 			(at 321.31 47.498 90)
 			(hide yes)
@@
 			)
 		)
-		(property "Footprint" "0402 (1005 Metric)"
+		(property "Footprint" "copy_ref:C_0402_1005Metric"
 			(at 87.3252 161.29 0)
 			(hide yes)
@@
 			)
 		)
-		(property "Footprint" "0402 (1005 Metric)"
+		(property "Footprint" "copy_ref:C_0402_1005Metric"
 			(at 194.0052 50.8 0)
 			(hide yes)
@@
 			)
 		)
-		(property "Footprint" "0402 (1005 Metric)"
+		(property "Footprint" "copy_ref:C_0402_1005Metric"
 			(at 77.7748 161.29 0)
 			(hide yes)
@@
 			)
 		)
-		(property "Footprint" "0402 (1005 Metric)"
+		(property "Footprint" "copy_ref:R_0402_1005Metric"
 			(at 331.978 140.97 90)
 			(hide yes)
@@
 			)
 		)
-		(property "Footprint" "0805 (2012 Metric)"
+		(property "Footprint" "copy_ref:L_0805_2012Metric"
 			(at 154.94 30.48 0)
 			(hide yes)
@@
 			)
 		)
-		(property "Footprint" "0402 (1005 Metric)"
+		(property "Footprint" "copy_ref:R_0402_1005Metric"
 			(at 142.24 28.702 90)
 			(hide yes)
@@
 			)
 		)
-		(property "Footprint" "SOT-23-3 (TO-236)"
+		(property "Footprint" "copy_ref:SOT-23-3"
 			(at 311.15 50.8 0)
 			(hide yes)
@@
 			)
 		)
-		(property "Footprint" "0402 (1005 Metric)"
+		(property "Footprint" "copy_ref:R_0402_1005Metric"
 			(at 76.708 139.7 90)
 			(hide yes)
@@
 			)
 		)
-		(property "Footprint" "0402 (1005 Metric)"
+		(property "Footprint" "copy_ref:R_0402_1005Metric"
 			(at 304.8 47.498 90)
 			(hide yes)
@@
 			)
 		)
-		(property "Footprint" "DO-214AC"
+		(property "Footprint" "dowload:DO-214AC"
 			(at 153.67 46.99 0)
 			(hide yes)
@@
 			)
 		)
-		(property "Footprint" "0402 (1005 Metric)"
+		(property "Footprint" "copy_ref:C_0402_1005Metric"
 			(at 96.2152 40.64 0)
 			(hide yes)
@@
 			)
 		)
-		(property "Footprint" "DO-214AC"
+		(property "Footprint" "dowload:DO-214AC"
 			(at 182.88 46.99 0)
 			(hide yes)
@@
 			)
 		)
-		(property "Footprint" "0402 (1005 Metric)"
+		(property "Footprint" "copy_ref:R_0402_1005Metric"
 			(at 142.24 27.178 90)
 			(hide yes)
@@
 			)
 		)
-		(property "Footprint" "0402 (1005 Metric)"
+		(property "Footprint" "copy_ref:C_0402_1005Metric"
 			(at 154.6352 167.64 0)
 			(hide yes)
