File: hardware/ntp-server-stm32/rb.kicad_sch (KiCad schematic)
At the start: 67 parts, among them Q15 BC847W, Q16 BC847W, Q17 BC857W, Q18 BC847W, Q19 BC847W, Q20 BC847W, U40 MIC28516T-E/PHA, U41 LMV393, U42 OPA320AIDBVT, U43 MCP41U83T-503E/ST, U44 INA228AQDGSRQ1, U45 MCP1502T-40E/CHY

Commit message: Standardize net/rail names: plain 3V3 style, _N active-low, voltage-format PG/alerts
22 net renames applied across all sheets and verified: removed/added net-name
sets match intent exactly and all node connectivity is preserved (kicad-cli
netlist re-parse).

Co-Authored-By: Claude Opus 4.8 (1M context) <noreply@anthropic.com>
Connections:
- net +3.3V renamed 3V3
- net +5V renamed 5V
Changed lines of the file:
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@@
 			)
 		)
-		(property "Value" "+5V"
+		(property "Value" "5V"
 			(at 212.09 213.36 0)
 			(show_name no)
@@
 			)
 		)
-		(property "Value" "+5V"
+		(property "Value" "5V"
 			(at 71.12 82.55 0)
 			(show_name no)
@@
 			)
 		)
-		(property "Value" "+5V"
+		(property "Value" "5V"
 			(at 186.69 129.54 0)
 			(show_name no)
@@
 			)
 		)
-		(property "Value" "+3.3V"
+		(property "Value" "3V3"
 			(at 104.14 16.51 0)
 			(show_name no)
@@
 			)
 		)
-		(property "Value" "+3.3V"
+		(property "Value" "3V3"
 			(at 149.86 82.55 0)
 			(show_name no)
@@
 			)
 		)
-		(property "Value" "+3.3V"
+		(property "Value" "3V3"
 			(at 66.04 134.62 0)
 			(show_name no)
@@
 			)
 		)
-		(property "Value" "+5V"
+		(property "Value" "5V"
 			(at 173.99 120.65 0)
 			(show_name no)
@@
 			)
 		)
-		(property "Value" "+5V"
+		(property "Value" "5V"
 			(at 93.98 187.96 0)
 			(show_name no)
@@
 			)
 		)
-		(property "Value" "+5V"
+		(property "Value" "5V"
 			(at 234.95 215.9 0)
 			(show_name no)
@@
 			)
 		)
-		(property "Value" "+3.3V"
+		(property "Value" "3V3"
 			(at 201.93 95.25 0)
 			(show_name no)
@@
 			)
 		)
-		(property "Value" "+5V"
+		(property "Value" "5V"
 			(at 153.67 199.39 0)
 			(show_name no)
@@
 			)
 		)
-		(property "Value" "+5V"
+		(property "Value" "5V"
 			(at 133.35 196.85 0)
 			(show_name no)
@@
 			)
 		)
-		(property "Value" "+5V"
+		(property "Value" "5V"
 			(at 196.85 134.62 0)
 			(show_name no)
@@
 			)
 		)
-		(property "Value" "+3.3V"
+		(property "Value" "3V3"
 			(at 46.99 140.97 0)
 			(show_name no)

Commit message: Standardize + complete BOM; write fields back into KiCad symbols
- New sts1000_bom.csv: rebuilt from authoritative Value field (source MPN/footprint/
  description were corrupted by copy-paste). 338 standardized, 78 MPN-from-value,
  50 kept, ~64 flagged (SELECT/REVIEW-HV/SHUNT-REVIEW) each with full spec.
- Resistors -> deterministic Panasonic ERJ-2RKF 0402 1% 1/10W (consolidated 1 part/value).
- Caps -> verified Murata GRM parts where value matches; clean spec + footprint otherwise.
- 1633 symbol field updates (Value/Footprint/Description/MPN/Mfr/Digikey) written to
  .kicad_sch; netlist re-parse confirms connectivity byte-identical.
- Add docs/sts1000_net_naming.md naming reference.

Co-Authored-By: Claude Opus 4.8 (1M context) <noreply@anthropic.com>
Parts:
- C119, C123, C124: footprint 402 -> C_0402_1005Metric; MANUFACTURER (none) -> Murata
- C120, C121, C122, C131, C132: footprint (none) -> C_0402_1005Metric; DIGIKEY_PART_NUMBER (none) -> 490-6328-2-ND; MANUFACTURER (none) -> Murata; MANUFACTURER_PART_NUMBER (none) -> GRM155R71C104KA88J
- C125: footprint 402 -> C_0402_1005Metric
- C126, C127, C128: footprint 1210 -> C_1210_3225Metric; MANUFACTURER (none) -> Murata
- C129: footprint (none) -> C_0603_1608Metric; DIGIKEY_PART_NUMBER (none) -> 490-GRM188Z71C225KE43DTR-ND; MANUFACTURER (none) -> Murata; MANUFACTURER_PART_NUMBER (none) -> GRM188Z71C225KE43D
- C130: footprint (none) -> C_0603_1608Metric
- C133, C134, C136: value 2.2uF 100V -> 2.2uF; footprint 805 -> C_0805_2012Metric; MANUFACTURER (none) -> Murata
- C135: value 1uF 100V -> 1uF; footprint 603 -> C_0603_1608Metric; MANUFACTURER (none) -> Murata
- C137: footprint 805 -> C_0805_2012Metric; MANUFACTURER (none) -> Murata
- C138: footprint 603 -> C_0603_1608Metric; MANUFACTURER (none) -> Murata
- D11: MANUFACTURER_PART_NUMBER (none) -> BAS16W
- L7: MANUFACTURER (none) -> Bourns Inc.
- Q15, Q16, Q18, Q19, Q20: MANUFACTURER_PART_NUMBER (none) -> BC847W
- Q17: MANUFACTURER_PART_NUMBER (none) -> BC857W
- R132, R133, R140: footprint 402 -> R_0402_1005Metric; MANUFACTURER (none) -> Panasonic
- R134: footprint 402 -> R_0402_1005Metric; MANUFACTURER (none) -> Panasonic; MANUFACTURER_PART_NUMBER ERJ-2RKF2051X -> ERJ-2RKF4121X
- R135, R137, R139, R145, R150, R155, R157, R158, R160, R161: footprint (none) -> R_0402_1005Metric; MANUFACTURER (none) -> Panasonic; MANUFACTURER_PART_NUMBER (none) -> ERJ-2RKF1002X
- R136: footprint (none) -> R_0402_1005Metric; MANUFACTURER (none) -> Panasonic; MANUFACTURER_PART_NUMBER (none) -> ERJ-2RKF1052X
- R138: footprint (none) -> R_0402_1005Metric; MANUFACTURER (none) -> Panasonic; MANUFACTURER_PART_NUMBER (none) -> ERJ-2RKF1203X
- R141: footprint (none) -> R_0402_1005Metric; MANUFACTURER (none) -> Panasonic; MANUFACTURER_PART_NUMBER (none) -> ERJ-2RKF1004X
- R142: footprint (none) -> R_0402_1005Metric; MANUFACTURER (none) -> Panasonic; MANUFACTURER_PART_NUMBER (none) -> ERJ-2RKF4702X
- R143: footprint 402 -> R_0402_1005Metric; MANUFACTURER (none) -> Panasonic; MANUFACTURER_PART_NUMBER ERJ-2RKF2051X -> ERJ-2RKF1002X
- R144: footprint 402 -> R_0402_1005Metric; MANUFACTURER (none) -> Panasonic; MANUFACTURER_PART_NUMBER ERJ-2RKF2492X -> ERJ-2RKF1072X
- R146, R152: footprint (none) -> R_0402_1005Metric; MANUFACTURER (none) -> Panasonic; MANUFACTURER_PART_NUMBER (none) -> ERJ-2RKF1003X
- R147: footprint 402 -> R_0402_1005Metric; MANUFACTURER (none) -> Panasonic; MANUFACTURER_PART_NUMBER ERJ-2RKF1502X -> ERJ-2RKF2002X
- R148: footprint 402 -> R_0402_1005Metric; MANUFACTURER (none) -> Panasonic; MANUFACTURER_PART_NUMBER ERJ-2RKF2051X -> ERJ-2RKF5760X
- R149: footprint 402 -> R_0402_1005Metric; MANUFACTURER (none) -> Panasonic; MANUFACTURER_PART_NUMBER ERJ-2RKF2003X -> ERJ-2RKF1002X
- R151: footprint (none) -> R_0402_1005Metric; MANUFACTURER (none) -> Panasonic; MANUFACTURER_PART_NUMBER (none) -> ERJ-2RKF4701X
- R153: footprint (none) -> R_0402_1005Metric; MANUFACTURER (none) -> Panasonic; MANUFACTURER_PART_NUMBER (none) -> ERJ-2RKF1802X
- R154: footprint (none) -> R_0402_1005Metric; MANUFACTURER (none) -> Panasonic; MANUFACTURER_PART_NUMBER (none) -> ERJ-2RKF3302X
- R156: footprint 402 -> R_0402_1005Metric; MANUFACTURER (none) -> Panasonic; MANUFACTURER_PART_NUMBER ERJ-2RKF2003X -> ERJ-2RKF4701X
- R162, R163: footprint 402 -> R_0402_1005Metric; MANUFACTURER (none) -> Panasonic; MANUFACTURER_PART_NUMBER ERJ-U02F2R20X -> ERJ-2RKF2R20X
- U40: MANUFACTURER (none) -> Microchip Technology
- U41: MANUFACTURER_PART_NUMBER (none) -> LMV393
- U42: MANUFACTURER_PART_NUMBER (none) -> OPA320AIDBVT
- U43: MANUFACTURER_PART_NUMBER (none) -> MCP41U83T-503E/ST
- U44: MANUFACTURER_PART_NUMBER (none) -> INA228AQDGSRQ1
- U45: MANUFACTURER_PART_NUMBER (none) -> MCP1502T-40E/CHY
