File: hardware/ntp-server-stm32/rb.kicad_sch (KiCad schematic)
At the start: 67 parts, among them Q15 BC847W, Q16 BC847W, Q17 BC857W, Q18 BC847W, Q19 BC847W, Q20 BC847W, U40 MIC28516T-E/PHA, U41 LMV393, U42 OPA320AIDBVT, U43 MCP41U83T-503E/ST, U44 INA228AQDGSRQ1, U45 MCP1502T-40E/CHY

Commit message: Updates
Parts:
- added C182: 1uF, 0603 (1608 Metric), symbol Device:C
- added D25: BZX84C12, SOT-23-3 (TO-236), symbol Device:D_Zener
- added Q25: SI7469DP-T1-E3, PowerPAK® SO-8, symbol SI7469DP-T1-E3:SI7469DP-T1-E3
- added Q26: BC847W, SOT-323, symbol Transistor_BJT:BC847W
- added R257: 100k, 0402 (1005 Metric), symbol Device:R
- added R258, R261, R262: 10k, 0402 (1005 Metric), symbol Device:R
- C119: footprint C_0402_1005Metric -> 0402 (1005 Metric); DIELECTRIC (none) -> X7R; DIGIKEY_PART_NUMBER 490-1313-2-ND -> 490-GRT155R71C103KE01JCT-ND; MANUFACTURER Murata -> Murata Electronics; MANUFACTURER_PART_NUMBER GRM155R71C103KA01D -> GRT155R71C103KE01J; TOLERANCE (none) -> 10%; VOLTAGE (none) -> 16V
- C120, C121, C122, C123, C124, C131, C132: footprint C_0402_1005Metric -> 0402 (1005 Metric); DIELECTRIC (none) -> X7R; DIGIKEY_PART_NUMBER 490-6328-2-ND -> 490-4759-1-ND; MANUFACTURER_PART_NUMBER GRM155R71C104KA88J -> GCM155R71C104KA55D; TOLERANCE (none) -> 10%; VOLTAGE (none) -> 16V
- C125: footprint C_0402_1005Metric -> 0402 (1005 Metric); DIELECTRIC (none) -> X7R; DIGIKEY_PART_NUMBER 490-6334-2-ND -> 490-14515-1-ND; MANUFACTURER (none) -> Murata Electronics; MANUFACTURER_PART_NUMBER GRM155R71C472KA01D -> GCM155R71H473KE02J; TOLERANCE (none) -> 10%; VOLTAGE (none) -> 50V
- C126, C127, C128: footprint C_1210_3225Metric -> Stacked SMD, 2 J-Lead; DIELECTRIC (none) -> X7S; DIGIKEY_PART_NUMBER 490-16309-2-ND -> 490-KCM55WR71H476MH13LCT-ND; MANUFACTURER Murata -> Murata Electronics; MANUFACTURER_PART_NUMBER GRM32EC81C476KE15K -> KCM55WR71H476MH13L; TOLERANCE (none) -> 10%; VOLTAGE (none) -> 50V
- C129, C138: footprint C_0603_1608Metric -> 0805 (2012 Metric); DIELECTRIC (none) -> X7R; DIGIKEY_PART_NUMBER 490-GRM188Z71C225KE43DTR-ND -> 490-GRT21BR71C225KE01LCT-ND; MANUFACTURER Murata -> Murata Electronics; MANUFACTURER_PART_NUMBER GRM188Z71C225KE43D -> GRT21BR71C225KE01L; TOLERANCE (none) -> 10%; VOLTAGE (none) -> 16V
- C130: footprint C_0603_1608Metric -> 0603 (1608 Metric); DIELECTRIC (none) -> X7R; DIGIKEY_PART_NUMBER (none) -> 399-17704-1-ND; MANUFACTURER (none) -> KEMET; MANUFACTURER_PART_NUMBER (none) -> C0603C105K4RACAUTO; TOLERANCE (none) -> 10%; VOLTAGE (none) -> 16V
- C133, C134, C136: footprint C_0805_2012Metric -> 2220 (5750 Metric); DIELECTRIC (none) -> X7T; DIGIKEY_PART_NUMBER 490-GRM21BD72A225ME01KTR-ND -> 445-7950-1-ND; MANUFACTURER Murata -> TDK; MANUFACTURER_PART_NUMBER GRM21BD72A225ME01K -> CGA9P3X7T2E225K250KA; TOLERANCE (none) -> 10%; VOLTAGE (none) -> 100V
- C135: footprint C_0603_1608Metric -> 0805 (2012 Metric); DIELECTRIC (none) -> X7T; DIGIKEY_PART_NUMBER 490-GRM188D72A105KE01WTR-ND -> 478-KAM21KR72A105KUCT-ND; MANUFACTURER Murata -> KYOCERA AVX; MANUFACTURER_PART_NUMBER GRM188D72A105KE01W -> 08051C105K4T2A; TOLERANCE (none) -> 10%; VOLTAGE (none) -> 100V
- C137: footprint C_0805_2012Metric -> 0805 (2012 Metric); DIELECTRIC (none) -> X7R; DIGIKEY_PART_NUMBER 490-GRM21BR71C475KE51KTR-ND -> 490-GRT21BR71C475KE13KCT-ND; MANUFACTURER Murata -> Murata Electronics; MANUFACTURER_PART_NUMBER GRM21BR71C475KE51K -> GRT21BR71C475KE13K; TOLERANCE (none) -> 10%; VOLTAGE (none) -> 16V
- D11: footprint Package_TO_SOT_SMD:SOT-323_SC-70 -> SOD-123; DIELECTRIC (none) -> Diode; DIGIKEY_PART_NUMBER (none) -> 353-BAS16WHE3-TPCT-ND; MANUFACTURER (none) -> MCC (Micro Commercial Components); MANUFACTURER_PART_NUMBER BAS16W -> BAS16WHE3-TP
- FB8: DIELECTRIC (none) -> Ferrite bead; MANUFACTURER Murata Electronics -> Murata; MANUFACTURER_PART_NUMBER BLM31KN601SN1L -> BLM31PG601SN1L; POWER (none) -> 3A
- L7: value 40uH -> 39uH; DIELECTRIC (none) -> Inductor; DIGIKEY_PART_NUMBER SRP1265A-6R8MTR-ND -> 732-7447709390CT-ND; MANUFACTURER Bourns Inc. -> Würth Elektronik; MANUFACTURER_PART_NUMBER SRP1265A-6R8M -> 7447709390
- Q15, Q16, Q18, Q19, Q20: footprint Package_TO_SOT_SMD:SOT-323_SC-70 -> SOT-323; DIELECTRIC (none) -> Transistor; DIGIKEY_PART_NUMBER (none) -> 1727-BC847W,135CT-ND; MANUFACTURER (none) -> Nexperia USA Inc.; MANUFACTURER_PART_NUMBER BC847W -> BC847W,135
- Q17: footprint Package_TO_SOT_SMD:SOT-323_SC-70 -> SOT-323; DIELECTRIC (none) -> Transistor; DIGIKEY_PART_NUMBER (none) -> 1727-BC857W,135CT-ND; MANUFACTURER (none) -> Nexperia USA Inc.; MANUFACTURER_PART_NUMBER BC857W -> BC857W,135
- R132: footprint R_0402_1005Metric -> 0402 (1005 Metric); DIELECTRIC (none) -> Thick-film; DIGIKEY_PART_NUMBER P200KLTR-ND -> P200KLCT-ND; MANUFACTURER Panasonic -> Panasonic Industry; POWER (none) -> 1/10W; TOLERANCE (none) -> 1%
- R133: footprint R_0402_1005Metric -> 0402 (1005 Metric); DIELECTRIC (none) -> Thick-film; DIGIKEY_PART_NUMBER P100KLTR-ND -> P100KLCT-ND; MANUFACTURER Panasonic -> Panasonic Industry; POWER (none) -> 1/10W; TOLERANCE (none) -> 1%
- R134: value 4.12k -> 3.01k; footprint R_0402_1005Metric -> 0402 (1005 Metric); DIELECTRIC (none) -> Thick-film; DIGIKEY_PART_NUMBER P2.05KLTR-ND -> 2019-RK73H1ETTP3011FCT-ND; MANUFACTURER Panasonic -> KOA Speer Electronics, Inc.; MANUFACTURER_PART_NUMBER ERJ-2RKF4121X -> RK73H1ETTP3011F; POWER (none) -> 1/10W; TOLERANCE (none) -> 1%
- R135, R137, R139, R145, R150, R155, R157, R158, R160, R161: footprint R_0402_1005Metric -> 0402 (1005 Metric); DIELECTRIC (none) -> Thick-film; DIGIKEY_PART_NUMBER (none) -> P10.0KLCT-ND; MANUFACTURER Panasonic -> Panasonic Industry; POWER (none) -> 1/10W; TOLERANCE (none) -> 1%
- R136: value 10.5k -> 4.99k; footprint R_0402_1005Metric -> 0402 (1005 Metric); DIELECTRIC (none) -> Thick-film; DIGIKEY_PART_NUMBER (none) -> P4.99KLCT-ND; MANUFACTURER Panasonic -> Panasonic Industry; MANUFACTURER_PART_NUMBER ERJ-2RKF1052X -> ERJ-2RKF4991X; POWER (none) -> 1/10W; TOLERANCE (none) -> 1%
- R138: footprint R_0402_1005Metric -> 0402 (1005 Metric); DIELECTRIC (none) -> Thick-film; DIGIKEY_PART_NUMBER (none) -> P120KLCT-ND; MANUFACTURER Panasonic -> Panasonic Industry; POWER (none) -> 1/10W; TOLERANCE (none) -> 1%
- R140: footprint R_0402_1005Metric -> 0402 (1005 Metric); DIELECTRIC (none) -> Thick-film; DIGIKEY_PART_NUMBER P2.21KLTR-ND -> P2.21KLCT-ND; MANUFACTURER Panasonic -> Panasonic Industry; POWER (none) -> 1/10W; TOLERANCE (none) -> 1%
- R141: footprint R_0402_1005Metric -> 0402 (1005 Metric); DIELECTRIC (none) -> Thick-film; DIGIKEY_PART_NUMBER (none) -> P1.00MLCT-ND; MANUFACTURER Panasonic -> Panasonic Industry; POWER (none) -> 1/10W; TOLERANCE (none) -> 1%
- R142, R144, R147, R153, R154: DIELECTRIC (none) -> Thick-film; POWER (none) -> 1/10W; TOLERANCE (none) -> 1%
- R143: footprint R_0402_1005Metric -> 0402 (1005 Metric); DIELECTRIC (none) -> Thick-film; DIGIKEY_PART_NUMBER P2.05KLTR-ND -> P10.0KLCT-ND; MANUFACTURER Panasonic -> Panasonic Industry; POWER (none) -> 1/10W; TOLERANCE (none) -> 1%
- R146, R152: footprint R_0402_1005Metric -> 0402 (1005 Metric); DIELECTRIC (none) -> Thick-film; DIGIKEY_PART_NUMBER (none) -> P100KLCT-ND; MANUFACTURER Panasonic -> Panasonic Industry; POWER (none) -> 1/10W; TOLERANCE (none) -> 1%
- R148: value 576 -> 604; DIELECTRIC (none) -> Thick-film; MANUFACTURER_PART_NUMBER ERJ-2RKF5760X -> ERJ-2RKF6040X; POWER (none) -> 1/10W; TOLERANCE (none) -> 1%
- R149: footprint R_0402_1005Metric -> 0402 (1005 Metric); DIELECTRIC (none) -> Thick-film; DIGIKEY_PART_NUMBER P200KLTR-ND -> P10.0KLCT-ND; MANUFACTURER Panasonic -> Panasonic Industry; POWER (none) -> 1/10W; TOLERANCE (none) -> 1%
- R151: footprint R_0402_1005Metric -> 0402 (1005 Metric); DIELECTRIC (none) -> Thick-film; DIGIKEY_PART_NUMBER (none) -> P4.70KLCT-ND; MANUFACTURER Panasonic -> Panasonic Industry; POWER (none) -> 1/10W; TOLERANCE (none) -> 1%
- R156: footprint R_0402_1005Metric -> 0402 (1005 Metric); DIELECTRIC (none) -> Thick-film; DIGIKEY_PART_NUMBER P200KLTR-ND -> P4.70KLCT-ND; MANUFACTURER Panasonic -> Panasonic Industry; POWER (none) -> 1/10W; TOLERANCE (none) -> 1%
- R159: DIELECTRIC (none) -> Metal-strip shunt; POWER (none) -> 1/4W; TOLERANCE (none) -> 0.5%
- R162, R163: footprint R_0402_1005Metric -> 0402 (1005 Metric); DIELECTRIC (none) -> Thick-film; MANUFACTURER Panasonic -> Panasonic Industry; MANUFACTURER_PART_NUMBER ERJ-2RKF2R20X -> ERJ-U02F2R20X; POWER (none) -> 1/10W; TOLERANCE (none) -> 1%
- U40: MANUFACTURER Microchip Technology -> Microchip
- U41: MANUFACTURER (none) -> Texas Instruments; MANUFACTURER_PART_NUMBER LMV393 -> LMV393IDGKR
- U42, U44: MANUFACTURER (none) -> Texas Instruments
- U43: MANUFACTURER (none) -> Microchip
- U45: value MCP1502T-40E/CHY -> MCP1502T-30E/CHY; MANUFACTURER (none) -> Microchip; MANUFACTURER_PART_NUMBER MCP1502T-40E/CHY -> MCP1502T-30E/CHY
Connections:
- net GND: now also C182.2, Q26.2 (E), R262.2
- net I2C_SCL: now also U44.2 (A0), U44.5 (SCL); no longer U44.4 (SDA)
- net I2C_SDA: now also U44.4 (SDA); no longer U44.2 (A0), U44.5 (SCL)
- net VCC_RB: now also D25.1 (K), Q25.1 (S), Q25.2 (S), Q25.3 (S), R257.1
- net VOUT_P renamed V_POE
- net VREF_4V096 renamed VREF_3V0
- net VREF_3V0: now also C182.1
- new net: D25.2 (A), Q25.4 (G), R257.2, R258.2
- new net: Q26.1 (B), R261.2, R262.1
- new net: Q26.3 (C), R258.1
- new net RB_VCC_GATE: R261.1
- new net VCC_RB_G: Q25.5 (D), Q25.6 (D), Q25.7 (D), Q25.8 (D)

Commit message: bom updates
Parts:
- R142: footprint R_0402_1005Metric -> 0402 (1005 Metric); DIGIKEY_PART_NUMBER (none) -> P47.0KLCT-ND; MANUFACTURER Panasonic -> Panasonic Industry
- R144: footprint R_0402_1005Metric -> 0402 (1005 Metric); DIGIKEY_PART_NUMBER P24.9KLTR-ND -> P10.7KLCT-ND; MANUFACTURER Panasonic -> Panasonic Industry
Changed lines of the file:
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@@
 			)
 		)
-		(property "Footprint" "R_0402_1005Metric"
+		(property "Footprint" "0402 (1005 Metric)"
 			(at 106.172 59.69 90)
 			(hide yes)
@@
 			)
 		)
-		(property "Description" "RES 10.7k 1% 1/10W 0402"
+		(property "Description" "RES SMD 10.7K OHM 1% 1/10W 0402"
 			(at 107.95 59.69 0)
 			(hide yes)
@@
 			)
 		)
-		(property "MANUFACTURER" "Panasonic"
+		(property "MANUFACTURER" "Panasonic Industry"
 			(at 0 0 0)
 			(hide yes)
@@
 			)
 		)
-		(property "DIGIKEY_PART_NUMBER" "P24.9KLTR-ND"
+		(property "DIGIKEY_PART_NUMBER" "P10.7KLCT-ND"
 			(at 107.95 59.69 0)
 			(hide yes)
@@
 			)
 		)
-		(property "Footprint" "R_0402_1005Metric"
+		(property "Footprint" "0402 (1005 Metric)"
 			(at 92.202 199.39 90)
 			(hide yes)
@@
 			)
 		)
-		(property "Datasheet" ""
+		(property "Datasheet" "https://industrial.panasonic.com/cdbs/www-data/pdf/RDA0000/AOA0000C304.pdf"
 			(at 93.98 199.39 0)
 			(hide yes)
@@
 			)
 		)
-		(property "Description" "RES 47k 1% 1/10W 0402"
+		(property "Description" "RES SMD 47K OHM 1% 1/10W 0402"
 			(at 93.98 199.39 0)
 			(hide yes)
@@
 			)
 		)
-		(property "MANUFACTURER" "Panasonic"
+		(property "MANUFACTURER" "Panasonic Industry"
 			(at 0 0 0)
 			(hide yes)
@@
 			(hide yes)
 			(show_name no)
+			(do_not_autoplace no)
+			(effects
+				(font
+					(size 1.27 1.27)
+				)
+			)
+		)
+		(property "DIGIKEY_PART_NUMBER" "P47.0KLCT-ND"
+			(at 93.98 199.39 0)
+			(hide yes)
+			(show_name no)

Commit message: Bom updates
Parts:
- FB8: footprint 1206 -> 1206 (3216 Metric)
- R147: footprint R_0402_1005Metric -> 0402 (1005 Metric); DIGIKEY_PART_NUMBER P15.0KLTR-ND -> 10-ERJ-H2RD2002XCT-ND; MANUFACTURER Panasonic -> Panasonic Industry; MANUFACTURER_PART_NUMBER ERJ-2RKF2002X -> ERJ-H2RD2002X
- R148: footprint R_0402_1005Metric -> 0402 (1005 Metric); DIGIKEY_PART_NUMBER P2.05KLTR-ND -> P604LCT-ND; MANUFACTURER Panasonic -> Panasonic Industry
- R153: footprint R_0402_1005Metric -> 0402 (1005 Metric); DIGIKEY_PART_NUMBER (none) -> P18.0KLCT-ND; MANUFACTURER Panasonic -> Panasonic Industry
- R154: footprint R_0402_1005Metric -> 0402 (1005 Metric); DIGIKEY_PART_NUMBER (none) -> P33.0KLCT-ND; MANUFACTURER Panasonic -> Panasonic Industry
- R159: value 20m -> 7m; footprint 0805 -> 2515 (6332 Metric); DIGIKEY_PART_NUMBER 273-KDV08DR150ETCT-ND -> WSLG-.007CT-ND; MANUFACTURER Ohmite -> Vishay Dale; MANUFACTURER_PART_NUMBER KDV08DR150ET -> WSL25127L000FEA
- U41: footprint (none) -> 8-VSSOP; DIGIKEY_PART_NUMBER (none) -> 296-13993-1-ND
- U42: DIGIKEY_PART_NUMBER (none) -> 296-29510-1-ND
- U43: DIGIKEY_PART_NUMBER (none) -> 150-MCP41U83T-503E/STCT-ND
- U44: DIGIKEY_PART_NUMBER (none) -> 296-INA228AQDGSRQ1CT-ND
- U45: DIGIKEY_PART_NUMBER (none) -> 150-MCP1502T-30E/CHYCT-ND
Changed lines of the file:
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@@
 			)
 		)
-		(property "Footprint" "R_0402_1005Metric"
+		(property "Footprint" "0402 (1005 Metric)"
 			(at 166.878 223.52 90)
 			(hide yes)
@@
 			)
 		)
-		(property "Datasheet" ""
+		(property "Datasheet" "https://industrial.panasonic.com/cdbs/www-data/pdf/RDA0000/AOA0000C304.pdf"
 			(at 165.1 223.52 0)
 			(hide yes)
@@
 			)
 		)
-		(property "Description" "RES 18k 1% 1/10W 0402"
+		(property "Description" "RES SMD 18K OHM 1% 1/10W 0402"
 			(at 165.1 223.52 0)
 			(hide yes)
@@
 			)
 		)
-		(property "MANUFACTURER" "Panasonic"
+		(property "MANUFACTURER" "Panasonic Industry"
 			(at 0 0 0)
 			(hide yes)
@@
 			)
 		)
+		(property "DIGIKEY_PART_NUMBER" "P18.0KLCT-ND"
+			(at 165.1 223.52 0)
+			(hide yes)
+			(show_name no)
+			(do_not_autoplace no)
+			(effects
+				(font
+					(size 1.27 1.27)
+				)
+			)
+		)
 		(pin "1"
 		)
@@
 			)
 		)
+		(property "DIGIKEY_PART_NUMBER" "150-MCP1502T-30E/CHYCT-ND"
+			(at 157.48 147.32 0)
+			(hide yes)
+			(show_name no)
+			(do_not_autoplace no)
+			(effects
+				(font
+					(size 1.27 1.27)
+				)
+			)
+		)
 		(pin "6"
 		)
@@
 			)
 		)
-		(property "Datasheet" ""
+		(property "Datasheet" "https://www.ti.com/general/docs/suppproductinfo.tsp?distId=10&gotoUrl=https%3A%2F%2Fwww.ti.com%2Flit%2Fgpn%2Fopa320"
 			(at 95.25 113.03 0)
 			(hide yes)
@@
 			)
 		)
+		(property "DIGIKEY_PART_NUMBER" "296-29510-1-ND"
+			(at 95.25 113.03 0)
+			(hide yes)
+			(show_name no)
+			(do_not_autoplace no)
+			(effects
+				(font
+					(size 1.27 1.27)
+				)
+			)
+		)
 		(pin "5"
 		)
@@
 			)
 		)
-		(property "Datasheet" "https://www.ti.com/lit/gpn/ina228-q1"
+		(property "Datasheet" "https://www.ti.com/lit/ds/symlink/ina228-q1.pdf"
 			(at 151.13 91.44 0)
 			(hide yes)
@@
 			)
 		)
-		(property "Description" "Current/power monitor 20-bit I2C"
+		(property "Description" "IC PWR MONITOR 10VSSOP"
 			(at 151.13 91.44 0)
 			(hide yes)
@@
 			)
 		)
+		(property "DIGIKEY_PART_NUMBER" "296-INA228AQDGSRQ1CT-ND"
+			(at 151.13 91.44 0)
+			(hide yes)
+			(show_name no)
+			(do_not_autoplace no)
+			(effects
+				(font
+					(size 1.27 1.27)
+				)
+			)
+		)
 		(pin "2"
 		)
@@
 			)
 		)
-		(property "Footprint" "R_0402_1005Metric"
+		(property "Footprint" "0402 (1005 Metric)"
 			(at 116.332 59.69 90)
 			(hide yes)
@@
 			)
 		)
-		(property "Datasheet" "https://industrial.panasonic.com/cdbs/www-data/pdf/RDA0000/AOA0000C304.pdf"
+		(property "Datasheet" "https://industrial.panasonic.com/cdbs/www-data/pdf/RDQ0000/ast-ind-151033.pdf"
 			(at 118.11 59.69 0)
 			(hide yes)
@@
 			)
 		)
-		(property "Description" "RES 20k 1% 1/10W 0402"
+		(property "Description" "RES 20K OHM 0.5% 1/10W 0402"
 			(at 118.11 59.69 0)
 			(hide yes)
@@
 			)
 		)
-		(property "MANUFACTURER" "Panasonic"
+		(property "MANUFACTURER" "Panasonic Industry"
 			(at 0 0 0)
 			(hide yes)
@@
 			)
 		)
-		(property "DIGIKEY_PART_NUMBER" "P15.0KLTR-ND"
+		(property "DIGIKEY_PART_NUMBER" "10-ERJ-H2RD2002XCT-ND"
 			(at 118.11 59.69 0)
 			(hide yes)
@@
 			)
 		)
-		(property "MANUFACTURER_PART_NUMBER" "ERJ-2RKF2002X"
+		(property "MANUFACTURER_PART_NUMBER" "ERJ-H2RD2002X"
 			(at 118.11 59.69 0)
 			(hide yes)
@@
 			)
 		)
-		(property "Footprint" "1206"
+		(property "Footprint" "1206 (3216 Metric)"
 			(at 213.868 224.79 90)
 			(hide yes)
@@
 			)
 		)
-		(property "Footprint" "R_0402_1005Metric"
+		(property "Footprint" "0402 (1005 Metric)"
 			(at 163.322 240.03 90)
 			(hide yes)
@@
 			)
 		)
-		(property "Datasheet" ""
+		(property "Datasheet" "https://industrial.panasonic.com/cdbs/www-data/pdf/RDA0000/AOA0000C304.pdf"
 			(at 165.1 240.03 0)
 			(hide yes)
@@
 			)
 		)
-		(property "Description" "RES 33k 1% 1/10W 0402"
+		(property "Description" "RES SMD 33K OHM 1% 1/10W 0402"
 			(at 165.1 240.03 0)
 			(hide yes)
@@
 			)
 		)
-		(property "MANUFACTURER" "Panasonic"
+		(property "MANUFACTURER" "Panasonic Industry"
 			(at 0 0 0)
 			(hide yes)
@@
 			)
 		)
+		(property "DIGIKEY_PART_NUMBER" "P33.0KLCT-ND"
+			(at 165.1 240.03 0)
+			(hide yes)
+			(show_name no)
+			(do_not_autoplace no)
+			(effects
+				(font
+					(size 1.27 1.27)
+				)
+			)
+		)
 		(pin "1"
 		)
@@
 			)
 		)
-		(property "Footprint" "R_0402_1005Metric"
+		(property "Footprint" "0402 (1005 Metric)"
 			(at 116.332 81.28 90)
 			(hide yes)
@@
 			)
 		)
-		(property "Description" "RES 604 1% 1/10W 0402"
+		(property "Description" "RES SMD 604 OHM 1% 1/10W 0402"
 			(at 118.11 81.28 0)
 			(hide yes)
@@
 			)
 		)
-		(property "MANUFACTURER" "Panasonic"
+		(property "MANUFACTURER" "Panasonic Industry"
 			(at 0 0 0)
 			(hide yes)
@@
 			)
 		)
-		(property "DIGIKEY_PART_NUMBER" "P2.05KLTR-ND"
+		(property "DIGIKEY_PART_NUMBER" "P604LCT-ND"
 			(at 118.11 81.28 0)
 			(hide yes)
@@
 			)
 		)
-		(property "Datasheet" "https://ww1.microchip.com/downloads/aemDocuments/documents/APID/ProductDocuments/DataSheets/MCP41U83-Data-Sheet-DS20007000.pdf"
+		(property "Datasheet" "https://ww1.microchip.com/downloads/aemDocuments/documents/MSLD/ProductDocuments/MCP41U83-Data-Sheet-DS20007000.pdf"
 			(at 106.68 173.99 0)
 			(hide yes)
@@
 			)
 		)
+		(property "DIGIKEY_PART_NUMBER" "150-MCP41U83T-503E/STCT-ND"
+			(at 106.68 156.21 0)
+			(hide yes)
+			(show_name no)
+			(do_not_autoplace no)
+			(effects
+				(font
+					(size 1.27 1.27)
+				)
+			)
+		)
 		(pin "11"
 		)
@@
 			)
 		)
-		(property "Value" "20m"
+		(property "Value" "7m"
 			(at 202.946 57.15 90)
 			(show_name no)
@@
 			)
 		)
-		(property "Footprint" "0805"
+		(property "Footprint" "2515 (6332 Metric)"
 			(at 200.66 52.832 90)
 			(hide yes)
@@
 			)
 		)
-		(property "Datasheet" "https://www.ohmite.com/assets/images/res-kdv.pdf"
+		(property "Datasheet" "https://www.vishay.com/docs/30100/wsl.pdf"
 			(at 200.66 54.61 0)
 			(hide yes)
@@
 			)
 		)
-		(property "Description" "RES 20m SENSE 0.5% 0805"
+		(property "Description" "RES 0.007 OHM 1% 1W 2512"
 			(at 200.66 54.61 90)
 			(hide yes)
@@
 			)
 		)
-		(property "DIGIKEY_PART_NUMBER" "273-KDV08DR150ETCT-ND"
+		(property "DIGIKEY_PART_NUMBER" "WSLG-.007CT-ND"
 			(at 200.66 54.61 90)
 			(hide yes)
@@
 			)
 		)
-		(property "MANUFACTURER_PART_NUMBER" "KDV08DR150ET"
+		(property "MANUFACTURER_PART_NUMBER" "WSL25127L000FEA"
 			(at 200.66 54.61 90)
 			(hide yes)
@@
 			)
 		)
-		(property "MANUFACTURER" "Ohmite"
+		(property "MANUFACTURER" "Vishay Dale"
 			(at 200.66 54.61 90)
 			(hide yes)
@@
 			)
 		)
-		(property "Footprint" ""
+		(property "Footprint" "8-VSSOP"
 			(at 246.38 224.79 0)
 			(hide yes)
@@
 			)
 		)
-		(property "Datasheet" "http://www.ti.com/lit/ds/symlink/lmv331.pdf"
+		(property "Datasheet" "https://www.ti.com/general/docs/suppproductinfo.tsp?distId=10&gotoUrl=https%3A%2F%2Fwww.ti.com%2Flit%2Fgpn%2Flmv393"
 			(at 246.38 224.79 0)
 			(hide yes)
@@
 			)
 		)
-		(property "Description" "Dual comparator low-voltage"
+		(property "Description" "IC COMPARATOR 2CH 8-VSSOP"
 			(at 246.38 224.79 0)
 			(hide yes)
@@
 			)
 		)
+		(property "DIGIKEY_PART_NUMBER" "296-13993-1-ND"
+			(at 246.38 224.79 0)
+			(hide yes)
+			(show_name no)
+			(do_not_autoplace no)
+			(effects
+				(font
+					(size 1.27 1.27)
+				)
+			)
+		)
 		(pin "5"
 		)
@@
 			)
 		)
-		(property "Footprint" ""
+		(property "Footprint" "8-VSSOP"
 			(at 220.98 240.03 0)
 			(hide yes)
@@
 			)
 		)
-		(property "Datasheet" "http://www.ti.com/lit/ds/symlink/lmv331.pdf"
+		(property "Datasheet" "https://www.ti.com/general/docs/suppproductinfo.tsp?distId=10&gotoUrl=https%3A%2F%2Fwww.ti.com%2Flit%2Fgpn%2Flmv393"
 			(at 220.98 240.03 0)
 			(hide yes)
@@
 			)
 		)
-		(property "Description" "Dual comparator low-voltage"
+		(property "Description" "IC COMPARATOR 2CH 8-VSSOP"
 			(at 220.98 240.03 0)
 			(hide yes)
@@
 			)
 		)
+		(property "DIGIKEY_PART_NUMBER" "296-13993-1-ND"
+			(at 220.98 240.03 0)
+			(hide yes)
+			(show_name no)
+			(do_not_autoplace no)
+			(effects
+				(font
+					(size 1.27 1.27)
+				)
+			)
+		)
 		(pin "5"
 		)
@@
 			)
 		)
-		(property "Footprint" ""
+		(property "Footprint" "8-VSSOP"
 			(at 85.09 219.71 0)
 			(hide yes)
@@
 			)
 		)
-		(property "Datasheet" "http://www.ti.com/lit/ds/symlink/lmv331.pdf"
+		(property "Datasheet" "https://www.ti.com/general/docs/suppproductinfo.tsp?distId=10&gotoUrl=https%3A%2F%2Fwww.ti.com%2Flit%2Fgpn%2Flmv393"
 			(at 85.09 219.71 0)
 			(hide yes)
@@
 			)
 		)
-		(property "Description" "Dual comparator low-voltage"
+		(property "Description" "IC COMPARATOR 2CH 8-VSSOP"
 			(at 85.09 219.71 0)
 			(hide yes)
@@
 			(hide yes)
 			(show_name no)
+			(do_not_autoplace no)
+			(effects
+				(font
+					(size 1.27 1.27)
+				)
+			)
+		)
+		(property "DIGIKEY_PART_NUMBER" "296-13993-1-ND"
+			(at 85.09 219.71 0)
+			(hide yes)
+			(show_name no)

Commit message: Bom updates
Parts:
- R159: footprint 2515 (6332 Metric) -> 2512 (6332 Metric)
- U44: footprint VSSOP10_DGS_TEX -> sts1000:VSSOP10_DGS_TEX
Changed lines of the file:
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@@
 			)
 		)
-		(property "Footprint" "VSSOP10_DGS_TEX"
+		(property "Footprint" "sts1000:VSSOP10_DGS_TEX"
 			(at 151.13 91.44 0)
 			(hide yes)
@@
 			)
 		)
-		(property "Footprint" "2515 (6332 Metric)"
+		(property "Footprint" "2512 (6332 Metric)"
 			(at 200.66 52.832 90)
 			(hide yes)

Commit message: Add files via upload
Updated, completed placement
Parts:
- C119, C120, C121, C122, C123, C124, C125, C131, C132: footprint 0402 (1005 Metric) -> copy_ref:C_0402_1005Metric
- C126, C127, C128: footprint Stacked SMD, 2 J-Lead -> dowload:KCM55WR71H476MH13L
- C129, C135, C137, C138: footprint 0805 (2012 Metric) -> copy_ref:C_0805_2012Metric
- C130, C182: footprint 0603 (1608 Metric) -> copy_ref:C_0603_1608Metric
- C133, C134, C136: footprint 2220 (5750 Metric) -> Capacitor_SMD:C_2220_5750Metric
- D11: footprint SOD-123 -> dowload:SOD-123
- D25: footprint SOT-23-3 (TO-236) -> copy_ref:SOT-23-3
- FB8: footprint 1206 (3216 Metric) -> copy_ref:1206
- L7: footprint (none) -> dowload:7447709390
- Q15, Q16, Q17, Q18, Q19, Q20, Q26: footprint SOT-323 -> Package_TO_SOT_SMD:SOT-323_SC-70
- Q25: footprint PowerPAK® SO-8 -> dowload:PowerPAKÂ® SO-8
- R132, R133, R134, R135, R136, R137, R138, R139, R140, R141, R142, R143, R144, R145, R146, R147, R148, R149, R150, R151, R152, R153, R154, R155, R156, R157, R158, R160, R161, R162, R163, R257, R258, R261, R262: footprint 0402 (1005 Metric) -> copy_ref:R_0402_1005Metric
- R159: footprint 2512 (6332 Metric) -> Resistor_SMD:R_2512_6332Metric
- U40: footprint 32-PowerVQFN -> copy_ref:MIC28516T-EPHA
- U41: footprint 8-VSSOP -> dowload:LMV393
- U45: footprint SOT-23-6 -> Package_TO_SOT_SMD:SOT-23-6
