File: hardware/ntp-server-stm32/refclock-input.kicad_sch (KiCad schematic)
At the start: 29 parts, among them U49 TMUX1101DCK, U50 LTC6752xS5, U51 LT3045xDD

Commit message: Standardize net/rail names: plain 3V3 style, _N active-low, voltage-format PG/alerts
22 net renames applied across all sheets and verified: removed/added net-name
sets match intent exactly and all node connectivity is preserved (kicad-cli
netlist re-parse).

Co-Authored-By: Claude Opus 4.8 (1M context) <noreply@anthropic.com>
Connections:
- net +3.0V_RF renamed 3V0_RF
- net +3.3V renamed 3V3
- net +5V renamed 5V
- net 3.0V_RF_LDO_PG renamed 3V0_RF_LDO_PG
Changed lines of the file:
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@@
 		)
 	)
-	(global_label "3.0V_RF_LDO_PG"
+	(global_label "3V0_RF_LDO_PG"
 		(shape output)
 		(at 334.01 100.33 0)
@@
 			)
 		)
-		(property "Value" "+3.0V_RF"
+		(property "Value" "3V0_RF"
 			(at 100.33 160.02 0)
 			(show_name no)
@@
 			)
 		)
-		(property "Value" "+3.0V_RF"
+		(property "Value" "3V0_RF"
 			(at 76.2 99.06 0)
 			(show_name no)
@@
 			)
 		)
-		(property "Value" "+3.0V_RF"
+		(property "Value" "3V0_RF"
 			(at 128.27 217.17 0)
 			(show_name no)
@@
 			)
 		)
-		(property "Value" "+5V"
+		(property "Value" "5V"
 			(at 262.89 59.69 0)
 			(show_name no)
@@
 			)
 		)
-		(property "Value" "+3.0V_RF"
+		(property "Value" "3V0_RF"
 			(at 110.49 86.36 0)
 			(show_name no)
@@
 			)
 		)
-		(property "Value" "+3.0V_RF"
+		(property "Value" "3V0_RF"
 			(at 181.61 67.31 0)
 			(show_name no)
@@
 			)
 		)
-		(property "Value" "+3.0V_RF"
+		(property "Value" "3V0_RF"
 			(at 341.63 45.72 0)
 			(show_name no)
@@
 			)
 		)
-		(property "Value" "+3.0V_RF"
+		(property "Value" "3V0_RF"
 			(at 138.43 124.46 0)
 			(show_name no)
@@
 			)
 		)
-		(property "Value" "+3.3V"
+		(property "Value" "3V3"
 			(at 87.63 218.44 0)
 			(show_name no)

Commit message: Standardize + complete BOM; write fields back into KiCad symbols
- New sts1000_bom.csv: rebuilt from authoritative Value field (source MPN/footprint/
  description were corrupted by copy-paste). 338 standardized, 78 MPN-from-value,
  50 kept, ~64 flagged (SELECT/REVIEW-HV/SHUNT-REVIEW) each with full spec.
- Resistors -> deterministic Panasonic ERJ-2RKF 0402 1% 1/10W (consolidated 1 part/value).
- Caps -> verified Murata GRM parts where value matches; clean spec + footprint otherwise.
- 1633 symbol field updates (Value/Footprint/Description/MPN/Mfr/Digikey) written to
  .kicad_sch; netlist re-parse confirms connectivity byte-identical.
- Add docs/sts1000_net_naming.md naming reference.

Co-Authored-By: Claude Opus 4.8 (1M context) <noreply@anthropic.com>
Parts:
- C149: value 100nF -> 0.1uF; footprint (none) -> C_0402_1005Metric; DIGIKEY_PART_NUMBER (none) -> 490-6328-2-ND; MANUFACTURER (none) -> Murata; MANUFACTURER_PART_NUMBER (none) -> GRM155R71C104KA88J
- C150: footprint (none) -> C_0402_1005Metric; DIGIKEY_PART_NUMBER (none) -> 490-6328-2-ND; MANUFACTURER (none) -> Murata; MANUFACTURER_PART_NUMBER (none) -> GRM155R71C104KA88J
- C151, C155: footprint (none) -> C_0402_1005Metric; DIGIKEY_PART_NUMBER (none) -> 490-1313-2-ND; MANUFACTURER (none) -> Murata; MANUFACTURER_PART_NUMBER (none) -> GRM155R71C103KA01D
- C152: footprint 0805 -> C_0603_1608Metric
- C153: footprint 0805 -> C_0402_1005Metric; DIGIKEY_PART_NUMBER 445-5972-1-ND -> 490-6328-2-ND; MANUFACTURER TDK -> Murata; MANUFACTURER_PART_NUMBER C2012X7R1E475K125AB -> GRM155R71C104KA88J
- C154: footprint 0805 -> C_0805_2012Metric; DIGIKEY_PART_NUMBER 445-5972-1-ND -> 490-GRM21BZ71C106KE15LTR-ND; MANUFACTURER TDK -> Murata; MANUFACTURER_PART_NUMBER C2012X7R1E475K125AB -> GRM21BZ71C106KE15L
- C156: footprint 1206 -> C_0805_2012Metric; DIGIKEY_PART_NUMBER 445-7705-1-ND -> 490-GRM21BZ71C106KE15LTR-ND; MANUFACTURER TDK -> Murata; MANUFACTURER_PART_NUMBER C3216X7R1E106K160AB -> GRM21BZ71C106KE15L
- D18, D19: MANUFACTURER_PART_NUMBER (none) -> BAT54S
- R174, R175: footprint (none) -> R_0402_1005Metric; MANUFACTURER (none) -> Panasonic; MANUFACTURER_PART_NUMBER (none) -> ERJ-2RKF4702X
- R176, R182: footprint (none) -> R_0402_1005Metric; MANUFACTURER (none) -> Panasonic; MANUFACTURER_PART_NUMBER (none) -> ERJ-2RKF1003X
- R177: footprint (none) -> R_0402_1005Metric; MANUFACTURER (none) -> Panasonic; MANUFACTURER_PART_NUMBER (none) -> ERJ-2RKF49R9X
- R178: footprint (none) -> R_0402_1005Metric; MANUFACTURER (none) -> Panasonic; MANUFACTURER_PART_NUMBER (none) -> ERJ-2RKF1000X
- R179, R180: footprint (none) -> R_0402_1005Metric; MANUFACTURER (none) -> Panasonic; MANUFACTURER_PART_NUMBER (none) -> ERJ-2RKF1002X
- R181: footprint (none) -> R_0402_1005Metric; MANUFACTURER (none) -> Panasonic; MANUFACTURER_PART_NUMBER (none) -> ERJ-2RKF1001X
- R183, R184: footprint (none) -> R_0402_1005Metric; MANUFACTURER (none) -> Panasonic; MANUFACTURER_PART_NUMBER (none) -> ERJ-2RKF33R0X
- R185: footprint (none) -> R_0402_1005Metric; MANUFACTURER (none) -> Panasonic; MANUFACTURER_PART_NUMBER (none) -> ERJ-2RKF1501X
- R186: footprint (none) -> R_0402_1005Metric; MANUFACTURER (none) -> Panasonic; MANUFACTURER_PART_NUMBER (none) -> ERJ-2RKF3012X
- U49: MANUFACTURER_PART_NUMBER (none) -> TMUX1101DCK
- U50: MANUFACTURER_PART_NUMBER (none) -> LTC6752xS5
- U51: MANUFACTURER_PART_NUMBER (none) -> LT3045xDD
