File: hardware/ntp-server-stm32/refclock-input.kicad_sch (KiCad schematic)
At the start: 29 parts, among them U49 TMUX1101DCK, U50 LTC6752xS5, U51 LT3045xDD

Commit message: Updates
Parts:
- added C183, C184: 0.1uF, 0402 (1005 Metric), symbol Device:C
- added R218: 49.9k, R_0402_1005Metric, symbol Device:R
- added R219: 402k, R_0402_1005Metric, symbol Device:R
- added R266: 10k, 0402 (1005 Metric), symbol Device:R
- C149, C150, C153: footprint C_0402_1005Metric -> 0402 (1005 Metric); DIELECTRIC (none) -> X7R; DIGIKEY_PART_NUMBER 490-6328-2-ND -> 490-4759-1-ND; MANUFACTURER_PART_NUMBER GRM155R71C104KA88J -> GCM155R71C104KA55D; TOLERANCE (none) -> 10%; VOLTAGE (none) -> 16V
- C151, C155: footprint C_0402_1005Metric -> 0402 (1005 Metric); DIELECTRIC (none) -> X7R; DIGIKEY_PART_NUMBER 490-1313-2-ND -> 490-GRT155R71C103KE01JCT-ND; MANUFACTURER Murata -> Murata Electronics; MANUFACTURER_PART_NUMBER GRM155R71C103KA01D -> GRT155R71C103KE01J; TOLERANCE (none) -> 10%; VOLTAGE (none) -> 16V
- C152: footprint C_0603_1608Metric -> 0603 (1608 Metric); DIELECTRIC (none) -> X7R; DIGIKEY_PART_NUMBER 445-5972-1-ND -> 399-17704-1-ND; MANUFACTURER TDK -> KEMET; MANUFACTURER_PART_NUMBER C2012X7R1E475K125AB -> C0603C105K4RACAUTO; TOLERANCE (none) -> 10%; VOLTAGE (none) -> 16V
- C154, C156: footprint C_0805_2012Metric -> 1206 (3216 Metric); DIELECTRIC (none) -> X7R; DIGIKEY_PART_NUMBER 490-GRM21BZ71C106KE15LTR-ND -> 1276-6797-1-ND; MANUFACTURER Murata -> Samsung Electro-Mechanics; MANUFACTURER_PART_NUMBER GRM21BZ71C106KE15L -> CL31B106KOHVPNE; TOLERANCE (none) -> 10%; VOLTAGE (none) -> 16V
- D18, D19: footprint Package_TO_SOT_SMD:SOT-23 -> SOT-23-3 (TO-236); DIELECTRIC (none) -> Diode; DIGIKEY_PART_NUMBER (none) -> 4878-BAT54SCT-ND; MANUFACTURER (none) -> Diotec Semiconductor
- D20, D21: footprint (none) -> SOT-23-3 (TO-236); DIELECTRIC (none) -> Diode; DIGIKEY_PART_NUMBER (none) -> BZX84C3V3LT1GOSCT-ND; MANUFACTURER (none) -> onsemi; MANUFACTURER_PART_NUMBER (none) -> BZX84C3V3LT1G
- FB9: DIELECTRIC (none) -> Ferrite bead; MANUFACTURER Murata Electronics -> Murata; MANUFACTURER_PART_NUMBER BLM31KN601SN1L -> BLM31PG601SN1L; POWER (none) -> 3A
- R174, R175, R183, R184, R186: DIELECTRIC (none) -> Thick-film; POWER (none) -> 1/10W; TOLERANCE (none) -> 1%
- R176, R182: footprint R_0402_1005Metric -> 0402 (1005 Metric); DIELECTRIC (none) -> Thick-film; DIGIKEY_PART_NUMBER (none) -> P100KLCT-ND; MANUFACTURER Panasonic -> Panasonic Industry; POWER (none) -> 1/10W; TOLERANCE (none) -> 1%
- R177: footprint R_0402_1005Metric -> 0402 (1005 Metric); DIELECTRIC (none) -> Thick-film; DIGIKEY_PART_NUMBER (none) -> P49.9LCT-ND; MANUFACTURER Panasonic -> Panasonic Industry; POWER (none) -> 1/10W; TOLERANCE (none) -> 1%
- R178: footprint R_0402_1005Metric -> 0402 (1005 Metric); DIELECTRIC (none) -> Thick-film; DIGIKEY_PART_NUMBER (none) -> P100LCT-ND; MANUFACTURER Panasonic -> Panasonic Industry; POWER (none) -> 1/10W; TOLERANCE (none) -> 1%
- R179, R180: footprint R_0402_1005Metric -> 0402 (1005 Metric); DIELECTRIC (none) -> Thick-film; DIGIKEY_PART_NUMBER (none) -> P10.0KLCT-ND; MANUFACTURER Panasonic -> Panasonic Industry; POWER (none) -> 1/10W; TOLERANCE (none) -> 1%
- R181: footprint R_0402_1005Metric -> 0402 (1005 Metric); DIELECTRIC (none) -> Thick-film; DIGIKEY_PART_NUMBER (none) -> P1.00KLCT-ND; MANUFACTURER Panasonic -> Panasonic Industry; POWER (none) -> 1/10W; TOLERANCE (none) -> 1%
- R185: footprint R_0402_1005Metric -> 0402 (1005 Metric); DIELECTRIC (none) -> Thick-film; DIGIKEY_PART_NUMBER (none) -> P1.50KLCT-ND; MANUFACTURER Panasonic -> Panasonic Industry; POWER (none) -> 1/10W; TOLERANCE (none) -> 1%
- U49: MANUFACTURER (none) -> Texas Instruments
- U50: MANUFACTURER (none) -> Analog Devices; MANUFACTURER_PART_NUMBER LTC6752xS5 -> LTC6752IS5#TRMPBF
- U51: MANUFACTURER (none) -> Analog Devices; MANUFACTURER_PART_NUMBER LT3045xDD -> LT3045EDD#TRPBF
Connections:
- net 3V0_RF: now also C184.1, R219.1
- net 3V0_RF_LDO_PG: now also R266.2
- net GND: now also C183.2, C184.2, R218.2
- net at C154.1, FB9.1, U51.1 (IN)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: no longer U51.6 (PGFB)
- net at R179.1, R180.2, R182.1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: now also C183.1
- new net: R218.1, R219.2, U51.6 (PGFB)
- new net 3V3_STM: R266.1
Other:
- moved on the sheet: C156

Commit message: bom updates
Parts:
- R174, R175: footprint R_0402_1005Metric -> 0402 (1005 Metric); DIGIKEY_PART_NUMBER (none) -> P47.0KLCT-ND; MANUFACTURER Panasonic -> Panasonic Industry
Changed lines of the file:
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@@
 			)
 		)
-		(property "Footprint" "R_0402_1005Metric"
+		(property "Footprint" "0402 (1005 Metric)"
 			(at 74.422 109.22 90)
 			(hide yes)
@@
 			)
 		)
-		(property "Datasheet" ""
+		(property "Datasheet" "https://industrial.panasonic.com/cdbs/www-data/pdf/RDA0000/AOA0000C304.pdf"
 			(at 76.2 109.22 0)
 			(hide yes)
@@
 			)
 		)
-		(property "Description" "RES 47k 1% 1/10W 0402"
+		(property "Description" "RES SMD 47K OHM 1% 1/10W 0402"
 			(at 76.2 109.22 0)
 			(hide yes)
@@
 			)
 		)
-		(property "MANUFACTURER" "Panasonic"
+		(property "MANUFACTURER" "Panasonic Industry"
 			(at 0 0 0)
 			(hide yes)
@@
 		(property "MANUFACTURER_PART_NUMBER" "ERJ-2RKF4702X"
 			(at 0 0 0)
+			(hide yes)
+			(show_name no)
+			(do_not_autoplace no)
+			(effects
+				(font
+					(size 1.27 1.27)
+				)
+			)
+		)
+		(property "DIGIKEY_PART_NUMBER" "P47.0KLCT-ND"
+			(at 76.2 109.22 0)
 			(hide yes)
 			(show_name no)
@@
 			)
 		)
-		(property "Footprint" "R_0402_1005Metric"
+		(property "Footprint" "0402 (1005 Metric)"
 			(at 74.422 119.38 90)
 			(hide yes)
@@
 			)
 		)
-		(property "Datasheet" ""
+		(property "Datasheet" "https://industrial.panasonic.com/cdbs/www-data/pdf/RDA0000/AOA0000C304.pdf"
 			(at 76.2 119.38 0)
 			(hide yes)
@@
 			)
 		)
-		(property "Description" "RES 47k 1% 1/10W 0402"
+		(property "Description" "RES SMD 47K OHM 1% 1/10W 0402"
 			(at 76.2 119.38 0)
 			(hide yes)
@@
 			)
 		)
-		(property "MANUFACTURER" "Panasonic"
+		(property "MANUFACTURER" "Panasonic Industry"
 			(at 0 0 0)
 			(hide yes)
@@
 			(hide yes)
 			(show_name no)
+			(do_not_autoplace no)
+			(effects
+				(font
+					(size 1.27 1.27)
+				)
+			)
+		)
+		(property "DIGIKEY_PART_NUMBER" "P47.0KLCT-ND"
+			(at 76.2 119.38 0)
+			(hide yes)
+			(show_name no)

Commit message: Bom updates
Parts:
- FB9: footprint 1206 -> 1206 (3216 Metric)
- R183, R184: footprint R_0402_1005Metric -> 0402 (1005 Metric); DIGIKEY_PART_NUMBER (none) -> P33.0LCT-ND; MANUFACTURER Panasonic -> Panasonic Industry
- R186: footprint R_0402_1005Metric -> 0402 (1005 Metric); DIGIKEY_PART_NUMBER (none) -> P30.1KLCT-ND; MANUFACTURER Panasonic -> Panasonic Industry
- R218: footprint R_0402_1005Metric -> 0402 (1005 Metric); DIGIKEY_PART_NUMBER (none) -> P49.9KLCT-ND; MANUFACTURER Panasonic -> Panasonic Industry
- R219: footprint R_0402_1005Metric -> 0402 (1005 Metric); DIGIKEY_PART_NUMBER (none) -> P402KLCT-ND; MANUFACTURER Panasonic -> Panasonic Industry
- U49: DIGIKEY_PART_NUMBER (none) -> 296-TMUX1101DCKRCT-ND
- U50: DIGIKEY_PART_NUMBER (none) -> 505-LTC6752IS5#TRMPBFCT-ND
- U51: DIGIKEY_PART_NUMBER (none) -> 505-LT3045EDD#TRPBFCT-ND
Changed lines of the file:
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@@
 			)
 		)
-		(property "Footprint" "R_0402_1005Metric"
+		(property "Footprint" "0402 (1005 Metric)"
 			(at 183.388 80.01 90)
 			(hide yes)
@@
 			)
 		)
-		(property "Datasheet" ""
+		(property "Datasheet" "https://industrial.panasonic.com/cdbs/www-data/pdf/RDA0000/AOA0000C304.pdf"
 			(at 181.61 80.01 0)
 			(hide yes)
@@
 			)
 		)
-		(property "Description" "RES 33 1% 1/10W 0402"
+		(property "Description" "RES SMD 33 OHM 1% 1/10W 0402"
 			(at 181.61 80.01 0)
 			(hide yes)
@@
 			)
 		)
-		(property "MANUFACTURER" "Panasonic"
+		(property "MANUFACTURER" "Panasonic Industry"
 			(at 0 0 0)
 			(hide yes)
@@
 			)
 		)
+		(property "DIGIKEY_PART_NUMBER" "P33.0LCT-ND"
+			(at 181.61 80.01 0)
+			(hide yes)
+			(show_name no)
+			(do_not_autoplace no)
+			(effects
+				(font
+					(size 1.27 1.27)
+				)
+			)
+		)
 		(pin "1"
 		)
@@
 			)
 		)
-		(property "Footprint" "R_0402_1005Metric"
+		(property "Footprint" "0402 (1005 Metric)"
 			(at 296.418 92.71 90)
 			(hide yes)
@@
 			)
 		)
-		(property "Datasheet" ""
+		(property "Datasheet" "https://industrial.panasonic.com/cdbs/www-data/pdf/RDA0000/AOA0000C304.pdf"
 			(at 294.64 92.71 0)
 			(hide yes)
@@
 			)
 		)
-		(property "Description" "RES 30.1k 1% 1/10W 0402"
+		(property "Description" "RES SMD 30.1K OHM 1% 1/10W 0402"
 			(at 294.64 92.71 0)
 			(hide yes)
@@
 			)
 		)
-		(property "MANUFACTURER" "Panasonic"
+		(property "MANUFACTURER" "Panasonic Industry"
 			(at 0 0 0)
 			(hide yes)
@@
 			)
 		)
+		(property "DIGIKEY_PART_NUMBER" "P30.1KLCT-ND"
+			(at 294.64 92.71 0)
+			(hide yes)
+			(show_name no)
+			(do_not_autoplace no)
+			(effects
+				(font
+					(size 1.27 1.27)
+				)
+			)
+		)
 		(pin "1"
 		)
@@
 			)
 		)
-		(property "Footprint" "1206"
+		(property "Footprint" "1206 (3216 Metric)"
 			(at 264.668 71.12 90)
 			(hide yes)
@@
 			)
 		)
-		(property "Footprint" "R_0402_1005Metric"
+		(property "Footprint" "0402 (1005 Metric)"
 			(at 345.948 92.71 90)
 			(hide yes)
@@
 			)
 		)
-		(property "Datasheet" ""
+		(property "Datasheet" "https://industrial.panasonic.com/cdbs/www-data/pdf/RDA0000/AOA0000C304.pdf"
 			(at 344.17 92.71 0)
 			(hide yes)
@@
 			)
 		)
-		(property "Description" "RES 49.9k 1% 1/10W 0402"
+		(property "Description" "RES SMD 49.9K OHM 1% 1/10W 0402"
 			(at 344.17 92.71 0)
 			(hide yes)
@@
 			)
 		)
-		(property "MANUFACTURER" "Panasonic"
+		(property "MANUFACTURER" "Panasonic Industry"
 			(at 49.53 0 0)
 			(hide yes)
@@
 			)
 		)
+		(property "DIGIKEY_PART_NUMBER" "P49.9KLCT-ND"
+			(at 344.17 92.71 0)
+			(hide yes)
+			(show_name no)
+			(do_not_autoplace no)
+			(effects
+				(font
+					(size 1.27 1.27)
+				)
+			)
+		)
 		(pin "1"
 		)
@@
 			)
 		)
+		(property "DIGIKEY_PART_NUMBER" "505-LTC6752IS5#TRMPBFCT-ND"
+			(at 184.15 116.84 0)
+			(hide yes)
+			(show_name no)
+			(do_not_autoplace no)
+			(effects
+				(font
+					(size 1.27 1.27)
+				)
+			)
+		)
 		(pin "1"
 		)
@@
 			)
 		)
-		(property "Footprint" "R_0402_1005Metric"
+		(property "Footprint" "0402 (1005 Metric)"
 			(at 345.948 82.55 90)
 			(hide yes)
@@
 			)
 		)
-		(property "Datasheet" ""
+		(property "Datasheet" "https://industrial.panasonic.com/cdbs/www-data/pdf/RDA0000/AOA0000C304.pdf"
 			(at 344.17 82.55 0)
 			(hide yes)
@@
 			)
 		)
-		(property "Description" "RES 402k 1% 1/10W 0402"
+		(property "Description" "RES SMD 402K OHM 1% 1/10W 0402"
 			(at 344.17 82.55 0)
 			(hide yes)
@@
 			)
 		)
-		(property "MANUFACTURER" "Panasonic"
+		(property "MANUFACTURER" "Panasonic Industry"
 			(at 49.53 -10.16 0)
 			(hide yes)
@@
 			)
 		)
+		(property "DIGIKEY_PART_NUMBER" "P402KLCT-ND"
+			(at 344.17 82.55 0)
+			(hide yes)
+			(show_name no)
+			(do_not_autoplace no)
+			(effects
+				(font
+					(size 1.27 1.27)
+				)
+			)
+		)
 		(pin "1"
 		)
@@
 			)
 		)
+		(property "DIGIKEY_PART_NUMBER" "296-TMUX1101DCKRCT-ND"
+			(at 125.73 231.14 0)
+			(hide yes)
+			(show_name no)
+			(do_not_autoplace no)
+			(effects
+				(font
+					(size 1.27 1.27)
+				)
+			)
+		)
 		(pin "4"
 		)
@@
 			)
 		)
-		(property "Description" "LDO 500mA ultralow-noise DFN-10"
+		(property "Description" "IC REG LIN POS ADJ 500MA 10DFN"
 			(at 316.23 80.01 0)
 			(hide yes)
@@
 			)
 		)
+		(property "DIGIKEY_PART_NUMBER" "505-LT3045EDD#TRPBFCT-ND"
+			(at 316.23 80.01 0)
+			(hide yes)
+			(show_name no)
+			(do_not_autoplace no)
+			(effects
+				(font
+					(size 1.27 1.27)
+				)
+			)
+		)
 		(pin "7"
 		)
@@
 			)
 		)
-		(property "Footprint" "R_0402_1005Metric"
+		(property "Footprint" "0402 (1005 Metric)"
 			(at 200.66 118.618 90)
 			(hide yes)
@@
 			)
 		)
-		(property "Datasheet" ""
+		(property "Datasheet" "https://industrial.panasonic.com/cdbs/www-data/pdf/RDA0000/AOA0000C304.pdf"
 			(at 200.66 116.84 0)
 			(hide yes)
@@
 			)
 		)
-		(property "Description" "RES 33 1% 1/10W 0402"
+		(property "Description" "RES SMD 33 OHM 1% 1/10W 0402"
 			(at 200.66 116.84 0)
 			(hide yes)
@@
 			)
 		)
-		(property "MANUFACTURER" "Panasonic"
+		(property "MANUFACTURER" "Panasonic Industry"
 			(at 0 0 0)
 			(hide yes)
@@
 			(hide yes)
 			(show_name no)
+			(do_not_autoplace no)
+			(effects
+				(font
+					(size 1.27 1.27)
+				)
+			)
+		)
+		(property "DIGIKEY_PART_NUMBER" "P33.0LCT-ND"
+			(at 200.66 116.84 90)
+			(hide yes)
+			(show_name no)

Commit message: Add files via upload
Updated, completed placement
Parts:
- C149, C150, C151, C153, C155, C183, C184: footprint 0402 (1005 Metric) -> copy_ref:C_0402_1005Metric
- C152: footprint 0603 (1608 Metric) -> copy_ref:C_0603_1608Metric
- C154, C156: footprint 1206 (3216 Metric) -> copy_ref:C_1206_3216Metric
- D18, D19, D20, D21: footprint SOT-23-3 (TO-236) -> copy_ref:SOT-23-3
- FB9: footprint 1206 (3216 Metric) -> copy_ref:1206
- R174, R175, R176, R177, R178, R179, R180, R181, R182, R183, R184, R185, R186, R218, R219, R266: footprint 0402 (1005 Metric) -> copy_ref:R_0402_1005Metric
Changed lines of the file:
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@@
 			)
 		)
-		(property "Footprint" "0402 (1005 Metric)"
+		(property "Footprint" "copy_ref:R_0402_1005Metric"
 			(at 74.422 109.22 90)
 			(hide yes)
@@
 			)
 		)
-		(property "Footprint" "0402 (1005 Metric)"
+		(property "Footprint" "copy_ref:R_0402_1005Metric"
 			(at 74.422 119.38 90)
 			(hide yes)
@@
 			)
 		)
-		(property "Footprint" "0402 (1005 Metric)"
+		(property "Footprint" "copy_ref:R_0402_1005Metric"
 			(at 88.9 132.588 90)
 			(hide yes)
@@
 			)
 		)
-		(property "Footprint" "1206 (3216 Metric)"
+		(property "Footprint" "copy_ref:C_1206_3216Metric"
 			(at 261.9248 95.25 0)
 			(hide yes)
@@
 			)
 		)
-		(property "Footprint" "0402 (1005 Metric)"
+		(property "Footprint" "copy_ref:R_0402_1005Metric"
 			(at 183.388 80.01 90)
 			(hide yes)
@@
 			)
 		)
-		(property "Footprint" "0402 (1005 Metric)"
+		(property "Footprint" "copy_ref:C_0402_1005Metric"
 			(at 199.0852 96.52 0)
 			(hide yes)
@@
 			)
 		)
-		(property "Footprint" "0402 (1005 Metric)"
+		(property "Footprint" "copy_ref:R_0402_1005Metric"
 			(at 296.418 92.71 90)
 			(hide yes)
@@
 			)
 		)
-		(property "Footprint" "0402 (1005 Metric)"
+		(property "Footprint" "copy_ref:R_0402_1005Metric"
 			(at 136.652 134.62 90)
 			(hide yes)
@@
 			)
 		)
-		(property "Footprint" "0402 (1005 Metric)"
+		(property "Footprint" "copy_ref:C_0402_1005Metric"
 			(at 143.51 113.3348 0)
 			(hide yes)
@@
 			)
 		)
-		(property "Footprint" "1206 (3216 Metric)"
+		(property "Footprint" "copy_ref:1206"
 			(at 264.668 71.12 90)
 			(hide yes)
@@
 			)
 		)
-		(property "Footprint" "0402 (1005 Metric)"
+		(property "Footprint" "copy_ref:R_0402_1005Metric"
 			(at 345.948 92.71 90)
 			(hide yes)
@@
 			)
 		)
-		(property "Footprint" "0402 (1005 Metric)"
+		(property "Footprint" "copy_ref:C_0402_1005Metric"
 			(at 72.39 113.3348 0)
 			(hide yes)
@@
 			)
 		)
-		(property "Footprint" "0402 (1005 Metric)"
+		(property "Footprint" "copy_ref:C_0402_1005Metric"
 			(at 149.5552 234.95 0)
 			(hide yes)
@@
 			)
 		)
-		(property "Footprint" "0402 (1005 Metric)"
+		(property "Footprint" "copy_ref:C_0402_1005Metric"
 			(at 301.9552 96.52 0)
 			(hide yes)
@@
 			)
 		)
-		(property "Footprint" "0402 (1005 Metric)"
+		(property "Footprint" "copy_ref:C_0402_1005Metric"
 			(at 101.6 129.8448 0)
 			(hide yes)
@@
 			)
 		)
-		(property "Footprint" "0402 (1005 Metric)"
+		(property "Footprint" "copy_ref:C_0402_1005Metric"
 			(at 171.1452 153.67 0)
 			(hide yes)
@@
 			)
 		)
-		(property "Footprint" "SOT-23-3 (TO-236)"
+		(property "Footprint" "copy_ref:SOT-23-3"
 			(at 175.26 92.71 0)
 			(hide yes)
@@
 			)
 		)
-		(property "Footprint" "0402 (1005 Metric)"
+		(property "Footprint" "copy_ref:R_0402_1005Metric"
 			(at 158.242 128.27 90)
 			(hide yes)
@@
 			)
 		)
-		(property "Footprint" "SOT-23-3 (TO-236)"
+		(property "Footprint" "copy_ref:SOT-23-3"
 			(at 93.345 165.735 0)
 			(hide yes)
@@
 			)
 		)
-		(property "Footprint" "0402 (1005 Metric)"
+		(property "Footprint" "copy_ref:R_0402_1005Metric"
 			(at 91.44 116.078 90)
 			(hide yes)
@@
 			)
 		)
-		(property "Footprint" "0402 (1005 Metric)"
+		(property "Footprint" "copy_ref:R_0402_1005Metric"
 			(at 345.948 82.55 90)
 			(hide yes)
@@
 			)
 		)
-		(property "Footprint" "0402 (1005 Metric)"
+		(property "Footprint" "copy_ref:R_0402_1005Metric"
 			(at 337.058 67.31 90)
 			(hide yes)
@@
 			)
 		)
-		(property "Footprint" "0402 (1005 Metric)"
+		(property "Footprint" "copy_ref:R_0402_1005Metric"
 			(at 276.098 92.71 90)
 			(hide yes)
@@
 			)
 		)
-		(property "Footprint" "0402 (1005 Metric)"
+		(property "Footprint" "copy_ref:R_0402_1005Metric"
 			(at 151.13 116.078 90)
 			(hide yes)
@@
 			)
 		)
-		(property "Footprint" "SOT-23-3 (TO-236)"
+		(property "Footprint" "copy_ref:SOT-23-3"
 			(at 110.49 99.06 0)
 			(hide yes)
@@
 			)
 		)
-		(property "Footprint" "0402 (1005 Metric)"
+		(property "Footprint" "copy_ref:R_0402_1005Metric"
 			(at 85.852 228.6 90)
 			(hide yes)
@@
 			)
 		)
-		(property "Footprint" "SOT-23-3 (TO-236)"
+		(property "Footprint" "copy_ref:SOT-23-3"
 			(at 103.505 92.075 0)
 			(hide yes)
@@
 			)
 		)
-		(property "Footprint" "0603 (1608 Metric)"
+		(property "Footprint" "copy_ref:C_0603_1608Metric"
 			(at 190.8048 96.52 0)
 			(hide yes)
@@
 			)
 		)
-		(property "Footprint" "0402 (1005 Metric)"
+		(property "Footprint" "copy_ref:R_0402_1005Metric"
 			(at 200.66 118.618 90)
 			(hide yes)
@@
 			)
 		)
-		(property "Footprint" "0402 (1005 Metric)"
+		(property "Footprint" "copy_ref:R_0402_1005Metric"
 			(at 136.652 144.78 90)
 			(hide yes)
@@
 			)
 		)
-		(property "Footprint" "1206 (3216 Metric)"
+		(property "Footprint" "copy_ref:C_1206_3216Metric"
 			(at 371.8052 86.36 0)
 			(hide yes)
