File: hardware/ntp-server-stm32/PoE.kicad_sch (KiCad schematic)
At the start: 57 parts, among them Q1 BC847W, Q2 FDMC8622, Q3 BC857W, Q4 BC847W, Q5 BC847W, U10 INA228AQDGSRQ1, U2 LMV393, U3 BC846BPDW1T1G, U4 BC846BPDW1T1G, U5 BC846BPDW1T1G, U6 BC846BPDW1T1G, U7 FDMQ8205A, U8 FDMQ8205A, U9 NCP1095DBR2

Commit message: Standardize net/rail names: plain 3V3 style, _N active-low, voltage-format PG/alerts
22 net renames applied across all sheets and verified: removed/added net-name
sets match intent exactly and all node connectivity is preserved (kicad-cli
netlist re-parse).

Co-Authored-By: Claude Opus 4.8 (1M context) <noreply@anthropic.com>
Connections:
- net +3.3V renamed 3V3
- net +5V renamed 5V
- net POE_PGO renamed POE_PG
Changed lines of the file:
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@@
 		)
 	)
-	(global_label "POE_PGO"
+	(global_label "POE_PG"
 		(shape output)
 		(at 256.54 57.15 0)
@@
 			)
 		)
-		(property "Value" "+5V"
+		(property "Value" "5V"
 			(at 92.71 231.14 0)
 			(show_name no)
@@
 			)
 		)
-		(property "Value" "+3.3V"
+		(property "Value" "3V3"
 			(at 385.826 76.2 0)
 			(show_name no)
@@
 			)
 		)
-		(property "Value" "+5V"
+		(property "Value" "5V"
 			(at 69.85 232.41 0)
 			(show_name no)
@@
 			)
 		)
-		(property "Value" "+3.3V"
+		(property "Value" "3V3"
 			(at 311.15 190.5 0)
 			(show_name no)
@@
 			)
 		)
-		(property "Value" "+3.3V"
+		(property "Value" "3V3"
 			(at 30.734 221.488 0)
 			(show_name no)
@@
 			)
 		)
-		(property "Value" "+3.3V"
+		(property "Value" "3V3"
 			(at 99.06 198.12 0)
 			(show_name no)
@@
 			)
 		)
-		(property "Value" "+3.3V"
+		(property "Value" "3V3"
 			(at 293.37 198.12 0)
 			(show_name no)

Commit message: Standardize + complete BOM; write fields back into KiCad symbols
- New sts1000_bom.csv: rebuilt from authoritative Value field (source MPN/footprint/
  description were corrupted by copy-paste). 338 standardized, 78 MPN-from-value,
  50 kept, ~64 flagged (SELECT/REVIEW-HV/SHUNT-REVIEW) each with full spec.
- Resistors -> deterministic Panasonic ERJ-2RKF 0402 1% 1/10W (consolidated 1 part/value).
- Caps -> verified Murata GRM parts where value matches; clean spec + footprint otherwise.
- 1633 symbol field updates (Value/Footprint/Description/MPN/Mfr/Digikey) written to
  .kicad_sch; netlist re-parse confirms connectivity byte-identical.
- Add docs/sts1000_net_naming.md naming reference.

Co-Authored-By: Claude Opus 4.8 (1M context) <noreply@anthropic.com>
Parts:
- C10: value 10uF 100V -> 10uF; footprint 1206 -> C_0805_2012Metric
- C11: footprint 402 -> C_0402_1005Metric
- C12, C4, C5: footprint (none) -> C_0402_1005Metric; DIGIKEY_PART_NUMBER (none) -> 490-6328-2-ND; MANUFACTURER (none) -> Murata; MANUFACTURER_PART_NUMBER (none) -> GRM155R71C104KA88J
- C3: footprint (none) -> C_0402_1005Metric; DIGIKEY_PART_NUMBER (none) -> 490-GRM1555C1H102FA01JTR-ND; MANUFACTURER (none) -> Murata; MANUFACTURER_PART_NUMBER (none) -> GRM1555C1H102FA01J
- C6: value 1nF 2% -> 1nF; footprint 402 -> C_0402_1005Metric
- C7, C9: footprint 402 -> C_0603_1608Metric
- C8: value 0.1uF 100V -> 0.1uF; footprint 1206 -> C_0402_1005Metric
- D1, D2, D3, Q2, U9: MANUFACTURER (none) -> onsemi
- Q1, Q4, Q5: MANUFACTURER_PART_NUMBER (none) -> BC847W
- Q3: MANUFACTURER_PART_NUMBER (none) -> BC857W
- R10, R11, R12, R9: footprint 402 -> R_0402_1005Metric; MANUFACTURER (none) -> Panasonic; MANUFACTURER_PART_NUMBER ERJ-U02J155X -> ERJ-2RKF1504X
- R13, R20: footprint 402 -> R_0402_1005Metric; MANUFACTURER (none) -> Panasonic
- R14: footprint 402 -> R_0402_1005Metric; MANUFACTURER (none) -> Panasonic; MANUFACTURER_PART_NUMBER ERJ-2RKF3320X -> ERJ-2RKF9090X
- R15: footprint 402 -> R_0402_1005Metric; MANUFACTURER (none) -> Panasonic; MANUFACTURER_PART_NUMBER RK73H1ETTP2612F -> ERJ-2RKF2612X
- R16: MANUFACTURER (none) -> YAGEO
- R17, R22, R23, R24, R26, R27, R28: footprint 1206 -> R_0402_1005Metric; MANUFACTURER (none) -> Panasonic; MANUFACTURER_PART_NUMBER RL1206FR-070R025L -> ERJ-2RKF1002X
- R18: footprint 1206 -> R_0402_1005Metric; MANUFACTURER (none) -> Panasonic; MANUFACTURER_PART_NUMBER RL1206FR-070R025L -> ERJ-2RKF2492X
- R19, R21, R29, R5, R8: footprint 1206 -> R_0402_1005Metric; MANUFACTURER (none) -> Panasonic; MANUFACTURER_PART_NUMBER RL1206FR-070R025L -> ERJ-2RKF1003X
- R2: footprint 1206 -> R_0402_1005Metric; MANUFACTURER (none) -> Panasonic; MANUFACTURER_PART_NUMBER RL1206FR-070R025L -> ERJ-2RKF1204X
- R25: footprint 1206 -> R_0402_1005Metric; MANUFACTURER (none) -> Panasonic; MANUFACTURER_PART_NUMBER RL1206FR-070R025L -> ERJ-2RKF1803X
- R3: footprint 1206 -> R_0402_1005Metric; MANUFACTURER (none) -> Panasonic; MANUFACTURER_PART_NUMBER RL1206FR-070R025L -> ERJ-2RKF3922X
- R4: footprint 1206 -> R_0402_1005Metric; MANUFACTURER (none) -> Panasonic; MANUFACTURER_PART_NUMBER RL1206FR-070R025L -> ERJ-2RKF1743X
- R6: footprint 1206 -> R_0402_1005Metric; MANUFACTURER (none) -> Panasonic; MANUFACTURER_PART_NUMBER RL1206FR-070R025L -> ERJ-2RKF2004X
- R7: footprint 1206 -> R_0402_1005Metric; MANUFACTURER (none) -> Panasonic; MANUFACTURER_PART_NUMBER RL1206FR-070R025L -> ERJ-2RKF1001X
- U10: MANUFACTURER_PART_NUMBER (none) -> INA228AQDGSRQ1
- U2: MANUFACTURER_PART_NUMBER (none) -> LMV393

Commit message: BOM: fix precision/sense resistor detection; add BOM status doc
Detect precision/sense resistors by value-tag + MPN series instead of the
corrupted Description field (R210/R211 22-ohm series resistors were false-flagged).
Add docs/sts1000_bom.md with standardization rules + sourcing-decision list.

Co-Authored-By: Claude Opus 4.8 (1M context) <noreply@anthropic.com>
Parts:
- R15: footprint R_0402_1005Metric -> 402; MANUFACTURER Panasonic -> KOA Speer Electronics, Inc.; MANUFACTURER_PART_NUMBER ERJ-2RKF2612X -> RK73H1ETTP2612F
Changed lines of the file:
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@@
 			)
 		)
-		(property "Footprint" "R_0402_1005Metric"
+		(property "Footprint" "402"
 			(at 210.058 74.93 90)
 			(hide yes)
@@
 			)
 		)
-		(property "Description" "RES SMD 26.1k OHM 1% 1/10W 0402"
+		(property "Description" "RES 26.1K OHM 1% 1/10W 0402"
 			(at 208.28 74.93 0)
 			(hide yes)
@@
 			)
 		)
-		(property "MANUFACTURER" "Panasonic"
+		(property "MANUFACTURER" "KOA Speer Electronics, Inc."
 			(at 0 0 0)
 			(hide yes)
@@
 			)
 		)
-		(property "MANUFACTURER_PART_NUMBER" "ERJ-2RKF2612X"
+		(property "MANUFACTURER_PART_NUMBER" "RK73H1ETTP2612F"
 			(at 208.28 74.93 0)
 			(hide yes)
