File: hardware/ntp-server-stm32/PoE.kicad_sch (KiCad schematic)
At the start: 57 parts, among them Q1 BC847W, Q2 FDMC8622, Q3 BC857W, Q4 BC847W, Q5 BC847W, U10 INA228AQDGSRQ1, U2 LMV393, U3 BC846BPDW1T1G, U4 BC846BPDW1T1G, U5 BC846BPDW1T1G, U6 BC846BPDW1T1G, U7 FDMQ8205A, U8 FDMQ8205A, U9 NCP1095DBR2

Commit message: Updates
Parts:
- added CR1: SMCJ58A, DO214AC_LTF, symbol SMCJ58A:SMCJ58A
- C10: footprint C_0805_2012Metric -> SMD, J-Lead; DIELECTRIC (none) -> X7S; DIGIKEY_PART_NUMBER 490-3542-2-ND -> 490-KCM55QR72A106KH01LCT-ND; MANUFACTURER (none) -> Murata Electronics; MANUFACTURER_PART_NUMBER GRM31CR72E104KW03L -> KCM55QR72A106KH01L; TOLERANCE (none) -> 10%; VOLTAGE (none) -> 100V
- C11: footprint C_0402_1005Metric -> 0402 (1005 Metric); DIELECTRIC (none) -> C0G; DIGIKEY_PART_NUMBER 490-GRM1555C1H102FA01JTR-ND -> 720-GA0402A470JXBAP31GCT-ND; MANUFACTURER (none) -> Vishay Vitramon; MANUFACTURER_PART_NUMBER GRM1555C1H102FA01J -> GA0402A470JXBAP31G; TOLERANCE (none) -> 5%; VOLTAGE (none) -> 100V
- C12, C4, C5: footprint C_0402_1005Metric -> 0402 (1005 Metric); DIELECTRIC (none) -> X7R; DIGIKEY_PART_NUMBER 490-6328-2-ND -> 490-4759-1-ND; MANUFACTURER_PART_NUMBER GRM155R71C104KA88J -> GCM155R71C104KA55D; TOLERANCE (none) -> 10%; VOLTAGE (none) -> 16V
- C3: footprint C_0402_1005Metric -> 0402 (1005 Metric); DIELECTRIC (none) -> C0G; DIGIKEY_PART_NUMBER 490-GRM1555C1H102FA01JTR-ND -> 399-C0402C102J5GECAUTOCT-ND; MANUFACTURER Murata -> KEMET; MANUFACTURER_PART_NUMBER GRM1555C1H102FA01J -> C0402C102J5GECAUTO; TOLERANCE (none) -> 5%; VOLTAGE (none) -> 50V
- C6: footprint C_0402_1005Metric -> 0402 (1005 Metric); DIELECTRIC (none) -> C0G; DIGIKEY_PART_NUMBER 490-GRM1555C1H102FA01JTR-ND -> 399-17168-1-ND; MANUFACTURER (none) -> KEMET; MANUFACTURER_PART_NUMBER GRM1555C1H102FA01J -> C0402C102K1GECAUTO; TOLERANCE (none) -> 5%; VOLTAGE (none) -> 100V
- C7, C9: footprint C_0603_1608Metric -> 0805 (2012 Metric); DIELECTRIC (none) -> X7T; DIGIKEY_PART_NUMBER 490-GRM1555C1H102FA01JTR-ND -> 478-KAM21KR72A105KUCT-ND; MANUFACTURER (none) -> KYOCERA AVX; MANUFACTURER_PART_NUMBER GRM1555C1H102FA01J -> 08051C105K4T2A; TOLERANCE (none) -> 10%; VOLTAGE (none) -> 100V
- C8: footprint C_0402_1005Metric -> 0603 (1608 Metric); DIELECTRIC (none) -> X7R; DIGIKEY_PART_NUMBER 490-3542-2-ND -> 490-13420-1-ND; MANUFACTURER (none) -> Murata; MANUFACTURER_PART_NUMBER GRM31CR72E104KW03L -> GCJ188R72A104KA01D; TOLERANCE (none) -> 10%; VOLTAGE (none) -> 100V
- D1, D2, D3: DIELECTRIC (none) -> Diode
- D4: value 12V -> BZX84C12; footprint (none) -> SOT-23-3 (TO-236); DIELECTRIC (none) -> Diode; DIGIKEY_PART_NUMBER (none) -> BZX84C12LT1GOSCT-ND; MANUFACTURER (none) -> onsemi; MANUFACTURER_PART_NUMBER (none) -> BZX84C12LT1G
- Q1, Q4, Q5: footprint Package_TO_SOT_SMD:SOT-323_SC-70 -> SOT-323; DIELECTRIC (none) -> Transistor; DIGIKEY_PART_NUMBER (none) -> 1727-BC847W,135CT-ND; MANUFACTURER (none) -> Nexperia USA Inc.; MANUFACTURER_PART_NUMBER BC847W -> BC847W,135
- Q2: DIELECTRIC (none) -> Transistor; DIGIKEY_PART_NUMBER FDMC8622TR-ND -> FDMC8622CT-ND
- Q3: footprint Package_TO_SOT_SMD:SOT-323_SC-70 -> SOT-323; DIELECTRIC (none) -> Transistor; DIGIKEY_PART_NUMBER (none) -> 1727-BC857W,135CT-ND; MANUFACTURER (none) -> Nexperia USA Inc.; MANUFACTURER_PART_NUMBER BC857W -> BC857W,135
- R10, R11, R12, R9: footprint R_0402_1005Metric -> 0402 (1005 Metric); DIELECTRIC (none) -> Thick-film; DIGIKEY_PART_NUMBER 10-ERJ-U02J155XCT-ND -> P1.5MJCT-ND; MANUFACTURER Panasonic -> Panasonic Industry; MANUFACTURER_PART_NUMBER ERJ-2RKF1504X -> ERJ-2GEJ155X; POWER (none) -> 1/10W; TOLERANCE (none) -> 1%
- R13: footprint R_0402_1005Metric -> 0402 (1005 Metric); DIELECTRIC (none) -> Thick-film; DIGIKEY_PART_NUMBER P232LTR-ND -> P232LCT-ND; MANUFACTURER Panasonic -> Panasonic Industry; POWER (none) -> 1/10W; TOLERANCE (none) -> 1%
- R14: footprint R_0402_1005Metric -> 0402 (1005 Metric); DIELECTRIC (none) -> Thick-film; DIGIKEY_PART_NUMBER P332LTR-ND -> P909LCT-ND; MANUFACTURER Panasonic -> Panasonic Industry; POWER (none) -> 1/10W; TOLERANCE (none) -> 1%
- R15: footprint 402 -> 0402 (1005 Metric); DIELECTRIC (none) -> Thick-film; DIGIKEY_PART_NUMBER 2019-RK73H1ETTP2612FTR-ND -> P26.1KLCT-ND; MANUFACTURER KOA Speer Electronics, Inc. -> Panasonic Industry; MANUFACTURER_PART_NUMBER RK73H1ETTP2612F -> ERJ-2RKF2612X; POWER (none) -> 1/10W; TOLERANCE (none) -> 1%
- R16: footprint 1206 -> 1206 (3216 Metric); DIELECTRIC (none) -> Metal-strip shunt; DIGIKEY_PART_NUMBER 311-.025LWTR-ND -> 273-MCS1632R025DERCT-ND; MANUFACTURER YAGEO -> Ohmite; MANUFACTURER_PART_NUMBER RL1206FR-070R025L -> MCS1632R025DER; POWER (none) -> 1/2W; TOLERANCE (none) -> 0.5%
- R17, R22, R23, R24, R26, R27, R28: footprint R_0402_1005Metric -> 0402 (1005 Metric); DIELECTRIC (none) -> Thick-film; DIGIKEY_PART_NUMBER 311-.025LWTR-ND -> P10.0KLCT-ND; MANUFACTURER Panasonic -> Panasonic Industry; POWER (none) -> 1/10W; TOLERANCE (none) -> 1%
- R18: footprint R_0402_1005Metric -> 0402 (1005 Metric); DIELECTRIC (none) -> Thick-film; DIGIKEY_PART_NUMBER 311-.025LWTR-ND -> P24.9KLCT-ND; MANUFACTURER Panasonic -> Panasonic Industry; POWER (none) -> 1/10W; TOLERANCE (none) -> 1%
- R19, R21, R29, R5, R8: footprint R_0402_1005Metric -> 0402 (1005 Metric); DIELECTRIC (none) -> Thick-film; DIGIKEY_PART_NUMBER 311-.025LWTR-ND -> P100KLCT-ND; MANUFACTURER Panasonic -> Panasonic Industry; POWER (none) -> 1/10W; TOLERANCE (none) -> 1%
- R2: footprint R_0402_1005Metric -> 0402 (1005 Metric); DIELECTRIC (none) -> Thick-film; DIGIKEY_PART_NUMBER 311-.025LWTR-ND -> 10-ERJ-U02F1204XCT-ND; MANUFACTURER Panasonic -> Panasonic Industry; MANUFACTURER_PART_NUMBER ERJ-2RKF1204X -> ERJ-U02F1204X; POWER (none) -> 1/10W; TOLERANCE (none) -> 1%
- R20: footprint R_0402_1005Metric -> 0402 (1005 Metric); DIELECTRIC (none) -> Thick-film; DIGIKEY_PART_NUMBER P10.0KLTR-ND -> P10.0KLCT-ND; MANUFACTURER Panasonic -> Panasonic Industry; POWER (none) -> 1/10W; TOLERANCE (none) -> 1%
- R25: footprint R_0402_1005Metric -> 0402 (1005 Metric); DIELECTRIC (none) -> Thick-film; DIGIKEY_PART_NUMBER 311-.025LWTR-ND -> P180KLCT-ND; MANUFACTURER Panasonic -> Panasonic Industry; POWER (none) -> 1/10W; TOLERANCE (none) -> 1%
- R3: footprint R_0402_1005Metric -> 0402 (1005 Metric); DIELECTRIC (none) -> Thick-film; DIGIKEY_PART_NUMBER 311-.025LWTR-ND -> P39.2KLCT-ND; MANUFACTURER Panasonic -> Panasonic Industry; POWER (none) -> 1/10W; TOLERANCE (none) -> 1%
- R30: footprint 0805 -> 1206 (3216 Metric); DIELECTRIC (none) -> Metal-strip shunt; DIGIKEY_PART_NUMBER 273-KDV08DR150ETCT-ND -> 273-KDV12DR150ETCT-ND; MANUFACTURER_PART_NUMBER KDV08DR150ET -> KDV12DR150ET; POWER (none) -> 1/4W; TOLERANCE (none) -> 0.5%
- R4: footprint R_0402_1005Metric -> 0402 (1005 Metric); DIELECTRIC (none) -> Thick-film; DIGIKEY_PART_NUMBER 311-.025LWTR-ND -> P174KLCT-ND; MANUFACTURER Panasonic -> Panasonic Industry; POWER (none) -> 1/10W; TOLERANCE (none) -> 1%
- R6: footprint R_0402_1005Metric -> 0402 (1005 Metric); DIELECTRIC (none) -> Thick-film; DIGIKEY_PART_NUMBER 311-.025LWTR-ND -> 10-ERJ-U02F2004XCT-ND; MANUFACTURER Panasonic -> Panasonic Industry; MANUFACTURER_PART_NUMBER ERJ-2RKF2004X -> ERJ-U02F2004X; POWER (none) -> 1/10W; TOLERANCE (none) -> 1%
- R7: footprint R_0402_1005Metric -> 0402 (1005 Metric); DIELECTRIC (none) -> Thick-film; DIGIKEY_PART_NUMBER 311-.025LWTR-ND -> P1.00KLCT-ND; MANUFACTURER Panasonic -> Panasonic Industry; POWER (none) -> 1/10W; TOLERANCE (none) -> 1%
- U10: MANUFACTURER (none) -> Texas Instruments
- U2: MANUFACTURER (none) -> Texas Instruments; MANUFACTURER_PART_NUMBER LMV393 -> LMV393IDGKR
- U3, U4, U5, U6: MANUFACTURER ON Semiconductor -> onsemi
- U7, U8: MANUFACTURER On Semiconductor -> onsemi
Connections:
- net I2C_SCL: now also U10.5 (SCL); no longer U10.4 (SDA)
- net I2C_SDA: now also U10.4 (SDA); no longer U10.5 (SCL)
- net KILL_N: now also R21.1
- net VOUT_N: now also CR1.2
- net VOUT_P: now also CR1.1; no longer R2.2
- net V_POE: now also R2.2
- net at C7.2, D4.1 (K), R18.1: now also Q3.2 (E), R21.2; no longer R21.1
- net at Q3.3 (C): now also C9.2, R25.1, R27.1; no longer R21.2
Other:
- moved on the sheet: C10, C6, C8, Q2, R13, R14, R15, R16, R20, R21, U9

Commit message: Bom updates
Parts:
- R30: value 150m -> 25m; DIGIKEY_PART_NUMBER 273-KDV12DR150ETCT-ND -> WSLC-.025CT-ND; MANUFACTURER Ohmite -> Vishay Dale; MANUFACTURER_PART_NUMBER KDV12DR150ET -> WSL1206R0250FEA
- U10: DIGIKEY_PART_NUMBER (none) -> 296-INA228AQDGSRQ1CT-ND
- U2: footprint (none) -> 8-VSSOP; DIGIKEY_PART_NUMBER (none) -> 296-13993-1-ND
Changed lines of the file:
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@@
 			)
 		)
-		(property "Description" "Dual NPN/PNP 65V 0.1A SC70-6"
+		(property "Description" "TRANS NPN/PNP 65V 0.1A SC88/SC70"
 			(at 120.65 109.22 0)
 			(hide yes)
@@
 			)
 		)
-		(property "Description" "PoE bridge rectifier (GreenBridge)"
+		(property "Description" "GREENBRIDGETM 2 SERIES OF HIGH-E"
 			(at 151.13 45.72 0)
 			(hide yes)
@@
 			)
 		)
-		(property "Description" "Dual NPN/PNP 65V 0.1A SC70-6"
+		(property "Description" "TRANS NPN/PNP 65V 0.1A SC88/SC70"
 			(at 119.38 38.1 0)
 			(hide yes)
@@
 			)
 		)
-		(property "Description" "Dual NPN/PNP 65V 0.1A SC70-6"
+		(property "Description" "TRANS NPN/PNP 65V 0.1A SC88/SC70"
 			(at 119.38 83.82 0)
 			(hide yes)
@@
 			)
 		)
-		(property "Description" "Dual NPN/PNP 65V 0.1A SC70-6"
+		(property "Description" "TRANS NPN/PNP 65V 0.1A SC88/SC70"
 			(at 119.38 68.58 0)
 			(hide yes)
@@
 			)
 		)
-		(property "Datasheet" "https://www.ti.com/lit/gpn/ina228-q1"
+		(property "Datasheet" "https://www.ti.com/lit/ds/symlink/ina228-q1.pdf"
 			(at 335.28 71.12 0)
 			(hide yes)
@@
 			)
 		)
-		(property "Description" "Current/power monitor 20-bit I2C"
+		(property "Description" "IC PWR MONITOR 10VSSOP"
 			(at 335.28 71.12 0)
 			(hide yes)
@@
 			)
 		)
+		(property "DIGIKEY_PART_NUMBER" "296-INA228AQDGSRQ1CT-ND"
+			(at 335.28 71.12 0)
+			(hide yes)
+			(show_name no)
+			(do_not_autoplace no)
+			(effects
+				(font
+					(size 1.27 1.27)
+				)
+			)
+		)
 		(pin "2"
 		)
@@
 			)
 		)
-		(property "Description" "Dual NPN/PNP 65V 0.1A SC70-6"
+		(property "Description" "TRANS NPN/PNP 65V 0.1A SC88/SC70"
 			(at 119.38 22.86 0)
 			(hide yes)
@@
 			)
 		)
-		(property "Footprint" ""
+		(property "Footprint" "8-VSSOP"
 			(at 113.03 236.22 0)
 			(hide yes)
@@
 			)
 		)
-		(property "Datasheet" "http://www.ti.com/lit/ds/symlink/lmv331.pdf"
+		(property "Datasheet" "https://www.ti.com/general/docs/suppproductinfo.tsp?distId=10&gotoUrl=https%3A%2F%2Fwww.ti.com%2Flit%2Fgpn%2Flmv393"
 			(at 113.03 236.22 0)
 			(hide yes)
@@
 			)
 		)
-		(property "Description" "Dual comparator low-voltage"
+		(property "Description" "IC COMPARATOR 2CH 8-VSSOP"
 			(at 113.03 236.22 0)
 			(hide yes)
@@
 			)
 		)
+		(property "DIGIKEY_PART_NUMBER" "296-13993-1-ND"
+			(at 113.03 236.22 0)
+			(hide yes)
+			(show_name no)
+			(do_not_autoplace no)
+			(effects
+				(font
+					(size 1.27 1.27)
+				)
+			)
+		)
 		(pin "7"
 		)
@@
 			)
 		)
-		(property "Description" "Dual NPN/PNP 65V 0.1A SC70-6"
+		(property "Description" "TRANS NPN/PNP 65V 0.1A SC88/SC70"
 			(at 120.65 124.46 0)
 			(hide yes)
@@
 			)
 		)
-		(property "Value" "150m"
+		(property "Value" "25m"
 			(at 387.096 46.99 90)
 			(show_name no)
@@
 			)
 		)
-		(property "Datasheet" "https://www.ohmite.com/assets/images/res-kdv.pdf"
+		(property "Datasheet" "https://www.vishay.com/docs/30100/wsl.pdf"
 			(at 384.81 44.45 0)
 			(hide yes)
@@
 			)
 		)
-		(property "Description" "RES 0.15 OHM 0.5% 1/2W 1206"
+		(property "Description" "RES 0.025 OHM 1% 1/4W 1206"
 			(at 384.81 44.45 90)
 			(hide yes)
@@
 			)
 		)
-		(property "DIGIKEY_PART_NUMBER" "273-KDV12DR150ETCT-ND"
+		(property "DIGIKEY_PART_NUMBER" "WSLC-.025CT-ND"
 			(at 384.81 44.45 90)
 			(hide yes)
@@
 			)
 		)
-		(property "MANUFACTURER_PART_NUMBER" "KDV12DR150ET"
+		(property "MANUFACTURER_PART_NUMBER" "WSL1206R0250FEA"
 			(at 384.81 44.45 90)
 			(hide yes)
@@
 			)
 		)
-		(property "MANUFACTURER" "Ohmite"
+		(property "MANUFACTURER" "Vishay Dale"
 			(at 384.81 44.45 90)
 			(hide yes)
@@
 			)
 		)
-		(property "Description" "PoE bridge rectifier (GreenBridge)"
+		(property "Description" "GREENBRIDGETM 2 SERIES OF HIGH-E"
 			(at 151.13 132.08 0)
 			(hide yes)
@@
 			)
 		)
-		(property "Description" "PoE-PD controller 16-TSSOP"
+		(property "Description" "IC POE CNTRL 1 CHANNEL 16TSSOP"
 			(at 226.06 54.61 0)
 			(hide yes)
@@
 			)
 		)
-		(property "Description" "Dual NPN/PNP 65V 0.1A SC70-6"
+		(property "Description" "TRANS NPN/PNP 65V 0.1A SC88/SC70"
 			(at 120.65 170.18 0)
 			(hide yes)
@@
 			)
 		)
-		(property "Footprint" ""
+		(property "Footprint" "8-VSSOP"
 			(at 73.66 217.17 0)
 			(hide yes)
@@
 			)
 		)
-		(property "Datasheet" "http://www.ti.com/lit/ds/symlink/lmv331.pdf"
+		(property "Datasheet" "https://www.ti.com/general/docs/suppproductinfo.tsp?distId=10&gotoUrl=https%3A%2F%2Fwww.ti.com%2Flit%2Fgpn%2Flmv393"
 			(at 73.66 217.17 0)
 			(hide yes)
@@
 			)
 		)
-		(property "Description" "Dual comparator low-voltage"
+		(property "Description" "IC COMPARATOR 2CH 8-VSSOP"
 			(at 73.66 217.17 0)
 			(hide yes)
@@
 			)
 		)
+		(property "DIGIKEY_PART_NUMBER" "296-13993-1-ND"
+			(at 73.66 217.17 0)
+			(hide yes)
+			(show_name no)
+			(do_not_autoplace no)
+			(effects
+				(font
+					(size 1.27 1.27)
+				)
+			)
+		)
 		(pin "7"
 		)
@@
 			)
 		)
-		(property "Description" "Dual NPN/PNP 65V 0.1A SC70-6"
+		(property "Description" "TRANS NPN/PNP 65V 0.1A SC88/SC70"
 			(at 120.65 154.94 0)
 			(hide yes)
@@
 			)
 		)
-		(property "Footprint" ""
+		(property "Footprint" "8-VSSOP"
 			(at 83.82 247.65 0)
 			(hide yes)
@@
 			)
 		)
-		(property "Datasheet" "http://www.ti.com/lit/ds/symlink/lmv331.pdf"
+		(property "Datasheet" "https://www.ti.com/general/docs/suppproductinfo.tsp?distId=10&gotoUrl=https%3A%2F%2Fwww.ti.com%2Flit%2Fgpn%2Flmv393"
 			(at 83.82 247.65 0)
 			(hide yes)
@@
 			)
 		)
-		(property "Description" "Dual comparator low-voltage"
+		(property "Description" "IC COMPARATOR 2CH 8-VSSOP"
 			(at 83.82 247.65 0)
 			(hide yes)
@@
 			(hide yes)
 			(show_name no)
+			(do_not_autoplace no)
+			(effects
+				(font
+					(size 1.27 1.27)
+				)
+			)
+		)
+		(property "DIGIKEY_PART_NUMBER" "296-13993-1-ND"
+			(at 83.82 247.65 0)
+			(hide yes)
+			(show_name no)

Commit message: Bom updates
Parts:
- CR1: footprint DO214AC_LTF -> sts1000:DO214AC_LTF
- R2: footprint 0402 (1005 Metric) -> 1206 (3216 Metric); DIGIKEY_PART_NUMBER 10-ERJ-U02F1204XCT-ND -> P1.20MFCT-ND; MANUFACTURER_PART_NUMBER ERJ-U02F1204X -> ERJ-8ENF1204V
- R20: footprint 0402 (1005 Metric) -> 1210 (3225 Metric); DIGIKEY_PART_NUMBER P10.0KLCT-ND -> P10.0KAACT-ND; MANUFACTURER_PART_NUMBER ERJ-2RKF1002X -> ERJ-14NF1002U
- U10: footprint VSSOP10_DGS_TEX -> sts1000:VSSOP10_DGS_TEX
Changed lines of the file:
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@@
 			)
 		)
-		(property "Footprint" "0402 (1005 Metric)"
+		(property "Footprint" "1210 (3225 Metric)"
 			(at 267.462 45.72 90)
 			(hide yes)
@@
 			)
 		)
-		(property "Description" "RES SMD 10K OHM 1% 1/10W 0402"
+		(property "Description" "RES SMD 10K OHM 1% 1/2W 1210"
 			(at 269.24 45.72 0)
 			(hide yes)
@@
 			)
 		)
-		(property "DIGIKEY_PART_NUMBER" "P10.0KLCT-ND"
+		(property "DIGIKEY_PART_NUMBER" "P10.0KAACT-ND"
 			(at 269.24 45.72 0)
 			(hide yes)
@@
 			)
 		)
-		(property "MANUFACTURER_PART_NUMBER" "ERJ-2RKF1002X"
+		(property "MANUFACTURER_PART_NUMBER" "ERJ-14NF1002U"
 			(at 269.24 45.72 0)
 			(hide yes)
@@
 			)
 		)
-		(property "Footprint" "VSSOP10_DGS_TEX"
+		(property "Footprint" "sts1000:VSSOP10_DGS_TEX"
 			(at 335.28 71.12 0)
 			(hide yes)
@@
 			)
 		)
-		(property "Footprint" "DO214AC_LTF"
+		(property "Footprint" "sts1000:DO214AC_LTF"
 			(at 182.88 53.34 0)
 			(hide yes)
@@
 			)
 		)
-		(property "Footprint" "0402 (1005 Metric)"
+		(property "Footprint" "1206 (3216 Metric)"
 			(at 28.702 195.58 90)
 			(hide yes)
@@
 			)
 		)
-		(property "Datasheet" "https://industrial.panasonic.com/cdbs/www-data/pdf/RDM0000/DMM0000COL9.pdf"
+		(property "Datasheet" "https://industrial.panasonic.com/cdbs/www-data/pdf/RDA0000/AOA0000C304.pdf"
 			(at 30.48 195.58 0)
 			(hide yes)
@@
 			)
 		)
-		(property "Description" "RES 1.2M OHM 1% 1/10W 0402"
+		(property "Description" "RES SMD 1.2M OHM 1% 1/4W 1206"
 			(at 30.48 195.58 90)
 			(hide yes)
@@
 			)
 		)
-		(property "DIGIKEY_PART_NUMBER" "10-ERJ-U02F1204XCT-ND"
+		(property "DIGIKEY_PART_NUMBER" "P1.20MFCT-ND"
 			(at 30.48 195.58 90)
 			(hide yes)
@@
 			)
 		)
-		(property "MANUFACTURER_PART_NUMBER" "ERJ-U02F1204X"
+		(property "MANUFACTURER_PART_NUMBER" "ERJ-8ENF1204V"
 			(at 30.48 195.58 90)
 			(hide yes)
