File: hardware/ntp-server-stm32/PoE.kicad_sch (KiCad schematic)
At the start: 58 parts, among them Q1 BC847W, Q2 FDMC8622, Q3 BC857W, Q4 BC847W, Q5 BC847W, U10 INA228AQDGSRQ1, U2 LMV393, U3 BC846BPDW1T1G, U4 BC846BPDW1T1G, U5 BC846BPDW1T1G, U6 BC846BPDW1T1G, U7 FDMQ8205A, U8 FDMQ8205A, U9 NCP1095DBR2

Commit message: Add files via upload
Updated, completed placement
Parts:
- C10: footprint SMD, J-Lead -> dowload:KCM55QR72A106KH01L
- C11, C12, C3, C4, C5, C6: footprint 0402 (1005 Metric) -> copy_ref:C_0402_1005Metric
- C7, C9: footprint 0805 (2012 Metric) -> copy_ref:C_0805_2012Metric
- C8: footprint 0603 (1608 Metric) -> copy_ref:C_0603_1608Metric
- D1: footprint SOT-23-3 -> Package_TO_SOT_SMD:SOT-23-3
- D4: footprint SOT-23-3 (TO-236) -> copy_ref:SOT-23-3
- Q1, Q3, Q4, Q5: footprint SOT-323 -> Package_TO_SOT_SMD:SOT-323_SC-70
- Q2: footprint 8-PowerWDFN -> dowload:8-PowerWDFN
- R10, R11, R12, R13, R14, R15, R17, R18, R19, R21, R22, R23, R24, R25, R26, R27, R28, R29, R3, R4, R5, R6, R7, R8, R9: footprint 0402 (1005 Metric) -> copy_ref:R_0402_1005Metric
- R16, R2, R30: footprint 1206 (3216 Metric) -> copy_ref:R_1206_3216Metric
- R20: footprint 1210 (3225 Metric) -> Resistor_SMD:R_1210_3225Metric
- U2: footprint 8-VSSOP -> dowload:LMV393
- U3, U4, U5, U6: footprint SOT-363 -> copy_ref:SOT-363_SC-70-6
- U7, U8: footprint 12-MLP -> copy_ref:IC_FDMQ8205A
- U9: footprint 16-TSSOP -> dowload:TSSOP-16_948F-01_OSI
Changed lines of the file:
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@@
 			)
 		)
-		(property "Footprint" "0402 (1005 Metric)"
+		(property "Footprint" "copy_ref:C_0402_1005Metric"
 			(at 339.3948 170.18 0)
 			(hide yes)
@@
 			)
 		)
-		(property "Footprint" "SOT-363"
+		(property "Footprint" "copy_ref:SOT-363_SC-70-6"
 			(at 120.65 109.22 0)
 			(hide yes)
@@
 			)
 		)
-		(property "Footprint" "12-MLP"
+		(property "Footprint" "copy_ref:IC_FDMQ8205A"
 			(at 151.13 43.18 0)
 			(hide yes)
@@
 			)
 		)
-		(property "Footprint" "0402 (1005 Metric)"
+		(property "Footprint" "copy_ref:R_0402_1005Metric"
 			(at 293.37 157.988 90)
 			(hide yes)
@@
 			)
 		)
-		(property "Footprint" "0402 (1005 Metric)"
+		(property "Footprint" "copy_ref:R_0402_1005Metric"
 			(at 291.592 209.55 90)
 			(hide yes)
@@
 			)
 		)
-		(property "Footprint" "SOT-23-3"
+		(property "Footprint" "Package_TO_SOT_SMD:SOT-23-3"
 			(at 82.55 72.39 0)
 			(hide yes)
@@
 			)
 		)
-		(property "Footprint" "0805 (2012 Metric)"
+		(property "Footprint" "copy_ref:C_0805_2012Metric"
 			(at 263.1948 144.78 0)
 			(hide yes)
@@
 			)
 		)
-		(property "Footprint" "0603 (1608 Metric)"
+		(property "Footprint" "copy_ref:C_0603_1608Metric"
 			(at 291.7952 58.42 0)
 			(hide yes)
@@
 			)
 		)
-		(property "Footprint" "0402 (1005 Metric)"
+		(property "Footprint" "copy_ref:R_0402_1005Metric"
 			(at 28.702 240.03 90)
 			(hide yes)
@@
 			)
 		)
-		(property "Footprint" "1206 (3216 Metric)"
+		(property "Footprint" "copy_ref:R_1206_3216Metric"
 			(at 255.27 85.852 90)
 			(hide yes)
@@
 			)
 		)
-		(property "Footprint" "SOT-363"
+		(property "Footprint" "copy_ref:SOT-363_SC-70-6"
 			(at 119.38 38.1 0)
 			(hide yes)
@@
 			)
 		)
-		(property "Footprint" "0402 (1005 Metric)"
+		(property "Footprint" "copy_ref:R_0402_1005Metric"
 			(at 242.57 215.392 90)
 			(hide yes)
@@
 			)
 		)
-		(property "Footprint" "0402 (1005 Metric)"
+		(property "Footprint" "copy_ref:R_0402_1005Metric"
 			(at 107.95 66.802 90)
 			(hide yes)
@@
 			)
 		)
-		(property "Footprint" "0402 (1005 Metric)"
+		(property "Footprint" "copy_ref:R_0402_1005Metric"
 			(at 281.432 149.86 90)
 			(hide yes)
@@
 			)
 		)
-		(property "Footprint" "0402 (1005 Metric)"
+		(property "Footprint" "copy_ref:R_0402_1005Metric"
 			(at 28.702 229.87 90)
 			(hide yes)
@@
 			)
 		)
-		(property "Footprint" "SOT-363"
+		(property "Footprint" "copy_ref:SOT-363_SC-70-6"
 			(at 119.38 83.82 0)
 			(hide yes)
@@
 			)
 		)
-		(property "Footprint" "SOT-363"
+		(property "Footprint" "copy_ref:SOT-363_SC-70-6"
 			(at 119.38 68.58 0)
 			(hide yes)
@@
 			)
 		)
-		(property "Footprint" "SOT-323"
+		(property "Footprint" "Package_TO_SOT_SMD:SOT-323_SC-70"
 			(at 308.61 154.305 0)
 			(hide yes)
@@
 			)
 		)
-		(property "Footprint" "0402 (1005 Metric)"
+		(property "Footprint" "copy_ref:R_0402_1005Metric"
 			(at 297.18 216.662 90)
 			(hide yes)
@@
 			)
 		)
-		(property "Footprint" "0805 (2012 Metric)"
+		(property "Footprint" "copy_ref:C_0805_2012Metric"
 			(at 294.9448 168.91 0)
 			(hide yes)
@@
 			)
 		)
-		(property "Footprint" "1210 (3225 Metric)"
+		(property "Footprint" "Resistor_SMD:R_1210_3225Metric"
 			(at 267.462 45.72 90)
 			(hide yes)
@@
 			)
 		)
-		(property "Footprint" "SOT-363"
+		(property "Footprint" "copy_ref:SOT-363_SC-70-6"
 			(at 119.38 22.86 0)
 			(hide yes)
@@
 			)
 		)
-		(property "Footprint" "0402 (1005 Metric)"
+		(property "Footprint" "copy_ref:R_0402_1005Metric"
 			(at 205.232 71.12 90)
 			(hide yes)
@@
 			)
 		)
-		(property "Footprint" "0402 (1005 Metric)"
+		(property "Footprint" "copy_ref:R_0402_1005Metric"
 			(at 307.848 172.72 90)
 			(hide yes)
@@
 			)
 		)
-		(property "Footprint" "0402 (1005 Metric)"
+		(property "Footprint" "copy_ref:R_0402_1005Metric"
 			(at 198.628 71.12 90)
 			(hide yes)
@@
 			)
 		)
-		(property "Footprint" "0402 (1005 Metric)"
+		(property "Footprint" "copy_ref:C_0402_1005Metric"
 			(at 46.0248 243.84 0)
 			(hide yes)
@@
 			)
 		)
-		(property "Footprint" "0402 (1005 Metric)"
+		(property "Footprint" "copy_ref:R_0402_1005Metric"
 			(at 318.77 165.862 90)
 			(hide yes)
@@
 			)
 		)
-		(property "Footprint" "0402 (1005 Metric)"
+		(property "Footprint" "copy_ref:R_0402_1005Metric"
 			(at 71.12 195.072 90)
 			(hide yes)
@@
 			)
 		)
-		(property "Footprint" "0402 (1005 Metric)"
+		(property "Footprint" "copy_ref:R_0402_1005Metric"
 			(at 329.438 173.99 90)
 			(hide yes)
@@
 			)
 		)
-		(property "Footprint" "0402 (1005 Metric)"
+		(property "Footprint" "copy_ref:R_0402_1005Metric"
 			(at 250.952 226.06 90)
 			(hide yes)
@@
 			)
 		)
-		(property "Footprint" "8-VSSOP"
+		(property "Footprint" "dowload:LMV393"
 			(at 113.03 236.22 0)
 			(hide yes)
@@
 			)
 		)
-		(property "Footprint" "SOT-323"
+		(property "Footprint" "Package_TO_SOT_SMD:SOT-323_SC-70"
 			(at 334.01 212.725 0)
 			(hide yes)
@@
 			)
 		)
-		(property "Footprint" "0402 (1005 Metric)"
+		(property "Footprint" "copy_ref:C_0402_1005Metric"
 			(at 68.8848 251.46 0)
 			(hide yes)
@@
 			)
 		)
-		(property "Footprint" "0402 (1005 Metric)"
+		(property "Footprint" "copy_ref:R_0402_1005Metric"
 			(at 109.22 126.238 90)
 			(hide yes)
@@
 			)
 		)
-		(property "Footprint" "0402 (1005 Metric)"
+		(property "Footprint" "copy_ref:R_0402_1005Metric"
 			(at 107.95 36.322 90)
 			(hide yes)
@@
 			)
 		)
-		(property "Footprint" "SOT-363"
+		(property "Footprint" "copy_ref:SOT-363_SC-70-6"
 			(at 120.65 124.46 0)
 			(hide yes)
@@
 			)
 		)
-		(property "Footprint" "0402 (1005 Metric)"
+		(property "Footprint" "copy_ref:C_0402_1005Metric"
 			(at 46.0248 223.52 0)
 			(hide yes)
@@
 			)
 		)
-		(property "Footprint" "SMD, J-Lead"
+		(property "Footprint" "dowload:KCM55QR72A106KH01L"
 			(at 313.3852 58.42 0)
 			(hide yes)
@@
 			)
 		)
-		(property "Footprint" "8-PowerWDFN"
+		(property "Footprint" "dowload:8-PowerWDFN"
 			(at 281.178 106.426 0)
 			(hide yes)
@@
 			)
 		)
-		(property "Footprint" "0402 (1005 Metric)"
+		(property "Footprint" "copy_ref:R_0402_1005Metric"
 			(at 225.298 69.85 90)
 			(hide yes)
@@
 			)
 		)
-		(property "Footprint" "1206 (3216 Metric)"
+		(property "Footprint" "copy_ref:R_1206_3216Metric"
 			(at 384.81 42.672 90)
 			(hide yes)
@@
 			)
 		)
-		(property "Footprint" "12-MLP"
+		(property "Footprint" "copy_ref:IC_FDMQ8205A"
 			(at 151.13 129.54 0)
 			(hide yes)
@@
 			)
 		)
-		(property "Footprint" "0402 (1005 Metric)"
+		(property "Footprint" "copy_ref:R_0402_1005Metric"
 			(at 109.22 156.718 90)
 			(hide yes)
@@
 			)
 		)
-		(property "Footprint" "SOT-323"
+		(property "Footprint" "Package_TO_SOT_SMD:SOT-323_SC-70"
 			(at 265.43 219.075 0)
 			(hide yes)
@@
 			)
 		)
-		(property "Footprint" "0402 (1005 Metric)"
+		(property "Footprint" "copy_ref:R_0402_1005Metric"
 			(at 97.282 209.55 90)
 			(hide yes)
@@
 			)
 		)
-		(property "Footprint" "SOT-23-3 (TO-236)"
+		(property "Footprint" "copy_ref:SOT-23-3"
 			(at 252.73 149.86 0)
 			(hide yes)
@@
 			)
 		)
-		(property "Footprint" "16-TSSOP"
+		(property "Footprint" "dowload:TSSOP-16_948F-01_OSI"
 			(at 226.06 54.61 0)
 			(hide yes)
@@
 			)
 		)
-		(property "Footprint" "0402 (1005 Metric)"
+		(property "Footprint" "copy_ref:R_0402_1005Metric"
 			(at 309.372 201.93 90)
 			(hide yes)
@@
 			)
 		)
-		(property "Footprint" "SOT-363"
+		(property "Footprint" "copy_ref:SOT-363_SC-70-6"
 			(at 120.65 170.18 0)
 			(hide yes)
@@
 			)
 		)
-		(property "Footprint" "0402 (1005 Metric)"
+		(property "Footprint" "copy_ref:C_0402_1005Metric"
 			(at 387.0452 88.9 0)
 			(hide yes)
@@
 			)
 		)
-		(property "Footprint" "0402 (1005 Metric)"
+		(property "Footprint" "copy_ref:R_0402_1005Metric"
 			(at 318.77 209.042 90)
 			(hide yes)
@@
 			)
 		)
-		(property "Footprint" "8-VSSOP"
+		(property "Footprint" "dowload:LMV393"
 			(at 73.66 217.17 0)
 			(hide yes)
@@
 			)
 		)
-		(property "Footprint" "SOT-363"
+		(property "Footprint" "copy_ref:SOT-363_SC-70-6"
 			(at 120.65 154.94 0)
 			(hide yes)
@@
 			)
 		)
-		(property "Footprint" "1206 (3216 Metric)"
+		(property "Footprint" "copy_ref:R_1206_3216Metric"
 			(at 28.702 195.58 90)
 			(hide yes)
@@
 			)
 		)
-		(property "Footprint" "0402 (1005 Metric)"
+		(property "Footprint" "copy_ref:R_0402_1005Metric"
 			(at 87.63 215.392 90)
 			(hide yes)
@@
 			)
 		)
-		(property "Footprint" "0402 (1005 Metric)"
+		(property "Footprint" "copy_ref:R_0402_1005Metric"
 			(at 28.702 205.74 90)
 			(hide yes)
@@
 			)
 		)
-		(property "Footprint" "0402 (1005 Metric)"
+		(property "Footprint" "copy_ref:R_0402_1005Metric"
 			(at 250.952 135.89 90)
 			(hide yes)
@@
 			)
 		)
-		(property "Footprint" "SOT-323"
+		(property "Footprint" "Package_TO_SOT_SMD:SOT-323_SC-70"
 			(at 313.69 220.345 0)
 			(hide yes)
@@
 			)
 		)
-		(property "Footprint" "0402 (1005 Metric)"
+		(property "Footprint" "copy_ref:C_0402_1005Metric"
 			(at 214.9348 72.39 0)
 			(hide yes)
@@
 			)
 		)
-		(property "Footprint" "8-VSSOP"
+		(property "Footprint" "dowload:LMV393"
 			(at 83.82 247.65 0)
 			(hide yes)
