File: hardware/ntp-server-stm32/spi-peripherals.kicad_sch (KiCad schematic)
At the start: 12 parts, among them U62 MX25L25645GM2I-08G, U63 PCA9306DCTT

Commit message: Updates
Parts:
- C179: footprint C_0402_1005Metric -> 0402 (1005 Metric); DIELECTRIC (none) -> X7R; DIGIKEY_PART_NUMBER 490-6328-2-ND -> 490-4759-1-ND; MANUFACTURER_PART_NUMBER GRM155R71C104KA88J -> GCM155R71C104KA55D; TOLERANCE (none) -> 10%; VOLTAGE (none) -> 16V
- R204, R205, R206, R207, R208, R209, R212: footprint R_0402_1005Metric -> 0402 (1005 Metric); DIELECTRIC (none) -> Thick-film; DIGIKEY_PART_NUMBER (none) -> P10.0KLCT-ND; MANUFACTURER Panasonic -> Panasonic Industry; POWER (none) -> 1/10W; TOLERANCE (none) -> 1%
- R210, R211: footprint R_0402_1005Metric -> 0402 (1005 Metric); DIELECTRIC (none) -> Thick-film; DIGIKEY_PART_NUMBER 273-KDV08DR150ETCT-ND -> P22.0LCT-ND; MANUFACTURER Panasonic -> Panasonic Industry; POWER (none) -> 1/10W; TOLERANCE (none) -> 1%
- U62: MANUFACTURER (none) -> Macronix
- U63: MANUFACTURER (none) -> Texas Instruments
Connections:
- net 3V3_STM: now also U62.8 (VCC); no longer U62. (VCC)
Other:
- note added: "Place resistors where traces branch away from U62 and U63 towards the connector"
- note removed: "Place resistors where traces branch away from U55 and U35 towards the connector"

Commit message: Bom updates
Parts:
- U62: footprint (none) -> 8-SOIC; DIGIKEY_PART_NUMBER (none) -> 1092-1234-ND
- U63: DIGIKEY_PART_NUMBER (none) -> 296-32200-1-ND
Changed lines of the file:
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@@
 			)
 		)
-		(property "Footprint" ""
+		(property "Footprint" "8-SOIC"
 			(at 129.54 86.36 0)
 			(hide yes)
@@
 			)
 		)
-		(property "Datasheet" ""
+		(property "Datasheet" "https://www.mxic.com.tw/Lists/Datasheet/Attachments/8906/MX25L25645G,%203V,%20256Mb,%20v2.0.pdf"
 			(at 129.54 86.36 0)
 			(hide yes)
@@
 		(property "MANUFACTURER_PART_NUMBER" "MX25L25645GM2I-08G"
 			(at 0 0 0)
+			(hide yes)
+			(show_name no)
+			(do_not_autoplace no)
+			(effects
+				(font
+					(size 1.27 1.27)
+				)
+			)
+		)
+		(property "DIGIKEY_PART_NUMBER" "1092-1234-ND"
+			(at 129.54 86.36 0)
 			(hide yes)
 			(show_name no)
@@
 			(hide yes)
 			(show_name no)
+			(do_not_autoplace no)
+			(effects
+				(font
+					(size 1.27 1.27)
+				)
+			)
+		)
+		(property "DIGIKEY_PART_NUMBER" "296-32200-1-ND"
+			(at 154.94 207.01 0)
+			(hide yes)
+			(show_name no)

Commit message: Bom updates
Parts:
- U63: footprint DCT8 -> sts1000:DCT8
Changed lines of the file:
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@@
 			)
 		)
-		(property "Footprint" "DCT8"
+		(property "Footprint" "sts1000:DCT8"
 			(at 154.94 207.01 0)
 			(hide yes)

Commit message: Add files via upload
Updated, completed placement
Parts:
- C179: footprint 0402 (1005 Metric) -> copy_ref:C_0402_1005Metric
- R204, R205, R206, R207, R208, R209, R210, R211, R212: footprint 0402 (1005 Metric) -> copy_ref:R_0402_1005Metric
- U62: footprint 8-SOIC -> copy_ref:SOIC-8_3.9x4.9mm_P1.27mm
Changed lines of the file:
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@@
 			)
 		)
-		(property "Footprint" "0402 (1005 Metric)"
+		(property "Footprint" "copy_ref:R_0402_1005Metric"
 			(at 152.4 109.982 90)
 			(hide yes)
@@
 			)
 		)
-		(property "Footprint" "0402 (1005 Metric)"
+		(property "Footprint" "copy_ref:R_0402_1005Metric"
 			(at 152.4 116.078 90)
 			(hide yes)
@@
 			)
 		)
-		(property "Footprint" "0402 (1005 Metric)"
+		(property "Footprint" "copy_ref:R_0402_1005Metric"
 			(at 107.442 226.06 90)
 			(hide yes)
@@
 			)
 		)
-		(property "Footprint" "0402 (1005 Metric)"
+		(property "Footprint" "copy_ref:R_0402_1005Metric"
 			(at 98.552 66.04 90)
 			(hide yes)
@@
 			)
 		)
-		(property "Footprint" "0402 (1005 Metric)"
+		(property "Footprint" "copy_ref:R_0402_1005Metric"
 			(at 97.282 201.93 90)
 			(hide yes)
@@
 			)
 		)
-		(property "Footprint" "0402 (1005 Metric)"
+		(property "Footprint" "copy_ref:R_0402_1005Metric"
 			(at 90.932 90.17 90)
 			(hide yes)
@@
 			)
 		)
-		(property "Footprint" "0402 (1005 Metric)"
+		(property "Footprint" "copy_ref:R_0402_1005Metric"
 			(at 107.442 201.93 90)
 			(hide yes)
@@
 			)
 		)
-		(property "Footprint" "0402 (1005 Metric)"
+		(property "Footprint" "copy_ref:R_0402_1005Metric"
 			(at 87.122 201.93 90)
 			(hide yes)
@@
 			)
 		)
-		(property "Footprint" "8-SOIC"
+		(property "Footprint" "copy_ref:SOIC-8_3.9x4.9mm_P1.27mm"
 			(at 129.54 86.36 0)
 			(hide yes)
@@
 			)
 		)
-		(property "Footprint" "0402 (1005 Metric)"
+		(property "Footprint" "copy_ref:C_0402_1005Metric"
 			(at 147.0152 62.23 0)
 			(hide yes)
@@
 			)
 		)
-		(property "Footprint" "0402 (1005 Metric)"
+		(property "Footprint" "copy_ref:R_0402_1005Metric"
 			(at 159.512 58.42 90)
 			(hide yes)
