File: hardware/ntp-server-stm32/ntp-server-stm32.kicad_pcb (KiCad board)
At the start: 6 copper layers, 101.3 x 138.2 mm, 615 parts, among them J1 0826-1X1T-HS-F, J10 OSTVN02A150, J15 SMA-J-P-H-RA-TH1, J16 OSTVN06A150, J17 1787179, J2 OSTVN04A150, J3 BG055-06A-1-0450-0530-0350-L-D, J5 USB4120-03-C, J6 622-009-260-033, J7 SMA-J-P-H-RA-TH1, J8 SMA-J-P-H-RA-TH1, J9 SMA-J-P-H-RA-TH1, Q1 BC847W, Q10 BC847W, Q11 NSS40300MZ4T1G, Q12 BC857W, Q13 BC857W, Q14 BC847W, Q15 BC847W, Q16 BC847W, Q17 BC857W, Q18 BC847W, Q19 BC847W, Q20 BC847W, Q21 BC847W, Q22 NSS40300MZ4T1G, Q23 BC847W, Q24 BC847W, Q26 BC847W, Q3 BC857W, Q4 BC847W, Q5 BC847W, Q6 BC847W, Q7 BC847W, Q8 BC847W, Q9 BC847W, U1 TPD4EUSB30, U10 INA228AQDGSRQ1, U11 LAN8742AI-CZ-TR, U12 STM32H563ZIT6, U13 LT3045xDD, U14 MCP1502T-33E/CHY, U15 TPD4E02B04DQAR, U16 TPD4E02B04DQAR, U17 TPD4E05U06DQAR, U18 TPD4E05U06DQAR, U19 TPD4E02B04DQAR, U2 LMV393, U20 TPD4E02B04DQAR, U21 ZED-F9T-00B, U22 LT3045xDD, U23 INA228AQDGSRQ1, U24 INA181A1IDBVR, U25 LMV393, U26 INA228AQDGSRQ1, U27 RT9742VGJ5, U3 BC846BPDW1T1G, U30 INA228AQDGSRQ1, U31 INA228AQDGSRQ1, U32 INA228AQDGSRQ1, U33 RT9742VGJ5, U34 TPS61094DSSR, U35 TPS61094DSSR, U36 OPA320AIDBVT, U37 INA228AQDGSRQ1, U39 TPS7A5201QRGRRQ1, U4 BC846BPDW1T1G, U41 LMV393, U42 OPA320AIDBVT, U43 MCP41U83T-503E/ST, U44 INA228AQDGSRQ1, U45 MCP1502T-30E/CHY, U46 SN65C3221EPWR, U47 PESD15VL2BT, U49 TMUX1101DCK, U5 BC846BPDW1T1G, U50 LTC6752xS5, U51 LT3045xDD, U52 74LVC1G157GW-Q100H, U53 74LVC1G34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

Commit message: Add files via upload
current placement
Parts:
- added C10: 10uF, dowload:KCM55QR72A106KH01L, F.Cu at (111.0, 164.8)
- added C126: 47uF, dowload:KCM55WR71H476MH13L, F.Cu at (25.4, 159.8)
- added C127: 47uF, dowload:KCM55WR71H476MH13L, F.Cu at (32.0, 159.8)
- added C128: 47uF, dowload:KCM55WR71H476MH13L, F.Cu at (38.6, 159.8)
- added C90: 3F, dowload:DSF305Q3R0, F.Cu at (109.2, 105.9)
- added C91: 3F, dowload:DSF305Q3R0, F.Cu at (97.8, 105.9)
- added D11: BAS16W, dowload:SOD-123, F.Cu at (55.8, 135.3)
- added D13: SMAJ15CA, dowload:DO-214AC, F.Cu at (135.0, 101.5)
- added D14: SMAJ15CA, dowload:DO-214AC, F.Cu at (142.3, 101.5)
- added D22: SMF5V0A, dowload:DO-219AB (SMF), B.Cu at (60.0, 93.6)
- added D23: SZESD7410MXWT5G, dowload:2-XDFN, F.Cu at (148.6, 135.1)
- added D26: SMAJ15CA, dowload:DO-214AC, F.Cu at (127.7, 101.5)
- added D8: SZESD7410MXWT5G, dowload:2-XDFN, F.Cu at (147.9, 102.1)
- added D9: SZESD7410MXWT5G, dowload:2-XDFN, F.Cu at (148.6, 118.7)
- added K1: G6K-2F-Y_DC3_OMR, dowload:G6K-2F-Y DC3, F.Cu at (122.7, 108.0)
- added K2: G6K-2F-Y_DC3_OMR, dowload:G6K-2F-Y DC3, F.Cu at (80.2, 176.8)
- added L2: 6.8uH, dowload:SRP1265A-6R8M, F.Cu at (58.4, 173.8)
- added L3: 2.2uH, dowload:DR73-2R2-R, F.Cu at (59.8, 157.6)
- added L4: 2.2uH, dowload:DR73-2R2-R, F.Cu at (110.2, 114.7)
- added L5: 2.2uH, dowload:DR73-2R2-R, F.Cu at (98.8, 114.7)
- added L6: 2.2uH, dowload:DR73-2R2-R, F.Cu at (38.5, 149.6)
- added L7: 39uH, dowload:7447709390, F.Cu at (48.4, 161.0)
- added Q2: FDMC8622, dowload:8-PowerWDFN, B.Cu at (97.0, 175.3)
- added Q25: SI7469DP-T1-E3, dowload:PowerPAKÂ® SO-8, F.Cu at (25.8, 178.6)
- added U28: MIC28516T-E/PHA, copy_ref:MIC28516T-EPHA, F.Cu at (70.2, 166.8)
- added U29: AP3441SHE-7B, dowload:AP3441SHE-7B_DIO-M, F.Cu at (66.6, 155.2)
- added U38: AP3441SHE-7B, dowload:AP3441SHE-7B_DIO-M, F.Cu at (31.6, 150.2)
- added U40: MIC28516T-E/PHA, copy_ref:MIC28516T-EPHA, F.Cu at (38.8, 170.8)
- added U48: APC-817C1, dowload:APC817C1SL, B.Cu at (118.6, 108.0)
- added U68: 74LVC2G17, dowload:74LVC2G17GW,125, F.Cu at (220.4, 208.4)
- added U71: 74LVC1G34, dowload:74LVC1G34GW_125, F.Cu at (107.9, 141.1)
- added Y1: 25MHz, dowload:445I23E25M00000, F.Cu at (108.7, 148.9)
- added Y2: 32.768kHz, dowload:ABS07-32.768KHZ-1-T, F.Cu at (94.1, 126.0)
- C137, C146, C147, C15, C172, C188, C189, C190, C191, C192, C40, C41, C6, C64, C8, C92, C93, CR1, D1, D16, D17, D2, D25, D3, FB11, Q11, Q24, Q26, R10, R11, R12, R13, R14, R143, R15, R16, R162, R163, R171, R172, R20, R228, R229, R230, R232, R233, R237, R238, R239, R240, R241, R242, R243, R244, R245, R246, R259, R260, R261, R262, R263, R264, R49, R64, R73, R9, U3, U4, U5, U58, U6, U9: moved to B.Cu
- U15, U16, U19, U20: value TPD4E02B04DQAR -> DQA0010A
- U2, U25, U41: value LMV393 -> DGK8
- U53: footprint Package_TO_SOT_SMD:SOT-23-5 -> dowload:74LVC1G34GW_125
- U67: value LMV393 -> DGK8; moved to B.Cu
- U7, U8: value FDMQ8205A -> MLP_4p5X5_ONS; moved to B.Cu
- Y3: footprint Oscillator:Oscillator_SMD_OCXO_ConnorWinfield_OH300 -> copy_ref:Oscillator_SMD_OCXO_ConnorWinfield_OH300
- moved C79 221.7 mm to (47.3, 214.9)
- moved C81 221.7 mm to (47.3, 217.9)
- moved C82 221.6 mm to (47.3, 221.0)
- moved R103 206.4 mm to (57.0, 218.4)
- moved D24 202.0 mm to (73.6, 177.2), turned to 90 degrees
- moved R1 201.9 mm to (129.8, 199.6)
- moved R259 200.9 mm to (73.6, 178.6)
- moved C1 200.5 mm to (131.9, 196.1)
- moved R260 200.4 mm to (73.6, 179.8)
- moved Q24 200.1 mm to (73.6, 176.3), turned to 90 degrees
- moved C18 199.4 mm to (103.9, 150.9), turned to 90 degrees
- moved R38 199.2 mm to (125.4, 180.5), turned to 180 degrees
- moved C15 197.0 mm to (107.3, 154.8), turned to -90 degrees
- moved R49 196.3 mm to (104.7, 154.1)
- moved R101 196.0 mm to (57.0, 216.4)
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Routing:
- net GPS_RF_IN: track 0.00 -> 18.2 mm
- net VOUT_N: track 0.00 -> 17.7 mm, vias 0 -> 8
- net VOUT_P: track 0.00 -> 14.8 mm, vias 0 -> 5
- net TRD0_P: track 0.00 -> 13.6 mm
- net TRD0_N: track 0.00 -> 12.8 mm
- net Net-(Q2-S): track 0.00 -> 9.85 mm, vias 0 -> 3
- net TRD1_P: track 0.00 -> 9.67 mm
- net TR3_TAP: track 0.00 -> 9.66 mm, vias 0 -> 3
- net TR1_TAP: track 0.00 -> 8.98 mm, vias 0 -> 3
- net TRD1_N: track 0.00 -> 8.92 mm
- net TR2_TAP: track 0.00 -> 7.53 mm, vias 0 -> 3
- net GBR: track 0.00 -> 6.88 mm
- net 10MHz_RF_IN: track 0.00 -> 6.76 mm
- net TR0_TAP: track 0.00 -> 6.35 mm, vias 0 -> 3
- net Net-(R11-Pad2): track 0.00 -> 5.61 mm
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Other:
- board size 101.3 x 138.2 mm -> 138.2 x 101.3 mm
