File: hardware/ntp-server-stm32/ntp-server-stm32.kicad_pcb (KiCad board)
At the start: 6 copper layers, 138.2 x 101.3 mm, 648 parts, among them J1 0826-1X1T-HS-F, J10 OSTVN02A150, J15 SMA-J-P-H-RA-TH1, J16 OSTVN06A150, J17 1787179, J2 OSTVN04A150, J3 BG055-06A-1-0450-0530-0350-L-D, J5 USB4120-03-C, J6 622-009-260-033, J7 SMA-J-P-H-RA-TH1, J8 SMA-J-P-H-RA-TH1, J9 SMA-J-P-H-RA-TH1, K1 G6K-2F-Y_DC3_OMR, K2 G6K-2F-Y_DC3_OMR, Q1 BC847W, Q10 BC847W, Q11 NSS40300MZ4T1G, Q12 BC857W, Q13 BC857W, Q14 BC847W, Q15 BC847W, Q16 BC847W, Q17 BC857W, Q18 BC847W, Q19 BC847W, Q2 FDMC8622, Q20 BC847W, Q21 BC847W, Q22 NSS40300MZ4T1G, Q23 BC847W, Q24 BC847W, Q25 SI7469DP-T1-E3, Q26 BC847W, Q3 BC857W, Q4 BC847W, Q5 BC847W, Q6 BC847W, Q7 BC847W, Q8 BC847W, Q9 BC847W, U1 TPD4EUSB30, U10 INA228AQDGSRQ1, U11 LAN8742AI-CZ-TR, U12 STM32H563ZIT6, U13 LT3045xDD, U14 MCP1502T-33E/CHY, U15 DQA0010A, U16 DQA0010A, U17 TPD4E05U06DQAR, U18 TPD4E05U06DQAR, U19 DQA0010A, U2 DGK8, U20 DQA0010A, U21 ZED-F9T-00B, U22 LT3045xDD, U23 INA228AQDGSRQ1, U24 INA181A1IDBVR, U25 DGK8, U26 INA228AQDGSRQ1, U27 RT9742VGJ5, U28 MIC28516T-E/PHA, U29 AP3441SHE-7B, U3 BC846BPDW1T1G, U30 INA228AQDGSRQ1, U31 INA228AQDGSRQ1, U32 INA228AQDGSRQ1, U33 RT9742VGJ5, U34 TPS61094DSSR, U35 TPS61094DSSR, U36 OPA320AIDBVT, U37 INA228AQDGSRQ1, U38 AP3441SHE-7B, U39 TPS7A5201QRGRRQ1, U4 BC846BPDW1T1G, U40 MIC28516T-E/PHA, U41 DGK8, U42 OPA320AIDBVT, U43 MCP41U83T-503E/ST, U44 INA228AQDGSRQ1, U45 MCP1502T-30E/CHY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

Commit message: Add files via upload
Updated, completed placement
Parts:
- C120, C122, C148, C161, C162, C163, C164, C165, C166, C167, C179, C182, C187, C2, C201, C202, C3, C4, C74, C78, C79, C82, D7, FB8, Q10, Q17, Q18, Q19, Q20, Q22, Q23, Q7, Q8, Q9, R101, R103, R108, R109, R110, R111, R116, R117, R134, R136, R137, R138, R139, R142, R150, R151, R152, R153, R154, R155, R156, R157, R158, R160, R161, R173, R2, R202, R203, R205, R207, R210, R211, R212, R216, R217, R221, R222, R223, R224, R225, R226, R227, R234, R235, R265, R3, R4, R46, R5, R53, R54, R55, R56, R57, R58, R59, R60, R61, R62, R63, R65, R66, R92, R94, U42, U62: moved to B.Cu
- C146, C147, C172, U58: moved to F.Cu
- U7, U8: value MLP_4p5X5_ONS -> FDMQ8205A; footprint dowload:FDMQ8205A -> copy_ref:IC_FDMQ8205A
- moved R201 210.6 mm to (27.7, 108.8), turned to 90 degrees
- moved R198 209.5 mm to (27.7, 110.9), turned to 90 degrees
- moved U55 203.9 mm to (30.1, 109.8), turned to -90 degrees
- moved C202 203.2 mm to (42.8, 183.5), turned to 90 degrees
- moved C201 203.1 mm to (44.0, 183.5), turned to 90 degrees
- moved C168 202.3 mm to (33.2, 110.1), turned to -90 degrees
- moved R254 199.9 mm to (42.8, 183.5), turned to -90 degrees
- moved R190 195.8 mm to (44.0, 183.5), turned to -90 degrees
- moved U54 195.5 mm to (37.6, 113.3), turned to 90 degrees
- moved R199 192.2 mm to (36.8, 108.1)
- moved U68 189.9 mm to (60.4, 106.2)
- moved U63 189.3 mm to (49.4, 105.1), turned to -90 degrees
- moved C193 188.3 mm to (63.3, 106.3)
- moved C169 187.4 mm to (40.1, 112.1), turned to -90 degrees
- moved FB12 186.6 mm to (41.6, 108.1), turned to 180 degrees
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Routing:
- net VCC_RB: track 0.00 -> 8.39 mm
- net Net-(U44-IN+): track 0.00 -> 6.99 mm
- net GND: vias 1 -> 24
