File: hardware/ntp-server-stm32/ntp-server-stm32.kicad_pcb (KiCad board)
At the start: 6 copper layers, 138.2 x 101.3 mm, 648 parts, among them J1 0826-1X1T-HS-F, J10 OSTVN02A150, J15 SMA-J-P-H-RA-TH1, J16 OSTVN06A150, J17 1787179, J2 OSTVN04A150, J3 BG055-06A-1-0450-0530-0350-L-D, J5 USB4120-03-C, J6 622-009-260-033, J7 SMA-J-P-H-RA-TH1, J8 SMA-J-P-H-RA-TH1, J9 SMA-J-P-H-RA-TH1, K1 G6K-2F-Y_DC3_OMR, K2 G6K-2F-Y_DC3_OMR, Q1 BC847W, Q10 BC847W, Q11 NSS40300MZ4T1G, Q12 BC857W, Q13 BC857W, Q14 BC847W, Q15 BC847W, Q16 BC847W, Q17 BC857W, Q18 BC847W, Q19 BC847W, Q2 FDMC8622, Q20 BC847W, Q21 BC847W, Q22 NSS40300MZ4T1G, Q23 BC847W, Q24 BC847W, Q25 SI7469DP-T1-E3, Q26 BC847W, Q3 BC857W, Q4 BC847W, Q5 BC847W, Q6 BC847W, Q7 BC847W, Q8 BC847W, Q9 BC847W, U1 TPD4EUSB30, U10 INA228AQDGSRQ1, U11 LAN8742AI-CZ-TR, U12 STM32H563ZIT6, U13 LT3045xDD, U14 MCP1502T-33E/CHY, U15 DQA0010A, U16 DQA0010A, U17 TPD4E05U06DQAR, U18 TPD4E05U06DQAR, U19 DQA0010A, U2 DGK8, U20 DQA0010A, U21 ZED-F9T-00B, U22 LT3045xDD, U23 INA228AQDGSRQ1, U24 INA181A1IDBVR, U25 DGK8, U26 INA228AQDGSRQ1, U27 RT9742VGJ5, U28 MIC28516T-E/PHA, U29 AP3441SHE-7B, U3 BC846BPDW1T1G, U30 INA228AQDGSRQ1, U31 INA228AQDGSRQ1, U32 INA228AQDGSRQ1, U33 RT9742VGJ5, U34 TPS61094DSSR, U35 TPS61094DSSR, U36 OPA320AIDBVT, U37 INA228AQDGSRQ1, U38 AP3441SHE-7B, U39 TPS7A5201QRGRRQ1, U4 BC846BPDW1T1G, U40 MIC28516T-E/PHA, U41 DGK8, U42 OPA320AIDBVT, U43 MCP41U83T-503E/ST, U44 INA228AQDGSRQ1, U45 MCP1502T-30E/CHY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

Commit message: Add files via upload
Completed PCB
Parts:
- C116, C172, C34, C36, D23, D9, R188, R254, R37, R95, U58: moved to B.Cu
- C179, C187, C201, C202, C8, CR1, Q22, Q23, R202, R203, R205, R207, R210, R211, R212, R216, R217, R234, R235, R46, R64, R65, R66, R94, U62: moved to F.Cu
- H1, H10, H11, H12, H13, H14, H2, H3, H4, H5, H6, H7, H8, H9: footprint copy_ref:MountingHole_3.2mm_M3 -> MountingHole:MountingHole_3.2mm_M3_Pad
- U32: value INA228AQDGSRQ1 -> RT9742VGJ5
- U52: footprint sts1000:SC-74_TSOP6_SOT457_NEX -> dowload:SOT-363-6_2P2X1P35_ONS
- moved R190 91.1 mm to (91.1, 105.5), turned to 90 degrees
- moved U16 83.2 mm to (35.0, 102.9), turned to -90 degrees
- moved C201 78.8 mm to (33.6, 105.4), turned to -90 degrees
- moved C202 78.5 mm to (34.7, 105.4), turned to -90 degrees
- moved R254 78.5 mm to (34.7, 105.4), turned to 90 degrees
- moved U58 51.0 mm to (60.9, 123.3)
- moved C172 50.8 mm to (60.4, 121.2), turned to 180 degrees
- moved R203 38.6 mm to (102.6, 135.9), turned to 180 degrees
- moved R202 37.3 mm to (102.6, 137.6), turned to 180 degrees
- moved C161 30.9 mm to (91.1, 105.5)
- moved R207 29.9 mm to (62.8, 150.4), turned to 90 degrees
- moved C1 26.7 mm to (146.7, 185.6), turned to -90 degrees
- moved R212 26.1 mm to (62.8, 146.9)
- moved R1 25.8 mm to (149.4, 184.6), turned to -90 degrees
- moved U62 23.0 mm to (67.2, 149.3), turned to 0 degrees
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Connections:
- net USB_DM renamed USB_D-
- net USB_DP renamed USB_D+
Routing:
- net GND: track 1.21 -> 1110.9 mm, vias 24 -> 671
- net I2C_SDA: track 0.00 -> 458.6 mm, vias 0 -> 15
- net I2C_SCL: track 0.00 -> 455.1 mm, vias 0 -> 15
- net 3V3: track 0.00 -> 269.1 mm, vias 0 -> 41
- net RTC_TAMPER: track 0.00 -> 229.7 mm, vias 0 -> 3
- net 5V_PSU_PG: track 0.00 -> 223.7 mm, vias 0 -> 7
- net 3V3_STM: track 0.00 -> 174.2 mm, vias 0 -> 61
- net INA_ALERT_5V_DISP: track 0.00 -> 156.6 mm, vias 0 -> 3
- net OCXO_PSU_PG: track 0.00 -> 137.2 mm, vias 0 -> 4
- net V_ANT_EN_FAULT: track 0.00 -> 136.9 mm, vias 0 -> 2
- net USB_VBUS_SENSE: track 0.00 -> 135.9 mm, vias 0 -> 4
- net 10MHz_CLK_OUT: track 0.00 -> 135.6 mm, vias 0 -> 2
- net 5V: track 0.00 -> 129.3 mm, vias 0 -> 47
- net MCU_NRST: track 0.00 -> 129.0 mm, vias 0 -> 3
- net USB_D+: track 0.00 -> 128.6 mm, vias 0 -> 4
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- added copper zone on In4.Cu, net 3V0_RF
- added copper zone on B.Cu, net 3V3
- added copper zone on F.Cu, net 3V3
- added copper zone on In2.Cu, net 3V3
- added copper zone on In3.Cu, net 3V3
- added copper zone on B.Cu, net 3V3_GPS
- added copper zone on In3.Cu, net 3V3_STM
- added copper zone on B.Cu, net 5V
- added copper zone on F.Cu, net 5V
- added copper zone on In4.Cu, net 5V
- added copper zone on B.Cu, net 5V_DISP
- added copper zone on F.Cu, net 5V_DISP
- added copper zone on In4.Cu, net 5V_DISP
- added copper zone on B.Cu, net GND
- added copper zone on F.Cu, net GND
- added copper zone on In1.Cu, net GND
- added copper zone on In4.Cu, net GND
- added copper zone on B.Cu, net GPS_VBAT
- added copper zone on F.Cu, net GPS_VBAT
- added copper zone on F.Cu, net Net-(C124-Pad2)
- added copper zone on F.Cu, net Net-(C68-Pad2)
- added copper zone on F.Cu, net Net-(D10-A)
- added copper zone on F.Cu, net Net-(D10-K)
- added copper zone on B.Cu, net Net-(Q2-S)
- added copper zone on F.Cu, net Net-(U22-OUT)
- added copper zone on F.Cu, net Net-(U26-IN+)
- added copper zone on F.Cu, net Net-(U26-IN-)
- added copper zone on F.Cu, net Net-(U29-LX)
- added copper zone on B.Cu, net Net-(U30-IN+)
- added copper zone on F.Cu, net Net-(U30-IN+)
- added copper zone on F.Cu, net Net-(U32-IN+)
- added copper zone on F.Cu, net Net-(U32-IN-)
- added copper zone on F.Cu, net Net-(U34-SUP)
- added copper zone on F.Cu, net Net-(U34-SW)
- added copper zone on F.Cu, net Net-(U35-SUP)
- added copper zone on F.Cu, net Net-(U35-SW)
- added copper zone on F.Cu, net Net-(U37-IN-)
- added copper zone on F.Cu, net Net-(U44-IN+)
- added copper zone on B.Cu, net STM_VBAT
- added copper zone on F.Cu, net STM_VBAT
- added copper zone on F.Cu, net VCC_RB
- added copper zone on F.Cu, net VCC_RB_G
- added copper zone on In3.Cu, net VCC_RB_G
- added copper zone on F.Cu, net VOUT_P
- added copper zone on F.Cu, net V_ANT
- added copper zone on F.Cu, net V_POE
- added copper zone on In3.Cu, net V_POE
Other:
- board text added: "1"
- board text added: "A"
- board text added: "B"
- board text added: "C"
