File: hardware/ntp-server-stm32/optical-encoder.kicad_sch (KiCad schematic)
At the start: 2 parts, among them U68 74LVC2G17

Commit message: Bom updates
Parts:
- U68: footprint (none) -> 6-TSSOP; DIGIKEY_PART_NUMBER (none) -> 1727-4218-1-ND
Changed lines of the file:
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@@
 			)
 		)
-		(property "Footprint" ""
+		(property "Footprint" "6-TSSOP"
 			(at 146.05 123.19 0)
 			(hide yes)
@@
 			)
 		)
-		(property "Datasheet" "http://www.ti.com/lit/sg/scyt129e/scyt129e.pdf"
+		(property "Datasheet" "https://assets.nexperia.com/documents/data-sheet/74LVC2G17.pdf"
 			(at 146.05 123.19 0)
 			(hide yes)
@@
 		(property "MANUFACTURER" "Nexperia"
 			(at 0 0 0)
+			(hide yes)
+			(show_name no)
+			(do_not_autoplace no)
+			(effects
+				(font
+					(size 1.27 1.27)
+				)
+			)
+		)
+		(property "DIGIKEY_PART_NUMBER" "1727-4218-1-ND"
+			(at 146.05 123.19 0)
 			(hide yes)
 			(show_name no)
@@
 			)
 		)
-		(property "Footprint" ""
+		(property "Footprint" "6-TSSOP"
 			(at 158.75 82.55 0)
 			(hide yes)
@@
 			)
 		)
-		(property "Datasheet" "http://www.ti.com/lit/sg/scyt129e/scyt129e.pdf"
+		(property "Datasheet" "https://assets.nexperia.com/documents/data-sheet/74LVC2G17.pdf"
 			(at 158.75 82.55 0)
 			(hide yes)
@@
 		(property "MANUFACTURER" "Nexperia"
 			(at 0 0 0)
+			(hide yes)
+			(show_name no)
+			(do_not_autoplace no)
+			(effects
+				(font
+					(size 1.27 1.27)
+				)
+			)
+		)
+		(property "DIGIKEY_PART_NUMBER" "1727-4218-1-ND"
+			(at 158.75 82.55 0)
 			(hide yes)
 			(show_name no)
@@
 			)
 		)
-		(property "Footprint" ""
+		(property "Footprint" "6-TSSOP"
 			(at 158.75 62.23 0)
 			(hide yes)
@@
 			)
 		)
-		(property "Datasheet" "http://www.ti.com/lit/sg/scyt129e/scyt129e.pdf"
+		(property "Datasheet" "https://assets.nexperia.com/documents/data-sheet/74LVC2G17.pdf"
 			(at 158.75 62.23 0)
 			(hide yes)
@@
 			(hide yes)
 			(show_name no)
+			(do_not_autoplace no)
+			(effects
+				(font
+					(size 1.27 1.27)
+				)
+			)
+		)
+		(property "DIGIKEY_PART_NUMBER" "1727-4218-1-ND"
+			(at 158.75 62.23 0)
+			(hide yes)
+			(show_name no)

Commit message: Add files via upload
Updated, completed placement
Parts:
- C193: footprint 0402 (1005 Metric) -> copy_ref:C_0402_1005Metric
- U68: footprint 6-TSSOP -> dowload:74LVC2G17GW,125
Changed lines of the file:
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@@
 			)
 		)
-		(property "Footprint" "0402 (1005 Metric)"
+		(property "Footprint" "copy_ref:C_0402_1005Metric"
 			(at 171.1452 121.92 0)
 			(hide yes)
@@
 			)
 		)
-		(property "Footprint" "6-TSSOP"
+		(property "Footprint" "dowload:74LVC2G17GW,125"
 			(at 146.05 123.19 0)
 			(hide yes)
@@
 			)
 		)
-		(property "Footprint" "6-TSSOP"
+		(property "Footprint" "dowload:74LVC2G17GW,125"
 			(at 158.75 82.55 0)
 			(hide yes)
@@
 			)
 		)
-		(property "Footprint" "6-TSSOP"
+		(property "Footprint" "dowload:74LVC2G17GW,125"
 			(at 158.75 62.23 0)
 			(hide yes)
