File: hardware/ntp-server-stm32/stm32.kicad_sch (KiCad schematic)
At the start: 35 parts, among them Q6 BC847W, Q7 BC847W, U12 STM32H563VIT6, U13 LT3045xDD, U14 MCP1502T-33E/CHY, Y2 32.768kHz

Commit message: Updates
Parts:
- removed R49: 10k, R_0402_1005Metric, symbol Device:R
- removed U12: STM32H563VIT6, 100-LQFP, symbol STM32H563VIT6:STM32H563VIT6
- added C194, C195, C196, C197, C198, C199: 0.1uF, 0402 (1005 Metric), symbol Device:C
- added R232: 1.21k, R_0402_1005Metric, symbol Device:R
- added R233, R263: 10k, 0402 (1005 Metric), symbol Device:R
- added R264: 174k, 0402 (1005 Metric), symbol Device:R
- added U12: STM32H563ZIT6, STM32H563ZIT6:QFP50P2200X2200X160-144N, symbol STM32H563ZIT6-2:STM32H563ZIT6
- C21, C22, C23, C24, C25, C26, C35: footprint C_0402_1005Metric -> 0402 (1005 Metric); DIELECTRIC (none) -> X7R; DIGIKEY_PART_NUMBER 490-6328-2-ND -> 490-4759-1-ND; MANUFACTURER_PART_NUMBER GRM155R71C104KA88J -> GCM155R71C104KA55D; TOLERANCE (none) -> 10%; VOLTAGE (none) -> 16V
- C27, C30, C33: footprint C_0805_2012Metric -> 0805 (2012 Metric); DIELECTRIC (none) -> X7R; DIGIKEY_PART_NUMBER 490-GRM21BR71C475KE51KTR-ND -> 490-GRT21BR71C475KE13KCT-ND; MANUFACTURER Murata -> Murata Electronics; MANUFACTURER_PART_NUMBER GRM21BR71C475KE51K -> GRT21BR71C475KE13K; TOLERANCE (none) -> 10%; VOLTAGE (none) -> 16V
- C28: footprint C_0603_1608Metric -> 0603 (1608 Metric); DIELECTRIC (none) -> X7R; DIGIKEY_PART_NUMBER (none) -> 399-17704-1-ND; MANUFACTURER (none) -> KEMET; MANUFACTURER_PART_NUMBER (none) -> C0603C105K4RACAUTO; TOLERANCE (none) -> 10%; VOLTAGE (none) -> 16V
- C29, C31: footprint C_0402_1005Metric -> 0402 (1005 Metric); DIELECTRIC (none) -> C0G; DIGIKEY_PART_NUMBER (none) -> 490-16460-1-ND; MANUFACTURER (none) -> Murata Electronics; MANUFACTURER_PART_NUMBER (none) -> GCM1555C1H120FA16D; TOLERANCE (none) -> 5%; VOLTAGE (none) -> 50V
- C32: footprint C_0805_2012Metric -> 1206 (3216 Metric); DIELECTRIC (none) -> X7R; DIGIKEY_PART_NUMBER 490-GRM21BZ71C106KE15LTR-ND -> 1276-6797-1-ND; MANUFACTURER Murata -> Samsung Electro-Mechanics; MANUFACTURER_PART_NUMBER GRM21BZ71C106KE15L -> CL31B106KOHVPNE; TOLERANCE (none) -> 10%; VOLTAGE (none) -> 16V
- C34, C36, C38, C39: footprint C_0603_1608Metric -> 0805 (2012 Metric); DIELECTRIC (none) -> X7R; DIGIKEY_PART_NUMBER 490-GRM188Z71C225KE43DTR-ND -> 490-GRT21BR71C225KE01LCT-ND; MANUFACTURER Murata -> Murata Electronics; MANUFACTURER_PART_NUMBER GRM188Z71C225KE43D -> GRT21BR71C225KE01L; TOLERANCE (none) -> 10%; VOLTAGE (none) -> 16V
- C37: value 1nF -> 0.1uF; footprint C_0402_1005Metric -> 1210 (3225 Metric); DIELECTRIC (none) -> C0G; DIGIKEY_PART_NUMBER 490-GRM1555C1H102FA01JTR-ND -> 399-15804-1-ND; MANUFACTURER Murata -> KEMET; MANUFACTURER_PART_NUMBER GRM1555C1H102FA01J -> C1210C104J5GACAUTO; TOLERANCE (none) -> 5%; VOLTAGE (none) -> 50V
- FB2: DIELECTRIC (none) -> Ferrite bead; MANUFACTURER Murata Electronics -> Murata; MANUFACTURER_PART_NUMBER BLM31KN601SN1L -> BLM31PG601SN1L; POWER (none) -> 3A
- Q6, Q7: footprint Package_TO_SOT_SMD:SOT-323_SC-70 -> SOT-323; DIELECTRIC (none) -> Transistor; DIGIKEY_PART_NUMBER (none) -> 1727-BC847W,135CT-ND; MANUFACTURER (none) -> Nexperia USA Inc.; MANUFACTURER_PART_NUMBER BC847W -> BC847W,135
- R46: footprint R_0402_1005Metric -> 0402 (1005 Metric); DIELECTRIC (none) -> Thick-film; DIGIKEY_PART_NUMBER (none) -> P1.50KLCT-ND; MANUFACTURER Panasonic -> Panasonic Industry; POWER (none) -> 1/10W; TOLERANCE (none) -> 1%
- R47: footprint R_0402_1005Metric -> 0402 (1005 Metric); DIELECTRIC (none) -> Thick-film; DIGIKEY_PART_NUMBER (none) -> P33.2KLCT-ND; MANUFACTURER Panasonic -> Panasonic Industry; POWER (none) -> 1/10W; TOLERANCE (none) -> 1%
- R48: footprint R_0402_1005Metric -> 0603 (1608 Metric); DIELECTRIC (none) -> Thick-film; DIGIKEY_PART_NUMBER (none) -> 541-3318-1-ND; MANUFACTURER Panasonic -> Vishay Dale; MANUFACTURER_PART_NUMBER ERJ-2RKF50R0X -> CRCW060350R0FKEA; POWER (none) -> 1/10W; TOLERANCE (none) -> 1%
- R50, R51, R52, R53, R54: footprint R_0402_1005Metric -> 0402 (1005 Metric); DIELECTRIC (none) -> Thick-film; DIGIKEY_PART_NUMBER (none) -> P10.0KLCT-ND; MANUFACTURER Panasonic -> Panasonic Industry; POWER (none) -> 1/10W; TOLERANCE (none) -> 1%
- U13: MANUFACTURER (none) -> Analog Devices; MANUFACTURER_PART_NUMBER LT3045xDD -> LT3045EDD#TRPBF
- U14: MANUFACTURER (none) -> Microchip
- Y2: MANUFACTURER Abracon LLC -> Abracon
Connections:
- net 3V3_STM: now also C194.1, C195.1, C196.1, C197.1, C198.1, C199.1, U12.108 (VDD__8), U12.121 (VDDIO2), U12.131 (VDD__9), U12.144 (VDD__10), U12.17 (VDD), U12.30 (VDD__1), U12.39 (VDD__2), U12.52 (VDD__3), U12.62 (VDD__4), U12.72 (VDD__5), U12.84 (VDD__6), U12.95 (VDD__7)
- net 3V3_STM_USB: now also U12.106 (VDDUSB)
- net 5V_PSU_PG: now also U12.88 (PG3)
- net ANT_BIAS_EN: now also U12.99 (PC9)
- net CLK_OUT: now also U12.23 (PH0-OSC_IN)
- net DISP_BL: now also U12.5 (PE6)
- net DISP_CS: now also U12.60 (PE9)
- net DISP_DC: now also U12.46 (PB0)
- net DISP_EN: now also U12.112 (PC11)
- net DISP_RST: now also U12.102 (PA10)
- net ETH_PPS_OUT: now also U12.135 (PB5)
- net EXTREF_MON: now also U12.75 (PB14)
- net FAN_PWM: now also U12.4 (PE5)
- net FAN_TACH: now also U12.110 (PA15(JTDI))
- net GND: now also C194.2, C195.2, C196.2, C197.2, C198.2, C199.2, R233.2, R263.2, U12.107 (VSS__7), U12.120 (VSS__8), U12.130 (VSS__9), U12.143 (VSS__10), U12.16 (VSS), U12.31 (VSSA), U12.38 (VSS__1), U12.51 (VSS__2), U12.61 (VSS__3), U12.71 (VSS__4), U12.83 (VSS__5), U12.94 (VSS__6)
- net GPS_ANT_OFF_MON: now also U12.118 (PD4)
- net GPS_DSEL: now also U12.123 (PD7)
- net GPS_EXTINT: now also U12.122 (PD6)
- net GPS_PPS: now also U12.34 (PA0)
- net GPS_PWR_EN: now also U12.98 (PC8)
- net GPS_RST_N: now also U12.80 (PD11)
- net GPS_RX: now also U12.77 (PD8)
- net GPS_RXD2: now also U12.115 (PD1)
- net GPS_SAFEBOOT_N: now also U12.86 (PD15)
- net GPS_TP2: now also U12.96 (PC6)
- net GPS_TX: now also U12.78 (PD9)
- net GPS_TXD2: now also U12.114 (PD0)
- net GPS_TXRDY: now also U12.119 (PD5)
- net I2C_SCL: now also U12.139 (PB8)
- net I2C_SDA: now also U12.140 (PB9)
- net LAN_RST_N: now also U12.79 (PD10)
- net LED_B: now also U12.85 (PD14)
- net LED_G: now also U12.82 (PD13)
- net LED_R: now also U12.81 (PD12)
- net MCU_NRST: now also U12.25 (~{RST})
- net MUX_SEL: now also U12.136 (PB6)
- net NOR_RST_N: now also U12.63 (PE10)
- net OCXO_V: now also U12.37 (PA3)
- net OCXO_VC: now also U12.40 (PA4)
- net PFI: now also U12.59 (PE8)
- net POE_KILL: now also U12.68 (PE15)
- net POE_LCF: now also U12.29 (PC3)
- net POE_NCL: now also U12.97 (PC7)
- net POE_NCM: now also U12.28 (PC2)
- net RB_LOCK: now also U12.74 (PB13)
- net RB_OV_DET: now also U12.2 (PE3)
- net RB_OV_RESET: now also U12.117 (PD3)
- net RB_PWR_EN: now also U12.137 (PB7)
- net RB_RS232_CMOS_SW: now also U12.3 (PE4)
- net RB_RX: now also U12.134 (PB4(NJTRST))
- net RB_TX: now also U12.58 (PE7)
- net REF_TERM_EN: now also U12.111 (PC10)
- net RMII_CRS_DV: now also U12.43 (PA7)
- net RMII_MDC: now also U12.27 (PC1)
- net RMII_MDIO: now also U12.36 (PA2)
- net RMII_REF_CLK: now also U12.35 (PA1)
- net RMII_RXD0: now also U12.44 (PC4)
- net RMII_RXD1: now also U12.45 (PC5)
- net RMII_RXER: now also U12.69 (PB10)
- net RMII_TXD0: now also U12.73 (PB12)
- net RMII_TXD1: now also U12.76 (PB15)
- net RMII_TX_EN: now also U12.41 (PA5)
- net RTC_TAMPER: now also U12.7 (PC13)
- net SPI_DPOT_CS: now also U12.116 (PD2)
- net SPI_MISO: now also U12.66 (PE13)
- net SPI_MOSI: now also U12.67 (PE14)
- net SPI_NSS: now also U12.64 (PE11)
- net SPI_SCK: now also U12.65 (PE12)
- net STM_VBAT: now also U12.6 (VBAT)
- net SWCLK: now also U12.109 (PA14(JTCK/SWCLK))
- net SWDIO: now also U12.105 (PA13(JTMS/SWDIO))
- net SWO: now also U12.133 (PB3(JTDO/TRACESWO))
- net USB_DM: now also U12.103 (PA11)
- net USB_DP: now also U12.104 (PA12)
- net USB_VBUS_SENSE: now also U12.1 (PE2)
- net VDDA: now also U12.33 (VDDA)
- net WDT_EN: now also U12.113 (PC12)
- net WDT_KICK: now also U12.48 (PB2)
- net at C31.1, Y2.2: now also U12.8 (PC14-OSC32_IN)
- net at R50.1: now also U12.138 (BOOT0)
- net VREF_3V3: now reaches C37.1, R48.1, U14.1 (OUT)
- net VREF_3V3: now also U12.32 (VREF+)
- net at C34.1: now also U12.142 (VCAP__1)
- net at C36.1: now also U12.70 (VCAP)
- net at C29.1, Y2.1: now also U12.9 (PC15-OSC32_OUT)
- new net: R232.2, R233.1, U12.90 (PG5)
- new net: R263.1, R264.2, U12.92 (PG7)
- new net 3V0_RF_LDO_PG: U12.87 (PG2)
- new net 3V3_GPS_LDO_PG: U12.56 (PG0)
- new net 3V3_PSU_PG: U12.89 (PG4)
- new net BKP_GPS_PG: U12.55 (PF15)
- new net BKP_STM_PG: U12.54 (PF14)
- new net BUTTON_1: U12.10 (PF0)
- new net BUTTON_2: U12.11 (PF1)
- new net BUTTON_3: U12.12 (PF2)
- new net BUTTON_4: U12.13 (PF3)
- new net BUTTON_5: U12.14 (PF4)
- new net BUTTON_6: U12.15 (PF5)
- new net BUTTON_7: U12.18 (PF6)
- new net DISP_TOUCH_INT: U12.19 (PF7)
- new net ENC_A: U12.100 (PA8)
- new net ENC_B: U12.101 (PA9)
- new net ENC_BUTTON: U12.49 (PF11)
- new net HOLDOVER_ALARM_RELAY: U12.42 (PA6)
- new net INA_ALERT_3V3: U12.126 (PG11)
- new net INA_ALERT_3V3_GPS: U12.127 (PG12)
- new net INA_ALERT_3V3_STM: U12.124 (PG9)
- new net INA_ALERT_5V_DISP: U12.125 (PG10)
- new net INA_ALERT_5V_PANEL: U12.53 (PF13)
- new net INA_ALERT_OCXO: U12.129 (PG14)
- new net INA_ALERT_VCC_RB: U12.132 (PG15)
- new net INA_ALERT_V_ANT: U12.128 (PG13)
- new net INA_ALERT_V_POE: U12.93 (PG8)
- new net OCXO_LDO_PG: U12.57 (PG1)
- new net OCXO_PSU_PG: R232.1
- new net PANEL_LED_EN: U12.26 (PC0)
- new net PANEL_LED_FAULT: U12.50 (PF12)
- new net PANEL_LED_PWM: U12.141 (PE0)
- new net POE_PG: R264.1
- new net PROX_WAKE: U12.22 (PF10)
- new net RB_PSU_PG: U12.91 (PG6)
- new net RB_VCC_GATE: U12.47 (PB1)
- new net V_ANT_EN_FAULT: U12.20 (PF8)
- new net V_DISP_EN_FAULT: U12.21 (PF9)
Other:
- note added: "<- 3.7V"
- note added: "<- ~56V"
- moved on the sheet: C21, C22, C23, C24, C25, C26, C27, C28, C29, C30, C31, C32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

Commit message: Bom updates
Parts:
- FB2: footprint 1206 -> 1206 (3216 Metric)
- R232: footprint R_0402_1005Metric -> 0402 (1005 Metric); DIGIKEY_PART_NUMBER (none) -> P1.21KLCT-ND; MANUFACTURER Panasonic -> Panasonic Industry
- U12: DIGIKEY_PART_NUMBER (none) -> 497-STM32H563ZIT6-ND
- U13: DIGIKEY_PART_NUMBER (none) -> 505-LT3045EDD#TRPBFCT-ND
- U14: DIGIKEY_PART_NUMBER (none) -> 150-MCP1502T-33E/CHYCT-ND
Changed lines of the file:
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@@
 			)
 		)
-		(property "Footprint" "1206"
+		(property "Footprint" "1206 (3216 Metric)"
 			(at 323.088 34.29 90)
 			(hide yes)
@@
 			)
 		)
-		(property "Footprint" "R_0402_1005Metric"
+		(property "Footprint" "0402 (1005 Metric)"
 			(at 321.31 144.018 90)
 			(hide yes)
@@
 			)
 		)
-		(property "Datasheet" ""
+		(property "Datasheet" "https://industrial.panasonic.com/cdbs/www-data/pdf/RDA0000/AOA0000C304.pdf"
 			(at 321.31 142.24 0)
 			(hide yes)
@@
 			)
 		)
-		(property "Description" "RES 1.21k 1% 1/10W 0402"
+		(property "Description" "RES SMD 1.21K OHM 1% 1/10W 0402"
 			(at 321.31 142.24 0)
 			(hide yes)
@@
 			)
 		)
-		(property "MANUFACTURER" "Panasonic"
+		(property "MANUFACTURER" "Panasonic Industry"
 			(at 419.1 370.84 0)
 			(hide yes)
@@
 			)
 		)
+		(property "DIGIKEY_PART_NUMBER" "P1.21KLCT-ND"
+			(at 321.31 142.24 90)
+			(hide yes)
+			(show_name no)
+			(do_not_autoplace no)
+			(effects
+				(font
+					(size 1.27 1.27)
+				)
+			)
+		)
 		(pin "1"
 		)
@@
 			)
 		)
-		(property "Datasheet" ""
+		(property "Datasheet" "https://www.st.com/resource/en/datasheet/stm32h562ag.pdf"
 			(at 207.01 106.68 0)
 			(hide yes)
@@
 			)
 		)
-		(property "Description" "MCU Cortex-M33 2MB LQFP144"
+		(property "Description" "IC MCU 32BIT 2MB FLASH 144LQFP"
 			(at 207.01 106.68 0)
 			(hide yes)
@@
 			)
 		)
+		(property "DIGIKEY_PART_NUMBER" "497-STM32H563ZIT6-ND"
+			(at 207.01 106.68 0)
+			(hide yes)
+			(show_name no)
+			(do_not_autoplace no)
+			(effects
+				(font
+					(size 1.27 1.27)
+				)
+			)
+		)
 		(pin "2"
 		)
@@
 			)
 		)
-		(property "Description" "Voltage ref 3.3V SOT-23-6"
+		(property "Description" "IC VREF SERIES 3.3V SOT23-6"
 			(at 281.94 214.63 0)
 			(hide yes)
@@
 			)
 		)
+		(property "DIGIKEY_PART_NUMBER" "150-MCP1502T-33E/CHYCT-ND"
+			(at 281.94 214.63 0)
+			(hide yes)
+			(show_name no)
+			(do_not_autoplace no)
+			(effects
+				(font
+					(size 1.27 1.27)
+				)
+			)
+		)
 		(pin "6"
 		)
@@
 			)
 		)
-		(property "Description" "LDO 500mA ultralow-noise DFN-10"
+		(property "Description" "IC REG LIN POS ADJ 500MA 10DFN"
 			(at 374.65 43.18 0)
 			(hide yes)
@@
 			)
 		)
+		(property "DIGIKEY_PART_NUMBER" "505-LT3045EDD#TRPBFCT-ND"
+			(at 374.65 43.18 0)
+			(hide yes)
+			(show_name no)
+			(do_not_autoplace no)
+			(effects
+				(font
+					(size 1.27 1.27)
+				)
+			)
+		)
 		(pin "7"
 		)
@@
 			)
 		)
-		(property "Datasheet" ""
+		(property "Datasheet" "https://www.st.com/resource/en/datasheet/stm32h562ag.pdf"
 			(at 68.58 74.93 0)
 			(hide yes)
@@
 			)
 		)
-		(property "Description" "MCU Cortex-M33 2MB LQFP144"
+		(property "Description" "IC MCU 32BIT 2MB FLASH 144LQFP"
 			(at 68.58 74.93 0)
 			(hide yes)
@@
 			)
 		)
+		(property "DIGIKEY_PART_NUMBER" "497-STM32H563ZIT6-ND"
+			(at 68.58 74.93 0)
+			(hide yes)
+			(show_name no)
+			(do_not_autoplace no)
+			(effects
+				(font
+					(size 1.27 1.27)
+				)
+			)
+		)

Commit message: Bom updates
Parts:
- R264: value 174k -> 162k; footprint 0402 (1005 Metric) -> 1206 (3216 Metric); DIGIKEY_PART_NUMBER P174KLCT-ND -> P162KFCT-ND; MANUFACTURER_PART_NUMBER ERJ-2RKF1743X -> ERJ-8ENF1623V
Changed lines of the file:
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@@
 			)
 		)
-		(property "Value" "174k"
+		(property "Value" "162k"
 			(at 289.56 151.13 90)
 			(show_name no)
@@
 			)
 		)
-		(property "Footprint" "0402 (1005 Metric)"
+		(property "Footprint" "1206 (3216 Metric)"
 			(at 289.56 145.542 90)
 			(hide yes)
@@
 			)
 		)
-		(property "Description" "RES SMD 174K OHM 1% 1/10W 0402"
+		(property "Description" "RES SMD 162K OHM 1% 1/4W 1206"
 			(at 289.56 147.32 0)
 			(hide yes)
@@
 			)
 		)
-		(property "MANUFACTURER_PART_NUMBER" "ERJ-2RKF1743X"
+		(property "MANUFACTURER_PART_NUMBER" "ERJ-8ENF1623V"
 			(at 387.35 -81.28 0)
 			(hide yes)
@@
 			)
 		)
-		(property "DIGIKEY_PART_NUMBER" "P174KLCT-ND"
+		(property "DIGIKEY_PART_NUMBER" "P162KFCT-ND"
 			(at 289.56 147.32 90)
 			(hide yes)

Commit message: Add files via upload
Updated, completed placement
Parts:
- C194, C195, C196, C197, C198, C199, C21, C22, C23, C24, C25, C26, C29, C31, C35: footprint 0402 (1005 Metric) -> copy_ref:C_0402_1005Metric
- C27, C30, C33, C34, C36, C38, C39: footprint 0805 (2012 Metric) -> copy_ref:C_0805_2012Metric
- C28: footprint 0603 (1608 Metric) -> copy_ref:C_0603_1608Metric
- C32: footprint 1206 (3216 Metric) -> copy_ref:C_1206_3216Metric
- C37: footprint 1210 (3225 Metric) -> copy_ref:C_1210_3225Metric
- FB2: footprint 1206 (3216 Metric) -> copy_ref:1206
- Q6, Q7: footprint SOT-323 -> Package_TO_SOT_SMD:SOT-323_SC-70
- R232, R233, R263, R46, R47, R50, R51, R52, R53, R54: footprint 0402 (1005 Metric) -> copy_ref:R_0402_1005Metric
- R264: footprint 1206 (3216 Metric) -> copy_ref:R_1206_3216Metric
- R48: footprint 0603 (1608 Metric) -> Resistor_SMD:R_0603_1608Metric
- U14: footprint SOT-23-6 -> Package_TO_SOT_SMD:SOT-23-6
- Y2: footprint (none) -> dowload:ABS07-32.768KHZ-1-T
Changed lines of the file:
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@@
 			)
 		)
-		(property "Footprint" "0402 (1005 Metric)"
+		(property "Footprint" "copy_ref:C_0402_1005Metric"
 			(at 20.0152 252.73 0)
 			(hide yes)
@@
 			)
 		)
-		(property "Footprint" "0402 (1005 Metric)"
+		(property "Footprint" "copy_ref:C_0402_1005Metric"
 			(at 32.7152 252.73 0)
 			(hide yes)
@@
 			)
 		)
-		(property "Footprint" "0402 (1005 Metric)"
+		(property "Footprint" "copy_ref:C_0402_1005Metric"
 			(at 138.1252 135.89 0)
 			(hide yes)
@@
 			)
 		)
-		(property "Footprint" "SOT-323"
+		(property "Footprint" "Package_TO_SOT_SMD:SOT-323_SC-70"
 			(at 256.54 222.885 0)
 			(hide yes)
@@
 			)
 		)
-		(property "Footprint" "0402 (1005 Metric)"
+		(property "Footprint" "copy_ref:R_0402_1005Metric"
 			(at 236.728 238.76 90)
 			(hide yes)
@@
 			)
 		)
-		(property "Footprint" "0805 (2012 Metric)"
+		(property "Footprint" "copy_ref:C_0805_2012Metric"
 			(at 197.8152 250.19 0)
 			(hide yes)
@@
 			)
 		)
-		(property "Footprint" "0805 (2012 Metric)"
+		(property "Footprint" "copy_ref:C_0805_2012Metric"
 			(at 264.4648 204.47 0)
 			(hide yes)
@@
 			)
 		)
-		(property "Footprint" "0402 (1005 Metric)"
+		(property "Footprint" "copy_ref:C_0402_1005Metric"
 			(at 210.5152 250.19 0)
 			(hide yes)
@@
 			)
 		)
-		(property "Footprint" "0402 (1005 Metric)"
+		(property "Footprint" "copy_ref:C_0402_1005Metric"
 			(at 58.1152 252.73 0)
 			(hide yes)
@@
 			)
 		)
-		(property "Footprint" "1206 (3216 Metric)"
+		(property "Footprint" "copy_ref:1206"
 			(at 323.088 34.29 90)
 			(hide yes)
@@
 			)
 		)
-		(property "Footprint" "0603 (1608 Metric)"
+		(property "Footprint" "Resistor_SMD:R_0603_1608Metric"
 			(at 304.038 215.9 90)
 			(hide yes)
@@
 			)
 		)
-		(property "Footprint" "0402 (1005 Metric)"
+		(property "Footprint" "copy_ref:R_0402_1005Metric"
 			(at 321.31 144.018 90)
 			(hide yes)
@@
 			)
 		)
-		(property "Footprint" "0402 (1005 Metric)"
+		(property "Footprint" "copy_ref:C_0402_1005Metric"
 			(at 148.2852 252.73 0)
 			(hide yes)
@@
 			)
 		)
-		(property "Footprint" "0402 (1005 Metric)"
+		(property "Footprint" "copy_ref:C_0402_1005Metric"
 			(at 70.8152 252.73 0)
 			(hide yes)
@@
 			)
 		)
-		(property "Footprint" "0402 (1005 Metric)"
+		(property "Footprint" "copy_ref:R_0402_1005Metric"
 			(at 284.988 152.4 90)
 			(hide yes)
@@
 			)
 		)
-		(property "Footprint" "0402 (1005 Metric)"
+		(property "Footprint" "copy_ref:C_0402_1005Metric"
 			(at 45.4152 252.73 0)
 			(hide yes)
@@
 			)
 		)
-		(property "Footprint" "0805 (2012 Metric)"
+		(property "Footprint" "copy_ref:C_0805_2012Metric"
 			(at 115.2652 63.5 0)
 			(hide yes)
@@
 			)
 		)
-		(property "Footprint" "0402 (1005 Metric)"
+		(property "Footprint" "copy_ref:R_0402_1005Metric"
 			(at 236.728 227.33 90)
 			(hide yes)
@@
 			)
 		)
-		(property "Footprint" "1206 (3216 Metric)"
+		(property "Footprint" "copy_ref:R_1206_3216Metric"
 			(at 289.56 145.542 90)
 			(hide yes)
@@
 			)
 		)
-		(property "Footprint" "0805 (2012 Metric)"
+		(property "Footprint" "copy_ref:C_0805_2012Metric"
 			(at 301.2948 227.33 0)
 			(hide yes)
@@
 			)
 		)
-		(property "Footprint" "0805 (2012 Metric)"
+		(property "Footprint" "copy_ref:C_0805_2012Metric"
 			(at 320.3448 58.42 0)
 			(hide yes)
@@
 			)
 		)
-		(property "Footprint" "0805 (2012 Metric)"
+		(property "Footprint" "copy_ref:C_0805_2012Metric"
 			(at 360.3752 59.69 0)
 			(hide yes)
@@
 			)
 		)
-		(property "Footprint" ""
+		(property "Footprint" "dowload:ABS07-32.768KHZ-1-T"
 			(at 130.81 124.46 0)
 			(hide yes)
@@
 			)
 		)
-		(property "Footprint" "0402 (1005 Metric)"
+		(property "Footprint" "copy_ref:R_0402_1005Metric"
 			(at 255.778 207.01 90)
 			(hide yes)
@@
 			)
 		)
-		(property "Footprint" "0402 (1005 Metric)"
+		(property "Footprint" "copy_ref:C_0402_1005Metric"
 			(at 121.6152 252.73 0)
 			(hide yes)
@@
 			)
 		)
-		(property "Footprint" "0603 (1608 Metric)"
+		(property "Footprint" "copy_ref:C_0603_1608Metric"
 			(at 180.0352 252.73 0)
 			(hide yes)
@@
 			)
 		)
-		(property "Footprint" "SOT-23-6"
+		(property "Footprint" "Package_TO_SOT_SMD:SOT-23-6"
 			(at 281.94 214.63 0)
 			(hide yes)
@@
 			)
 		)
-		(property "Footprint" "0402 (1005 Metric)"
+		(property "Footprint" "copy_ref:C_0402_1005Metric"
 			(at 108.9152 252.73 0)
 			(hide yes)
@@
 			)
 		)
-		(property "Footprint" "0402 (1005 Metric)"
+		(property "Footprint" "copy_ref:C_0402_1005Metric"
 			(at 124.1552 135.89 0)
 			(hide yes)
@@
 			)
 		)
-		(property "Footprint" "0402 (1005 Metric)"
+		(property "Footprint" "copy_ref:R_0402_1005Metric"
 			(at 316.738 147.32 90)
 			(hide yes)
@@
 			)
 		)
-		(property "Footprint" "SOT-323"
+		(property "Footprint" "Package_TO_SOT_SMD:SOT-323_SC-70"
 			(at 246.38 235.585 0)
 			(hide yes)
@@
 			)
 		)
-		(property "Footprint" "0805 (2012 Metric)"
+		(property "Footprint" "copy_ref:C_0805_2012Metric"
 			(at 129.2352 63.5 0)
 			(hide yes)
@@
 			)
 		)
-		(property "Footprint" "0402 (1005 Metric)"
+		(property "Footprint" "copy_ref:R_0402_1005Metric"
 			(at 354.838 55.88 90)
 			(hide yes)
@@
 			)
 		)
-		(property "Footprint" "0402 (1005 Metric)"
+		(property "Footprint" "copy_ref:C_0402_1005Metric"
 			(at 96.2152 252.73 0)
 			(hide yes)
@@
 			)
 		)
-		(property "Footprint" "1206 (3216 Metric)"
+		(property "Footprint" "copy_ref:C_1206_3216Metric"
 			(at 401.0152 49.53 0)
 			(hide yes)
@@
 			)
 		)
-		(property "Footprint" "0402 (1005 Metric)"
+		(property "Footprint" "copy_ref:C_0402_1005Metric"
 			(at 83.5152 252.73 0)
 			(hide yes)
@@
 			)
 		)
-		(property "Footprint" "0402 (1005 Metric)"
+		(property "Footprint" "copy_ref:C_0402_1005Metric"
 			(at 134.3152 252.73 0)
 			(hide yes)
@@
 			)
 		)
-		(property "Footprint" "0402 (1005 Metric)"
+		(property "Footprint" "copy_ref:R_0402_1005Metric"
 			(at 334.518 55.88 90)
 			(hide yes)
@@
 			)
 		)
-		(property "Footprint" "0402 (1005 Metric)"
+		(property "Footprint" "copy_ref:R_0402_1005Metric"
 			(at 245.618 212.09 90)
 			(hide yes)
@@
 			)
 		)
-		(property "Footprint" "1210 (3225 Metric)"
+		(property "Footprint" "copy_ref:C_1210_3225Metric"
 			(at 313.9948 220.98 0)
 			(hide yes)
@@
 			)
 		)
-		(property "Footprint" "0402 (1005 Metric)"
+		(property "Footprint" "copy_ref:C_0402_1005Metric"
 			(at 167.3352 252.73 0)
 			(hide yes)
@@
 			)
 		)
-		(property "Footprint" "0402 (1005 Metric)"
+		(property "Footprint" "copy_ref:R_0402_1005Metric"
 			(at 23.368 73.66 90)
 			(hide yes)
