File: hardware/ntp-server-stm32/wdt.kicad_sch (KiCad schematic)
At the start: 4 parts, among them U64 TPS3430WDRC

Commit message: Updates
Parts:
- added D24: BAT54J, SOD-323F, symbol Diode:BAT54J
- added K2: G6K-2F-Y DC3, symbol Relay:G6K-2
- added Q24: BC847W, SOT-323, symbol Transistor_BJT:BC847W
- added R259: 10k, 0402 (1005 Metric), symbol Device:R
- added R260: 470, R_0402_1005Metric, symbol Device:R
- C180, C181: footprint C_0402_1005Metric -> 0402 (1005 Metric); DIELECTRIC (none) -> X7R; DIGIKEY_PART_NUMBER 490-6328-2-ND -> 490-4759-1-ND; MANUFACTURER_PART_NUMBER GRM155R71C104KA88J -> GCM155R71C104KA55D; TOLERANCE (none) -> 10%; VOLTAGE (none) -> 16V
- R213: footprint R_0402_1005Metric -> 0402 (1005 Metric); DIELECTRIC (none) -> Thick-film; DIGIKEY_PART_NUMBER (none) -> P100KLCT-ND; MANUFACTURER Panasonic -> Panasonic Industry; POWER (none) -> 1/10W; TOLERANCE (none) -> 1%
- U64: MANUFACTURER (none) -> Texas Instruments
Connections:
- net GND: now also Q24.2 (E), R259.1
- new net: D24.2 (A), K2.8, Q24.3 (C)
- new net: Q24.1 (B), R259.2, R260.2
- new net 3V3: D24.1 (K), K2.1
- new net HOLDOVER_ALARM_C1: K2.3
- new net HOLDOVER_ALARM_C2: K2.6
- new net HOLDOVER_ALARM_NC1: K2.2
- new net HOLDOVER_ALARM_NC2: K2.7
- new net HOLDOVER_ALARM_NO1: K2.4
- new net HOLDOVER_ALARM_NO2: K2.5
- new net HOLDOVER_ALARM_RELAY: R260.1

Commit message: Bom updates
Parts:
- R260: footprint R_0402_1005Metric -> 0402 (1005 Metric); DIGIKEY_PART_NUMBER (none) -> P470LCT-ND; MANUFACTURER Panasonic -> Panasonic Industry
- U64: DIGIKEY_PART_NUMBER (none) -> 296-51907-1-ND
Changed lines of the file:
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@@
+			)
+		)
+		(property "DIGIKEY_PART_NUMBER" "296-51907-1-ND"
+			(at 163.83 106.68 0)
+			(hide yes)
+			(show_name no)
+			(do_not_autoplace no)
+			(effects
+				(font
+					(size 1.27 1.27)
+				)
 			)
 		)
@@
 			)
 		)
-		(property "Footprint" "R_0402_1005Metric"
+		(property "Footprint" "0402 (1005 Metric)"
 			(at 338.328 95.25 90)
 			(hide yes)
@@
 			)
 		)
-		(property "Datasheet" ""
+		(property "Datasheet" "https://industrial.panasonic.com/cdbs/www-data/pdf/RDA0000/AOA0000C304.pdf"
 			(at 336.55 95.25 0)
 			(hide yes)
@@
 			)
 		)
-		(property "Description" "RES 470 1% 1/10W 0402"
+		(property "Description" "RES SMD 470 OHM 1% 1/10W 0402"
 			(at 336.55 95.25 0)
 			(hide yes)
@@
 			)
 		)
-		(property "MANUFACTURER" "Panasonic"
+		(property "MANUFACTURER" "Panasonic Industry"
 			(at 101.6 -3.81 0)
 			(hide yes)
@@
 			(hide yes)
 			(show_name no)
+			(do_not_autoplace no)
+			(effects
+				(font
+					(size 1.27 1.27)
+				)
+			)
+		)
+		(property "DIGIKEY_PART_NUMBER" "P470LCT-ND"
+			(at 336.55 95.25 0)
+			(hide yes)
+			(show_name no)

Commit message: Add files via upload
Updated, completed placement
Parts:
- C180, C181: footprint 0402 (1005 Metric) -> copy_ref:C_0402_1005Metric
- D24: footprint SOD-323F -> Diode_SMD:D_SOD-323F
- K2: footprint (none) -> dowload:G6K-2F-Y DC3
- Q24: footprint SOT-323 -> Package_TO_SOT_SMD:SOT-323_SC-70
- R213, R259, R260: footprint 0402 (1005 Metric) -> copy_ref:R_0402_1005Metric
Changed lines of the file:
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@@
 			)
 		)
-		(property "Footprint" "0402 (1005 Metric)"
+		(property "Footprint" "copy_ref:R_0402_1005Metric"
 			(at 143.002 118.11 90)
 			(hide yes)
@@
 			)
 		)
-		(property "Footprint" "0402 (1005 Metric)"
+		(property "Footprint" "copy_ref:C_0402_1005Metric"
 			(at 129.2352 66.04 0)
 			(hide yes)
@@
 			)
 		)
-		(property "Footprint" "SOD-323F"
+		(property "Footprint" "Diode_SMD:D_SOD-323F"
 			(at 295.91 89.535 0)
 			(hide yes)
@@
 			)
 		)
-		(property "Footprint" "SOT-323"
+		(property "Footprint" "Package_TO_SOT_SMD:SOT-323_SC-70"
 			(at 317.5 93.345 0)
 			(hide yes)
@@
 			)
 		)
-		(property "Footprint" ""
+		(property "Footprint" "dowload:G6K-2F-Y DC3"
 			(at 295.91 109.22 0)
 			(hide yes)
@@
 			)
 		)
-		(property "Footprint" "0402 (1005 Metric)"
+		(property "Footprint" "copy_ref:R_0402_1005Metric"
 			(at 338.328 95.25 90)
 			(hide yes)
@@
 			)
 		)
-		(property "Footprint" "0402 (1005 Metric)"
+		(property "Footprint" "copy_ref:R_0402_1005Metric"
 			(at 329.692 96.52 90)
 			(hide yes)
@@
 			)
 		)
-		(property "Footprint" "0402 (1005 Metric)"
+		(property "Footprint" "copy_ref:C_0402_1005Metric"
 			(at 113.9952 66.04 0)
 			(hide yes)
