File: hardware/ntp-server-stm32/clock-mux.kicad_sch (KiCad schematic)
At the start: 10 parts, among them U52 74LVC1G157GW-Q100H, U53 74LVC1G34

Commit message: Updates
Parts:
- added C203: 0.1uF, 0402 (1005 Metric), symbol Device:C
- added C206: 10nF, 0402 (1005 Metric), symbol Device:C
- added R255, R256: 33, R_0402_1005Metric, symbol Device:R
- added U71: 74LVC1G34, symbol 74xGxx:74LVC1G34
- C157: footprint C_0603_1608Metric -> 0603 (1608 Metric); DIELECTRIC (none) -> X7R; DIGIKEY_PART_NUMBER 445-5972-1-ND -> 399-17704-1-ND; MANUFACTURER TDK -> KEMET; MANUFACTURER_PART_NUMBER C2012X7R1E475K125AB -> C0603C105K4RACAUTO; TOLERANCE (none) -> 10%; VOLTAGE (none) -> 16V
- C158, C159, C160: footprint C_0402_1005Metric -> 0402 (1005 Metric); DIELECTRIC (none) -> X7R; DIGIKEY_PART_NUMBER 490-6328-2-ND -> 490-4759-1-ND; MANUFACTURER_PART_NUMBER GRM155R71C104KA88J -> GCM155R71C104KA55D; TOLERANCE (none) -> 10%; VOLTAGE (none) -> 16V
- FB10: DIELECTRIC (none) -> Ferrite bead; MANUFACTURER Murata Electronics -> Murata; MANUFACTURER_PART_NUMBER BLM31KN601SN1L -> BLM31PG601SN1L; POWER (none) -> 3A
- R187, R189: footprint R_0402_1005Metric -> 0402 (1005 Metric); DIELECTRIC (none) -> Thick-film; DIGIKEY_PART_NUMBER (none) -> P22.0LCT-ND; MANUFACTURER Panasonic -> Panasonic Industry; POWER (none) -> 1/10W; TOLERANCE (none) -> 1%
- R188: footprint R_0402_1005Metric -> 0402 (1005 Metric); DIELECTRIC (none) -> Thick-film; DIGIKEY_PART_NUMBER (none) -> P100KLCT-ND; MANUFACTURER Panasonic -> Panasonic Industry; POWER (none) -> 1/10W; TOLERANCE (none) -> 1%
- U52: MANUFACTURER (none) -> Nexperia
- U53: MANUFACTURER (none) -> Nexperia; MANUFACTURER_PART_NUMBER 74LVC1G34 -> 74LVC1G34GW,125
Connections:
- net GND: now also C203.2, C206.2, U71.3 (GND)
- new net: R256.1, U71.2
- new net: R255.2, U71.4
- new net 1PPS_OUT: R255.1
- new net 5V: C203.1, C206.1, U71.5 (VCC)
- new net ETH_PPS_OUT: R256.2
- no-connect marks 1 -> 2

Commit message: Bom updates
Parts:
- FB10: footprint 1206 -> 1206 (3216 Metric)
- R255, R256: footprint R_0402_1005Metric -> 0402 (1005 Metric); DIGIKEY_PART_NUMBER (none) -> P33.0LCT-ND; MANUFACTURER Panasonic -> Panasonic Industry
- U52: DIGIKEY_PART_NUMBER (none) -> 1727-74LVC1G157GW-Q100HCT-ND
- U53, U71: DIGIKEY_PART_NUMBER (none) -> 1727-6074-1-ND
Changed lines of the file:
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@@
+			)
+		)
+		(property "DIGIKEY_PART_NUMBER" "1727-6074-1-ND"
+			(at 219.71 224.79 0)
+			(hide yes)
+			(show_name no)
+			(do_not_autoplace no)
+			(effects
+				(font
+					(size 1.27 1.27)
+				)
 			)
 		)
@@
 			)
 		)
+		(property "DIGIKEY_PART_NUMBER" "1727-74LVC1G157GW-Q100HCT-ND"
+			(at 147.32 113.03 0)
+			(hide yes)
+			(show_name no)
+			(do_not_autoplace no)
+			(effects
+				(font
+					(size 1.27 1.27)
+				)
+			)
+		)
 		(pin "3"
 		)
@@
 			)
 		)
-		(property "Footprint" "R_0402_1005Metric"
+		(property "Footprint" "0402 (1005 Metric)"
 			(at 196.85 226.568 90)
 			(hide yes)
@@
 			)
 		)
-		(property "Datasheet" ""
+		(property "Datasheet" "https://industrial.panasonic.com/cdbs/www-data/pdf/RDA0000/AOA0000C304.pdf"
 			(at 196.85 224.79 0)
 			(hide yes)
@@
 			)
 		)
-		(property "Description" "RES 33 1% 1/10W 0402"
+		(property "Description" "RES SMD 33 OHM 1% 1/10W 0402"
 			(at 196.85 224.79 0)
 			(hide yes)
@@
 			)
 		)
-		(property "MANUFACTURER" "Panasonic"
+		(property "MANUFACTURER" "Panasonic Industry"
 			(at -2.54 106.68 0)
 			(hide yes)
@@
 		(property "MANUFACTURER_PART_NUMBER" "ERJ-2RKF33R0X"
 			(at -2.54 106.68 0)
+			(hide yes)
+			(show_name no)
+			(do_not_autoplace no)
+			(effects
+				(font
+					(size 1.27 1.27)
+				)
+			)
+		)
+		(property "DIGIKEY_PART_NUMBER" "P33.0LCT-ND"
+			(at 196.85 224.79 90)
 			(hide yes)
 			(show_name no)
@@
 			)
 		)
-		(property "Footprint" "1206"
+		(property "Footprint" "1206 (3216 Metric)"
 			(at 133.858 78.74 90)
 			(hide yes)
@@
 			)
 		)
-		(property "Footprint" "R_0402_1005Metric"
+		(property "Footprint" "0402 (1005 Metric)"
 			(at 242.57 226.568 90)
 			(hide yes)
@@
 			)
 		)
-		(property "Datasheet" ""
+		(property "Datasheet" "https://industrial.panasonic.com/cdbs/www-data/pdf/RDA0000/AOA0000C304.pdf"
 			(at 242.57 224.79 0)
 			(hide yes)
@@
 			)
 		)
-		(property "Description" "RES 33 1% 1/10W 0402"
+		(property "Description" "RES SMD 33 OHM 1% 1/10W 0402"
 			(at 242.57 224.79 0)
 			(hide yes)
@@
 			)
 		)
-		(property "MANUFACTURER" "Panasonic"
+		(property "MANUFACTURER" "Panasonic Industry"
 			(at 0 62.23 0)
 			(hide yes)
@@
 		(property "MANUFACTURER_PART_NUMBER" "ERJ-2RKF33R0X"
 			(at 0 62.23 0)
+			(hide yes)
+			(show_name no)
+			(do_not_autoplace no)
+			(effects
+				(font
+					(size 1.27 1.27)
+				)
+			)
+		)
+		(property "DIGIKEY_PART_NUMBER" "P33.0LCT-ND"
+			(at 242.57 224.79 90)
 			(hide yes)
 			(show_name no)
@@
 			(hide yes)
 			(show_name no)
+			(do_not_autoplace no)
+			(effects
+				(font
+					(size 1.27 1.27)
+				)
+			)
+		)
+		(property "DIGIKEY_PART_NUMBER" "1727-6074-1-ND"
+			(at 219.71 162.56 0)
+			(hide yes)
+			(show_name no)

Commit message: Bom updates
Parts:
- U52: footprint SC-74_TSOP6_SOT457_NEX -> sts1000:SC-74_TSOP6_SOT457_NEX
Changed lines of the file:
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@@
 			)
 		)
-		(property "Footprint" "SC-74_TSOP6_SOT457_NEX"
+		(property "Footprint" "sts1000:SC-74_TSOP6_SOT457_NEX"
 			(at 147.32 113.03 0)
 			(hide yes)

Commit message: Add files via upload
Updated, completed placement
Parts:
- C157: footprint 0603 (1608 Metric) -> copy_ref:C_0603_1608Metric
- C158, C159, C160, C203, C206: footprint 0402 (1005 Metric) -> copy_ref:C_0402_1005Metric
- FB10: footprint 1206 (3216 Metric) -> copy_ref:1206
- R187, R188, R189, R255, R256: footprint 0402 (1005 Metric) -> copy_ref:R_0402_1005Metric
- U53, U71: footprint (none) -> dowload:74LVC1G34GW_125
Changed lines of the file:
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@@
 			)
 		)
-		(property "Footprint" "0402 (1005 Metric)"
+		(property "Footprint" "copy_ref:R_0402_1005Metric"
 			(at 199.39 119.888 90)
 			(hide yes)
@@
 			)
 		)
-		(property "Footprint" ""
+		(property "Footprint" "dowload:74LVC1G34GW_125"
 			(at 219.71 224.79 0)
 			(hide yes)
@@
 			)
 		)
-		(property "Footprint" "0402 (1005 Metric)"
+		(property "Footprint" "copy_ref:C_0402_1005Metric"
 			(at 257.81 161.5948 0)
 			(hide yes)
@@
 			)
 		)
-		(property "Footprint" "0402 (1005 Metric)"
+		(property "Footprint" "copy_ref:R_0402_1005Metric"
 			(at 242.57 164.338 90)
 			(hide yes)
@@
 			)
 		)
-		(property "Footprint" "0603 (1608 Metric)"
+		(property "Footprint" "copy_ref:C_0603_1608Metric"
 			(at 133.0452 97.79 0)
 			(hide yes)
@@
 			)
 		)
-		(property "Footprint" "0402 (1005 Metric)"
+		(property "Footprint" "copy_ref:R_0402_1005Metric"
 			(at 196.85 226.568 90)
 			(hide yes)
@@
 			)
 		)
-		(property "Footprint" "1206 (3216 Metric)"
+		(property "Footprint" "copy_ref:1206"
 			(at 133.858 78.74 90)
 			(hide yes)
@@
 			)
 		)
-		(property "Footprint" "0402 (1005 Metric)"
+		(property "Footprint" "copy_ref:C_0402_1005Metric"
 			(at 237.1852 210.82 0)
 			(hide yes)
@@
 			)
 		)
-		(property "Footprint" "0402 (1005 Metric)"
+		(property "Footprint" "copy_ref:R_0402_1005Metric"
 			(at 242.57 226.568 90)
 			(hide yes)
@@
 			)
 		)
-		(property "Footprint" ""
+		(property "Footprint" "dowload:74LVC1G34GW_125"
 			(at 219.71 162.56 0)
 			(hide yes)
@@
 			)
 		)
-		(property "Footprint" "0402 (1005 Metric)"
+		(property "Footprint" "copy_ref:R_0402_1005Metric"
 			(at 241.808 118.11 90)
 			(hide yes)
@@
 			)
 		)
-		(property "Footprint" "0402 (1005 Metric)"
+		(property "Footprint" "copy_ref:C_0402_1005Metric"
 			(at 223.2152 212.09 0)
 			(hide yes)
@@
 			)
 		)
-		(property "Footprint" "0402 (1005 Metric)"
+		(property "Footprint" "copy_ref:C_0402_1005Metric"
 			(at 223.2152 149.86 0)
 			(hide yes)
@@
 			)
 		)
-		(property "Footprint" "0402 (1005 Metric)"
+		(property "Footprint" "copy_ref:C_0402_1005Metric"
 			(at 202.8952 97.79 0)
 			(hide yes)

Commit message: PCB / 3D updates
Parts:
- U52: footprint sts1000:SC-74_TSOP6_SOT457_NEX -> dowload:SOT-363-6_2P2X1P35_ONS
Changed lines of the file:
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@@
 			)
 		)
-		(property "Footprint" "sts1000:SC-74_TSOP6_SOT457_NEX"
+		(property "Footprint" "dowload:SOT-363-6_2P2X1P35_ONS"
 			(at 147.32 113.03 0)
 			(hide yes)
