File: hardware/ntp-server-stm32/connectors.kicad_sch (KiCad schematic)
At the start: 31 parts, among them J10 Conn_01x02_Pin, J11 Conn_01x08_Pin, J2 Conn_01x04_Pin, J3 Conn_01x06_Pin, J4 Conn_01x14_Pin, J5 USB4120-03-C_REVA6, J6 DE9_Socket_MountingHoles, J7 Conn_Coaxial, J8 Conn_Coaxial, J9 Conn_Coaxial, U15 TPD4E02B04DQAR, U16 TPD4E02B04DQAR, U17 TPD4E05U06DQAR, U18 TPD4E05U06DQAR, U19 TPD4E02B04DQAR, U20 TPD4E02B04DQAR

Commit message: Updates
Parts:
- removed C44: 1nF, C_0402_1005Metric, symbol Device:C
- removed J11: Conn_01x08_Pin, symbol Connector:Conn_01x08_Pin
- removed J4: Conn_01x14_Pin, symbol Connector:Conn_01x14_Pin
- removed TP1: TestPoint, symbol Connector:TestPoint
- added C186: 4.7nF, 1812 (4532 Metric), symbol Device:C
- added C188: 0.1uF, 0402 (1005 Metric), symbol Device:C
- added D22: SMF5V0A, DO-219AB (SMF), symbol Diode:SMF5V0A
- added D23: SZESD7410MXWT5G, 2-XDFN, symbol ntp-server-stm32:SZESD7410MXWT5G
- added D26: SMAJ15CA, DO-214AC, symbol Diode:SMAJ15CA
- added J15: SMA-J-P-H-RA-TH1, symbol Connector:Conn_Coaxial
- added J16: OSTVN06A150, symbol Connector:Conn_01x06_Pin
- added J17: 1787179, symbol Connector_Generic:Conn_02x18_Top_Bottom
- added L10: PGB1010603MR, 0603 (1608 Metric), symbol PGB1010603MR:PGB1010603MR
- added R231: 1M, 0402 (1005 Metric), symbol Device:R
- added U65, U66, U69, U70: TPD4E05U06DQAR, DQA0010A, symbol TPD4E05U06DQAR:TPD4E05U06DQAR
- C40: footprint C_0603_1608Metric -> 0603 (1608 Metric); DIELECTRIC (none) -> X7R; DIGIKEY_PART_NUMBER (none) -> 399-17704-1-ND; MANUFACTURER (none) -> KEMET; MANUFACTURER_PART_NUMBER (none) -> C0603C105K4RACAUTO; TOLERANCE (none) -> 10%; VOLTAGE (none) -> 16V
- C41, C43: footprint C_0402_1005Metric -> 0402 (1005 Metric); DIELECTRIC (none) -> X7R; DIGIKEY_PART_NUMBER 490-6328-2-ND -> 490-4759-1-ND; MANUFACTURER_PART_NUMBER GRM155R71C104KA88J -> GCM155R71C104KA55D; TOLERANCE (none) -> 10%; VOLTAGE (none) -> 16V
- C42: footprint C_0402_1005Metric -> 1812 (4532 Metric); DIELECTRIC (none) -> X7R; DIGIKEY_PART_NUMBER 490-6334-2-ND -> 399-16791-1-ND; MANUFACTURER Murata -> KEMET; MANUFACTURER_PART_NUMBER GRM155R71C472KA01D -> C1812C472KGRACAUTO; TOLERANCE (none) -> 10%; VOLTAGE (none) -> 2kV
- D6: footprint Diode_SMD:D_SMF -> DO-219AB (SMF); DIELECTRIC (none) -> Diode; DIGIKEY_PART_NUMBER (none) -> 112-SMF5V0A-HE3_A08CT-ND; MANUFACTURER (none) -> Vishay; MANUFACTURER_PART_NUMBER SMF5V0A -> SMF5V0A-HE3_A08
- D7: value 1.5SMCxxA -> 1.5SMCJ28A; footprint Diode_SMD:D_SMC -> DO-214AB (SMC); DIELECTRIC (none) -> Diode; DIGIKEY_PART_NUMBER (none) -> 4878-1.5SMCJ28ACT-ND; MANUFACTURER (none) -> Diotec Semiconductor; MANUFACTURER_PART_NUMBER (none) -> 1.5SMCJ28A
- D8, D9: footprint (none) -> 2-XDFN; DIELECTRIC (none) -> Diode; DIGIKEY_PART_NUMBER (none) -> 488-SZESD7410MXWT5GCT-ND; MANUFACTURER (none) -> onsemi
- J10: value Conn_01x02_Pin -> OSTVN02A150; DIGIKEY_PART_NUMBER (none) -> ED10561-ND; MANUFACTURER (none) -> On Shore Technology Inc.; MANUFACTURER_PART_NUMBER (none) -> OSTVN02A150
- J2: value Conn_01x04_Pin -> OSTVN04A150; DIGIKEY_PART_NUMBER (none) -> ED10563-ND; MANUFACTURER (none) -> On Shore Technology Inc.; MANUFACTURER_PART_NUMBER (none) -> OSTVN04A150
- J3: value Conn_01x06_Pin -> BG055-06A-1-0450-0530-0350-L-D
- J5: value USB4120-03-C_REVA6 -> USB4120-03-C; DIGIKEY_PART_NUMBER (none) -> 2073-USB4120-03-CCT-ND; MANUFACTURER Global Connector Technology -> GCT; MANUFACTURER_PART_NUMBER USB4120-03-C_REVA6 -> USB4120-03-C
- J6: value DE9_Socket_MountingHoles -> 622-009-260-033; DIGIKEY_PART_NUMBER (none) -> 151-622-009-260-033-ND; MANUFACTURER (none) -> EDAC Inc.; MANUFACTURER_PART_NUMBER (none) -> 622-009-260-033
- J7, J8, J9: value Conn_Coaxial -> SMA-J-P-H-RA-TH1; DIGIKEY_PART_NUMBER (none) -> SAM8856-ND; MANUFACTURER (none) -> Samtec Inc.; MANUFACTURER_PART_NUMBER (none) -> SMA-J-P-H-RA-TH1
- R64, R66: footprint R_0402_1005Metric -> 0402 (1005 Metric); DIELECTRIC (none) -> Thick-film; DIGIKEY_PART_NUMBER (none) -> P5.10KLCT-ND; MANUFACTURER Panasonic -> Panasonic Industry; POWER (none) -> 1/10W; TOLERANCE (none) -> 1%
- R65: footprint R_0402_1005Metric -> 0402 (1005 Metric); DIELECTRIC (none) -> Thick-film; DIGIKEY_PART_NUMBER (none) -> P1.00MLCT-ND; MANUFACTURER Panasonic -> Panasonic Industry; POWER (none) -> 1/10W; TOLERANCE (none) -> 1%
- R67: footprint R_0402_1005Metric -> 0402 (1005 Metric); DIELECTRIC (none) -> Thick-film; DIGIKEY_PART_NUMBER (none) -> P121KLCT-ND; MANUFACTURER Panasonic -> Panasonic Industry; POWER (none) -> 1/10W; TOLERANCE (none) -> 1%
- R68: footprint R_0402_1005Metric -> 0402 (1005 Metric); DIELECTRIC (none) -> Thick-film; DIGIKEY_PART_NUMBER (none) -> P100KLCT-ND; MANUFACTURER Panasonic -> Panasonic Industry; POWER (none) -> 1/10W; TOLERANCE (none) -> 1%
- U15, U16, U17, U18, U19, U20: MANUFACTURER (none) -> Texas Instruments
Connections:
- net 5V: now also C188.1, D22.1 (A1), J17.28 (Pin_28)
- net 5V_DISP: now also J17.16 (Pin_16)
- net BUTTON_1: now also J17.1 (Pin_1)
- net BUTTON_2: now also J17.19 (Pin_19)
- net BUTTON_3: now also J17.2 (Pin_2)
- net BUTTON_4: now also J17.20 (Pin_20)
- net BUTTON_5: now also J17.21 (Pin_21)
- net BUTTON_6: now also J17.4 (Pin_4)
- net BUTTON_7: now also J17.22 (Pin_22)
- net DISP_BL: now also J17.14 (Pin_14)
- net DISP_CS: now also J17.12 (Pin_12)
- net DISP_DC: now also J17.31 (Pin_31)
- net DISP_RST: now also J17.30 (Pin_30)
- net DISP_TOUCH_INT: now also J17.33 (Pin_33)
- net GND: now also C186.2, C188.2, D22.2 (A2), D23.2, D26.1 (A1), J15.2 (Ext), J17.10 (Pin_10), J17.13 (Pin_13), J17.3 (Pin_3), J17.35 (Pin_35), J17.36 (Pin_36), L10.2, R231.2, U65.3 (GND), U65.8 (GND), U66.3 (GND), U66.8 (GND), U69.3 (GND), U69.8 (GND), U70.3 (GND), U70.8 (GND); no longer J6.SH (PAD)
- net GPS_RF_IN: now also L10.1
- net I2C_DISP_SCL: now also J17.32 (Pin_32)
- net I2C_DISP_SDA: now also J17.15 (Pin_15)
- net RB_LOCK_IN: now also D26.2 (A2)
- net RTC_TAMPER: now also U16.5 (D2-), U16.6 (NC); no longer U20.5 (D2-), U20.6 (NC)
- net SPI_MOSI_DISP: now also J17.34 (Pin_34)
- net SPI_SCK_DISP: now also J17.17 (Pin_17)
- net USB_VBUS: no longer R67.1
- net USB_VBUS_SENSE: now also R67.1
- net USB_CC1: now reaches J5.A5 (CC1)
- net USB_CC1: now also R66.1, U65.1 (D1+), U65.10 (NC); no longer R64.1
- net USB_CC2: now reaches J5.B5 (CC2)
- net USB_CC2: now also R64.1, U65.2 (D1-), U65.9 (NC); no longer R66.1
- net PROX_WAKE: now reaches U16.4 (D2+)
- net PROX_WAKE: now also U16.7 (NC), J17.18 (Pin_18)
- net VCC_RB renamed VCC_RB_G
- new net: C186.1, J6.SH (PAD), R231.1
- new net 1PPS_OUT: D23.1, J15.1 (In)
- new net ENC_A_IN: J17.11 (Pin_11), U69.4 (D2+), U69.7 (NC)
- new net ENC_BUTTON: J17.9 (Pin_9), U69.1 (D1+), U69.10 (NC)
- new net ENC_B_IN: J17.27 (Pin_27), U69.2 (D1-), U69.9 (NC)
- new net HOLDOVER_ALARM_C1: J16.2 (Pin_2)
- new net HOLDOVER_ALARM_C2: J16.5 (Pin_5)
- new net HOLDOVER_ALARM_NC1: J16.3 (Pin_3)
- new net HOLDOVER_ALARM_NC2: J16.6 (Pin_6)
- new net HOLDOVER_ALARM_NO1: J16.1 (Pin_1)
- new net HOLDOVER_ALARM_NO2: J16.4 (Pin_4)
- new net PANEL_LEDS_P: J17.26 (Pin_26), U70.5 (D2-), U70.6 (NC)
- new net PANEL_LED_RED_N_1: J17.8 (Pin_8), U70.4 (D2+), U70.7 (NC)
- new net PANEL_LED_WHITE_N_1: J17.5 (Pin_5), U66.1 (D1+), U66.10 (NC)
- new net PANEL_LED_WHITE_N_2: J17.23 (Pin_23), U66.2 (D1-), U66.9 (NC)
- new net PANEL_LED_WHITE_N_3: J17.6 (Pin_6), U66.4 (D2+), U66.7 (NC)
- new net PANEL_LED_WHITE_N_4: J17.24 (Pin_24), U66.5 (D2-), U66.6 (NC)
- new net PANEL_LED_WHITE_N_5: J17.7 (Pin_7), U70.1 (D1+), U70.10 (NC)
- new net PANEL_LED_WHITE_N_6: J17.25 (Pin_25), U70.2 (D1-), U70.9 (NC)
- no-connect marks 13 -> 17
Other:
- note added: "BOTTOM"
- note added: "Place ALL Components on this sheet CLOSE to their connectors"
- note added: "TOP"
- note removed: "Place close to connector"
- moved on the sheet: C40, C41, C42, C43, D6, D7, D8, D9, J10, J2, J5, J6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

Commit message: Bom updates
Parts:
- U15, U16, U19, U20: footprint DQA0010A -> 10-USON; DIGIKEY_PART_NUMBER (none) -> 296-43875-1-ND
- U17, U18, U65, U66, U69, U70: footprint DQA0010A -> 10-USON; DIGIKEY_PART_NUMBER (none) -> 296-35765-1-ND
Changed lines of the file:
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@@
 			)
 		)
-		(property "Footprint" "DQA0010A"
+		(property "Footprint" "10-USON"
 			(at 292.1 81.28 0)
 			(hide yes)
@@
 			)
 		)
-		(property "Description" "4-ch ESD array"
+		(property "Description" "TVS DIODE 3.6VWM 8.8VC 10USON"
 			(at 292.1 81.28 0)
 			(hide yes)
@@
 			)
 		)
+		(property "DIGIKEY_PART_NUMBER" "296-43875-1-ND"
+			(at 292.1 81.28 0)
+			(hide yes)
+			(show_name no)
+			(do_not_autoplace no)
+			(effects
+				(font
+					(size 1.27 1.27)
+				)
+			)
+		)
 		(pin "9"
 		)
@@
 			)
 		)
-		(property "Footprint" "DQA0010A"
+		(property "Footprint" "10-USON"
 			(at 292.1 125.73 0)
 			(hide yes)
@@
 			)
 		)
-		(property "Description" "4-ch ESD array USB/IO"
+		(property "Description" "TVS DIODE 5.5VWM 14VC 10USON"
 			(at 292.1 125.73 0)
 			(hide yes)
@@
 			)
 		)
+		(property "DIGIKEY_PART_NUMBER" "296-35765-1-ND"
+			(at 292.1 125.73 0)
+			(hide yes)
+			(show_name no)
+			(do_not_autoplace no)
+			(effects
+				(font
+					(size 1.27 1.27)
+				)
+			)
+		)
 		(pin "2"
 		)
@@
 			)
 		)
-		(property "Footprint" "DQA0010A"
+		(property "Footprint" "10-USON"
 			(at 217.17 151.13 0)
 			(hide yes)
@@
 			)
 		)
-		(property "Description" "4-ch ESD array USB/IO"
+		(property "Description" "TVS DIODE 5.5VWM 14VC 10USON"
 			(at 217.17 151.13 0)
 			(hide yes)
@@
 			)
 		)
+		(property "DIGIKEY_PART_NUMBER" "296-35765-1-ND"
+			(at 217.17 151.13 0)
+			(hide yes)
+			(show_name no)
+			(do_not_autoplace no)
+			(effects
+				(font
+					(size 1.27 1.27)
+				)
+			)
+		)
 		(pin "2"
 		)
@@
 			)
 		)
-		(property "Footprint" "DQA0010A"
+		(property "Footprint" "10-USON"
 			(at 292.1 171.45 0)
 			(hide yes)
@@
 			)
 		)
-		(property "Description" "4-ch ESD array USB/IO"
+		(property "Description" "TVS DIODE 5.5VWM 14VC 10USON"
 			(at 292.1 171.45 0)
 			(hide yes)
@@
 			)
 		)
+		(property "DIGIKEY_PART_NUMBER" "296-35765-1-ND"
+			(at 292.1 171.45 0)
+			(hide yes)
+			(show_name no)
+			(do_not_autoplace no)
+			(effects
+				(font
+					(size 1.27 1.27)
+				)
+			)
+		)
 		(pin "2"
 		)
@@
 			)
 		)
-		(property "Footprint" "DQA0010A"
+		(property "Footprint" "10-USON"
 			(at 374.65 125.73 0)
 			(hide yes)
@@
 			)
 		)
-		(property "Description" "4-ch ESD array USB/IO"
+		(property "Description" "TVS DIODE 5.5VWM 14VC 10USON"
 			(at 374.65 125.73 0)
 			(hide yes)
@@
 			)
 		)
+		(property "DIGIKEY_PART_NUMBER" "296-35765-1-ND"
+			(at 374.65 125.73 0)
+			(hide yes)
+			(show_name no)
+			(do_not_autoplace no)
+			(effects
+				(font
+					(size 1.27 1.27)
+				)
+			)
+		)
 		(pin "2"
 		)
@@
 			)
 		)
-		(property "Footprint" "DQA0010A"
+		(property "Footprint" "10-USON"
 			(at 374.65 40.64 0)
 			(hide yes)
@@
 			)
 		)
-		(property "Description" "4-ch ESD array USB/IO"
+		(property "Description" "TVS DIODE 5.5VWM 14VC 10USON"
 			(at 374.65 40.64 0)
 			(hide yes)
@@
 			)
 		)
+		(property "DIGIKEY_PART_NUMBER" "296-35765-1-ND"
+			(at 374.65 40.64 0)
+			(hide yes)
+			(show_name no)
+			(do_not_autoplace no)
+			(effects
+				(font
+					(size 1.27 1.27)
+				)
+			)
+		)
 		(pin "2"
 		)
@@
 			)
 		)
-		(property "Footprint" "DQA0010A"
+		(property "Footprint" "10-USON"
 			(at 374.65 171.45 0)
 			(hide yes)
@@
 			)
 		)
-		(property "Description" "4-ch ESD array"
+		(property "Description" "TVS DIODE 3.6VWM 8.8VC 10USON"
 			(at 374.65 171.45 0)
 			(hide yes)
@@
 			)
 		)
+		(property "DIGIKEY_PART_NUMBER" "296-43875-1-ND"
+			(at 374.65 171.45 0)
+			(hide yes)
+			(show_name no)
+			(do_not_autoplace no)
+			(effects
+				(font
+					(size 1.27 1.27)
+				)
+			)
+		)
 		(pin "1"
 		)
@@
 			)
 		)
-		(property "Footprint" "DQA0010A"
+		(property "Footprint" "10-USON"
 			(at 153.67 151.13 0)
 			(hide yes)
@@
 			)
 		)
-		(property "Description" "4-ch ESD array USB/IO"
+		(property "Description" "TVS DIODE 5.5VWM 14VC 10USON"
 			(at 153.67 151.13 0)
 			(hide yes)
@@
 			)
 		)
+		(property "DIGIKEY_PART_NUMBER" "296-35765-1-ND"
+			(at 153.67 151.13 0)
+			(hide yes)
+			(show_name no)
+			(do_not_autoplace no)
+			(effects
+				(font
+					(size 1.27 1.27)
+				)
+			)
+		)
 		(pin "2"
 		)
@@
 			)
 		)
-		(property "Footprint" "DQA0010A"
+		(property "Footprint" "10-USON"
 			(at 374.65 81.28 0)
 			(hide yes)
@@
 			)
 		)
-		(property "Description" "4-ch ESD array"
+		(property "Description" "TVS DIODE 3.6VWM 8.8VC 10USON"
 			(at 374.65 81.28 0)
 			(hide yes)
@@
 			)
 		)
+		(property "DIGIKEY_PART_NUMBER" "296-43875-1-ND"
+			(at 374.65 81.28 0)
+			(hide yes)
+			(show_name no)
+			(do_not_autoplace no)
+			(effects
+				(font
+					(size 1.27 1.27)
+				)
+			)
+		)
 		(pin "1"
 		)
@@
 			)
 		)
-		(property "Footprint" "DQA0010A"
+		(property "Footprint" "10-USON"
 			(at 290.83 40.64 0)
 			(hide yes)
@@
 			)
 		)
-		(property "Description" "4-ch ESD array"
+		(property "Description" "TVS DIODE 3.6VWM 8.8VC 10USON"
 			(at 290.83 40.64 0)
 			(hide yes)
@@
 			(hide yes)
 			(show_name no)
+			(do_not_autoplace no)
+			(effects
+				(font
+					(size 1.27 1.27)
+				)
+			)
+		)
+		(property "DIGIKEY_PART_NUMBER" "296-43875-1-ND"
+			(at 290.83 40.64 0)
+			(hide yes)
+			(show_name no)

Commit message: Bom updates
Connections:
- no-connect marks 17 -> 18
Changed lines of the file:
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@@
+	)
+	(no_connect
+		(at 180.34 222.25)
 	)
 	(no_connect

Commit message: Add files via upload
Updated, completed placement
Parts:
- C186, C42: footprint 1812 (4532 Metric) -> Capacitor_SMD:C_1812_4532Metric
- C188, C41, C43: footprint 0402 (1005 Metric) -> copy_ref:C_0402_1005Metric
- C40: footprint 0603 (1608 Metric) -> copy_ref:C_0603_1608Metric
- D22: footprint DO-219AB (SMF) -> dowload:DO-219AB (SMF)
- D23, D8, D9: footprint 2-XDFN -> dowload:2-XDFN
- D26: footprint DO-214AC -> dowload:DO-214AC
- D6: footprint DO-219AB (SMF) -> Diode_SMD:D_SMF
- D7: footprint DO-214AB (SMC) -> Diode_SMD:D_SMC
- J10: footprint (none) -> dowload:CONN_OSTVN02A150_OST
- J15, J7, J8, J9: footprint (none) -> dowload:SAMTEC_SMA-J-P-X-RA-TH1
- J16: footprint (none) -> dowload:CONN_OSTVN06A150_OST
- J17: footprint (none) -> dowload:PHOENIX_1787179
- J2: footprint (none) -> dowload:CONN_OSTVN04A150_OST
- J3: footprint Library:GCT_BG055-06A-1-0450-0530-0350-L-D -> dowload:GCT_BG055-06A-1-0450-0530-0350-L-D
- J6: footprint (none) -> copy_ref:DB9_Socket
- L10: footprint 0603 (1608 Metric) -> Inductor_SMD:L_0603_1608Metric
- R231, R64, R65, R66, R67, R68: footprint 0402 (1005 Metric) -> copy_ref:R_0402_1005Metric
- U15, U16, U17, U18, U19, U20: footprint 10-USON -> dowload:TPD4E02B04DQAR
- U65, U66, U69, U70: footprint 10-USON -> copy_ref:USON-10_2.5x1.0mm_P0.5mm
Changed lines of the file:
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@@
 			)
 		)
-		(property "Footprint" ""
+		(property "Footprint" "dowload:SAMTEC_SMA-J-P-X-RA-TH1"
 			(at 63.5 234.95 0)
 			(hide yes)
@@
 			)
 		)
-		(property "Footprint" "DO-214AC"
+		(property "Footprint" "dowload:DO-214AC"
 			(at 52.07 95.25 0)
 			(hide yes)
@@
 			)
 		)
-		(property "Footprint" "10-USON"
+		(property "Footprint" "dowload:TPD4E02B04DQAR"
 			(at 292.1 81.28 0)
 			(hide yes)
@@
 			)
 		)
-		(property "Footprint" "1812 (4532 Metric)"
+		(property "Footprint" "Capacitor_SMD:C_1812_4532Metric"
 			(at 102.5652 119.38 0)
 			(hide yes)
@@
 			)
 		)
-		(property "Footprint" ""
+		(property "Footprint" "dowload:SAMTEC_SMA-J-P-X-RA-TH1"
 			(at 63.5 201.93 0)
 			(hide yes)
@@
 			)
 		)
-		(property "Footprint" "2-XDFN"
+		(property "Footprint" "dowload:2-XDFN"
 			(at 57.15 254 0)
 			(hide yes)
@@
 			)
 		)
-		(property "Footprint" ""
+		(property "Footprint" "dowload:CONN_OSTVN06A150_OST"
 			(at 356.87 210.82 0)
 			(hide yes)
@@
 			)
 		)
-		(property "Footprint" "10-USON"
+		(property "Footprint" "copy_ref:USON-10_2.5x1.0mm_P0.5mm"
 			(at 292.1 125.73 0)
 			(hide yes)
@@
 			)
 		)
-		(property "Footprint" "0603 (1608 Metric)"
+		(property "Footprint" "Inductor_SMD:L_0603_1608Metric"
 			(at 49.53 218.44 0)
 			(hide yes)
@@
 			)
 		)
-		(property "Footprint" ""
+		(property "Footprint" "dowload:PHOENIX_1787179"
 			(at 172.72 217.17 0)
 			(hide yes)
@@
 			)
 		)
-		(property "Footprint" "10-USON"
+		(property "Footprint" "copy_ref:USON-10_2.5x1.0mm_P0.5mm"
 			(at 217.17 151.13 0)
 			(hide yes)
@@
 			)
 		)
-		(property "Footprint" "DO-219AB (SMF)"
+		(property "Footprint" "Diode_SMD:D_SMF"
 			(at 111.76 240.03 0)
 			(hide yes)
@@
 			)
 		)
-		(property "Footprint" "0402 (1005 Metric)"
+		(property "Footprint" "copy_ref:R_0402_1005Metric"
 			(at 163.83 24.638 90)
 			(hide yes)
@@
 			)
 		)
-		(property "Footprint" "0402 (1005 Metric)"
+		(property "Footprint" "copy_ref:R_0402_1005Metric"
 			(at 95.758 115.57 90)
 			(hide yes)
@@
 			)
 		)
-		(property "Footprint" "0402 (1005 Metric)"
+		(property "Footprint" "copy_ref:R_0402_1005Metric"
 			(at 141.478 69.85 90)
 			(hide yes)
@@
 			)
 		)
-		(property "Footprint" ""
+		(property "Footprint" "dowload:CONN_OSTVN02A150_OST"
 			(at 265.43 236.22 0)
 			(hide yes)
@@
 			)
 		)
-		(property "Footprint" "DO-214AB (SMC)"
+		(property "Footprint" "Diode_SMD:D_SMC"
 			(at 76.2 80.01 0)
 			(hide yes)
@@
 			)
 		)
-		(property "Footprint" "10-USON"
+		(property "Footprint" "copy_ref:USON-10_2.5x1.0mm_P0.5mm"
 			(at 292.1 171.45 0)
 			(hide yes)
@@
 			)
 		)
-		(property "Footprint" "0603 (1608 Metric)"
+		(property "Footprint" "copy_ref:C_0603_1608Metric"
 			(at 118.4148 243.84 0)
 			(hide yes)
@@
 			)
 		)
-		(property "Footprint" "0402 (1005 Metric)"
+		(property "Footprint" "copy_ref:R_0402_1005Metric"
 			(at 173.228 29.21 90)
 			(hide yes)
@@
 			)
 		)
-		(property "Footprint" ""
+		(property "Footprint" "copy_ref:DB9_Socket"
 			(at 93.98 88.9 0)
 			(hide yes)
@@
 			)
 		)
-		(property "Footprint" "0402 (1005 Metric)"
+		(property "Footprint" "copy_ref:C_0402_1005Metric"
 			(at 219.4052 228.6 0)
 			(hide yes)
@@
 			)
 		)
-		(property "Footprint" ""
+		(property "Footprint" "dowload:CONN_OSTVN04A150_OST"
 			(at 76.2 36.83 0)
 			(hide yes)
@@
 			)
 		)
-		(property "Footprint" "2-XDFN"
+		(property "Footprint" "dowload:2-XDFN"
 			(at 57.15 190.5 0)
 			(hide yes)
@@
 			)
 		)
-		(property "Footprint" "10-USON"
+		(property "Footprint" "dowload:TPD4E02B04DQAR"
 			(at 374.65 125.73 0)
 			(hide yes)
@@
 			)
 		)
-		(property "Footprint" "10-USON"
+		(property "Footprint" "copy_ref:USON-10_2.5x1.0mm_P0.5mm"
 			(at 374.65 40.64 0)
 			(hide yes)
@@
 			)
 		)
-		(property "Footprint" "0402 (1005 Metric)"
+		(property "Footprint" "copy_ref:R_0402_1005Metric"
 			(at 205.232 78.74 90)
 			(hide yes)
@@
 			)
 		)
-		(property "Footprint" "10-USON"
+		(property "Footprint" "dowload:TPD4E02B04DQAR"
 			(at 374.65 171.45 0)
 			(hide yes)
@@
 			)
 		)
-		(property "Footprint" "10-USON"
+		(property "Footprint" "dowload:TPD4E02B04DQAR"
 			(at 153.67 151.13 0)
 			(hide yes)
@@
 			)
 		)
-		(property "Footprint" "0402 (1005 Metric)"
+		(property "Footprint" "copy_ref:R_0402_1005Metric"
 			(at 150.368 104.14 90)
 			(hide yes)
@@
 			)
 		)
-		(property "Footprint" "2-XDFN"
+		(property "Footprint" "dowload:2-XDFN"
 			(at 57.15 165.1 0)
 			(hide yes)
@@
 			)
 		)
-		(property "Footprint" "10-USON"
+		(property "Footprint" "dowload:TPD4E02B04DQAR"
 			(at 374.65 81.28 0)
 			(hide yes)
@@
 			)
 		)
-		(property "Footprint" "0402 (1005 Metric)"
+		(property "Footprint" "copy_ref:C_0402_1005Metric"
 			(at 126.6952 243.84 0)
 			(hide yes)
@@
 			)
 		)
-		(property "Footprint" ""
+		(property "Footprint" "dowload:SAMTEC_SMA-J-P-X-RA-TH1"
 			(at 63.5 171.45 0)
 			(hide yes)
@@
 			)
 		)
-		(property "Footprint" ""
+		(property "Footprint" "dowload:SAMTEC_SMA-J-P-X-RA-TH1"
 			(at 63.5 146.05 0)
 			(hide yes)
@@
 			)
 		)
-		(property "Footprint" "Library:GCT_BG055-06A-1-0450-0530-0350-L-D"
+		(property "Footprint" "dowload:GCT_BG055-06A-1-0450-0530-0350-L-D"
 			(at 27.94 40.64 0)
 			(hide yes)
@@
 			)
 		)
-		(property "Footprint" "0402 (1005 Metric)"
+		(property "Footprint" "copy_ref:C_0402_1005Metric"
 			(at 182.5752 33.02 0)
 			(hide yes)
@@
 			)
 		)
-		(property "Footprint" "10-USON"
+		(property "Footprint" "dowload:TPD4E02B04DQAR"
 			(at 290.83 40.64 0)
 			(hide yes)
@@
 			)
 		)
-		(property "Footprint" "DO-219AB (SMF)"
+		(property "Footprint" "dowload:DO-219AB (SMF)"
 			(at 217.17 224.79 0)
 			(hide yes)
@@
 			)
 		)
-		(property "Footprint" "1812 (4532 Metric)"
+		(property "Footprint" "Capacitor_SMD:C_1812_4532Metric"
 			(at 157.1752 107.95 0)
 			(hide yes)

Commit message: PCB / 3D updates
Connections:
- net USB_DM renamed USB_D-
- net USB_DP renamed USB_D+
Changed lines of the file:
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@@
 	(wire
 		(pts
+			(xy 220.98 57.15) (xy 226.06 57.15)
+		)
+		(stroke
+			(width 0)
+			(type default)
+		)
+	)
+	(wire
+		(pts
 			(xy 160.02 53.34) (xy 158.75 53.34)
 		)
@@
 	(wire
 		(pts
+			(xy 220.98 59.69) (xy 226.06 59.69)
+		)
+		(stroke
+			(width 0)
+			(type default)
+		)
+	)
+	(wire
+		(pts
 			(xy 392.43 45.72) (xy 394.97 45.72)
 		)
@@
 		)
 	)
+	(global_label "USB_D+"
+		(shape bidirectional)
+		(at 226.06 57.15 0)
+		(fields_autoplaced yes)
+		(effects
+			(font
+				(size 1.27 1.27)
+			)
+			(justify left)
+		)
+		(property "Intersheetrefs" "${INTERSHEET_REFS}"
+			(at 237.7765 57.15 0)
+			(hide yes)
+			(show_name no)
+			(do_not_autoplace no)
+			(effects
+				(font
+					(size 1.27 1.27)
+				)
+				(justify left)
+			)
+		)
+	)
 	(global_label "BUTTON_3"
 		(shape input)
@@
 		)
 	)
+	(global_label "USB_DP"
+		(shape bidirectional)
+		(at 220.98 57.15 180)
+		(fields_autoplaced yes)
+		(effects
+			(font
+				(size 1.27 1.27)
+			)
+			(justify right)
+		)
+		(property "Intersheetrefs" "${INTERSHEET_REFS}"
+			(at 209.5659 57.15 0)
+			(hide yes)
+			(show_name no)
+			(do_not_autoplace no)
+			(effects
+				(font
+					(size 1.27 1.27)
+				)
+				(justify right)
+			)
+		)
+	)
 	(global_label "PANEL_LED_WHITE_N_4"
 		(shape input)
@@
 		)
 	)
+	(global_label "USB_DM"
+		(shape bidirectional)
+		(at 220.98 59.69 180)
+		(fields_autoplaced yes)
+		(effects
+			(font
+				(size 1.27 1.27)
+			)
+			(justify right)
+		)
+		(property "Intersheetrefs" "${INTERSHEET_REFS}"
+			(at 209.3845 59.69 0)
+			(hide yes)
+			(show_name no)
+			(do_not_autoplace no)
+			(effects
+				(font
+					(size 1.27 1.27)
+				)
+				(justify right)
+			)
+		)
+	)
 	(global_label "USB_DP"
 		(shape bidirectional)
@@
 			)
 		)
+	)
+	(global_label "USB_D-"
+		(shape bidirectional)
+		(at 226.06 59.69 0)
+		(fields_autoplaced yes)
+		(effects
+			(font
+				(size 1.27 1.27)
+			)
+			(justify left)
+		)
+		(property "Intersheetrefs" "${INTERSHEET_REFS}"
+			(at 237.7765 59.69 0)
+			(hide yes)
+			(show_name no)
+			(do_not_autoplace no)
+			(effects
+				(font
+					(size 1.27 1.27)
+				)
+				(justify left)
+			)
+		)
