File: hardware/ntp-server-stm32/ntp-server-stm32.kicad_sch (KiCad schematic)
At the start: 14 parts

Commit message: Updates
Other:
- sheet I2C GPIO renamed GPIO (page 17)
- added sheet Optical Encoder (optical-encoder.kicad_sch)
Changed lines of the file:
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@@
+	)
+	(sheet
+		(at 257.81 140.97)
+		(size 12.7 12.7)
+		(exclude_from_sim no)
+		(in_bom yes)
+		(on_board yes)
+		(dnp no)
+		(fields_autoplaced yes)
+		(stroke
+			(width 0.1524)
+			(type solid)
+		)
+		(fill
+			(color 0 0 0 0)
+		)
+		(property "Sheetname" "Optical Encoder"
+			(at 257.81 140.2584 0)
+			(show_name no)
+			(do_not_autoplace no)
+			(effects
+				(font
+					(size 1.27 1.27)
+				)
+				(justify left bottom)
+			)
+		)
+		(property "Sheetfile" "optical-encoder.kicad_sch"
+			(at 257.81 154.2546 0)
+			(show_name no)
+			(do_not_autoplace no)
+			(effects
+				(font
+					(size 1.27 1.27)
+				)
+				(justify left top)
+			)
+		)
+		(instances
+			(project "ntp-server-stm32"
+				(path "/4c8fa883-5b85-4079-9006-ac22e5786016"
+					(page "22")
+				)
+			)
+		)
 	)
 	(sheet
@@
 			(color 0 0 0 0)
 		)
-		(property "Sheetname" "I2C GPIO"
+		(property "Sheetname" "GPIO (page 17)"
 			(at 375.92 19.6084 0)
 			(show_name no)

Commit message: Add files via upload
Updated, completed placement
Parts:
- H1, H10, H11, H12, H13, H14, H2, H3, H4, H5, H6, H7, H8, H9: footprint (none) -> copy_ref:MountingHole_3.2mm_M3
Changed lines of the file:
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@@
 			)
 		)
-		(property "Footprint" ""
+		(property "Footprint" "copy_ref:MountingHole_3.2mm_M3"
 			(at 22.86 220.98 0)
 			(hide yes)
@@
 			)
 		)
-		(property "Footprint" ""
+		(property "Footprint" "copy_ref:MountingHole_3.2mm_M3"
 			(at 22.86 241.3 0)
 			(hide yes)
@@
 			)
 		)
-		(property "Footprint" ""
+		(property "Footprint" "copy_ref:MountingHole_3.2mm_M3"
 			(at 52.07 236.22 0)
 			(hide yes)
@@
 			)
 		)
-		(property "Footprint" ""
+		(property "Footprint" "copy_ref:MountingHole_3.2mm_M3"
 			(at 52.07 231.14 0)
 			(hide yes)
@@
 			)
 		)
-		(property "Footprint" ""
+		(property "Footprint" "copy_ref:MountingHole_3.2mm_M3"
 			(at 52.07 241.3 0)
 			(hide yes)
@@
 			)
 		)
-		(property "Footprint" ""
+		(property "Footprint" "copy_ref:MountingHole_3.2mm_M3"
 			(at 22.86 256.54 0)
 			(hide yes)
@@
 			)
 		)
-		(property "Footprint" ""
+		(property "Footprint" "copy_ref:MountingHole_3.2mm_M3"
 			(at 22.86 236.22 0)
 			(hide yes)
@@
 			)
 		)
-		(property "Footprint" ""
+		(property "Footprint" "copy_ref:MountingHole_3.2mm_M3"
 			(at 52.07 220.98 0)
 			(hide yes)
@@
 			)
 		)
-		(property "Footprint" ""
+		(property "Footprint" "copy_ref:MountingHole_3.2mm_M3"
 			(at 22.86 231.14 0)
 			(hide yes)
@@
 			)
 		)
-		(property "Footprint" ""
+		(property "Footprint" "copy_ref:MountingHole_3.2mm_M3"
 			(at 52.07 246.38 0)
 			(hide yes)
@@
 			)
 		)
-		(property "Footprint" ""
+		(property "Footprint" "copy_ref:MountingHole_3.2mm_M3"
 			(at 22.86 226.06 0)
 			(hide yes)
@@
 			)
 		)
-		(property "Footprint" ""
+		(property "Footprint" "copy_ref:MountingHole_3.2mm_M3"
 			(at 22.86 251.46 0)
 			(hide yes)
@@
 			)
 		)
-		(property "Footprint" ""
+		(property "Footprint" "copy_ref:MountingHole_3.2mm_M3"
 			(at 52.07 226.06 0)
 			(hide yes)
@@
 			)
 		)
-		(property "Footprint" ""
+		(property "Footprint" "copy_ref:MountingHole_3.2mm_M3"
 			(at 22.86 246.38 0)
 			(hide yes)

Commit message: PCB / 3D updates
Parts:
- H1, H10, H11, H12, H13, H14, H2, H3, H4, H5, H6, H7, H8, H9: footprint copy_ref:MountingHole_3.2mm_M3 -> MountingHole:MountingHole_3.2mm_M3_Pad
Other:
- moved on the sheet: H1
Changed lines of the file:
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@@
 	(symbol
 		(lib_id "Mechanical:MountingHole")
-		(at 22.86 220.98 0)
+		(at 22.86 218.44 0)
 		(unit 1)
 		(body_style 1)
@@
 		(fields_autoplaced yes)
 		(property "Reference" "H1"
+			(at 25.4 217.1699 0)
+			(show_name no)
+			(do_not_autoplace no)
+			(effects
+				(font
+					(size 1.27 1.27)
+				)
+				(justify left)
+			)
+		)
+		(property "Value" "0.125\" Mounting Hole"
 			(at 25.4 219.7099 0)
 			(show_name no)
@@
 			)
 		)
-		(property "Value" "0.125\" Mounting Hole"
-			(at 25.4 222.2499 0)
-			(show_name no)
-			(do_not_autoplace no)
-			(effects
-				(font
-					(size 1.27 1.27)
-				)
-				(justify left)
-			)
-		)
-		(property "Footprint" "copy_ref:MountingHole_3.2mm_M3"
-			(at 22.86 220.98 0)
-			(hide yes)
-			(show_name no)
-			(do_not_autoplace no)
-			(effects
-				(font
-					(size 1.27 1.27)
-				)
-			)
-		)
-		(property "Datasheet" ""
-			(at 22.86 220.98 0)
-			(hide yes)
-			(show_name no)
-			(do_not_autoplace no)
-			(effects
-				(font
-					(size 1.27 1.27)
-				)
-			)
-		)
-		(property "Description" "Mounting Hole without connection"
-			(at 22.86 220.98 0)
+		(property "Footprint" "MountingHole:MountingHole_3.2mm_M3_Pad"
+			(at 22.86 218.44 0)
+			(hide yes)
+			(show_name no)
+			(do_not_autoplace no)
+			(effects
+				(font
+					(size 1.27 1.27)
+				)
+			)
+		)
+		(property "Datasheet" ""
+			(at 22.86 218.44 0)
+			(hide yes)
+			(show_name no)
+			(do_not_autoplace no)
+			(effects
+				(font
+					(size 1.27 1.27)
+				)
+			)
+		)
+		(property "Description" "Mounting Hole without connection"
+			(at 22.86 218.44 0)
 			(hide yes)
 			(show_name no)
@@
 			)
 		)
-		(property "Footprint" "copy_ref:MountingHole_3.2mm_M3"
+		(property "Footprint" "MountingHole:MountingHole_3.2mm_M3_Pad"
 			(at 22.86 241.3 0)
 			(hide yes)
@@
 			)
 		)
-		(property "Footprint" "copy_ref:MountingHole_3.2mm_M3"
+		(property "Footprint" "MountingHole:MountingHole_3.2mm_M3_Pad"
 			(at 52.07 236.22 0)
 			(hide yes)
@@
 			)
 		)
-		(property "Footprint" "copy_ref:MountingHole_3.2mm_M3"
+		(property "Footprint" "MountingHole:MountingHole_3.2mm_M3_Pad"
 			(at 52.07 231.14 0)
 			(hide yes)
@@
 			)
 		)
-		(property "Footprint" "copy_ref:MountingHole_3.2mm_M3"
+		(property "Footprint" "MountingHole:MountingHole_3.2mm_M3_Pad"
 			(at 52.07 241.3 0)
 			(hide yes)
@@
 			)
 		)
-		(property "Footprint" "copy_ref:MountingHole_3.2mm_M3"
+		(property "Footprint" "MountingHole:MountingHole_3.2mm_M3_Pad"
 			(at 22.86 256.54 0)
 			(hide yes)
@@
 			)
 		)
-		(property "Footprint" "copy_ref:MountingHole_3.2mm_M3"
+		(property "Footprint" "MountingHole:MountingHole_3.2mm_M3_Pad"
 			(at 22.86 236.22 0)
 			(hide yes)
@@
 			)
 		)
-		(property "Footprint" "copy_ref:MountingHole_3.2mm_M3"
+		(property "Footprint" "MountingHole:MountingHole_3.2mm_M3_Pad"
 			(at 52.07 220.98 0)
 			(hide yes)
@@
 			)
 		)
-		(property "Footprint" "copy_ref:MountingHole_3.2mm_M3"
+		(property "Footprint" "MountingHole:MountingHole_3.2mm_M3_Pad"
 			(at 22.86 231.14 0)
 			(hide yes)
@@
 			)
 		)
-		(property "Footprint" "copy_ref:MountingHole_3.2mm_M3"
+		(property "Footprint" "MountingHole:MountingHole_3.2mm_M3_Pad"
 			(at 52.07 246.38 0)
 			(hide yes)
@@
 			)
 		)
-		(property "Footprint" "copy_ref:MountingHole_3.2mm_M3"
+		(property "Footprint" "MountingHole:MountingHole_3.2mm_M3_Pad"
 			(at 22.86 226.06 0)
 			(hide yes)
@@
 			)
 		)
-		(property "Footprint" "copy_ref:MountingHole_3.2mm_M3"
+		(property "Footprint" "MountingHole:MountingHole_3.2mm_M3_Pad"
 			(at 22.86 251.46 0)
 			(hide yes)
@@
 			)
 		)
-		(property "Footprint" "copy_ref:MountingHole_3.2mm_M3"
+		(property "Footprint" "MountingHole:MountingHole_3.2mm_M3_Pad"
 			(at 52.07 226.06 0)
 			(hide yes)
@@
 			)
 		)
-		(property "Footprint" "copy_ref:MountingHole_3.2mm_M3"
+		(property "Footprint" "MountingHole:MountingHole_3.2mm_M3_Pad"
 			(at 22.86 246.38 0)
 			(hide yes)
